Commit message: Fixes to get diff drive working for ros2 control

File: ros_control_demo_example_2/description/ros2_control/diffbot.ros2_control.xacro (robot description, xacro)
@@ -6,5 +6,5 @@
         <plugin>ros2_control_demo_example_2/DiffBotSystemHardware</plugin>
         <param name="example_param_hw_start_duration_sec">0</param>
-        <param name="example_param_hw_stop_duration_sec">3.0</param>
+        <param name="example_param_hw_stop_duration_sec">0.1</param>
       </hardware>
       <joint name="${prefix}left_wheel_joint">

File: ros_control_demo_example_2/description/urdf/diffbot_description.urdf.xacro (robot description, xacro)
@@ -5,10 +5,10 @@
   <xacro:property name="PI" value="3.1415926535897931"/>
   <xacro:property name="base_mass" value="0.3" /> <!-- arbitrary value for base mass -->
-  <xacro:property name="base_width" value="0.1" />
-  <xacro:property name="base_length" value="0.1" />
-  <xacro:property name="base_height" value="0.05" />
+  <xacro:property name="base_width" value="0.125" />
+  <xacro:property name="base_length" value="0.22" />
+  <xacro:property name="base_height" value="0.1" />
   <xacro:property name="wheel_mass" value="0.3" /> <!-- arbitrary value for wheel mass -->
-  <xacro:property name="wheel_len" value="0.020" />
-  <xacro:property name="wheel_radius" value="0.015" />
+  <xacro:property name="wheel_len" value="0.01" />
+  <xacro:property name="wheel_radius" value="0.003" />
   <xacro:property name="caster_wheel_mass" value="0.1" /> <!-- arbitrary value for caster wheel mass -->
   <xacro:property name="caster_wheel_radius" value="0.015" />
