Commit message: sonar wip

File: urdf/diffdrive.xacro (robot description, xacro)
@@ -9,6 +9,6 @@
       <leftJoint>joint_left_wheel</leftJoint>
       <rightJoint>joint_right_wheel</rightJoint>
-      <wheelSeparation>5</wheelSeparation>
-      <wheelDiameter>2</wheelDiameter>
+      <wheelSeparation>0.15</wheelSeparation>
+      <wheelDiameter>${0.0325*2}</wheelDiameter>
       <torque>20</torque>
       <commandTopic>

File: urdf/lidar.xacro (robot description, xacro)
@@ -10,5 +10,5 @@
     <sensor name="lidar" type="ray">
       <pose>0 0 0 0 0 0</pose>
-      <visualize>true</visualize>
+      <visualize>false</visualize>
       <update_rate>15</update_rate>
       <ray>
@@ -32,8 +32,8 @@
         </noise>
       </ray>
-      <plugin name="laser_controller"
+      <plugin name="ultra_controller"
       filename="libgazebo_ros_laser.so">
         <topicName>/mirte/scan</topicName>
-        <frameName>lidar_link</frameName>
+        <frameName>lidar_link2</frameName>
       </plugin>
     </sensor>

File: urdf/mirte.xacro (robot description, xacro)
@@ -4,6 +4,6 @@
   <xacro:include filename="$(find mirte_gazebo)/urdf/macros.xacro" />
   <xacro:include filename="$(find mirte_gazebo)/urdf/ros_control.xacro" />
-  <xacro:include filename="$(find mirte_gazebo)/urdf/lidar.xacro" />
-  <xacro:include filename="$(find mirte_gazebo)/urdf/camera.xacro" />
+  <!-- <xacro:include filename="$(find mirte_gazebo)/urdf/lidar.xacro" /> -->
+  <!-- <xacro:include filename="$(find mirte_gazebo)/urdf/camera.xacro" /> -->
    <xacro:include filename="$(find mirte_gazebo)/urdf/ultrasonic.xacro"/>
   <xacro:property name="yaml_param_file"
@@ -77,7 +77,8 @@
     <origin rpy="0 0 .45" xyz="0.085 0.04 0.022" />
   </xacro:ultrasonic_sensor>
+<!--
   <xacro:ultrasonic_sensor name="right">
     <origin rpy="0 0 -0.45" xyz="0.085 -0.04 0.022" />
-  </xacro:ultrasonic_sensor>
+  </xacro:ultrasonic_sensor> -->
   <gazebo>
     <plugin name="gazebo_ros_control"

File: urdf/ultrasonic.xacro (robot description, xacro)
@@ -2,4 +2,5 @@
 <robot xmlns:xacro="http://www.ros.org/wiki/xacro">
   <xacro:macro name="ultrasonic_sensor" params="name *origin">
+<xacro:property name="sonar_angle_max" value="${radians(15)}" />
     <joint name="sonar_${name}" type="fixed">
       <axis xyz="0 1 0" />
@@ -31,19 +32,19 @@
     <gazebo reference="base_sonar_${name}">
       <sensor type="ray" name="range_sensor_${name}">
-        <visualize>false</visualize>
+        <visualize>true</visualize>
         <ray>
           <scan>
             <horizontal>
               <!-- for some reason 1 does not work, we neex 2x2 -->
-              <samples>2</samples>
+              <samples>4</samples>
               <resolution>1</resolution>
-              <min_angle>-0.26</min_angle>
-              <max_angle>0.26</max_angle>
+              <min_angle>${-sonar_angle_max/2}</min_angle>
+              <max_angle>${sonar_angle_max/2}</max_angle>
             </horizontal>
             <vertical>
-              <samples>2</samples>
+              <samples>4</samples>
               <resolution>1</resolution>
-              <min_angle>-0.014835</min_angle>
-              <max_angle>0.014835</max_angle>
+              <min_angle>0</min_angle> <!-- Don't look to much at the floor-->
+              <max_angle>${sonar_angle_max/4}</max_angle>
             </vertical>
           </scan>
@@ -62,16 +63,26 @@
         <!-- Using gazebo's update rate instead of plugin's -->
         <update_rate>30</update_rate>
-        <plugin name="gazebo_ros_range_controller_${name}"
-        filename="libgazebo_ros_ray_sensor.so">
-          <!-- Change namespace and output topic so published topic is /rrbot/laser/scan -->
-          <ros>
-            <namespace>/mirte</namespace>
-            <remapping>~/out:=distance/${name}</remapping>
-          </ros>
-          <!-- Set output to sensor_msgs/Range to get same output type as gazebo_ros_range -->
-          <output_type>sensor_msgs/Range</output_type>
-          <!-- <frame_name> ommited, will default to range_link -->
-          <radiation_type>ultrasound</radiation_type>
-        </plugin>
+          <plugin name="laser_controller"
+      filename="libgazebo_ros_laser.so">
+        <topicName>/mirte/scan2</topicName>
+              <output_type>sensor_msgs/Range</output_type>
+      <radiation_type>ultrasound</radiation_type>
+        <frameName>base_sonar_${name}</frameName>
+      </plugin>
+<!--         <plugin name="gazebo_ros_head_hokuyo_controlle" filename="libgazebo_ros_range_sensor.so" >
+  <ros>
+    <remapping>~/out:=/jemoeder</remapping>
+  </ros>
+   <output_type>sensor_msgs/LaserScan</output_type>
+</plugin>
+-->
+        <!-- <plugin name="ultrasonic_sensor_1" filename="libgazebo_ros_ray_sensor.so">
+    <ros>
+        <remapping>~/out:=ultrasonic_sensor_1</remapping>
+      </ros>
+      <output_type>sensor_msgs/Range</output_type>
+      <radiation_type>ultrasound</radiation_type>
+      <frame_name>ultrasonic_1_link</frame_name>
+    </plugin>  -->
       </sensor>
     </gazebo>
