Commit message: Add intensity sensor

File: urdf/materials.xacro (robot description, xacro)
@@ -6,4 +6,7 @@
   <material name="blue">
     <color rgba="0.203125 0.23828125 0.28515625 1.0"/>
+  </material>
+  <material name="yellow">
+    <color rgba="1 1 0 1.0"/>
   </material>
   <material name="green">
@@ -59,3 +62,13 @@
     <material>Gazebo/Red</material>
   </gazebo>
+  <gazebo reference="base_ir_left">
+    <mu1>0.2</mu1>
+    <mu2>0.2</mu2>
+    <material>Gazebo/Purple</material>
+  </gazebo>
+  <gazebo reference="base_ir_right">
+    <mu1>0.2</mu1>
+    <mu2>0.2</mu2>
+    <material>Gazebo/Purple</material>
+  </gazebo>
 </robot>

File: urdf/mirte.xacro (robot description, xacro)
@@ -5,4 +5,5 @@
   <xacro:include filename="$(find mirte_gazebo)/urdf/ros_control.xacro"/>
   <xacro:include filename="$(find mirte_gazebo)/urdf/lidar.xacro"/>
+  <xacro:include filename="$(find mirte_gazebo)/urdf/ir.xacro"/>
   <!-- <xacro:include filename="$(find mirte_gazebo)/urdf/camera.xacro" /> -->
   <xacro:include filename="$(find mirte_gazebo)/urdf/ultrasonic.xacro"/>
@@ -59,10 +60,16 @@
     </joint_options>
   </xacro:wheel>
-  <xacro:ultrasonic_sensor name="left">
+  <!-- <xacro:ultrasonic_sensor name="left">
     <origin rpy="0 0 .45" xyz="0.085 0.04 0.022"/>
   </xacro:ultrasonic_sensor>
   <xacro:ultrasonic_sensor name="right">
     <origin rpy="0 0 -0.45" xyz="0.085 -0.04 0.022"/>
-  </xacro:ultrasonic_sensor>
+  </xacro:ultrasonic_sensor> -->
+  <xacro:ir_sensor name="left">
+    <origin rpy="0 ${radians(90)} 0" xyz="0.0785 0.022 0.002"/>
+  </xacro:ir_sensor>
+  <xacro:ir_sensor name="right">
+    <origin rpy="0 ${radians(90)} 0" xyz="0.0785 -0.022 0.002"/>
+  </xacro:ir_sensor>
   <gazebo>
     <plugin name="gazebo_ros_control" filename="libgazebo_ros_control.so">
