Commit message: World spawning done

File: urdf/duckietown.xacro (robot description, xacro)
@@ -1,4 +1,5 @@
 <?xml version="1.0"?>
-<robot xmlns:xacro="http://www.ros.org/wiki/xacro" name="duckietown">
+<model xmlns:xacro="http://www.ros.org/wiki/xacro" name="duckietown">
+  <static>true</static>
   <xacro:include filename="$(find mirte_gazebo)/urdf/tile.xacro"/>
   <!-- this dummy base is used to link all tiles to -->
@@ -94,3 +95,3 @@
   <xacro:tile name="tile_7_8" material="DT/asphalt" size="0.6" x="7" y="8" yaw="0"/>
   <xacro:tile name="tile_8_8" material="DT/asphalt" size="0.6" x="8" y="8" yaw="0"/>
-</robot>
+</model>

File: urdf/tileWorld.xacro (robot description, xacro)
@@ -1,73 +1,71 @@
 <?xml version="1.0"?>
 <robot xmlns:xacro="http://www.ros.org/wiki/xacro">
-    <xacro:macro name="tileWorld" params="name material size x y yaw=0">
-        <model name='unit_box_${name}'>
-            <static>1</static>
-            <pose>${x * size} ${y * size} 0. 0 -0 ${pi / 180 * yaw}</pose>
-            <link name='link'>
-                <inertial>
-                    <mass>1</mass>
-                    <inertia>
-                        <ixx>0.</ixx>
-                        <ixy>0</ixy>
-                        <ixz>0</ixz>
-                        <iyy>0</iyy>
-                        <iyz>0</iyz>
-                        <izz>0</izz>
-                    </inertia>
-                    <pose>0 0 0 0 -0 0</pose>
-                </inertial>
-                <collision name='collision'>
-                    <geometry>
-                        <box>
-                            <size>${size} ${size} 0.01</size>
-                        </box>
-                    </geometry>
-                    <max_contacts>10</max_contacts>
-                    <surface>
-                        <contact>
-                            <ode />
-                        </contact>
-                        <bounce />
-                        <friction>
-                            <torsional>
-                                <ode />
-                            </torsional>
-                            <ode />
-                        </friction>
-                    </surface>
-                </collision>
-                <visual name='visual'>
-                    <geometry>
-                        <box>
-                            <size>${size} ${size} 0.01</size>
-                        </box>
-                    </geometry>
-                    <material>
-                        <script>
-                            <name>${material}</name>
-                            <uri>file://$(find mirte_gazebo)/media/materials/scripts/duckietown.material</uri>
-                        </script>
-                    </material>
-                </visual>
-                <self_collide>0</self_collide>
-                <enable_wind>0</enable_wind>
-                <kinematic>0</kinematic>
-            </link>
-        </model>
-    </xacro:macro>
-    <xacro:macro name="tileState" params="name material size x y yaw=0">
-        <model name='unit_box_${name}'>
-            <!-- <origin xyz="${x * size} ${y * size} 0" rpy="0 0 ${pi / 180 * yaw}"/> -->
-            <pose>${x * size} ${y * size} 0 -1e-05 -0 ${pi / 180 * yaw}</pose>
-            <size>${size} ${size} 0.01</size>
-            <link name='link'>
-                <!-- <origin xyz="${x * size} ${y * size} 0" rpy="0 0 ${pi / 180 * yaw}"/> -->
-                <pose>${x * size} ${y * size}  0 -1e-05 -0 ${pi / 180 * yaw}</pose>
-                <velocity>0 0 0 0 -0 0</velocity>
-                <acceleration>0.00 0.00 -9.78158 -0.00 0.0 1e-06</acceleration>
-                <wrench>0.000 0.00 -9.78158 0 -0 0</wrench>
-            </link>
-        </model>
-    </xacro:macro>
+  <xacro:macro name="tileWorld" params="name material size x y yaw=0">
+    <model name="unit_box_${name}">
+      <static>1</static>
+      <pose>${x * size} ${y * size} 0. 0 -0 ${pi / 180 * yaw}</pose>
+      <link name="link">
+        <inertial>
+          <mass>1</mass>
+          <inertia>
+            <ixx>0.</ixx>
+            <ixy>0</ixy>
+            <ixz>0</ixz>
+            <iyy>0</iyy>
+            <iyz>0</iyz>
+            <izz>0</izz>
+          </inertia>
+          <pose>0 0 0 0 -0 0</pose>
+        </inertial>
+        <collision name="collision">
+          <geometry>
+            <box>
+              <size>${size} ${size} 0.01</size>
+            </box>
+          </geometry>
+          <max_contacts>10</max_contacts>
+          <surface>
+            <contact>
+              <ode/>
+            </contact>
+            <bounce/>
+            <friction>
+              <torsional>
+                <ode/>
+              </torsional>
+              <ode/>
+            </friction>
+          </surface>
+        </collision>
+        <visual name="visual">
+          <geometry>
+            <box>
+              <size>${size} ${size} 0.01</size>
+            </box>
+          </geometry>
+          <material>
+            <script>
+              <name>${material}</name>
+              <uri>file://$(find mirte_gazebo)/media/materials/scripts/duckietown.material</uri>
+            </script>
+          </material>
+        </visual>
+        <self_collide>0</self_collide>
+        <enable_wind>0</enable_wind>
+        <kinematic>0</kinematic>
+      </link>
+    </model>
+  </xacro:macro>
+  <xacro:macro name="tileState" params="name material size x y yaw=0">
+    <model name="unit_box_${name}">
+      <pose>${x * size} ${y * size} 0 -1e-05 -0 ${pi / 180 * yaw}</pose>
+      <size>${size} ${size} 0.01</size>
+      <link name="link">
+        <pose>${x * size} ${y * size}  0 -1e-05 -0 ${pi / 180 * yaw}</pose>
+        <velocity>0 0 0 0 -0 0</velocity>
+        <acceleration>0.00 0.00 -9.78158 -0.00 0.0 1e-06</acceleration>
+        <wrench>0.000 0.00 -9.78158 0 -0 0</wrench>
+      </link>
+    </model>
+  </xacro:macro>
 </robot>
