Commit message: Stylecheck fixes

File: urdf/realsense-RS200.macro.xacro (robot description, xacro)
@@ -120,5 +120,5 @@
         <pose frame="">0 -0.06 0.004 0 0 0</pose>
         <camera name="${prefix}rs200_camera">
-         <horizontal_fov>1.047</horizontal_fov>
+          <horizontal_fov>1.047</horizontal_fov>
           <!-- <!-<horizontal_fov>2.5</horizontal_fov>/ -->
           <!-- <horizontal_fov>1.5</horizontal_fov> -->
@@ -142,8 +142,8 @@
         <visualize>0</visualize>
       </sensor>
-       <sensor name="${prefix}ired2" type="camera">
+      <sensor name="${prefix}ired2" type="camera">
         <pose frame="">0 0.01 0.004 0 0 0</pose>
         <camera name="${prefix}rs200_camera">
-           <horizontal_fov>1.047</horizontal_fov>
+          <horizontal_fov>1.047</horizontal_fov>
           <!-- <horizontal_fov>2.5</horizontal_fov> -->
           <image>

File: urdf/realsense-depth.xacro (robot description, xacro)
@@ -17,34 +17,33 @@
     <link name="${prefix}rs200_camera">
       <visual>
-        <origin rpy="0 0 0" xyz="0 0 0" />
+        <origin rpy="0 0 0" xyz="0 0 0"/>
         <geometry>
-          <mesh
-            filename="package://realsense_gazebo_plugin/models/realsense_camera/meshes/realsense.dae" />
+          <mesh filename="package://realsense_gazebo_plugin/models/realsense_camera/meshes/realsense.dae"/>
         </geometry>
       </visual>
       <collision>
         <geometry>
-          <box size="0.0078 0.130 0.0192" />
+          <box size="0.0078 0.130 0.0192"/>
         </geometry>
       </collision>
       <inertial>
-        <mass value="0.0615752" />
-        <origin rpy="0 0 0" xyz="0 0 0" />
-        <inertia ixx="9.108e-05" ixy="0" ixz="0" iyy="2.51e-06" iyz="0" izz="8.931e-05" />
+        <mass value="0.0615752"/>
+        <origin rpy="0 0 0" xyz="0 0 0"/>
+        <inertia ixx="9.108e-05" ixy="0" ixz="0" iyy="2.51e-06" iyz="0" izz="8.931e-05"/>
       </inertial>
     </link>
     <!-- Connect camera to parent frame-->
     <joint name="${prefix}realsense_joint" type="fixed">
-      <parent link="${parent}" />
-      <child link="${prefix}rs200_camera" />
-      <xacro:insert_block name="origin" />
+      <parent link="${parent}"/>
+      <child link="${prefix}rs200_camera"/>
+      <xacro:insert_block name="origin"/>
     </joint>
     <!-- Virtual links representing the cameras positons and orientations-->
-    <link name="${prefix}depth" />
+    <link name="${prefix}depth"/>
     <!-- Joints positioning the virtual links with respect to the camera main link-->
     <joint name="${prefix}depth_joint" type="fixed">
-      <parent link="${prefix}rs200_camera" />
-      <child link="${prefix}depth" />
-      <origin xyz="0 -0 0.004" rpy="0 0 0" />
+      <parent link="${prefix}rs200_camera"/>
+      <child link="${prefix}depth"/>
+      <origin xyz="0 -0 0.004" rpy="0 0 0"/>
     </joint>
     <gazebo reference="${prefix}depth">

File: urdf/realsense-lidar.xacro (robot description, xacro)
@@ -17,34 +17,33 @@
     <link name="${prefix}rs200_camera">
       <visual>
-        <origin rpy="0 0 0" xyz="0 0 0" />
+        <origin rpy="0 0 0" xyz="0 0 0"/>
         <geometry>
-          <mesh
-            filename="package://realsense_gazebo_plugin/models/realsense_camera/meshes/realsense.dae" />
+          <mesh filename="package://realsense_gazebo_plugin/models/realsense_camera/meshes/realsense.dae"/>
         </geometry>
       </visual>
       <collision>
         <geometry>
-          <box size="0.0078 0.130 0.0192" />
+          <box size="0.0078 0.130 0.0192"/>
         </geometry>
       </collision>
       <inertial>
-        <mass value="0.0615752" />
-        <origin rpy="0 0 0" xyz="0 0 0" />
-        <inertia ixx="9.108e-05" ixy="0" ixz="0" iyy="2.51e-06" iyz="0" izz="8.931e-05" />
+        <mass value="0.0615752"/>
+        <origin rpy="0 0 0" xyz="0 0 0"/>
+        <inertia ixx="9.108e-05" ixy="0" ixz="0" iyy="2.51e-06" iyz="0" izz="8.931e-05"/>
       </inertial>
     </link>
     <!-- Connect camera to parent frame-->
     <joint name="${prefix}realsense_joint" type="fixed">
-      <parent link="${parent}" />
-      <child link="${prefix}rs200_camera" />
-      <xacro:insert_block name="origin" />
+      <parent link="${parent}"/>
+      <child link="${prefix}rs200_camera"/>
+      <xacro:insert_block name="origin"/>
     </joint>
     <!-- Virtual links representing the cameras positons and orientations-->
-    <link name="${prefix}depth" />
+    <link name="${prefix}depth"/>
     <!-- Joints positioning the virtual links with respect to the camera main link-->
     <joint name="${prefix}depth_joint" type="fixed">
-      <parent link="${prefix}rs200_camera" />
-      <child link="${prefix}depth" />
-      <origin xyz="0 -0.03 0.004" rpy="0 0 0" />
+      <parent link="${prefix}rs200_camera"/>
+      <child link="${prefix}depth"/>
+      <origin xyz="0 -0.03 0.004" rpy="0 0 0"/>
     </joint>
     <gazebo reference="${prefix}depth">
