Commit message: Little cleanup

File: urdf/mirte.xacro (robot description, xacro)
@@ -1,7 +1,8 @@
 <?xml version="1.0" ?>
 <robot name="mirte" xmlns:xacro="http://www.ros.org/wiki/xacro">
-  <xacro:include filename="materials.xacro"/>
-  <xacro:include filename="macros.xacro"/>
-  <xacro:property name="yaml_param_file" value="../config/robot_dimensions.yaml" />
+  <xacro:include filename="$(find mirte_gazebo)/urdf/materials.xacro"/>
+  <xacro:include filename="$(find mirte_gazebo)/urdf/macros.xacro"/>
+  <xacro:include filename="$(find mirte_gazebo)/urdf/ros2_control.xacro"/>
+  <xacro:property name="yaml_param_file" value="$(find mirte_gazebo)/config/mirte_dimensions.yaml" />
   <xacro:property name="params" value="${load_yaml(yaml_param_file)}"/>
   <link name="link_chassis">
@@ -49,8 +50,9 @@
         <box size="0.01 0.05 0.037"/>
       </geometry>
-    </visual>    <inertial>
-      <mass value="1e-5" />
+    </visual>
+    <inertial>
+      <mass value="0.0" />
       <origin xyz="0 0 0" rpy="0 0 0"/>
-      <inertia ixx="1e-6" ixy="0" ixz="0" iyy="1e-6" iyz="0" izz="1e-6" />
+      <inertia ixx="0.0" ixy="0.0" ixz="0.0" iyy="0.0" iyz="0.0" izz="0.0" />
     </inertial>
  </link>
@@ -58,4 +60,5 @@
     <origin rpy=" 0 0 0" xyz="${params['caster_wheel_center_x_offset']} ${params['caster_wheel_center_y_offset']} ${params['caster_wheel_center_z_offset']}"/>
   </xacro:caster>
+  <!-- NOTE: xacro parser adds joint_ -->
   <xacro:wheel name="left_wheel" parent="link_chassis" radius="${params['wheel_radius']}" mass="${params['wheel_mass']}">
     <origin rpy="0 0 0" xyz="${params['wheel_center_x_offset']} ${params['wheel_center_y_offset']} ${params['wheel_center_z_offset']}"/>
@@ -65,4 +68,5 @@
     </joint_options>
   </xacro:wheel>
+  <!-- NOTE: xacro parser adds joint_ -->
   <xacro:wheel name="right_wheel" parent="link_chassis" radius="${params['wheel_radius']}" mass="${params['wheel_mass']}">
     <origin rpy="0 0 0" xyz="${params['wheel_center_x_offset']} ${-1*params['wheel_center_y_offset']} ${params['wheel_center_z_offset']}"/>

Commit message: Added meshes

File: urdf/mirte.xacro (robot description, xacro)
@@ -17,6 +17,5 @@
     <collision name="collision_chassis">
       <geometry>
-        <box size="${params['base_len']} ${params['base_width']} ${params['base_height']}"/>
-        <!-- <mesh filename="package://mirte_gazebo/meshes/mirte_base.stl" scale="0.001 0.001 0.001"/> -->
+        <mesh filename="file://$(find mirte_gazebo)/meshes/mirte_base.stl" scale="0.001 0.001 0.001"/> -->
       </geometry>
     </collision>
@@ -24,6 +23,5 @@
       <origin rpy="0 0 0" xyz="0 0 0"/>
       <geometry>
-        <box size="${params['base_len']} ${params['base_width']} ${params['base_height']}"/>
-        <!-- <mesh filename="package://mirte_gazebo/meshes/mirte_base.stl" scale="0.001 0.001 0.001"/> -->
+        <mesh filename="file://$(find mirte_gazebo)/meshes/mirte_base.stl" scale="0.001 0.001 0.001"/>
       </geometry>
       <material name="blue"/>

Commit message: Fixes for ROS1 first launch

File: urdf/mirte.xacro (robot description, xacro)
@@ -18,5 +18,5 @@
     <collision name="collision_chassis">
       <geometry>
-        <mesh filename="file://$(find mirte_gazebo)/meshes/mirte_base.stl" scale="0.001 0.001 0.001"/> -->
+        <mesh filename="file://$(find mirte_gazebo)/meshes/mirte_base.stl" scale="0.001 0.001 0.001"/>
       </geometry>
     </collision>

Commit message: Add launch arguments

File: urdf/mirte.xacro (robot description, xacro)
@@ -1,11 +1,27 @@
 <?xml version="1.0"?>
 <robot xmlns:xacro="http://www.ros.org/wiki/xacro" name="mirte">
+  <xacro:arg name="sonar_enable" default="true"/>
+  <xacro:arg name="intensity_enable" default="true"/>
+  <xacro:arg name="camera_enable" default="true"/>
+  <xacro:arg name="lidar_enable" default="true"/>
   <xacro:include filename="$(find mirte_gazebo)/urdf/materials.xacro"/>
   <xacro:include filename="$(find mirte_gazebo)/urdf/macros.xacro"/>
   <xacro:include filename="$(find mirte_gazebo)/urdf/ros_control.xacro"/>
-  <xacro:include filename="$(find mirte_gazebo)/urdf/lidar.xacro"/>
-  <xacro:include filename="$(find mirte_gazebo)/urdf/ir.xacro"/>
-  <!-- <xacro:include filename="$(find mirte_gazebo)/urdf/camera.xacro" /> -->
-  <xacro:include filename="$(find mirte_gazebo)/urdf/ultrasonic.xacro"/>
+  <test value="$(arg sonar_enable)" name="sonar_enable"/>
+  <test value="$(arg intensity_enable)" name="intensity_enable"/>
+  <test value="$(arg camera_enable)" name="camera_enable"/>
+  <test value="$(arg lidar_enable)" name="lidar_enable"/>
+  <xacro:if value="$(arg lidar_enable)">
+    <xacro:include filename="$(find mirte_gazebo)/urdf/lidar.xacro"/>
+  </xacro:if>
+  <xacro:if value="$(arg intensity_enable)">
+    <xacro:include filename="$(find mirte_gazebo)/urdf/ir.xacro"/>
+  </xacro:if>
+  <xacro:if value="$(arg camera_enable)">
+    <xacro:include filename="$(find mirte_gazebo)/urdf/camera.xacro"/>
+  </xacro:if>
+  <xacro:if value="$(arg sonar_enable)">
+    <xacro:include filename="$(find mirte_gazebo)/urdf/ultrasonic.xacro"/>
+  </xacro:if>
   <xacro:property name="yaml_param_file" value="$(find mirte_gazebo)/config/mirte_dimensions.yaml"/>
   <xacro:property name="params" value="${xacro.load_yaml(yaml_param_file)}"/>
@@ -60,16 +76,20 @@
     </joint_options>
   </xacro:wheel>
-  <!-- <xacro:ultrasonic_sensor name="left">
-    <origin rpy="0 0 .45" xyz="0.085 0.04 0.022"/>
-  </xacro:ultrasonic_sensor>
-  <xacro:ultrasonic_sensor name="right">
-    <origin rpy="0 0 -0.45" xyz="0.085 -0.04 0.022"/>
-  </xacro:ultrasonic_sensor> -->
-  <xacro:ir_sensor name="left">
-    <origin rpy="0 ${radians(90)} 0" xyz="0.0785 0.022 0.002"/>
-  </xacro:ir_sensor>
-  <xacro:ir_sensor name="right">
-    <origin rpy="0 ${radians(90)} 0" xyz="0.0785 -0.022 0.002"/>
-  </xacro:ir_sensor>
+  <xacro:if value="$(arg sonar_enable)">
+    <xacro:ultrasonic_sensor name="left">
+      <origin rpy="0 0 .45" xyz="0.085 0.04 0.022"/>
+    </xacro:ultrasonic_sensor>
+    <xacro:ultrasonic_sensor name="right">
+      <origin rpy="0 0 -0.45" xyz="0.085 -0.04 0.022"/>
+    </xacro:ultrasonic_sensor>
+  </xacro:if>
+  <xacro:if value="$(arg intensity_enable)">
+    <xacro:ir_sensor name="left">
+      <origin rpy="0 ${radians(90)} 0" xyz="0.0785 0.022 0.002"/>
+    </xacro:ir_sensor>
+    <xacro:ir_sensor name="right">
+      <origin rpy="0 ${radians(90)} 0" xyz="0.0785 -0.022 0.002"/>
+    </xacro:ir_sensor>
+  </xacro:if>
   <gazebo>
     <plugin name="gazebo_ros_control" filename="libgazebo_ros_control.so">

Commit message: New mirte_base and collision stl

File: urdf/mirte.xacro (robot description, xacro)
@@ -39,5 +39,5 @@
     <collision name="collision_chassis">
       <geometry>
-        <mesh filename="file://$(find mirte_gazebo)/meshes/mirte_base.stl" scale="0.001 0.001 0.001" rpy="0 0 1.57079633"/>
+        <mesh filename="file://$(find mirte_gazebo)/meshes/mirte_base_coll.stl" scale="0.001 0.001 0.001" rpy="0 0 1.57079633"/>
       </geometry>
     </collision>

Commit message: simplify stls for faster rendering

File: urdf/mirte.xacro (robot description, xacro)
@@ -39,5 +39,5 @@
     <collision name="collision_chassis">
       <geometry>
-        <mesh filename="file://$(find mirte_gazebo)/meshes/mirte_base_coll.stl" scale="0.001 0.001 0.001" rpy="0 0 1.57079633"/>
+        <mesh filename="file://$(find mirte_gazebo)/meshes/mirte_base.stl" scale="0.001 0.001 0.001" rpy="0 0 1.57079633"/>
       </geometry>
     </collision>

Commit message: Add collision sensor mirte & realsense

File: urdf/mirte.xacro (robot description, xacro)
@@ -52,4 +52,18 @@
   <gazebo reference="link_chassis">
     <gravity>0</gravity>
+  </gazebo>
+  <gazebo reference="link_chassis">
+    <sensor name="gripper_contact_sensor" type="contact">
+      <always_on>true</always_on>
+      <update_rate>30.0</update_rate>
+      <contact>
+        <collision>base_link_fixed_joint_lump__collision_chassis_collision</collision>
+        <!-- See https://github.com/gazebosim/sdformat/issues/333 for why the strange naming. Get the correct name by running xacro mirte.xacro > test.txt && gz sdf -p test.txt > robot.xml and look for the name-->
+      </contact>
+      <plugin name="gripper_bumper" filename="libgazebo_ros_bumper.so">
+        <bumperTopicName>gripper_contact_sensor_state</bumperTopicName>
+        <frameName>gripper</frameName>
+      </plugin>
+    </sensor>
   </gazebo>
   <link name="base_link"/>

File: urdf/realsense-depth.xacro (robot description, xacro)
@@ -22,5 +22,5 @@
         </geometry>
       </visual>
-      <collision>
+      <collision name="realsense_collision">
         <geometry>
           <box size="0.0078 0.130 0.0192"/>
@@ -47,4 +47,24 @@
       <origin xyz="0 -0 0.004" rpy="0 0 0"/>
     </joint>
+    <gazebo reference="${prefix}rs200_camera">
+      <sensor name="realsense_contact" type="contact">
+        <always_on>true</always_on>
+        <update_rate>30.0</update_rate>
+        <contact>
+          <xacro:property name="lidar" value="$(arg lidar_enable)"/>
+          <xacro:property name="ir" value="$(arg intensity_enable)"/>
+          <test2 name="lidar" value="$(arg lidar_enable)"/>
+          <test2 name="ir" value="$(arg intensity_enable)"/>
+          <arg val="2 + 2xir + lidar"/>
+          <!-- See https://github.com/gazebosim/sdformat/issues/333 for why the strange naming. Get the correct name by running xacro mirte.xacro > test.xml && gz sdf -p test.xml > robot.xml and look for the name-->
+          <!-- This strange calculation should make sure that when adding/removing lidar and ir sensors, the collision name still is correct -->
+          <collision>base_link_fixed_joint_lump__realsense_collision_collision_${lidar + 2*ir + 2}</collision>
+        </contact>
+        <plugin name="gripper_bumper" filename="libgazebo_ros_bumper.so">
+          <bumperTopicName>realsense_bumper</bumperTopicName>
+          <frameName>${prefix}rs200_camera</frameName>
+        </plugin>
+      </sensor>
+    </gazebo>
     <gazebo reference="${prefix}depth">
       <sensor name="depth_camera" type="depth">
