Commit message: Added 2 sonars

File: urdf/lidar.xacro (robot description, xacro)
@@ -10,5 +10,5 @@
         <sensor name="lidar" type="ray">
             <pose> 0 0 0 0 0 0 </pose>
-            <visualize>true</visualize>
+            <visualize>false</visualize>
             <update_rate>15</update_rate>
             <ray>

File: urdf/materials.xacro (robot description, xacro)
@@ -24,4 +24,7 @@
   <material name="white">
     <color rgba="1.0 1.0 1.0 1.0"/>
+  </material>
+  <material name="wood">
+    <color rgba="1.0 0.0 1.0 1.0"/>
   </material>
   <gazebo reference="link_chassis">

File: urdf/mirte.xacro (robot description, xacro)
@@ -6,4 +6,5 @@
   <xacro:include filename="$(find mirte_gazebo)/urdf/lidar.xacro"/>
   <xacro:include filename="$(find mirte_gazebo)/urdf/camera.xacro"/>
+  <xacro:include filename="$(find mirte_gazebo)/urdf/ultrasonic.xacro"/>
   <xacro:property name="yaml_param_file" value="$(find mirte_gazebo)/config/mirte_dimensions.yaml" />
   <xacro:property name="params" value="${load_yaml(yaml_param_file)}"/>
@@ -33,28 +34,4 @@
     <child link="link_chassis"/>
   </joint>
-<joint name="sonar_front_joint" type="fixed">
-    <axis xyz="0 1 0" />
-    <origin rpy="0 0 0" xyz="0.093 0 0.02" />
-    <parent link="link_chassis"/>
-    <child link="base_sonar_front"/>
-</joint>
-<link name="base_sonar_front">
-    <collision>
-      <origin xyz="0 0 0" rpy="0 0 0"/>
-      <geometry>
-        <box size="0.01 0.05 0.037"/>
-      </geometry>
-    </collision>    <visual>
-      <origin xyz="0 0 0" rpy="0 0 0"/>
-      <geometry>
-        <box size="0.01 0.05 0.037"/>
-      </geometry>
-    </visual>
-    <inertial>
-      <mass value="0.0" />
-      <origin xyz="0 0 0" rpy="0 0 0"/>
-      <inertia ixx="0.0" ixy="0.0" ixz="0.0" iyy="0.0" iyz="0.0" izz="0.0" />
-    </inertial>
- </link>
   <xacro:caster name="caster_wheel_back" parent="link_chassis" radius="${params['caster_wheel_radius']}" mass="${params['caster_wheel_mass']}">
     <origin rpy=" 0 0 0" xyz="${params['caster_wheel_center_x_offset']} ${params['caster_wheel_center_y_offset']} ${params['caster_wheel_center_z_offset']}"/>
@@ -76,48 +53,9 @@
     </joint_options>
   </xacro:wheel>
-<!--
- <gazebo>
-   <plugin name="gazebo_ros_control" filename="libgazebo_ros_control.so">
-     <robotNamespace>/mirte</robotNamespace>
-     <robotSimType>gazebo_ros_control/DefaultRobotHWSim</robotSimType>
-   </plugin>
- </gazebo>
-<gazebo reference="base_sonar_front">
-   <sensor type="ray" name="TeraRanger">
-      <pose>0 0 0 0 0 0</pose>
-      <visualize>false</visualize>
-      <update_rate>12</update_rate>
-      <ray>
-         <scan>
-            <horizontal>
-               <samples>1</samples>
-               <resolution>1</resolution>
-               <min_angle>-0.14835</min_angle>
-               <max_angle>0.14835</max_angle>
-            </horizontal>
-            <vertical>
-               <samples>1</samples>
-               <resolution>1</resolution>
-               <min_angle>-0.014835</min_angle>
-               <max_angle>0.014835</max_angle>
-            </vertical>
-         </scan>
-         <range>
-            <min>0.01</min>
-            <max>2</max>
-            <resolution>0.01</resolution>
-         </range>
-      </ray>
-      <plugin filename="libgazebo_ros_range.so" name="gazebo_ros_range">
-         <gaussianNoise>0.005</gaussianNoise>
-         <alwaysOn>true</alwaysOn>
-         <updateRate>12</updateRate>
-         <topicName>sensor/ir_front</topicName>
-         <frameName>base_sonar_front</frameName>
-         <radiation>ULTRASOUND</radiation>
-         <fov>0.2967</fov>
-      </plugin>
-   </sensor>
-   </gazebo>
--->
+  <xacro:ultrasonic_sensor name="left">
+    <origin rpy="0 0 .45" xyz="0.085 0.04 0.022" />
+  </xacro:ultrasonic_sensor>
+  <xacro:ultrasonic_sensor name="right">
+    <origin rpy="0 0 -0.45" xyz="0.085 -0.04 0.022" />
+  </xacro:ultrasonic_sensor>
 </robot>

Commit message: Add lidar

File: urdf/lidar.xacro (robot description, xacro)
@@ -2,5 +2,5 @@
 <robot xmlns:xacro="http://www.ros.org/wiki/xacro">
   <joint name="lidar" type="fixed">
-    <origin rpy="0 0 0" xyz="0 0 0.6" />
+    <origin rpy="0 0 0" xyz="0 0 0.1" />
     <parent link="link_chassis" />
     <child link="lidar_link" />
@@ -10,5 +10,5 @@
     <sensor name="lidar" type="ray">
       <pose>0 0 0 0 0 0</pose>
-      <visualize>false</visualize>
+      <visualize>true</visualize>
       <update_rate>15</update_rate>
       <ray>
@@ -22,5 +22,5 @@
         </scan>
         <range>
-          <min>2</min>
+          <min>0.1</min>
           <max>12</max>
           <resolution>0.1</resolution>

File: urdf/mirte.xacro (robot description, xacro)
@@ -3,8 +3,8 @@
   <xacro:include filename="$(find mirte_gazebo)/urdf/materials.xacro" />
   <xacro:include filename="$(find mirte_gazebo)/urdf/macros.xacro" />
-  <!-- <xacro:include filename="$(find mirte_gazebo)/urdf/ros_control.xacro" /> -->
+  <xacro:include filename="$(find mirte_gazebo)/urdf/ros_control.xacro" />
   <xacro:include filename="$(find mirte_gazebo)/urdf/lidar.xacro" />
   <xacro:include filename="$(find mirte_gazebo)/urdf/camera.xacro" />
-  <!--  <xacro:include filename="$(find mirte_gazebo)/urdf/ultrasonic.xacro"/> -->
+   <xacro:include filename="$(find mirte_gazebo)/urdf/ultrasonic.xacro"/>
   <xacro:property name="yaml_param_file"
   value="$(find mirte_gazebo)/config/mirte_dimensions.yaml" />
@@ -74,5 +74,4 @@
     </joint_options>
   </xacro:wheel>
-  <!--
   <xacro:ultrasonic_sensor name="left">
     <origin rpy="0 0 .45" xyz="0.085 0.04 0.022" />
@@ -81,11 +80,9 @@
     <origin rpy="0 0 -0.45" xyz="0.085 -0.04 0.022" />
   </xacro:ultrasonic_sensor>
--->
   <gazebo>
     <plugin name="gazebo_ros_control"
     filename="libgazebo_ros_control.so">
       <robotNamespace>/mirte-control</robotNamespace>
-      <parameters>$(find
-      mirte_gazebo)/config/mirte_diff_drive.yaml</parameters>
+      <parameters>$(find mirte_gazebo)/config/mirte_diff_drive.yaml</parameters>
     </plugin>
     <plugin name="gazebo_ros_controller_manager"

Commit message: Add lidar stl on top

File: urdf/lidar.xacro (robot description, xacro)
@@ -2,14 +2,27 @@
 <robot xmlns:xacro="http://www.ros.org/wiki/xacro">
   <joint name="lidar" type="fixed">
-    <origin rpy="0 0 0" xyz="0 0 0.1"/>
+    <origin rpy="0 0 0" xyz="0.012 0 0.105"/>
     <parent link="link_chassis"/>
     <child link="lidar_link"/>
   </joint>
-  <link name="lidar_link"/>
+  <link name="lidar_link">
+  <visual>
+    <origin rpy="0 0 0" xyz="0 0 -0.03"/>
+    <geometry>
+      <mesh filename="file://$(find mirte_gazebo)/meshes/lidar.stl" scale="0.001 0.001 0.001" rpy="0 0 1.57079633"/>
+    </geometry>
+  </visual>
+  <collision>
+    <origin rpy="0 0 0" xyz="0 0 -0.03"/>
+    <geometry>
+      <mesh filename="file://$(find mirte_gazebo)/meshes/lidar.stl" scale="0.001 0.001 0.001" rpy="0 0 1.57079633"/>
+    </geometry>
+  </collision>
+  </link>
   <gazebo reference="lidar_link">
     <sensor name="lidar" type="ray">
       <pose>0 0 0 0 0 0</pose>
       <visualize>false</visualize>
-      <update_rate>15</update_rate>
+      <update_rate>10</update_rate>
       <ray>
         <scan>
@@ -22,7 +35,7 @@
         </scan>
         <range>
-          <min>0.2</min>
+          <min>0.15</min> <!-- bit more than the actual min range of the lidar, but otherwise it will detect the mirte itself-->
           <max>12</max>
-          <resolution>0.1</resolution>
+          <resolution>0.01</resolution>
         </range>
         <noise>

Commit message: Fix lidar styling

File: urdf/lidar.xacro (robot description, xacro)
@@ -7,16 +7,16 @@
   </joint>
   <link name="lidar_link">
-  <visual>
-    <origin rpy="0 0 0" xyz="0 0 -0.03"/>
-    <geometry>
-      <mesh filename="file://$(find mirte_gazebo)/meshes/lidar.stl" scale="0.001 0.001 0.001" rpy="0 0 1.57079633"/>
-    </geometry>
-  </visual>
-  <collision>
-    <origin rpy="0 0 0" xyz="0 0 -0.03"/>
-    <geometry>
-      <mesh filename="file://$(find mirte_gazebo)/meshes/lidar.stl" scale="0.001 0.001 0.001" rpy="0 0 1.57079633"/>
-    </geometry>
-  </collision>
+    <visual>
+      <origin rpy="0 0 0" xyz="0 0 -0.03"/>
+      <geometry>
+        <mesh filename="file://$(find mirte_gazebo)/meshes/lidar.stl" scale="0.001 0.001 0.001" rpy="0 0 1.57079633"/>
+      </geometry>
+    </visual>
+    <collision>
+      <origin rpy="0 0 0" xyz="0 0 -0.03"/>
+      <geometry>
+        <mesh filename="file://$(find mirte_gazebo)/meshes/lidar.stl" scale="0.001 0.001 0.001" rpy="0 0 1.57079633"/>
+      </geometry>
+    </collision>
   </link>
   <gazebo reference="lidar_link">
@@ -35,5 +35,6 @@
         </scan>
         <range>
-          <min>0.15</min> <!-- bit more than the actual min range of the lidar, but otherwise it will detect the mirte itself-->
+          <min>0.15</min>
+          <!-- bit more than the actual min range of the lidar, but otherwise it will detect the mirte itself-->
           <max>12</max>
           <resolution>0.01</resolution>

Commit message: start rsp

File: urdf/lidar.xacro (robot description, xacro)
@@ -2,52 +2,56 @@
 <robot xmlns:xacro="http://www.ros.org/wiki/xacro">
   <joint name="lidar" type="fixed">
-    <origin rpy="0 0 0" xyz="0.012 0 0.105"/>
-    <parent link="link_chassis"/>
-    <child link="lidar_link"/>
+    <origin rpy="0 0 0" xyz="0.012 0 1.105" />
+    <parent link="link_chassis" />
+    <child link="lidar_link" />
   </joint>
   <link name="lidar_link">
     <visual>
-      <origin rpy="0 0 0" xyz="0 0 -0.03"/>
+      <origin rpy="0 0 0" xyz="0 0 -0.03" />
       <geometry>
-        <mesh filename="file://$(find mirte_gazebo)/meshes/lidar.stl" scale="0.001 0.001 0.001" rpy="0 0 1.57079633"/>
+        <mesh filename="file://$(find mirte_gazebo)/meshes/lidar.stl" scale="0.001 0.001 0.001"
+          rpy="0 0 1.57079633" />
       </geometry>
     </visual>
     <collision>
-      <origin rpy="0 0 0" xyz="0 0 -0.03"/>
+      <origin rpy="0 0 0" xyz="0 0 -0.03" />
       <geometry>
-        <mesh filename="file://$(find mirte_gazebo)/meshes/lidar.stl" scale="0.001 0.001 0.001" rpy="0 0 1.57079633"/>
+        <mesh filename="file://$(find mirte_gazebo)/meshes/lidar.stl" scale="0.001 0.001 0.001"
+          rpy="0 0 1.57079633" />
       </geometry>
     </collision>
   </link>
   <gazebo reference="lidar_link">
-    <sensor name="lidar" type="ray">
-      <pose>0 0 0 0 0 0</pose>
-      <visualize>false</visualize>
-      <update_rate>10</update_rate>
+    <sensor name='center_laser_sensor' type='ray'>
       <ray>
         <scan>
           <horizontal>
-            <samples>720</samples>
+            <samples>512</samples>
             <resolution>1</resolution>
             <min_angle>-3.14</min_angle>
             <max_angle>3.14</max_angle>
           </horizontal>
+          <vertical>
+            <samples>16</samples>
+            <min_angle>-0.1</min_angle>
+            <max_angle>-0.35</max_angle>
+          </vertical>
         </scan>
         <range>
-          <min>0.15</min>
-          <!-- bit more than the actual min range of the lidar, but otherwise it will detect the mirte itself-->
-          <max>12</max>
+          <min>0.2</min>
+          <max>30</max>
           <resolution>0.01</resolution>
         </range>
-        <noise>
-          <type>gaussian</type>
-          <mean>0.0</mean>
-          <stddev>0.01</stddev>
-        </noise>
       </ray>
-      <plugin name="ultra_controller" filename="libgazebo_ros_laser.so">
-        <topicName>/mirte/scan</topicName>
+      <plugin name='center_laser' filename='libgazebo_ros_block_laser.so'>
+        <topicName>/prius/center_laser/scan</topicName>
         <frameName>lidar_link</frameName>
+        <gaussianNoise>0.01</gaussianNoise>
+        <robotNamespace>/</robotNamespace>
       </plugin>
+      <always_on>1</always_on>
+      <update_rate>10</update_rate>
+      <visualize>1</visualize>
+      <pose frame=''>0 0.4 1.8 0 0 -1.5707</pose>
     </sensor>
   </gazebo>

Commit message: revert lidar + add duckie material

File: urdf/lidar.xacro (robot description, xacro)
@@ -2,56 +2,52 @@
 <robot xmlns:xacro="http://www.ros.org/wiki/xacro">
   <joint name="lidar" type="fixed">
-    <origin rpy="0 0 0" xyz="0.012 0 1.105" />
-    <parent link="link_chassis" />
-    <child link="lidar_link" />
+    <origin rpy="0 0 0" xyz="0.012 0 0.105"/>
+    <parent link="link_chassis"/>
+    <child link="lidar_link"/>
   </joint>
   <link name="lidar_link">
     <visual>
-      <origin rpy="0 0 0" xyz="0 0 -0.03" />
+      <origin rpy="0 0 0" xyz="0 0 -0.03"/>
       <geometry>
-        <mesh filename="file://$(find mirte_gazebo)/meshes/lidar.stl" scale="0.001 0.001 0.001"
-          rpy="0 0 1.57079633" />
+        <mesh filename="file://$(find mirte_gazebo)/meshes/lidar.stl" scale="0.001 0.001 0.001" rpy="0 0 1.57079633"/>
       </geometry>
     </visual>
     <collision>
-      <origin rpy="0 0 0" xyz="0 0 -0.03" />
+      <origin rpy="0 0 0" xyz="0 0 -0.03"/>
       <geometry>
-        <mesh filename="file://$(find mirte_gazebo)/meshes/lidar.stl" scale="0.001 0.001 0.001"
-          rpy="0 0 1.57079633" />
+        <mesh filename="file://$(find mirte_gazebo)/meshes/lidar.stl" scale="0.001 0.001 0.001" rpy="0 0 1.57079633"/>
       </geometry>
     </collision>
   </link>
   <gazebo reference="lidar_link">
-    <sensor name='center_laser_sensor' type='ray'>
+    <sensor name="lidar" type="ray">
+      <pose>0 0 0 0 0 0</pose>
+      <visualize>true</visualize>
+      <update_rate>10</update_rate>
       <ray>
         <scan>
           <horizontal>
-            <samples>512</samples>
+            <samples>720</samples>
             <resolution>1</resolution>
             <min_angle>-3.14</min_angle>
             <max_angle>3.14</max_angle>
           </horizontal>
-          <vertical>
-            <samples>16</samples>
-            <min_angle>-0.1</min_angle>
-            <max_angle>-0.35</max_angle>
-          </vertical>
         </scan>
         <range>
-          <min>0.2</min>
-          <max>30</max>
+          <min>0.15</min>
+          <!-- bit more than the actual min range of the lidar, but otherwise it will detect the mirte itself-->
+          <max>12</max>
           <resolution>0.01</resolution>
         </range>
+        <noise>
+          <type>gaussian</type>
+          <mean>0.0</mean>
+          <stddev>0.01</stddev>
+        </noise>
       </ray>
-      <plugin name='center_laser' filename='libgazebo_ros_block_laser.so'>
-        <topicName>/prius/center_laser/scan</topicName>
+      <plugin name="ultra_controller" filename="libgazebo_ros_laser.so">
+        <topicName>/mirte/scan</topicName>
         <frameName>lidar_link</frameName>
-        <gaussianNoise>0.01</gaussianNoise>
-        <robotNamespace>/</robotNamespace>
       </plugin>
-      <always_on>1</always_on>
-      <update_rate>10</update_rate>
-      <visualize>1</visualize>
-      <pose frame=''>0 0.4 1.8 0 0 -1.5707</pose>
     </sensor>
   </gazebo>

Commit message: werkende lidar

File: urdf/lidar.xacro (robot description, xacro)
@@ -2,29 +2,34 @@
 <robot xmlns:xacro="http://www.ros.org/wiki/xacro">
   <joint name="lidar" type="fixed">
-    <origin rpy="0 0 0" xyz="0.012 0 0.105"/>
-    <parent link="link_chassis"/>
-    <child link="lidar_link"/>
+    <!-- <origin rpy="0 0 0" xyz=""/> -->
+    <pose>0.012 0 0.105 0 0 0</pose>
+    <parent>link_chassis</parent>
+    <child>lidar_link</child>
   </joint>
   <link name="lidar_link">
-    <visual>
+      <pose>0.012 0 0.105 0 0 0</pose>
+    <visual name="vis_lidar">
       <origin rpy="0 0 0" xyz="0 0 -0.03"/>
       <geometry>
-        <mesh filename="file://$(find mirte_gazebo)/meshes/lidar.stl" scale="0.001 0.001 0.001" rpy="0 0 1.57079633"/>
+        <mesh>
+        <uri>file://$(find mirte_gazebo)/meshes/lidar.stl</uri><scale>0.001 0.001 0.001</scale> <rpy>0 0 1.57079633</rpy></mesh>
       </geometry>
     </visual>
-    <collision>
+    <collision  name="coll_lidar">
       <origin rpy="0 0 0" xyz="0 0 -0.03"/>
       <geometry>
-        <mesh filename="file://$(find mirte_gazebo)/meshes/lidar.stl" scale="0.001 0.001 0.001" rpy="0 0 1.57079633"/>
+        <mesh>
+        <uri>file://$(find mirte_gazebo)/meshes/lidar.stl</uri><scale>0.001 0.001 0.001</scale> <rpy>0 0 1.57079633</rpy></mesh>
       </geometry>
     </collision>
-  </link>
-  <gazebo reference="lidar_link">
-    <sensor name="lidar" type="ray">
-      <pose>0 0 0 0 0 0</pose>
-      <visualize>true</visualize>
-      <update_rate>10</update_rate>
-      <ray>
-        <scan>
+  <!-- <sensor name="hls_lfcd_lds" type="gpu_lidar">
+  <always_on>true</always_on>
+  <visualize>true</visualize>
+    <pose>0.012 0 0.205 0 0 0</pose>
+  <update_rate>5</update_rate>
+  <topic>scan</topic>
+  <gz_frame_id>base_scan</gz_frame_id>
+  <lidar>
+<scan>
           <horizontal>
             <samples>720</samples>
@@ -36,5 +41,5 @@
         <range>
           <min>0.15</min>
-          <!-- bit more than the actual min range of the lidar, but otherwise it will detect the mirte itself-->
+          <!- - bit more than the actual min range of the lidar, but otherwise it will detect the mirte itself- ->
           <max>12</max>
           <resolution>0.01</resolution>
@@ -44,5 +49,41 @@
           <mean>0.0</mean>
           <stddev>0.01</stddev>
-        </noise>
+        </noise>  </lidar>
+</sensor> -->
+<sensor name="hls_lfcd_lds" type="gpu_lidar">
+        <always_on>true</always_on>
+        <visualize>true</visualize>
+        <pose>-0.064 0 0.221 0 0 0</pose>
+        <update_rate>5</update_rate>
+        <topic>scan</topic>
+        <gz_frame_id>lidar_link</gz_frame_id>
+        <lidar>
+          <scan>
+            <horizontal>
+              <samples>360</samples>
+              <resolution>1.000000</resolution>
+              <min_angle>0.000000</min_angle>
+              <max_angle>6.280000</max_angle>
+            </horizontal>
+          </scan>
+          <range>
+            <min>0.120000</min>
+            <max>3.5</max>
+            <resolution>0.015000</resolution>
+          </range>
+          <noise>
+            <type>gaussian</type>
+            <mean>0.0</mean>
+            <stddev>0.01</stddev>
+          </noise>
+        </lidar>
+      </sensor>
+  </link>
+  <!-- <gazebo reference="lidar_link">
+    <sensor name="lidar" type="ray">
+      <pose>0 0 0 0 0 0</pose>
+      <visualize>true</visualize>
+      <update_rate>10</update_rate>
+      <ray>
       </ray>
       <plugin name="ultra_controller" filename="libgazebo_ros_laser.so">
@@ -51,4 +92,4 @@
       </plugin>
     </sensor>
-  </gazebo>
+  </gazebo> -->
 </robot>

File: urdf/macros.xacro (robot description, xacro)
@@ -32,11 +32,11 @@
     </inertial>
   </xacro:macro>
-  <xacro:macro name="wheel" params="name parent radius mass visualRot *pose **content">
+  <xacro:macro name="wheel" params="name parent radius mass visualRot  *pose **content">
     <link name="link_${name}">
-    <pose>0 1.5707 1.5707 0 0 0</pose>
+  <xacro:insert_block name="pose"/>
       <xacro:inertia_cylinder r="${radius}" h="0.015" mass="${mass}">
       </xacro:inertia_cylinder>
       <collision name="link_${name}_collision">
-        <origin> <rpy>0 1.5707 1.5707</rpy><xyz>0 0 0</xyz></origin>
+        <!-- <origin> <rpy>0 1.5707 1.5707</rpy><xyz>0 0 0</xyz></origin> -->
         <geometry>
           <cylinder>
@@ -61,7 +61,7 @@
       </visual> -->
       <visual name="link_${name}_visual">
-        <origin rpy="0 1.5707 ${1.5707 + visualRot*pi}" xyz="-0 0.0 0"/>
+        <!-- <origin rpy="0 1.5707 ${1.5707 + visualRot*pi}" xyz="-0 0.0 0"/> -->
         <geometry>
-        <pose>0 0 ${pi*0 + visualRot*pi}</pose>
+        <!-- <pose>0 0 ${pi*0 + visualRot*pi}</pose> -->
         <mesh>
         <uri>file://$(find mirte_gazebo)/meshes/wheel.stl</uri>
@@ -91,8 +91,8 @@
     </transmission>
   </xacro:macro>
-  <xacro:macro name="caster" params="name parent radius mass *origin">
+  <xacro:macro name="caster" params="name parent radius mass *pose">
     <link name="link_${name}">
+            <xacro:insert_block name="pose"/>
       <collision name="link_${name}_collision">
-        <xacro:insert_block name="origin"/>
         <geometry>
           <sphere> <radius>${radius}</radius></sphere>
@@ -108,5 +108,6 @@
       </collision>
       <visual name="vis_${name}_sphere">
-        <xacro:insert_block name="origin"/>
+              <origin/>
+        <!-- <xacro:insert_block name="origin"/> -->
         <geometry>
           <sphere> <radius>${radius}</radius></sphere>
@@ -116,5 +117,6 @@
       </visual>
       <xacro:inertia_sphere r="${radius}" mass="${mass}">
-        <xacro:insert_block name="origin"/>
+        <!-- <xacro:insert_block name="origin"/> -->
+        <origin/>
       </xacro:inertia_sphere>
     </link>

File: urdf/mirte.xacro (robot description, xacro)
@@ -79,9 +79,10 @@
   </joint>
   <xacro:caster name="caster_wheel_back" parent="link_chassis" radius="${params['caster_wheel_radius']}" mass="${params['caster_wheel_mass']}">
-    <origin rpy="0 0 0" xyz="${params['caster_wheel_center_x_offset']} ${params['caster_wheel_center_y_offset']} ${params['caster_wheel_center_z_offset']}"/>
+  <pose>${params['caster_wheel_center_x_offset']} ${params['caster_wheel_center_y_offset']} ${params['caster_wheel_center_z_offset']} 0 0 0</pose>
   </xacro:caster>
   <!-- NOTE: xacro parser adds joint_ -->
   <xacro:wheel name="left_wheel" parent="link_chassis" radius="${params['wheel_radius']}" visualRot="1" mass="${params['wheel_mass']}">
-    <origin><rpy>0 0 0</rpy><xyz>${params['wheel_center_x_offset']} ${params['wheel_center_y_offset']} ${params['wheel_center_z_offset']}</xyz></origin>
+        <pose>${params['wheel_center_x_offset']} ${params['wheel_center_y_offset']} ${params['wheel_center_z_offset']} ${pi/2} ${pi/2} 0</pose>
+    <!-- <origin><rpy>0 0 0</rpy><xyz>${params['wheel_center_x_offset']} ${params['wheel_center_y_offset']} ${params['wheel_center_z_offset']}</xyz></origin> -->
     <joint_options>
       <limit effort="10" velocity="8"/>
@@ -91,5 +92,5 @@
   <!-- NOTE: xacro parser adds joint_ -->
   <xacro:wheel name="right_wheel" parent="link_chassis" radius="${params['wheel_radius']}" mass="${params['wheel_mass']}" visualRot="0">
-      <pose>${params['wheel_center_x_offset']} ${-1*params['wheel_center_y_offset']} ${params['wheel_center_z_offset']} 0 0 0</pose>
+      <pose>${params['wheel_center_x_offset']} ${-1*params['wheel_center_y_offset']} ${params['wheel_center_z_offset']} ${pi/2} ${pi/2} ${pi}</pose>
       <!-- <origin><rpy>0 0 0</rpy><xyz></xyz></origin> -->
     <!-- <origin rpy="0 0 0" xyz="${params['wheel_center_x_offset']} ${-1*params['wheel_center_y_offset']} ${params['wheel_center_z_offset']}"/> -->
