Commit message: style updates

File: urdf/lidar.xacro (robot description, xacro)
@@ -8,20 +8,26 @@
   </joint>
   <link name="lidar_link">
-      <pose>0.012 0 0.105 0 0 0</pose>
+    <pose>0.012 0 0.105 0 0 0</pose>
     <visual name="vis_lidar">
       <origin rpy="0 0 0" xyz="0 0 -0.03"/>
       <geometry>
         <mesh>
-        <uri>file://$(find mirte_gazebo)/meshes/lidar.stl</uri><scale>0.001 0.001 0.001</scale> <rpy>0 0 1.57079633</rpy></mesh>
+          <uri>file://$(find mirte_gazebo)/meshes/lidar.stl</uri>
+          <scale>0.001 0.001 0.001</scale>
+          <rpy>0 0 1.57079633</rpy>
+        </mesh>
       </geometry>
     </visual>
-    <collision  name="coll_lidar">
+    <collision name="coll_lidar">
       <origin rpy="0 0 0" xyz="0 0 -0.03"/>
       <geometry>
         <mesh>
-        <uri>file://$(find mirte_gazebo)/meshes/lidar.stl</uri><scale>0.001 0.001 0.001</scale> <rpy>0 0 1.57079633</rpy></mesh>
+          <uri>file://$(find mirte_gazebo)/meshes/lidar.stl</uri>
+          <scale>0.001 0.001 0.001</scale>
+          <rpy>0 0 1.57079633</rpy>
+        </mesh>
       </geometry>
     </collision>
-  <!-- <sensor name="hls_lfcd_lds" type="gpu_lidar">
+    <!-- <sensor name="hls_lfcd_lds" type="gpu_lidar">
   <always_on>true</always_on>
   <visualize>true</visualize>
@@ -51,32 +57,32 @@
         </noise>  </lidar>
 </sensor> -->
-<sensor name="hls_lfcd_lds" type="gpu_lidar">
-        <always_on>true</always_on>
-        <visualize>true</visualize>
-        <pose>-0.064 0 0.221 0 0 0</pose>
-        <update_rate>5</update_rate>
-        <topic>scan</topic>
-        <gz_frame_id>lidar_link</gz_frame_id>
-        <lidar>
-          <scan>
-            <horizontal>
-              <samples>360</samples>
-              <resolution>1.000000</resolution>
-              <min_angle>0.000000</min_angle>
-              <max_angle>6.280000</max_angle>
-            </horizontal>
-          </scan>
-          <range>
-            <min>0.120000</min>
-            <max>3.5</max>
-            <resolution>0.015000</resolution>
-          </range>
-          <noise>
-            <type>gaussian</type>
-            <mean>0.0</mean>
-            <stddev>0.01</stddev>
-          </noise>
-        </lidar>
-      </sensor>
+    <sensor name="hls_lfcd_lds" type="gpu_lidar">
+      <always_on>true</always_on>
+      <visualize>true</visualize>
+      <pose>-0.064 0 0.221 0 0 0</pose>
+      <update_rate>5</update_rate>
+      <topic>scan</topic>
+      <gz_frame_id>lidar_link</gz_frame_id>
+      <lidar>
+        <scan>
+          <horizontal>
+            <samples>360</samples>
+            <resolution>1.000000</resolution>
+            <min_angle>0.000000</min_angle>
+            <max_angle>6.280000</max_angle>
+          </horizontal>
+        </scan>
+        <range>
+          <min>0.120000</min>
+          <max>3.5</max>
+          <resolution>0.015000</resolution>
+        </range>
+        <noise>
+          <type>gaussian</type>
+          <mean>0.0</mean>
+          <stddev>0.01</stddev>
+        </noise>
+      </lidar>
+    </sensor>
   </link>
   <!-- <gazebo reference="lidar_link">

File: urdf/macros.xacro (robot description, xacro)
@@ -3,8 +3,15 @@
   <xacro:macro name="inertia_box" params="x y z mass *origin">
     <inertial>
-      <mass><value>${mass}</value></mass>
+      <mass>
+        <value>${mass}</value>
+      </mass>
       <xacro:insert_block name="origin"/>
       <inertia>
-      <ixx>${mass / 12.0 * (y*y + z*z)}</ixx><ixy>0.0</ixy><ixz>0.0</ixz><iyy>${mass / 12.0 * (z*z + x*x)}</iyy><iyz>0.0</iyz><izz>${mass / 12.0 * (y*y + x*x)}</izz>
+        <ixx>${mass / 12.0 * (y*y + z*z)}</ixx>
+        <ixy>0.0</ixy>
+        <ixz>0.0</ixz>
+        <iyy>${mass / 12.0 * (z*z + x*x)}</iyy>
+        <iyz>0.0</iyz>
+        <izz>${mass / 12.0 * (y*y + x*x)}</izz>
       </inertia>
     </inertial>
@@ -12,7 +19,15 @@
   <xacro:macro name="inertia_cylinder" params="r h mass">
     <inertial>
-      <mass><value>${mass}</value></mass>
+      <mass>
+        <value>${mass}</value>
+      </mass>
       <!-- <xacro:insert_block name="origin"/> -->
-      <inertia><ixx>${mass / 12 * (3*r*r + h*h)}</ixx><ixy>0</ixy><ixz>0</ixz><iyy>${mass / 12 * (3*r*r + h*h)}</iyy><iyz>0</iyz><izz>${mass / 2 * r * r}</izz>
+      <inertia>
+        <ixx>${mass / 12 * (3*r*r + h*h)}</ixx>
+        <ixy>0</ixy>
+        <ixz>0</ixz>
+        <iyy>${mass / 12 * (3*r*r + h*h)}</iyy>
+        <iyz>0</iyz>
+        <izz>${mass / 2 * r * r}</izz>
       </inertia>
     </inertial>
@@ -20,19 +35,21 @@
   <xacro:macro name="inertia_sphere" params="r mass *origin">
     <inertial>
-      <mass><value>${mass}</value></mass>
+      <mass>
+        <value>${mass}</value>
+      </mass>
       <xacro:insert_block name="origin"/>
       <inertia>
-       <ixx>${2/5 * mass * r*r}</ixx>
-       <ixy>0</ixy>
-       <ixz>0</ixz>
-       <iyy>${2/5 * mass * r*r}</iyy>
-       <iyz>0</iyz>
-       <izz>${2/5 * mass * r*r}</izz>
-       </inertia>
+        <ixx>${2/5 * mass * r*r}</ixx>
+        <ixy>0</ixy>
+        <ixz>0</ixz>
+        <iyy>${2/5 * mass * r*r}</iyy>
+        <iyz>0</iyz>
+        <izz>${2/5 * mass * r*r}</izz>
+      </inertia>
     </inertial>
   </xacro:macro>
   <xacro:macro name="wheel" params="name parent radius mass visualRot  *pose **content">
     <link name="link_${name}">
-  <xacro:insert_block name="pose"/>
+      <xacro:insert_block name="pose"/>
       <xacro:inertia_cylinder r="${radius}" h="0.015" mass="${mass}">
       </xacro:inertia_cylinder>
@@ -41,5 +58,6 @@
         <geometry>
           <cylinder>
-          <length>0.015</length> <radius>${radius}</radius>
+            <length>0.015</length>
+            <radius>${radius}</radius>
           </cylinder>
         </geometry>
@@ -63,9 +81,9 @@
         <!-- <origin rpy="0 1.5707 ${1.5707 + visualRot*pi}" xyz="-0 0.0 0"/> -->
         <geometry>
-        <!-- <pose>0 0 ${pi*0 + visualRot*pi}</pose> -->
-        <mesh>
-        <uri>file://$(find mirte_gazebo)/meshes/wheel.stl</uri>
-        <scale>1 1 1</scale>
-        </mesh>
+          <!-- <pose>0 0 ${pi*0 + visualRot*pi}</pose> -->
+          <mesh>
+            <uri>file://$(find mirte_gazebo)/meshes/wheel.stl</uri>
+            <scale>1 1 1</scale>
+          </mesh>
         </geometry>
       </visual>
@@ -75,5 +93,8 @@
       <child>link_${name}</child>
       <parent>${parent}</parent>
-      <axis><rpy>0 0 0</rpy><xyz>0 1 0</xyz></axis>
+      <axis>
+        <rpy>0 0 0</rpy>
+        <xyz>0 1 0</xyz>
+      </axis>
       <xacro:insert_block name="content"/>
     </joint>
@@ -93,8 +114,10 @@
   <xacro:macro name="caster" params="name parent radius mass *pose">
     <link name="link_${name}">
-            <xacro:insert_block name="pose"/>
+      <xacro:insert_block name="pose"/>
       <collision name="link_${name}_collision">
         <geometry>
-          <sphere> <radius>${radius}</radius></sphere>
+          <sphere>
+            <radius>${radius}</radius>
+          </sphere>
         </geometry>
         <surface>
@@ -108,11 +131,14 @@
       </collision>
       <visual name="vis_${name}_sphere">
-              <origin/>
+        <origin/>
         <!-- <xacro:insert_block name="origin"/> -->
         <geometry>
-          <sphere> <radius>${radius}</radius></sphere>
+          <sphere>
+            <radius>${radius}</radius>
+          </sphere>
         </geometry>
         <material>
-        <name>red</name></material>
+          <name>red</name>
+        </material>
       </visual>
       <xacro:inertia_sphere r="${radius}" mass="${mass}">

File: urdf/mirte.xacro (robot description, xacro)
@@ -1,64 +1,70 @@
 <?xml version="1.0"?>
-<sdf xmlns:xacro="http://www.ros.org/wiki/xacro"  version="1.9">
-<model name="mirte">
-  <xacro:arg name="sonar_enable" default="false"/>
-  <xacro:arg name="intensity_enable" default="false"/>
-  <xacro:arg name="camera_enable" default="false"/>
-  <xacro:arg name="lidar_enable" default="false"/>
-  <xacro:arg name="realsense_enable" default="false"/>
-  <!-- <xacro:include filename="$(find mirte_gazebo)/urdf/materials.xacro"/> -->
-  <xacro:include filename="$(find mirte_gazebo)/urdf/macros.xacro"/>
-  <!-- <xacro:include filename="$(find mirte_gazebo)/urdf/ros_control.xacro"/> -->
-  <test value="$(arg sonar_enable)" name="sonar_enable"/>
-  <test value="$(arg intensity_enable)" name="intensity_enable"/>
-  <test value="$(arg camera_enable)" name="camera_enable"/>
-  <test value="$(arg lidar_enable)" name="lidar_enable"/>
-  <xacro:if value="$(arg lidar_enable)">
-    <xacro:include filename="$(find mirte_gazebo)/urdf/lidar.xacro"/>
-  </xacro:if>
-  <xacro:if value="$(arg intensity_enable)">
-    <xacro:include filename="$(find mirte_gazebo)/urdf/ir.xacro"/>
-  </xacro:if>
-  <xacro:if value="$(arg camera_enable)">
-    <xacro:include filename="$(find mirte_gazebo)/urdf/camera.xacro"/>
-  </xacro:if>
-  <xacro:if value="$(arg sonar_enable)">
-    <xacro:include filename="$(find mirte_gazebo)/urdf/ultrasonic.xacro"/>
-  </xacro:if>
-  <xacro:if value="$(arg realsense_enable)">
-    <xacro:include filename="$(find mirte_gazebo)/urdf/realsense.xacro"/>
-  </xacro:if>
-  <xacro:property name="yaml_param_file" value="$(find mirte_gazebo)/config/mirte_dimensions.yaml"/>
-  <xacro:property name="params" value="${xacro.load_yaml(yaml_param_file)}"/>
-  <link name="link_chassis">
-    <!-- pose and inertial -->
-    <pose>0 0 0.015 0 0 0</pose>
-    <xacro:inertia_box x="${params['base_len']}" y="${params['base_width']}" z="${params['base_height']}" mass="${params['base_mass']}">
-      <origin>
-       <rpy>0 0 0</rpy><xyz>0 0 0.015</xyz></origin>
-    </xacro:inertia_box>
-    <!-- body -->
-    <collision name="collision_chassis">
-      <geometry>
-      <pose>0 0 1.57079633</pose>
-        <mesh>
-        <uri>file://$(find mirte_gazebo)/meshes/mirte_base.stl</uri>
-        <scale>0.001 0.001 0.001</scale>
-        </mesh>
-      </geometry>
-    </collision>
-    <visual name="mirte-base">
-    <origin>
-       <rpy>0 0 0</rpy><xyz>0 0 0</xyz></origin>
-      <geometry>
-      <pose>0 0 1.57079633</pose>
-        <mesh>
-        <uri>file://$(find mirte_gazebo)/meshes/mirte_base.stl</uri>
-        <scale>0.001 0.001 0.001</scale>
-        </mesh>
-      </geometry>
-      <material><name>blue</name></material>
-    </visual>
-    <!-- <sensor name="chassis_contact_sensor" type="contact">
+<sdf xmlns:xacro="http://www.ros.org/wiki/xacro" version="1.9">
+  <model name="mirte">
+    <xacro:arg name="sonar_enable" default="false"/>
+    <xacro:arg name="intensity_enable" default="false"/>
+    <xacro:arg name="camera_enable" default="false"/>
+    <xacro:arg name="lidar_enable" default="false"/>
+    <xacro:arg name="realsense_enable" default="false"/>
+    <!-- <xacro:include filename="$(find mirte_gazebo)/urdf/materials.xacro"/> -->
+    <xacro:include filename="$(find mirte_gazebo)/urdf/macros.xacro"/>
+    <!-- <xacro:include filename="$(find mirte_gazebo)/urdf/ros_control.xacro"/> -->
+    <test value="$(arg sonar_enable)" name="sonar_enable"/>
+    <test value="$(arg intensity_enable)" name="intensity_enable"/>
+    <test value="$(arg camera_enable)" name="camera_enable"/>
+    <test value="$(arg lidar_enable)" name="lidar_enable"/>
+    <xacro:if value="$(arg lidar_enable)">
+      <xacro:include filename="$(find mirte_gazebo)/urdf/lidar.xacro"/>
+    </xacro:if>
+    <xacro:if value="$(arg intensity_enable)">
+      <xacro:include filename="$(find mirte_gazebo)/urdf/ir.xacro"/>
+    </xacro:if>
+    <xacro:if value="$(arg camera_enable)">
+      <xacro:include filename="$(find mirte_gazebo)/urdf/camera.xacro"/>
+    </xacro:if>
+    <xacro:if value="$(arg sonar_enable)">
+      <xacro:include filename="$(find mirte_gazebo)/urdf/ultrasonic.xacro"/>
+    </xacro:if>
+    <xacro:if value="$(arg realsense_enable)">
+      <xacro:include filename="$(find mirte_gazebo)/urdf/realsense.xacro"/>
+    </xacro:if>
+    <xacro:property name="yaml_param_file" value="$(find mirte_gazebo)/config/mirte_dimensions.yaml"/>
+    <xacro:property name="params" value="${xacro.load_yaml(yaml_param_file)}"/>
+    <link name="link_chassis">
+      <!-- pose and inertial -->
+      <pose>0 0 0.015 0 0 0</pose>
+      <xacro:inertia_box x="${params['base_len']}" y="${params['base_width']}" z="${params['base_height']}" mass="${params['base_mass']}">
+        <origin>
+          <rpy>0 0 0</rpy>
+          <xyz>0 0 0.015</xyz>
+        </origin>
+      </xacro:inertia_box>
+      <!-- body -->
+      <collision name="collision_chassis">
+        <geometry>
+          <pose>0 0 1.57079633</pose>
+          <mesh>
+            <uri>file://$(find mirte_gazebo)/meshes/mirte_base.stl</uri>
+            <scale>0.001 0.001 0.001</scale>
+          </mesh>
+        </geometry>
+      </collision>
+      <visual name="mirte-base">
+        <origin>
+          <rpy>0 0 0</rpy>
+          <xyz>0 0 0</xyz>
+        </origin>
+        <geometry>
+          <pose>0 0 1.57079633</pose>
+          <mesh>
+            <uri>file://$(find mirte_gazebo)/meshes/mirte_base.stl</uri>
+            <scale>0.001 0.001 0.001</scale>
+          </mesh>
+        </geometry>
+        <material>
+          <name>blue</name>
+        </material>
+      </visual>
+      <!-- <sensor name="chassis_contact_sensor" type="contact">
       <always_on>true</always_on>
       <update_rate>30.0</update_rate>
@@ -72,49 +78,49 @@
       </plugin> - ->
     </sensor> -->
-</link>
-  <link name="base_link"/>
-  <joint name="base_joint" type="fixed">
-    <parent>base_link</parent>
-    <child>link_chassis</child>
-  </joint>
-  <xacro:caster name="caster_wheel_back" parent="link_chassis" radius="${params['caster_wheel_radius']}" mass="${params['caster_wheel_mass']}">
-  <pose>${params['caster_wheel_center_x_offset']} ${params['caster_wheel_center_y_offset']} ${params['caster_wheel_center_z_offset']} 0 0 0</pose>
-  </xacro:caster>
-  <!-- NOTE: xacro parser adds joint_ -->
-  <xacro:wheel name="left_wheel" parent="link_chassis" radius="${params['wheel_radius']}" visualRot="1" mass="${params['wheel_mass']}">
-        <pose>${params['wheel_center_x_offset']} ${params['wheel_center_y_offset']} ${params['wheel_center_z_offset']} ${pi/2} ${pi/2} 0</pose>
-    <!-- <origin><rpy>0 0 0</rpy><xyz>${params['wheel_center_x_offset']} ${params['wheel_center_y_offset']} ${params['wheel_center_z_offset']}</xyz></origin> -->
-    <joint_options>
-      <limit effort="10" velocity="8"/>
-      <dynamics damping="0.0" friction="0.0"/>
-    </joint_options>
-  </xacro:wheel>
-  <!-- NOTE: xacro parser adds joint_ -->
-  <xacro:wheel name="right_wheel" parent="link_chassis" radius="${params['wheel_radius']}" mass="${params['wheel_mass']}" visualRot="0">
+    </link>
+    <link name="base_link"/>
+    <joint name="base_joint" type="fixed">
+      <parent>base_link</parent>
+      <child>link_chassis</child>
+    </joint>
+    <xacro:caster name="caster_wheel_back" parent="link_chassis" radius="${params['caster_wheel_radius']}" mass="${params['caster_wheel_mass']}">
+      <pose>${params['caster_wheel_center_x_offset']} ${params['caster_wheel_center_y_offset']} ${params['caster_wheel_center_z_offset']} 0 0 0</pose>
+    </xacro:caster>
+    <!-- NOTE: xacro parser adds joint_ -->
+    <xacro:wheel name="left_wheel" parent="link_chassis" radius="${params['wheel_radius']}" visualRot="1" mass="${params['wheel_mass']}">
+      <pose>${params['wheel_center_x_offset']} ${params['wheel_center_y_offset']} ${params['wheel_center_z_offset']} ${pi/2} ${pi/2} 0</pose>
+      <!-- <origin><rpy>0 0 0</rpy><xyz>${params['wheel_center_x_offset']} ${params['wheel_center_y_offset']} ${params['wheel_center_z_offset']}</xyz></origin> -->
+      <joint_options>
+        <limit effort="10" velocity="8"/>
+        <dynamics damping="0.0" friction="0.0"/>
+      </joint_options>
+    </xacro:wheel>
+    <!-- NOTE: xacro parser adds joint_ -->
+    <xacro:wheel name="right_wheel" parent="link_chassis" radius="${params['wheel_radius']}" mass="${params['wheel_mass']}" visualRot="0">
       <pose>${params['wheel_center_x_offset']} ${-1*params['wheel_center_y_offset']} ${params['wheel_center_z_offset']} ${pi/2} ${pi/2} ${pi}</pose>
       <!-- <origin><rpy>0 0 0</rpy><xyz></xyz></origin> -->
-    <!-- <origin rpy="0 0 0" xyz="${params['wheel_center_x_offset']} ${-1*params['wheel_center_y_offset']} ${params['wheel_center_z_offset']}"/> -->
-    <joint_options>
-      <limit effort="10" velocity="8"/>
-      <dynamics damping="0.0" friction="0.0"/>
-    </joint_options>
-  </xacro:wheel>
-  <xacro:if value="$(arg sonar_enable)">
-    <xacro:ultrasonic_sensor name="left">
-      <origin rpy="0 0 .45" xyz="0.085 0.04 0.022"/>
-    </xacro:ultrasonic_sensor>
-    <xacro:ultrasonic_sensor name="right">
-      <origin rpy="0 0 -0.45" xyz="0.085 -0.04 0.022"/>
-    </xacro:ultrasonic_sensor>
-  </xacro:if>
-  <xacro:if value="$(arg intensity_enable)">
-    <xacro:ir_sensor name="left">
-      <origin rpy="0 ${radians(90)} 0" xyz="0.0785 0.022 0.002"/>
-    </xacro:ir_sensor>
-    <xacro:ir_sensor name="right">
-      <origin rpy="0 ${radians(90)} 0" xyz="0.0785 -0.022 0.002"/>
-    </xacro:ir_sensor>
-  </xacro:if>
-  <!-- <gazebo>
+      <!-- <origin rpy="0 0 0" xyz="${params['wheel_center_x_offset']} ${-1*params['wheel_center_y_offset']} ${params['wheel_center_z_offset']}"/> -->
+      <joint_options>
+        <limit effort="10" velocity="8"/>
+        <dynamics damping="0.0" friction="0.0"/>
+      </joint_options>
+    </xacro:wheel>
+    <xacro:if value="$(arg sonar_enable)">
+      <xacro:ultrasonic_sensor name="left">
+        <origin rpy="0 0 .45" xyz="0.085 0.04 0.022"/>
+      </xacro:ultrasonic_sensor>
+      <xacro:ultrasonic_sensor name="right">
+        <origin rpy="0 0 -0.45" xyz="0.085 -0.04 0.022"/>
+      </xacro:ultrasonic_sensor>
+    </xacro:if>
+    <xacro:if value="$(arg intensity_enable)">
+      <xacro:ir_sensor name="left">
+        <origin rpy="0 ${radians(90)} 0" xyz="0.0785 0.022 0.002"/>
+      </xacro:ir_sensor>
+      <xacro:ir_sensor name="right">
+        <origin rpy="0 ${radians(90)} 0" xyz="0.0785 -0.022 0.002"/>
+      </xacro:ir_sensor>
+    </xacro:if>
+    <!-- <gazebo>
     <plugin name="gazebo_ros_control" filename="libgazebo_ros_control.so">
       <robotNamespace>/mirte</robotNamespace>
@@ -123,5 +129,5 @@
     <!-- <plugin name="gazebo_ros_controller_manager" filename="libgazebo_ros_controller_manager.so"/> - ->
   </gazebo> -->
-  <!-- <xacro:include filename="$(find mirte_gazebo)/urdf/diffdrive.xacro"/>
+    <!-- <xacro:include filename="$(find mirte_gazebo)/urdf/diffdrive.xacro"/>
   <gazebo>
     <plugin name="p3d" filename="libgazebo_ros_p3d.so">

File: urdf/tileWorld.xacro (robot description, xacro)
@@ -45,6 +45,6 @@
           </geometry>
           <material>
-      <albedo_map>file://$(find mirte_gazebo)/media/materials/textures/${material}.png</albedo_map>
-    <!-- <ambient>1 0 0 1</ambient>
+            <albedo_map>file://$(find mirte_gazebo)/media/materials/textures/${material}.png</albedo_map>
+            <!-- <ambient>1 0 0 1</ambient>
   <diffuse>1 0 0 1</diffuse>
   <specular>0.1 0.1 0.1 1</specular> -->

Commit message: werkende pointcloud

File: urdf/lidar.xacro (robot description, xacro)
@@ -29,32 +29,4 @@
       </geometry>
     </collision>
-    <!-- <sensor name="hls_lfcd_lds" type="gpu_lidar">
-  <always_on>true</always_on>
-  <visualize>true</visualize>
-    <pose>0.012 0 0.205 0 0 0</pose>
-  <update_rate>5</update_rate>
-  <topic>scan</topic>
-  <gz_frame_id>base_scan</gz_frame_id>
-  <lidar>
-<scan>
-          <horizontal>
-            <samples>720</samples>
-            <resolution>1</resolution>
-            <min_angle>-3.14</min_angle>
-            <max_angle>3.14</max_angle>
-          </horizontal>
-        </scan>
-        <range>
-          <min>0.15</min>
-          <!- - bit more than the actual min range of the lidar, but otherwise it will detect the mirte itself- ->
-          <max>12</max>
-          <resolution>0.01</resolution>
-        </range>
-        <noise>
-          <type>gaussian</type>
-          <mean>0.0</mean>
-          <stddev>0.01</stddev>
-        </noise>  </lidar>
-</sensor> -->
     <sensor name="hls_lfcd_lds" type="gpu_lidar">
       <always_on>true</always_on>

File: urdf/mirte.xacro (robot description, xacro)
@@ -20,7 +20,7 @@
       <xacro:include filename="$(find mirte_gazebo)/urdf/ir.xacro"/>
     </xacro:if>
-    <xacro:if value="$(arg camera_enable)">
+    <!-- <xacro:if value="$(arg camera_enable)">
       <xacro:include filename="$(find mirte_gazebo)/urdf/camera.xacro"/>
-    </xacro:if>
+    </xacro:if> -->
     <xacro:if value="$(arg sonar_enable)">
       <xacro:include filename="$(find mirte_gazebo)/urdf/ultrasonic.xacro"/>

File: urdf/realsense-depth.xacro (robot description, xacro)
@@ -43,5 +43,4 @@
     </joint>
     <!-- Virtual links representing the cameras positons and orientations-->
-    <link name="${prefix}depth"/>
     <!-- Joints positioning the virtual links with respect to the camera main link-->
     <joint name="${prefix}depth_joint" type="fixed">
@@ -72,4 +71,5 @@
     </gazebo> -->
     <!-- <gazebo reference="${prefix}depth"> -->
+    <link name="${prefix}depth">
     <sensor name="camera_sensor_depth" type="camera">
   <always_on>true</always_on>
@@ -91,5 +91,5 @@
           </clip>  </camera>
 </sensor>
-      <sensor name="depth_camera1" type="depth_camera">
+      <sensor name="depth_camera1" type="depth">
           <update_rate>10</update_rate>
           <topic>depth_camera</topic>
@@ -107,4 +107,5 @@
           </camera>
           </sensor>
+          </link>
         <!-- <plugin name="depth_camera_controller" filename="libgazebo_ros_depth_camera.so">
           <alwaysOn>1</alwaysOn>
