Commit message: start fix tiles

File: urdf/tileWorld.xacro (robot description, xacro)
@@ -1,62 +1,31 @@
 <?xml version="1.0"?>
 <robot xmlns:xacro="http://www.ros.org/wiki/xacro">
-  <xacro:macro name="tileWorld" params="name material size x y yaw=0">
+  <xacro:macro name="tileWorld" params="name material size x y yaw=0 z_offset=0 model_scale=1 scale=1">
     <model name="unit_box_${name}">
+         <model name="model_${name}">
       <static>1</static>
-      <pose>${x * size} ${y * size} 0. 0 -0 ${pi / 180 * yaw}</pose>
-      <link name="link">
-        <!-- <inertial>
-          <mass>1</mass>
-          <inertia>
-            <ixx>0.</ixx>
-            <ixy>0</ixy>
-            <ixz>0</ixz>
-            <iyy>0</iyy>
-            <iyz>0</iyz>
-            <izz>0</izz>
-          </inertia>
-          <pose>0 0 0 0 -0 0</pose>
-        </inertial> -->
-        <collision name="collision">
-          <geometry>
-            <box>
-              <size>${size} ${size} 0.01</size>
-            </box>
-          </geometry>
-          <max_contacts>10</max_contacts>
-          <surface>
-            <contact>
-              <ode/>
-            </contact>
-            <bounce/>
-            <friction>
-              <torsional>
-                <ode/>
-              </torsional>
-              <ode/>
-            </friction>
-          </surface>
-        </collision>
-        <visual name="visual">
-          <geometry>
-            <box>
-              <size>${size} ${size} 0.01</size>
-            </box>
-          </geometry>
-          <material>
-            <albedo_map>file://$(find mirte_gazebo)/media/materials/textures/${material}.png</albedo_map>
-            <!-- <ambient>1 0 0 1</ambient>
-  <diffuse>1 0 0 1</diffuse>
-  <specular>0.1 0.1 0.1 1</specular> -->
-            <!-- <script>
-              <name>${material}</name>
-              <uri>file://$(find mirte_gazebo)/media/materials/scripts/duckietown.material</uri>
-            </script> -->
-          </material>
-        </visual>
-        <self_collide>0</self_collide>
-        <enable_wind>0</enable_wind>
-        <kinematic>0</kinematic>
-      </link>
+                <pose>${x * size} ${y * size} ${z_offset*size * model_scale * scale + 0.01} ${radians(90)} -0  ${radians(yaw)}</pose>
+    <link name="link_${name}">
+      <collision name="collision_${name}">
+        <geometry>
+          <mesh>
+      <scale>${size * model_scale * scale} ${size * model_scale * scale} ${size * model_scale * scale}</scale>
+            <!-- <scale>0.0254 0.0254 0.0254</scale> -->
+            <uri>model://${material}/meshes/${material}.obj</uri>
+          </mesh>
+        </geometry>
+      </collision>
+      <visual name="visual_${name}">
+        <geometry>
+          <mesh>
+      <pose>${x * size} ${y * size} ${z_offset*size * model_scale * scale + 0.01} ${radians(90)} -0  ${radians(yaw)}</pose>
+      <scale>${size * model_scale * scale} ${size * model_scale * scale} ${size * model_scale * scale}</scale>
+            <!-- <scale>0.0254 0.0254 0.0254</scale> -->
+            <uri>model://${material}/meshes/${material}.obj</uri>
+          </mesh>
+        </geometry>
+      </visual>
+    </link>
+  </model>
     </model>
   </xacro:macro>
