Commit message: Copy over realsense model to remove need for realsense_gazebo_plugin

File: urdf/realsense-depth.xacro (robot description, xacro)
@@ -9,5 +9,5 @@
             * Virtual depth coordinate frame
         Configured to work with Gazebo if desired.
-    Modified by Arend-Jan van Hilten to not visualize the color image, copied from
+    Modified by Arend-Jan van Hilten to not use the other sensors and change depth cam to gazebo depth cam, copied from
 https://github.com/SyrianSpock/realsense_gazebo_plugin
 -->
@@ -19,5 +19,5 @@
         <origin rpy="0 0 0" xyz="0 0 0"/>
         <geometry>
-          <mesh filename="package://realsense_gazebo_plugin/models/realsense_camera/meshes/realsense.dae"/>
+          <mesh filename="package://mirte_gazebo/models/realsense_camera/meshes/realsense.dae"/>
         </geometry>
       </visual>

Commit message: add light + default cam

File: urdf/realsense-depth.xacro (robot description, xacro)
@@ -43,5 +43,5 @@
       </collision>
       <inertial>
-        <mass value="0.0"/>
+        <!-- <mass value="0.0"/> -->
         <!-- <origin rpy="0 0 0" xyz="0 0 0"/> -->
         <inertia>
