Commit message: fixes, but not working yet

File: urdf/macros.xacro (robot description, xacro)
@@ -38,6 +38,5 @@
         <origin rpy="0 1.5707 1.5707" xyz="0 0 0" />
         <geometry>
-          <mesh filename="file://$(find mirte_gazebo)/meshes/mirte_wheel.stl"
-          scale="0.001 0.001 0.001" rpy="0 0 1.57079633" />
+         <cylinder length="0.015" radius="${radius}"/>
         </geometry>
       </collision>
@@ -94,5 +93,5 @@
     </link>
     <gazebo reference="link_${name}">
-      <gravity>1</gravity>
+      <gravity>0</gravity>
     </gazebo>
     <joint name="fixed" type="fixed">

File: urdf/mirte.xacro (robot description, xacro)
@@ -3,5 +3,5 @@
   <xacro:include filename="$(find mirte_gazebo)/urdf/materials.xacro" />
   <xacro:include filename="$(find mirte_gazebo)/urdf/macros.xacro" />
-  <xacro:include filename="$(find mirte_gazebo)/urdf/ros_control.xacro" />
+  <!-- <xacro:include filename="$(find mirte_gazebo)/urdf/ros_control.xacro" /> -->
   <xacro:include filename="$(find mirte_gazebo)/urdf/lidar.xacro" />
   <xacro:include filename="$(find mirte_gazebo)/urdf/camera.xacro" />
@@ -10,5 +10,5 @@
   value="$(find mirte_gazebo)/config/mirte_dimensions.yaml" />
   <xacro:property name="params"
-  value="${load_yaml(yaml_param_file)}" />
+  value="${xacro.load_yaml(yaml_param_file)}" />
   <link name="link_chassis">
     <!-- pose and inertial -->
@@ -83,9 +83,10 @@
 -->
   <gazebo>
-    <!-- <plugin name="gazebo_ros_control" filename="libgazebo_ros_control.so">
+    <plugin name="gazebo_ros_control" filename="libgazebo_ros_control.so">
     <robotNamespace>/mirte-control</robotNamespace>
-  </plugin> -->
-    <plugin name="gazebo_ros_controller_manager"
-    filename="libgazebo_ros_controller_manager.so" />
+    <parameters>$(find mirte_gazebo)/config/mirte_diff_drive.yaml</parameters>
+  </plugin>
+    <!-- <plugin name="gazebo_ros_controller_manager"
+    filename="libgazebo_ros_controller_manager.so" /> -->
   </gazebo>
   <xacro:include filename="$(find mirte_gazebo)/urdf/diffdrive.xacro" />

Commit message: working control

File: urdf/macros.xacro (robot description, xacro)
@@ -29,5 +29,5 @@
   </xacro:macro>
   <xacro:macro name="wheel"
-  params="name parent radius mass *origin **content">
+  params="name parent radius mass visualRot *origin **content">
     <link name="link_${name}">
       <xacro:inertia_cylinder r="${radius}" h="0.015"
@@ -38,12 +38,20 @@
         <origin rpy="0 1.5707 1.5707" xyz="0 0 0" />
         <geometry>
-         <cylinder length="0.015" radius="${radius}"/>
+          <cylinder length="0.015" radius="${radius}" />
         </geometry>
       </collision>
+      <!-- <visual name="link_${name}_visual">
+        <origin rpy="0 1.5707 1.5707"  xyz="-0 0 0" />
+        <geometry>
+          <cylinder color="pink" length="0.015" radius="${radius}"/>
+        </geometry>
+        <material name="red" />
+      </visual> -->
       <visual name="link_${name}_visual">
-        <origin rpy="0 1.5707 1.5707" xyz="0 0 0" />
+        <origin rpy="0 1.5707 ${1.5707 + visualRot*pi}"
+        xyz="-0 0.0 0" />
         <geometry>
-          <mesh filename="file://$(find mirte_gazebo)/meshes/mirte_wheel.stl"
-          scale="0.001 0.001 0.001" rpy="0 0 1.57079633" />
+          <mesh filename="file://$(find mirte_gazebo)/meshes/wheel.stl"
+          scale="1 1 1" rpy="0 0 ${pi*0 + visualRot*pi}" />
         </geometry>
       </visual>

File: urdf/mirte.xacro (robot description, xacro)
@@ -54,5 +54,5 @@
   <!-- NOTE: xacro parser adds joint_ -->
   <xacro:wheel name="left_wheel" parent="link_chassis"
-  radius="${params['wheel_radius']}"
+  radius="${params['wheel_radius']}" visualRot="1"
   mass="${params['wheel_mass']}">
     <origin rpy="0 0 0"
@@ -65,7 +65,7 @@
   <!-- NOTE: xacro parser adds joint_ -->
   <xacro:wheel name="right_wheel" parent="link_chassis"
-  radius="${params['wheel_radius']}"
-  mass="${params['wheel_mass']}">
-    <origin rpy="3.14 0 0"
+  radius="${params['wheel_radius']}" mass="${params['wheel_mass']}"
+  visualRot="0">
+    <origin rpy="0 0 0"
     xyz="${params['wheel_center_x_offset']} ${-1*params['wheel_center_y_offset']} ${params['wheel_center_z_offset']}" />
     <joint_options>
@@ -83,10 +83,12 @@
 -->
   <gazebo>
-    <plugin name="gazebo_ros_control" filename="libgazebo_ros_control.so">
-    <robotNamespace>/mirte-control</robotNamespace>
-    <parameters>$(find mirte_gazebo)/config/mirte_diff_drive.yaml</parameters>
-  </plugin>
-    <!-- <plugin name="gazebo_ros_controller_manager"
-    filename="libgazebo_ros_controller_manager.so" /> -->
+    <plugin name="gazebo_ros_control"
+    filename="libgazebo_ros_control.so">
+      <robotNamespace>/mirte-control</robotNamespace>
+      <parameters>$(find
+      mirte_gazebo)/config/mirte_diff_drive.yaml</parameters>
+    </plugin>
+    <plugin name="gazebo_ros_controller_manager"
+    filename="libgazebo_ros_controller_manager.so" />
   </gazebo>
   <xacro:include filename="$(find mirte_gazebo)/urdf/diffdrive.xacro" />

Commit message: Wider 'realsense' + fixes rsp

File: urdf/macros.xacro (robot description, xacro)
@@ -32,4 +32,12 @@
           <cylinder length="0.015" radius="${radius}"/>
         </geometry>
+        <!-- <surface>
+          <friction>
+            <ode>
+              <mu>1</mu>
+              <mu2>1</mu2>
+            </ode>
+          </friction>
+        </surface> -->
       </collision>
       <!-- <visual name="link_${name}_visual">
@@ -66,5 +74,5 @@
         <hardwareInterface>
           hardware_interface/VelocityJointInterface</hardwareInterface>
-        <mechanicalReduction>120</mechanicalReduction>
+        <mechanicalReduction>1</mechanicalReduction>
       </actuator>
     </transmission>
@@ -77,4 +85,12 @@
           <sphere radius="${radius}"/>
         </geometry>
+        <surface>
+          <friction>
+            <ode>
+              <mu>0.01</mu>
+              <mu2>0.01</mu2>
+            </ode>
+          </friction>
+        </surface>
       </collision>
       <visual>

File: urdf/realsense-depth.xacro (robot description, xacro)
@@ -46,13 +46,13 @@
       <parent link="${prefix}rs200_camera" />
       <child link="${prefix}depth" />
-      <origin xyz="0 -0.03 0.004" rpy="0 0 0" />
+      <origin xyz="0 -0 0.004" rpy="0 0 0" />
     </joint>
     <gazebo reference="${prefix}depth">
       <sensor name="depth_camera" type="depth">
         <always_on>true</always_on>
-        <visualize>true</visualize>
-        <update_rate>5</update_rate>
+        <visualize>False</visualize>
+        <update_rate>10</update_rate>
         <camera name="camera">
-          <horizontal_fov>1.5</horizontal_fov>
+          <horizontal_fov>2.5</horizontal_fov>
           <image>
             <width>640</width>

Commit message: start gazebo fortress

File: urdf/macros.xacro (robot description, xacro)
@@ -3,32 +3,44 @@
   <xacro:macro name="inertia_box" params="x y z mass *origin">
     <inertial>
-      <mass value="${mass}"/>
+      <mass><value>${mass}</value></mass>
       <xacro:insert_block name="origin"/>
-      <inertia ixx="${mass / 12.0 * (y*y + z*z)}" ixy="0.0" ixz="0.0" iyy="${mass / 12.0 * (z*z + x*x)}" iyz="0.0" izz="${mass / 12.0 * (y*y + x*x)}"/>
+      <inertia>
+      <ixx>${mass / 12.0 * (y*y + z*z)}</ixx><ixy>0.0</ixy><ixz>0.0</ixz><iyy>${mass / 12.0 * (z*z + x*x)}</iyy><iyz>0.0</iyz><izz>${mass / 12.0 * (y*y + x*x)}</izz>
+      </inertia>
     </inertial>
   </xacro:macro>
-  <xacro:macro name="inertia_cylinder" params="r h mass *origin">
+  <xacro:macro name="inertia_cylinder" params="r h mass">
     <inertial>
-      <mass value="${mass}"/>
-      <xacro:insert_block name="origin"/>
-      <inertia ixx="${mass / 12 * (3*r*r + h*h)}" ixy="0" ixz="0" iyy="${mass / 12 * (3*r*r + h*h)}" iyz="0" izz="${mass / 2 * r * r}"/>
+      <mass><value>${mass}</value></mass>
+      <!-- <xacro:insert_block name="origin"/> -->
+      <inertia><ixx>${mass / 12 * (3*r*r + h*h)}</ixx><ixy>0</ixy><ixz>0</ixz><iyy>${mass / 12 * (3*r*r + h*h)}</iyy><iyz>0</iyz><izz>${mass / 2 * r * r}</izz>
+      </inertia>
     </inertial>
   </xacro:macro>
   <xacro:macro name="inertia_sphere" params="r mass *origin">
     <inertial>
-      <mass value="${mass}"/>
+      <mass><value>${mass}</value></mass>
       <xacro:insert_block name="origin"/>
-      <inertia ixx="${2/5 * mass * r*r}" ixy="0" ixz="0" iyy="${2/5 * mass * r*r}" iyz="0" izz="${2/5 * mass * r*r}"/>
+      <inertia>
+       <ixx>${2/5 * mass * r*r}</ixx>
+       <ixy>0</ixy>
+       <ixz>0</ixz>
+       <iyy>${2/5 * mass * r*r}</iyy>
+       <iyz>0</iyz>
+       <izz>${2/5 * mass * r*r}</izz>
+       </inertia>
     </inertial>
   </xacro:macro>
-  <xacro:macro name="wheel" params="name parent radius mass visualRot *origin **content">
+  <xacro:macro name="wheel" params="name parent radius mass visualRot *pose **content">
     <link name="link_${name}">
+    <pose>0 1.5707 1.5707 0 0 0</pose>
       <xacro:inertia_cylinder r="${radius}" h="0.015" mass="${mass}">
-        <origin rpy="0 1.5707 1.5707" xyz="0 0 0"/>
       </xacro:inertia_cylinder>
       <collision name="link_${name}_collision">
-        <origin rpy="0 1.5707 1.5707" xyz="0 0 0"/>
+        <origin> <rpy>0 1.5707 1.5707</rpy><xyz>0 0 0</xyz></origin>
         <geometry>
-          <cylinder length="0.015" radius="${radius}"/>
+          <cylinder>
+          <length>0.015</length> <radius>${radius}</radius>
+          </cylinder>
         </geometry>
         <!-- <surface>
@@ -51,16 +63,17 @@
         <origin rpy="0 1.5707 ${1.5707 + visualRot*pi}" xyz="-0 0.0 0"/>
         <geometry>
-          <mesh filename="file://$(find mirte_gazebo)/meshes/wheel.stl" scale="1 1 1" rpy="0 0 ${pi*0 + visualRot*pi}"/>
+        <pose>0 0 ${pi*0 + visualRot*pi}</pose>
+        <mesh>
+        <uri>file://$(find mirte_gazebo)/meshes/wheel.stl</uri>
+        <scale>1 1 1</scale>
+        </mesh>
         </geometry>
       </visual>
     </link>
-    <gazebo reference="link_${name}">
-      <gravity>0</gravity>
-    </gazebo>
-    <joint name="joint_${name}" type="continuous">
-      <xacro:insert_block name="origin"/>
-      <child link="link_${name}"/>
-      <parent link="${parent}"/>
-      <axis rpy="0 0 0" xyz="0 1 0"/>
+    <joint name="joint_${name}" type="revolute">
+      <!-- <xacro:insert_block name="origposein"/> -->
+      <child>link_${name}</child>
+      <parent>${parent}</parent>
+      <axis><rpy>0 0 0</rpy><xyz>0 1 0</xyz></axis>
       <xacro:insert_block name="content"/>
     </joint>
@@ -80,8 +93,8 @@
   <xacro:macro name="caster" params="name parent radius mass *origin">
     <link name="link_${name}">
-      <collision>
+      <collision name="link_${name}_collision">
         <xacro:insert_block name="origin"/>
         <geometry>
-          <sphere radius="${radius}"/>
+          <sphere> <radius>${radius}</radius></sphere>
         </geometry>
         <surface>
@@ -94,10 +107,11 @@
         </surface>
       </collision>
-      <visual>
+      <visual name="vis_${name}_sphere">
         <xacro:insert_block name="origin"/>
         <geometry>
-          <sphere radius="${radius}"/>
+          <sphere> <radius>${radius}</radius></sphere>
         </geometry>
-        <material name="red"/>
+        <material>
+        <name>red</name></material>
       </visual>
       <xacro:inertia_sphere r="${radius}" mass="${mass}">
@@ -109,6 +123,6 @@
     </gazebo>
     <joint name="fixed" type="fixed">
-      <parent link="${parent}"/>
-      <child link="link_${name}"/>
+      <parent>${parent}</parent>
+      <child>link_${name}</child>
     </joint>
   </xacro:macro>

File: urdf/mirte.xacro (robot description, xacro)
@@ -1,12 +1,13 @@
 <?xml version="1.0"?>
-<robot xmlns:xacro="http://www.ros.org/wiki/xacro" name="mirte">
-  <xacro:arg name="sonar_enable" default="true"/>
-  <xacro:arg name="intensity_enable" default="true"/>
-  <xacro:arg name="camera_enable" default="true"/>
-  <xacro:arg name="lidar_enable" default="true"/>
-  <xacro:arg name="realsense_enable" default="true"/>
-  <xacro:include filename="$(find mirte_gazebo)/urdf/materials.xacro"/>
+<sdf xmlns:xacro="http://www.ros.org/wiki/xacro"  version="1.9">
+<model name="mirte">
+  <xacro:arg name="sonar_enable" default="false"/>
+  <xacro:arg name="intensity_enable" default="false"/>
+  <xacro:arg name="camera_enable" default="false"/>
+  <xacro:arg name="lidar_enable" default="false"/>
+  <xacro:arg name="realsense_enable" default="false"/>
+  <!-- <xacro:include filename="$(find mirte_gazebo)/urdf/materials.xacro"/> -->
   <xacro:include filename="$(find mirte_gazebo)/urdf/macros.xacro"/>
-  <xacro:include filename="$(find mirte_gazebo)/urdf/ros_control.xacro"/>
+  <!-- <xacro:include filename="$(find mirte_gazebo)/urdf/ros_control.xacro"/> -->
   <test value="$(arg sonar_enable)" name="sonar_enable"/>
   <test value="$(arg intensity_enable)" name="intensity_enable"/>
@@ -34,44 +35,46 @@
     <pose>0 0 0.015 0 0 0</pose>
     <xacro:inertia_box x="${params['base_len']}" y="${params['base_width']}" z="${params['base_height']}" mass="${params['base_mass']}">
-      <origin rpy="0 0 0" xyz="0 0 0.015"/>
+      <origin>
+       <rpy>0 0 0</rpy><xyz>0 0 0.015</xyz></origin>
     </xacro:inertia_box>
     <!-- body -->
     <collision name="collision_chassis">
       <geometry>
-        <mesh filename="file://$(find mirte_gazebo)/meshes/mirte_base.stl" scale="0.001 0.001 0.001" rpy="0 0 1.57079633"/>
+      <pose>0 0 1.57079633</pose>
+        <mesh>
+        <uri>file://$(find mirte_gazebo)/meshes/mirte_base.stl</uri>
+        <scale>0.001 0.001 0.001</scale>
+        </mesh>
       </geometry>
     </collision>
-    <visual>
-      <origin rpy="0 0 0" xyz="0 0 0"/>
+    <visual name="mirte-base">
+    <origin>
+       <rpy>0 0 0</rpy><xyz>0 0 0</xyz></origin>
       <geometry>
-        <mesh filename="file://$(find mirte_gazebo)/meshes/mirte_base.stl" scale="0.001 0.001 0.001" rpy="0 0 1.57079633"/>
+      <pose>0 0 1.57079633</pose>
+        <mesh>
+        <uri>file://$(find mirte_gazebo)/meshes/mirte_base.stl</uri>
+        <scale>0.001 0.001 0.001</scale>
+        </mesh>
       </geometry>
-      <material name="blue"/>
+      <material><name>blue</name></material>
     </visual>
-  </link>
-  <gazebo reference="link_chassis">
-    <gravity>0</gravity>
-  </gazebo>
-  <gazebo reference="link_chassis">
-    <sensor name="chassis_contact_sensor" type="contact">
+    <!-- <sensor name="chassis_contact_sensor" type="contact">
       <always_on>true</always_on>
       <update_rate>30.0</update_rate>
       <contact>
-        <collision>base_link_fixed_joint_lump__collision_chassis_collision</collision>
-        <!-- See https://github.com/gazebosim/sdformat/issues/333 for why the strange naming. Get the correct name by running xacro mirte.xacro > test.txt && gz sdf -p test.txt > robot.xml and look for the name-->
+        <collision><name>base_link_fixed_joint_lump__collision_chassis_collision</name></collision>
+        <!- - See https://github.com/gazebosim/sdformat/issues/333 for why the strange naming. Get the correct name by running xacro mirte.xacro > test.txt && gz sdf -p test.txt > robot.xml and look for the name- ->
       </contact>
-      <plugin name="gripper_bumper" filename="libgazebo_ros_bumper.so">
+      <!- - <plugin name="gripper_bumper" filename="libgazebo_ros_bumper.so">
         <bumperTopicName>contact</bumperTopicName>
         <frameName>link_chassis</frameName>
-      </plugin>
-    </sensor>
-  </gazebo>
+      </plugin> - ->
+    </sensor> -->
+</link>
   <link name="base_link"/>
-  <gazebo reference="base_link">
-    <gravity>0</gravity>
-  </gazebo>
   <joint name="base_joint" type="fixed">
-    <parent link="base_link"/>
-    <child link="link_chassis"/>
+    <parent>base_link</parent>
+    <child>link_chassis</child>
   </joint>
   <xacro:caster name="caster_wheel_back" parent="link_chassis" radius="${params['caster_wheel_radius']}" mass="${params['caster_wheel_mass']}">
@@ -80,5 +83,5 @@
   <!-- NOTE: xacro parser adds joint_ -->
   <xacro:wheel name="left_wheel" parent="link_chassis" radius="${params['wheel_radius']}" visualRot="1" mass="${params['wheel_mass']}">
-    <origin rpy="0 0 0" xyz="${params['wheel_center_x_offset']} ${params['wheel_center_y_offset']} ${params['wheel_center_z_offset']}"/>
+    <origin><rpy>0 0 0</rpy><xyz>${params['wheel_center_x_offset']} ${params['wheel_center_y_offset']} ${params['wheel_center_z_offset']}</xyz></origin>
     <joint_options>
       <limit effort="10" velocity="8"/>
@@ -88,5 +91,7 @@
   <!-- NOTE: xacro parser adds joint_ -->
   <xacro:wheel name="right_wheel" parent="link_chassis" radius="${params['wheel_radius']}" mass="${params['wheel_mass']}" visualRot="0">
-    <origin rpy="0 0 0" xyz="${params['wheel_center_x_offset']} ${-1*params['wheel_center_y_offset']} ${params['wheel_center_z_offset']}"/>
+      <pose>${params['wheel_center_x_offset']} ${-1*params['wheel_center_y_offset']} ${params['wheel_center_z_offset']} 0 0 0</pose>
+      <!-- <origin><rpy>0 0 0</rpy><xyz></xyz></origin> -->
+    <!-- <origin rpy="0 0 0" xyz="${params['wheel_center_x_offset']} ${-1*params['wheel_center_y_offset']} ${params['wheel_center_z_offset']}"/> -->
     <joint_options>
       <limit effort="10" velocity="8"/>
@@ -110,15 +115,15 @@
     </xacro:ir_sensor>
   </xacro:if>
-  <gazebo>
+  <!-- <gazebo>
     <plugin name="gazebo_ros_control" filename="libgazebo_ros_control.so">
       <robotNamespace>/mirte</robotNamespace>
-      <!-- <parameters>$(find mirte_gazebo)/config/mirte_diff_drive.yaml</parameters> -->
-    </plugin>
-    <!-- <plugin name="gazebo_ros_controller_manager" filename="libgazebo_ros_controller_manager.so"/> -->
-  </gazebo>
-  <xacro:include filename="$(find mirte_gazebo)/urdf/diffdrive.xacro"/>
+      <!- - <parameters>$(find mirte_gazebo)/config/mirte_diff_drive.yaml</parameters> -->
+    <!-- </plugin> -->
+    <!-- <plugin name="gazebo_ros_controller_manager" filename="libgazebo_ros_controller_manager.so"/> - ->
+  </gazebo> -->
+  <!-- <xacro:include filename="$(find mirte_gazebo)/urdf/diffdrive.xacro"/>
   <gazebo>
     <plugin name="p3d" filename="libgazebo_ros_p3d.so">
-      <!-- <robotNamespace>/prius</robotNamespace> -->
+      <!- -  <robotNamespace>/prius</robotNamespace> - ->
       <bodyName>base_link</bodyName>
       <topicName>base_pose_ground_truth</topicName>
@@ -126,4 +131,5 @@
       <updateRate>10.0</updateRate>
     </plugin>
-  </gazebo>
-</robot>
+  </gazebo> -->
+  </model>
+</sdf>

File: urdf/tileWorld.xacro (robot description, xacro)
@@ -6,5 +6,5 @@
       <pose>${x * size} ${y * size} 0. 0 -0 ${pi / 180 * yaw}</pose>
       <link name="link">
-        <inertial>
+        <!-- <inertial>
           <mass>1</mass>
           <inertia>
@@ -17,5 +17,5 @@
           </inertia>
           <pose>0 0 0 0 -0 0</pose>
-        </inertial>
+        </inertial> -->
         <collision name="collision">
           <geometry>
@@ -45,8 +45,12 @@
           </geometry>
           <material>
-            <script>
+      <albedo_map>file://$(find mirte_gazebo)/media/materials/textures/${material}.png</albedo_map>
+    <!-- <ambient>1 0 0 1</ambient>
+  <diffuse>1 0 0 1</diffuse>
+  <specular>0.1 0.1 0.1 1</specular> -->
+            <!-- <script>
               <name>${material}</name>
               <uri>file://$(find mirte_gazebo)/media/materials/scripts/duckietown.material</uri>
-            </script>
+            </script> -->
           </material>
         </visual>
