Commit message: realsense fixes

File: urdf/macros.xacro (robot description, xacro)
@@ -114,4 +114,12 @@
   <xacro:macro name="caster" params="name parent radius mass *pose">
     <link name="link_${name}">
+    <inertial>
+        <mass>
+        4.0</mass>
+        <!-- <origin rpy="0 0 0" xyz="0 0 0"/> -->
+        <inertia>
+         <ixx>9.108e-05</ixx> <ixy>0</ixy><ixz>0</ixz><iyy>2.51e-06</iyy><iyz>0</iyz><izz>8.931e-05</izz>
+         </inertia>
+      </inertial>
       <xacro:insert_block name="pose"/>
       <collision name="link_${name}_collision">

File: urdf/realsense-RS200.macro.xacro (robot description, xacro)
@@ -1,3 +1,4 @@
 <?xml version="1.0"?>
+THIS FILE IS NOT IN USE
 <!--Develped by Daniel Ordonez 22.05.2018 - daniels.ordonez@gmail.com
     INFORMATION:
@@ -16,7 +17,13 @@
     <link name="${prefix}rs200_camera">
       <visual>
-        <origin rpy="0 0 0" xyz="0 0 0"/>
-        <geometry>
-          <mesh filename="package://realsense_gazebo_plugin/models/realsense_camera/meshes/realsense.dae"/>
+    <geometry>
+        <!-- <geometry> -->
+              <mesh>
+                <!-- <scale>0.0254 0.0254 0.0254</scale> -->
+                <uri>model://curve_left_1/meshes/curve_left_1.obj</uri>
+                <!-- <uri>model://realsense_camera/meshes/realsense.obj</uri> -->
+              </mesh>
+            <!-- </geometry> -->
+          <!-- <mesh filename="model://realsense_camera/meshes/realsense.dae"/> -->
         </geometry>
       </visual>

File: urdf/realsense-depth.xacro (robot description, xacro)
@@ -13,12 +13,26 @@
 -->
 <robot xmlns:xacro="http://ros.org/wiki/xacro">
-  <xacro:macro name="realsense-depth" params="prefix parent *origin">
+  <xacro:macro name="realsense-depth" params="prefix parent">
     <!-- Camera link -->
     <link name="${prefix}rs200_camera">
+            <!-- <origin rpy="${pi/2} ${pi/2} ${pi/2}" xyz="0 0 0"/> -->
+          <pose>0.1 0 0.035 0 0 0</pose>
       <visual name="vis_${prefix}_rs200_cam">
-        <origin rpy="0 0 0" xyz="0 0 0"/>
+      <pose>0 0 0 ${pi/2} 0 0</pose>
+       <!-- <origin>
+          <rpy>${pi/2} 0 0</rpy>
+          <xyz>0 0 0</xyz>
+        </origin>     -->
         <geometry>
-          <mesh>
-           <filename>package://mirte_gazebo/models/realsense_camera/meshes/realsense.dae</filename></mesh>
+                <!-- <origin rpy="${pi/2} ${pi/2} ${pi/2}" xyz="0 0 0"/> -->
+        <!-- <geometry> -->
+              <mesh>
+                              <!-- <origin rpy="${pi/2} ${pi/2} ${pi/2}" xyz="0 0 0"/> -->
+                <!-- <scale>0.0254 0.0254 0.0254</scale> -->
+                <!-- <uri>model://curve_left_1/meshes/curve_left_1.obj</uri> -->
+                <uri>model://realsense_camera/meshes/realsense.obj</uri>
+              </mesh>
+            <!-- </geometry> -->
+          <!-- <mesh filename="model://realsense_camera/meshes/realsense.dae"/> -->
         </geometry>
       </visual>
@@ -29,6 +43,6 @@
       </collision>
       <inertial>
-        <mass value="0.0615752"/>
-        <origin rpy="0 0 0" xyz="0 0 0"/>
+        <mass value="0.0"/>
+        <!-- <origin rpy="0 0 0" xyz="0 0 0"/> -->
         <inertia>
          <ixx>9.108e-05</ixx> <ixy>0</ixy><ixz>0</ixz><iyy>2.51e-06</iyy><iyz>0</iyz><izz>8.931e-05</izz>
@@ -40,5 +54,5 @@
       <parent>${parent}</parent>
       <child>${prefix}rs200_camera</child>
-      <xacro:insert_block name="origin"/>
+      <!-- <xacro:insert_block name="origin"/> -->
     </joint>
     <!-- Virtual links representing the cameras positons and orientations-->
@@ -47,5 +61,5 @@
       <parent>${prefix}rs200_camera</parent>
       <child>${prefix}depth</child>
-      <origin xyz="0 -0 0.004" rpy="0 0 0"/>
+      <!-- <origin xyz="0 -0 0.004" rpy="0 0 0"/> -->
     </joint>
     <!-- <gazebo reference="${prefix}rs200_camera"> -->

File: urdf/realsense.xacro (robot description, xacro)
@@ -3,5 +3,4 @@
   <xacro:include filename="$(find mirte_gazebo)/urdf/realsense-depth.xacro"/>
   <xacro:realsense-depth prefix="mirte_" parent="link_chassis">
-    <origin xyz="0.1 0 0.035" rpy="0 0 0"/>
   </xacro:realsense-depth>
 </robot>

Commit message: colors etc, headless

File: urdf/macros.xacro (robot description, xacro)
@@ -83,5 +83,5 @@
           <!-- <pose>0 0 ${pi*0 + visualRot*pi}</pose> -->
           <mesh>
-            <uri>file://$(find mirte_gazebo)/meshes/wheel.stl</uri>
+            <uri>models://wheel/wheel.obj</uri>
             <scale>1 1 1</scale>
           </mesh>

File: urdf/mirte.xacro (robot description, xacro)
@@ -58,11 +58,9 @@
           <pose>0 0 1.57079633</pose>
           <mesh>
-            <uri>file://$(find mirte_gazebo)/meshes/mirte_base.stl</uri>
+            <uri>model://mirte_base/mirte_base.obj</uri>
+            <color>0 0 1 1</color>
             <scale>0.001 0.001 0.001</scale>
           </mesh>
         </geometry>
-        <material>
-          <name>blue</name>
-        </material>
       </visual>
       <!-- <sensor name="chassis_contact_sensor" type="contact">

Commit message: fix pointcloud

File: urdf/macros.xacro (robot description, xacro)
@@ -52,5 +52,5 @@
     <link name="link_${name}">
       <xacro:insert_block name="pose"/>
-      <xacro:inertia_cylinder r="${radius}" h="0.015" mass="${mass}">
+      <xacro:inertia_cylinder r="${radius}" h="0.015" mass="1">
       </xacro:inertia_cylinder>
       <collision name="link_${name}_collision">
@@ -115,9 +115,8 @@
     <link name="link_${name}">
     <inertial>
-        <mass>
-        4.0</mass>
+        <mass>10.0</mass>
         <!-- <origin rpy="0 0 0" xyz="0 0 0"/> -->
         <inertia>
-         <ixx>9.108e-05</ixx> <ixy>0</ixy><ixz>0</ixz><iyy>2.51e-06</iyy><iyz>0</iyz><izz>8.931e-05</izz>
+         <!-- <ixx>9.108e-05</ixx> <ixy>0</ixy><ixz>0</ixz><iyy>2.51e-06</iyy><iyz>0</iyz><izz>8.931e-05</izz> -->
          </inertia>
       </inertial>

File: urdf/realsense-depth.xacro (robot description, xacro)
@@ -87,9 +87,9 @@
     <!-- <gazebo reference="${prefix}depth"> -->
     <link name="${prefix}depth">
-              <pose>0.1 0 0.045 0 0 0</pose>
+              <pose>0.13 0 0.045 0 0 0</pose>
     <sensor name="camera_sensor_depth" type="camera">
   <always_on>true</always_on>
   <visualize>true</visualize>
-  <update_rate>30</update_rate>
+  <update_rate>10</update_rate>
   <topic>camera/image_raw</topic>
   <gz_frame_id>camera_rgb_frame</gz_frame_id>
@@ -107,20 +107,40 @@
           </clip>  </camera>
 </sensor>
-      <sensor name="depth_camera1" type="depth">
+   <sensor name="depth_camera1" type="depth_camera">
+  <always_on>true</always_on>
+  <visualize>true</visualize>
+  <update_rate>10</update_rate>
+  <topic>depth_camera</topic>
+  <gz_frame_id>camera_rgb_frame</gz_frame_id>
+  <camera name="intel_realsense_r200_depth">
+    <!-- <camera_info_topic>camera/camera_info</camera_info_topic> -->
+<horizontal_fov>2.5</horizontal_fov>
+          <image>
+            <width>640</width>
+            <height>480</height>
+            <format>R8G8B8</format>
+          </image>
+          <clip>
+            <near>0.02</near>
+            <far>2</far>
+          </clip>  </camera>
+</sensor>
+      <!-- <sensor name="depth_camera1" type="camera">
           <update_rate>10</update_rate>
-          <topic>depth_camera</topic>
+          <!- - <topic>depth_camera</topic> - ->
+          <topic>camera/image_raw</topic>
           <camera>
-            <horizontal_fov>1.05</horizontal_fov>
+            <horizontal_fov>2.5</horizontal_fov>
             <image>
-              <width>256</width>
-              <height>256</height>
-              <format>R_FLOAT32</format>
+              <width>512</width>
+              <height>512</height>
+              <!- - <format>R_FLOAT32</format> - ->
             </image>
             <clip>
-              <near>0.1</near>
-              <far>10.0</far>
+              <near>0.001</near>
+              <far>2</far>
             </clip>
           </camera>
-          </sensor>
+          </sensor> -->
           </link>
         <!-- <plugin name="depth_camera_controller" filename="libgazebo_ros_depth_camera.so">
