Commit message: Fix stylings

File: urdf/duckieModels.xacro (robot description, xacro)
@@ -2,156 +2,156 @@
 <robot xmlns:xacro="http://www.ros.org/wiki/xacro">
   <xacro:macro name="duckieModel" params="name type size x y yaw=0 static=1 scale=1">
-<model name='model_${name}'>
-  <xacro:property name="model_scale" value="${1}"/>
-  <xacro:property name="z_offset" value="${0}"/>
-    <!-- START GENERATED SCALES AND OFFSETS-->
-    <xacro:if value="${type == 'sign_blank'}">
-      <xacro:property name="model_scale" value="${0.19415283233733935}"/>
-      <xacro:property name="z_offset" value="${0}"/>
-      </xacro:if>
-    <xacro:if value="${type == 'building'}">
-      <xacro:property name="model_scale" value="${0.2898550724637681}"/>
-      <xacro:property name="z_offset" value="${0}"/>
-      </xacro:if>
-    <xacro:if value="${type == 'house'}">
-      <xacro:property name="model_scale" value="${0.20755956855837843}"/>
-      <xacro:property name="z_offset" value="${0.024247}"/>
-      </xacro:if>
-    <xacro:if value="${type == 'cone'}">
-      <xacro:property name="model_scale" value="${0.03172296965063494}"/>
-      <xacro:property name="z_offset" value="${0}"/>
-      </xacro:if>
-    <xacro:if value="${type == 'truck'}">
-      <xacro:property name="model_scale" value="${0.1927574101731193}"/>
-      <xacro:property name="z_offset" value="${1.072166}"/>
-      </xacro:if>
-    <xacro:if value="${type == 'tree'}">
-      <xacro:property name="model_scale" value="${0.28054126509522415}"/>
-      <xacro:property name="z_offset" value="${0.003644}"/>
-      </xacro:if>
-    <xacro:if value="${type == 'duckiebot'}">
-      <xacro:property name="model_scale" value="${8.126777732629012}"/>
-      <xacro:property name="z_offset" value="${0.03311}"/>
-      </xacro:if>
-    <xacro:if value="${type == 'sign_left_T_intersect'}">
-      <xacro:property name="model_scale" value="${4.34593654932638}"/>
-      <xacro:property name="z_offset" value="${0}"/>
-      </xacro:if>
-    <xacro:if value="${type == 'sign_4_way_intersect'}">
-      <xacro:property name="model_scale" value="${4.34593654932638}"/>
-      <xacro:property name="z_offset" value="${0}"/>
-      </xacro:if>
-    <xacro:if value="${type == 'sign_yield'}">
-      <xacro:property name="model_scale" value="${4.34593654932638}"/>
-      <xacro:property name="z_offset" value="${0}"/>
-      </xacro:if>
-    <xacro:if value="${type == 'sign_no_right_turn'}">
-      <xacro:property name="model_scale" value="${4.34593654932638}"/>
-      <xacro:property name="z_offset" value="${0}"/>
-      </xacro:if>
-    <xacro:if value="${type == 'sign_duck_crossing'}">
-      <xacro:property name="model_scale" value="${4.34593654932638}"/>
-      <xacro:property name="z_offset" value="${0}"/>
-      </xacro:if>
-    <xacro:if value="${type == 'sign_no_left_turn'}">
-      <xacro:property name="model_scale" value="${4.34593654932638}"/>
-      <xacro:property name="z_offset" value="${0}"/>
-      </xacro:if>
-    <xacro:if value="${type == 'sign_stop'}">
-      <xacro:property name="model_scale" value="${4.34593654932638}"/>
-      <xacro:property name="z_offset" value="${0}"/>
-      </xacro:if>
-    <xacro:if value="${type == 'sign_do_not_enter'}">
-      <xacro:property name="model_scale" value="${4.34593654932638}"/>
-      <xacro:property name="z_offset" value="${0}"/>
-      </xacro:if>
-    <xacro:if value="${type == 'bus'}">
-      <xacro:property name="model_scale" value="${0.22667415295835838}"/>
-      <xacro:property name="z_offset" value="${-4.396879}"/>
-      </xacro:if>
-    <xacro:if value="${type == 'sign_t_light_ahead'}">
-      <xacro:property name="model_scale" value="${4.34593654932638}"/>
-      <xacro:property name="z_offset" value="${0}"/>
-      </xacro:if>
-    <xacro:if value="${type == 'sign_right_T_intersect'}">
-      <xacro:property name="model_scale" value="${4.34593654932638}"/>
-      <xacro:property name="z_offset" value="${0}"/>
-      </xacro:if>
-    <xacro:if value="${type == 'sign_pedestrian'}">
-      <xacro:property name="model_scale" value="${4.34593654932638}"/>
-      <xacro:property name="z_offset" value="${0}"/>
-      </xacro:if>
-    <xacro:if value="${type == 'sign_oneway_left'}">
-      <xacro:property name="model_scale" value="${4.34593654932638}"/>
-      <xacro:property name="z_offset" value="${0}"/>
-      </xacro:if>
-    <xacro:if value="${type == 'trafficlight'}">
-      <xacro:property name="model_scale" value="${2.7362925425083047}"/>
-      <xacro:property name="z_offset" value="${0.014439}"/>
-      </xacro:if>
-    <xacro:if value="${type == 'sign_oneway_right'}">
-      <xacro:property name="model_scale" value="${4.34593654932638}"/>
-      <xacro:property name="z_offset" value="${0}"/>
-      </xacro:if>
-    <xacro:if value="${type == 'sign_T_intersect'}">
-      <xacro:property name="model_scale" value="${4.34593654932638}"/>
-      <xacro:property name="z_offset" value="${0}"/>
-      </xacro:if>
-    <xacro:if value="${type == 'duckie'}">
-      <xacro:property name="model_scale" value="${0.6585788789802037}"/>
-      <xacro:property name="z_offset" value="${-0.113989}"/>
-      </xacro:if>
-    <xacro:if value="${type == 'barrier'}">
-      <xacro:property name="model_scale" value="${0.8748906386701663}"/>
-      <xacro:property name="z_offset" value="${0}"/>
+    <model name="model_${name}">
+      <xacro:property name="model_scale" value="${1}"/>
+      <xacro:property name="z_offset" value="${0}"/>
+      <!-- START GENERATED SCALES AND OFFSETS-->
+      <xacro:if value="${type == 'sign_blank'}">
+        <xacro:property name="model_scale" value="${0.19415283233733935}"/>
+        <xacro:property name="z_offset" value="${0}"/>
+      </xacro:if>
+      <xacro:if value="${type == 'building'}">
+        <xacro:property name="model_scale" value="${0.2898550724637681}"/>
+        <xacro:property name="z_offset" value="${0}"/>
+      </xacro:if>
+      <xacro:if value="${type == 'house'}">
+        <xacro:property name="model_scale" value="${0.20755956855837843}"/>
+        <xacro:property name="z_offset" value="${0.024247}"/>
+      </xacro:if>
+      <xacro:if value="${type == 'cone'}">
+        <xacro:property name="model_scale" value="${0.03172296965063494}"/>
+        <xacro:property name="z_offset" value="${0}"/>
+      </xacro:if>
+      <xacro:if value="${type == 'truck'}">
+        <xacro:property name="model_scale" value="${0.1927574101731193}"/>
+        <xacro:property name="z_offset" value="${1.072166}"/>
+      </xacro:if>
+      <xacro:if value="${type == 'tree'}">
+        <xacro:property name="model_scale" value="${0.28054126509522415}"/>
+        <xacro:property name="z_offset" value="${0.003644}"/>
+      </xacro:if>
+      <xacro:if value="${type == 'duckiebot'}">
+        <xacro:property name="model_scale" value="${8.126777732629012}"/>
+        <xacro:property name="z_offset" value="${0.03311}"/>
+      </xacro:if>
+      <xacro:if value="${type == 'sign_left_T_intersect'}">
+        <xacro:property name="model_scale" value="${4.34593654932638}"/>
+        <xacro:property name="z_offset" value="${0}"/>
+      </xacro:if>
+      <xacro:if value="${type == 'sign_4_way_intersect'}">
+        <xacro:property name="model_scale" value="${4.34593654932638}"/>
+        <xacro:property name="z_offset" value="${0}"/>
+      </xacro:if>
+      <xacro:if value="${type == 'sign_yield'}">
+        <xacro:property name="model_scale" value="${4.34593654932638}"/>
+        <xacro:property name="z_offset" value="${0}"/>
+      </xacro:if>
+      <xacro:if value="${type == 'sign_no_right_turn'}">
+        <xacro:property name="model_scale" value="${4.34593654932638}"/>
+        <xacro:property name="z_offset" value="${0}"/>
+      </xacro:if>
+      <xacro:if value="${type == 'sign_duck_crossing'}">
+        <xacro:property name="model_scale" value="${4.34593654932638}"/>
+        <xacro:property name="z_offset" value="${0}"/>
+      </xacro:if>
+      <xacro:if value="${type == 'sign_no_left_turn'}">
+        <xacro:property name="model_scale" value="${4.34593654932638}"/>
+        <xacro:property name="z_offset" value="${0}"/>
+      </xacro:if>
+      <xacro:if value="${type == 'sign_stop'}">
+        <xacro:property name="model_scale" value="${4.34593654932638}"/>
+        <xacro:property name="z_offset" value="${0}"/>
+      </xacro:if>
+      <xacro:if value="${type == 'sign_do_not_enter'}">
+        <xacro:property name="model_scale" value="${4.34593654932638}"/>
+        <xacro:property name="z_offset" value="${0}"/>
+      </xacro:if>
+      <xacro:if value="${type == 'bus'}">
+        <xacro:property name="model_scale" value="${0.22667415295835838}"/>
+        <xacro:property name="z_offset" value="${-4.396879}"/>
+      </xacro:if>
+      <xacro:if value="${type == 'sign_t_light_ahead'}">
+        <xacro:property name="model_scale" value="${4.34593654932638}"/>
+        <xacro:property name="z_offset" value="${0}"/>
+      </xacro:if>
+      <xacro:if value="${type == 'sign_right_T_intersect'}">
+        <xacro:property name="model_scale" value="${4.34593654932638}"/>
+        <xacro:property name="z_offset" value="${0}"/>
+      </xacro:if>
+      <xacro:if value="${type == 'sign_pedestrian'}">
+        <xacro:property name="model_scale" value="${4.34593654932638}"/>
+        <xacro:property name="z_offset" value="${0}"/>
+      </xacro:if>
+      <xacro:if value="${type == 'sign_oneway_left'}">
+        <xacro:property name="model_scale" value="${4.34593654932638}"/>
+        <xacro:property name="z_offset" value="${0}"/>
+      </xacro:if>
+      <xacro:if value="${type == 'trafficlight'}">
+        <xacro:property name="model_scale" value="${2.7362925425083047}"/>
+        <xacro:property name="z_offset" value="${0.014439}"/>
+      </xacro:if>
+      <xacro:if value="${type == 'sign_oneway_right'}">
+        <xacro:property name="model_scale" value="${4.34593654932638}"/>
+        <xacro:property name="z_offset" value="${0}"/>
+      </xacro:if>
+      <xacro:if value="${type == 'sign_T_intersect'}">
+        <xacro:property name="model_scale" value="${4.34593654932638}"/>
+        <xacro:property name="z_offset" value="${0}"/>
+      </xacro:if>
+      <xacro:if value="${type == 'duckie'}">
+        <xacro:property name="model_scale" value="${0.6585788789802037}"/>
+        <xacro:property name="z_offset" value="${-0.113989}"/>
+      </xacro:if>
+      <xacro:if value="${type == 'barrier'}">
+        <xacro:property name="model_scale" value="${0.8748906386701663}"/>
+        <xacro:property name="z_offset" value="${0}"/>
       </xacro:if>
       <!-- END GENERATED -->
-    <static>${static}</static>
-            <origin xyz="${size} ${y * size} 0"/>
-            <pose>${x * size} ${y * size} ${z_offset*size * model_scale * scale + 0.01} ${radians(90)} -0  ${radians(yaw)}</pose>
-    <link name='link'>
-      <collision name='collision'>
-        <geometry>
-          <mesh>
-            <scale>${size * model_scale * scale} ${size * model_scale * scale} ${size * model_scale * scale}</scale>
-            <uri>file://$(find mirte_gazebo)/models/${type}/meshes/${type}.obj</uri>
-        </mesh>
-        </geometry>
-        <max_contacts>10</max_contacts>
-        <surface>
-          <contact>
-            <ode/>
-          </contact>
-          <bounce/>
-          <friction>
-            <torsional>
+      <static>${static}</static>
+      <origin xyz="${size} ${y * size} 0"/>
+      <pose>${x * size} ${y * size} ${z_offset*size * model_scale * scale + 0.01} ${radians(90)} -0  ${radians(yaw)}</pose>
+      <link name="link">
+        <collision name="collision">
+          <geometry>
+            <mesh>
+              <scale>${size * model_scale * scale} ${size * model_scale * scale} ${size * model_scale * scale}</scale>
+              <uri>file://$(find mirte_gazebo)/models/${type}/meshes/${type}.obj</uri>
+            </mesh>
+          </geometry>
+          <max_contacts>10</max_contacts>
+          <surface>
+            <contact>
               <ode/>
-            </torsional>
-            <ode/>
-          </friction>
-        </surface>
-      </collision>
-      <visual name='visual'>
-        <!-- <origin xyz="${x * size} ${y * size} 0"/> -->
-        <geometry>
-          <mesh>
-            <scale>${size * model_scale * scale} ${size * model_scale * scale} ${size * model_scale * scale}</scale>
-            <uri>file://$(find mirte_gazebo)/models/${type}/meshes/${type}.obj</uri>
-            <!-- <pose>${x * size} ${y * size}  ${z_offset*size * model_scale * scale + 0.01} ${radians(90)} -0 0</pose> -->
-        </mesh>
-        </geometry>
-        <material>
-          <script>
-            <name>${type}/${type}</name>
-            <uri>file://$(find mirte_gazebo)/models/${type}/materials/scripts/${type}.material</uri>
-          </script>
-        </material>
-      </visual>
-      <self_collide>0</self_collide>
-      <enable_wind>0</enable_wind>
-      <kinematic>0</kinematic>
-    </link>
-    <!-- <pose>${x * size} ${y * size}  ${z_offset*size * model_scale * scale + 0.01} ${radians(90)} -0 0</pose> -->
-</model>
+            </contact>
+            <bounce/>
+            <friction>
+              <torsional>
+                <ode/>
+              </torsional>
+              <ode/>
+            </friction>
+          </surface>
+        </collision>
+        <visual name="visual">
+          <!-- <origin xyz="${x * size} ${y * size} 0"/> -->
+          <geometry>
+            <mesh>
+              <scale>${size * model_scale * scale} ${size * model_scale * scale} ${size * model_scale * scale}</scale>
+              <uri>file://$(find mirte_gazebo)/models/${type}/meshes/${type}.obj</uri>
+              <!-- <pose>${x * size} ${y * size}  ${z_offset*size * model_scale * scale + 0.01} ${radians(90)} -0 0</pose> -->
+            </mesh>
+          </geometry>
+          <material>
+            <script>
+              <name>${type}/${type}</name>
+              <uri>file://$(find mirte_gazebo)/models/${type}/materials/scripts/${type}.material</uri>
+            </script>
+          </material>
+        </visual>
+        <self_collide>0</self_collide>
+        <enable_wind>0</enable_wind>
+        <kinematic>0</kinematic>
+      </link>
+      <!-- <pose>${x * size} ${y * size}  ${z_offset*size * model_scale * scale + 0.01} ${radians(90)} -0 0</pose> -->
+    </model>
   </xacro:macro>
   <xacro:macro name="duckieState" params="name type size x y yaw=0 static=1 scale=1">
@@ -160,114 +160,114 @@
     <!-- START GENERATED SCALES AND OFFSETS-->
     <xacro:if value="${type == 'sign_blank'}">
-    <xacro:property name="model_scale" value="${0.19415283233733935}"/>
-    <xacro:property name="z_offset" value="${0}"/>
-    </xacro:if>
-  <xacro:if value="${type == 'building'}">
-    <xacro:property name="model_scale" value="${0.2898550724637681}"/>
-    <xacro:property name="z_offset" value="${0}"/>
-    </xacro:if>
-  <xacro:if value="${type == 'house'}">
-    <xacro:property name="model_scale" value="${0.20755956855837843}"/>
-    <xacro:property name="z_offset" value="${0.024247}"/>
-    </xacro:if>
-  <xacro:if value="${type == 'cone'}">
-    <xacro:property name="model_scale" value="${0.03172296965063494}"/>
-    <xacro:property name="z_offset" value="${0}"/>
-    </xacro:if>
-  <xacro:if value="${type == 'truck'}">
-    <xacro:property name="model_scale" value="${0.1927574101731193}"/>
-    <xacro:property name="z_offset" value="${1.072166}"/>
-    </xacro:if>
-  <xacro:if value="${type == 'tree'}">
-    <xacro:property name="model_scale" value="${0.28054126509522415}"/>
-    <xacro:property name="z_offset" value="${0.003644}"/>
-    </xacro:if>
-  <xacro:if value="${type == 'duckiebot'}">
-    <xacro:property name="model_scale" value="${8.126777732629012}"/>
-    <xacro:property name="z_offset" value="${0.03311}"/>
-    </xacro:if>
-  <xacro:if value="${type == 'sign_left_T_intersect'}">
-    <xacro:property name="model_scale" value="${4.34593654932638}"/>
-    <xacro:property name="z_offset" value="${0}"/>
-    </xacro:if>
-  <xacro:if value="${type == 'sign_4_way_intersect'}">
-    <xacro:property name="model_scale" value="${4.34593654932638}"/>
-    <xacro:property name="z_offset" value="${0}"/>
-    </xacro:if>
-  <xacro:if value="${type == 'sign_yield'}">
-    <xacro:property name="model_scale" value="${4.34593654932638}"/>
-    <xacro:property name="z_offset" value="${0}"/>
-    </xacro:if>
-  <xacro:if value="${type == 'sign_no_right_turn'}">
-    <xacro:property name="model_scale" value="${4.34593654932638}"/>
-    <xacro:property name="z_offset" value="${0}"/>
-    </xacro:if>
-  <xacro:if value="${type == 'sign_duck_crossing'}">
-    <xacro:property name="model_scale" value="${4.34593654932638}"/>
-    <xacro:property name="z_offset" value="${0}"/>
-    </xacro:if>
-  <xacro:if value="${type == 'sign_no_left_turn'}">
-    <xacro:property name="model_scale" value="${4.34593654932638}"/>
-    <xacro:property name="z_offset" value="${0}"/>
-    </xacro:if>
-  <xacro:if value="${type == 'sign_stop'}">
-    <xacro:property name="model_scale" value="${4.34593654932638}"/>
-    <xacro:property name="z_offset" value="${0}"/>
-    </xacro:if>
-  <xacro:if value="${type == 'sign_do_not_enter'}">
-    <xacro:property name="model_scale" value="${4.34593654932638}"/>
-    <xacro:property name="z_offset" value="${0}"/>
-    </xacro:if>
-  <xacro:if value="${type == 'bus'}">
-    <xacro:property name="model_scale" value="${0.22667415295835838}"/>
-    <xacro:property name="z_offset" value="${-4.396879}"/>
-    </xacro:if>
-  <xacro:if value="${type == 'sign_t_light_ahead'}">
-    <xacro:property name="model_scale" value="${4.34593654932638}"/>
-    <xacro:property name="z_offset" value="${0}"/>
-    </xacro:if>
-  <xacro:if value="${type == 'sign_right_T_intersect'}">
-    <xacro:property name="model_scale" value="${4.34593654932638}"/>
-    <xacro:property name="z_offset" value="${0}"/>
-    </xacro:if>
-  <xacro:if value="${type == 'sign_pedestrian'}">
-    <xacro:property name="model_scale" value="${4.34593654932638}"/>
-    <xacro:property name="z_offset" value="${0}"/>
-    </xacro:if>
-  <xacro:if value="${type == 'sign_oneway_left'}">
-    <xacro:property name="model_scale" value="${4.34593654932638}"/>
-    <xacro:property name="z_offset" value="${0}"/>
-    </xacro:if>
-  <xacro:if value="${type == 'trafficlight'}">
-    <xacro:property name="model_scale" value="${2.7362925425083047}"/>
-    <xacro:property name="z_offset" value="${0.014439}"/>
-    </xacro:if>
-  <xacro:if value="${type == 'sign_oneway_right'}">
-    <xacro:property name="model_scale" value="${4.34593654932638}"/>
-    <xacro:property name="z_offset" value="${0}"/>
-    </xacro:if>
-  <xacro:if value="${type == 'sign_T_intersect'}">
-    <xacro:property name="model_scale" value="${4.34593654932638}"/>
-    <xacro:property name="z_offset" value="${0}"/>
-    </xacro:if>
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
Commit message: move cone up a bit

File: urdf/duckieModels.xacro (robot description, xacro)
@@ -290,5 +290,5 @@
       <xacro:if value="${type == 'cone'}">
         <xacro:property name="model_scale" value="${0.03172296965063494}"/>
-        <xacro:property name="z_offset" value="${0}"/>
+        <xacro:property name="z_offset" value="${3.5}"/>
       </xacro:if>
       <xacro:if value="${type == 'truck'}">
