Commit message: Working camera and lidar in rviz

File: urdf/camera.xacro (robot description, xacro)
@@ -17,5 +17,5 @@
         </image>
         <clip>
-          <near>0.02</near>
+          <near>0.0001</near>
           <far>300</far>
         </clip>

File: urdf/mirte.xacro (robot description, xacro)
@@ -30,7 +30,7 @@
     </visual>
   </link>
-  <link name="footprint" />
+  <link name="base_link" />
   <joint name="base_joint" type="fixed">
-    <parent link="footprint"/>
+    <parent link="base_link"/>
     <child link="link_chassis"/>
   </joint>

Commit message: Backported simulation to ROS1

File: urdf/camera.xacro (robot description, xacro)
@@ -1,5 +1,5 @@
 <robot xmlns:xacro="http://www.ros.org/wiki/xacro">
     <joint name="joint_camera" type="fixed">
-        <origin xyz="4 0 0" rpy="0 0 0" />
+        <origin xyz="0.1 0 0.035" rpy="0 0 0" />
         <parent link="link_chassis" />
         <child link="camera_link" />

File: urdf/lidar.xacro (robot description, xacro)
@@ -23,14 +23,16 @@
                 <range>
                     <min>2</min>
-                    <max>20</max>
+                    <max>12</max>
                     <resolution>0.1</resolution>
                 </range>
+                <noise>
+                  <type>gaussian</type>
+                  <mean>0.0</mean>
+                  <stddev>0.01</stddev>
+                </noise>
             </ray>
-            <plugin name="laser_controller" filename="libgazebo_ros_ray_sensor.so">
-                <ros>
-                    <remapping>~/out:=scan</remapping>
-                </ros>
-                <output_type>sensor_msgs/LaserScan</output_type>
-                <frame_name>lidar_link</frame_name>
+            <plugin name="laser_controller" filename="libgazebo_ros_laser.so">
+                <topicName>/mirte/scan</topicName>
+                <frameName>lidar_link</frameName>
             </plugin>
         </sensor>

File: urdf/macros.xacro (robot description, xacro)
@@ -40,4 +40,7 @@
       </visual>
     </link>
+    <gazebo reference="link_${name}">
+       <gravity>0</gravity>
+    </gazebo>
     <joint name="joint_${name}" type="continuous">
       <xacro:insert_block name="origin" />
@@ -54,5 +57,5 @@
      <actuator name="motor_${name}">
        <hardwareInterface>hardware_interface/VelocityJointInterface</hardwareInterface>
-       <mechanicalReduction>1</mechanicalReduction>
+       <mechanicalReduction>120</mechanicalReduction>
      </actuator>
    </transmission>
@@ -77,4 +80,7 @@
      </xacro:inertia_sphere>
    </link>
+   <gazebo reference="link_${name}">
+    <gravity>0</gravity>
+  </gazebo>
    <joint name="fixed" type="fixed">
      <parent link="${parent}"/>

File: urdf/mirte.xacro (robot description, xacro)
@@ -3,8 +3,8 @@
   <xacro:include filename="$(find mirte_gazebo)/urdf/materials.xacro"/>
   <xacro:include filename="$(find mirte_gazebo)/urdf/macros.xacro"/>
-  <xacro:include filename="$(find mirte_gazebo)/urdf/ros2_control.xacro"/>
+  <xacro:include filename="$(find mirte_gazebo)/urdf/ros_control.xacro"/>
   <xacro:include filename="$(find mirte_gazebo)/urdf/lidar.xacro"/>
   <xacro:include filename="$(find mirte_gazebo)/urdf/camera.xacro"/>
-  <xacro:include filename="$(find mirte_gazebo)/urdf/ultrasonic.xacro"/>
+<!--  <xacro:include filename="$(find mirte_gazebo)/urdf/ultrasonic.xacro"/> -->
   <xacro:property name="yaml_param_file" value="$(find mirte_gazebo)/config/mirte_dimensions.yaml" />
   <xacro:property name="params" value="${load_yaml(yaml_param_file)}"/>
@@ -29,5 +29,11 @@
     </visual>
   </link>
+  <gazebo reference="link_chassis">
+    <gravity>0</gravity>
+  </gazebo>
   <link name="base_link" />
+  <gazebo reference="base_link">
+    <gravity>0</gravity>
+  </gazebo>
   <joint name="base_joint" type="fixed">
     <parent link="base_link"/>
@@ -53,4 +59,5 @@
     </joint_options>
   </xacro:wheel>
+<!--
   <xacro:ultrasonic_sensor name="left">
     <origin rpy="0 0 .45" xyz="0.085 0.04 0.022" />
@@ -59,3 +66,4 @@
     <origin rpy="0 0 -0.45" xyz="0.085 -0.04 0.022" />
   </xacro:ultrasonic_sensor>
+-->
 </robot>
