Commit message: Add duckytown generation + start sim

File: urdf/camera.xacro (robot description, xacro)
@@ -1,9 +1,9 @@
 <robot xmlns:xacro="http://www.ros.org/wiki/xacro">
-    <joint name="joint_camera" type="fixed">
-        <origin xyz="0.1 0 0.035" rpy="0 0 0" />
-        <parent link="link_chassis" />
-        <child link="camera_link" />
-    </joint>
-    <link name="camera_link"></link>
+  <joint name="joint_camera" type="fixed">
+    <origin xyz="0.1 0 0.035" rpy="0 0 0" />
+    <parent link="link_chassis" />
+    <child link="camera_link" />
+  </joint>
+  <link name="camera_link"></link>
   <gazebo reference="camera_link">
     <sensor type="camera" name="camera1">

File: urdf/duckietown.xacro (robot description, xacro)
@@ -1,15 +1,96 @@
-<?xml version="1.0" ?>
+<?xml version="1.0"?>
 <robot name="duckietown" xmlns:xacro="http://www.ros.org/wiki/xacro">
-  <xacro:include filename="$(find mirte_gazebo)/urdf/tile.xacro"/>
+  <xacro:include filename="$(find mirte_gazebo)/urdf/tile.xacro" />
   <!-- this dummy base is used to link all tiles to -->
   <link name="dummy_link">
     <inertial>
       <mass value="10.0" />
-      <inertia  ixx="1.0" ixy="0.0"  ixz="0.0"  iyy="1.0"  iyz="0.0"  izz="1.0" />
+      <inertia ixx="1.0" ixy="0.0" ixz="0.0" iyy="1.0" iyz="0.0" izz="1.0" />
     </inertial>
   </link>
-  <xacro:tile name="straight_1" material="DT/Straight" size="0.6" x="0" y="0"/>
+  <!-- <xacro:tile name="straight_1" material="DT/Straight" size="0.6" x="0" y="0"/>
   <xacro:tile name="curve_1" material="DT/Curve" size="0.6" x="1" y="0" yaw="90"/>
   <xacro:tile name="curve_2" material="DT/Curve" size="0.6" x="1" y="-1"/>
-  <xacro:tile name="straight_2" material="DT/Straight" size="0.6" x="0" y="-1"/>
+  <xacro:tile name="straight_2" material="DT/Straight" size="0.6" x="0" y="-1"/> -->
+  <xacro:tile name="tile_0_0" material="DT/asphalt" size="0.6" x="0" y="0" yaw="0" />
+  <xacro:tile name="tile_1_0" material="DT/asphalt" size="0.6" x="1" y="0" yaw="0" />
+  <xacro:tile name="tile_2_0" material="DT/asphalt" size="0.6" x="2" y="0" yaw="0" />
+  <xacro:tile name="tile_3_0" material="DT/asphalt" size="0.6" x="3" y="0" yaw="0" />
+  <xacro:tile name="tile_4_0" material="DT/asphalt" size="0.6" x="4" y="0" yaw="0" />
+  <xacro:tile name="tile_5_0" material="DT/asphalt" size="0.6" x="5" y="0" yaw="0" />
+  <xacro:tile name="tile_6_0" material="DT/asphalt" size="0.6" x="6" y="0" yaw="0" />
+  <xacro:tile name="tile_7_0" material="DT/asphalt" size="0.6" x="7" y="0" yaw="0" />
+  <xacro:tile name="tile_8_0" material="DT/asphalt" size="0.6" x="8" y="0" yaw="0" />
+  <xacro:tile name="tile_0_1" material="DT/asphalt" size="0.6" x="0" y="1" yaw="0" />
+  <xacro:tile name="tile_1_1" material="DT/curve_left" size="0.6" x="1" y="1" yaw="270" />
+  <xacro:tile name="tile_2_1" material="DT/curve_left" size="0.6" x="2" y="1" yaw="0" />
+  <xacro:tile name="tile_3_1" material="DT/asphalt" size="0.6" x="3" y="1" yaw="0" />
+  <xacro:tile name="tile_4_1" material="DT/curve_left" size="0.6" x="4" y="1" yaw="270" />
+  <xacro:tile name="tile_5_1" material="DT/straight" size="0.6" x="5" y="1" yaw="270" />
+  <xacro:tile name="tile_6_1" material="DT/straight" size="0.6" x="6" y="1" yaw="270" />
+  <xacro:tile name="tile_7_1" material="DT/curve_left" size="0.6" x="7" y="1" yaw="0" />
+  <xacro:tile name="tile_8_1" material="DT/asphalt" size="0.6" x="8" y="1" yaw="0" />
+  <xacro:tile name="tile_0_2" material="DT/asphalt" size="0.6" x="0" y="2" yaw="0" />
+  <xacro:tile name="tile_1_2" material="DT/straight" size="0.6" x="1" y="2" yaw="180" />
+  <xacro:tile name="tile_2_2" material="DT/curve_right" size="0.6" x="2" y="2" yaw="270" />
+  <xacro:tile name="tile_3_2" material="DT/straight" size="0.6" x="3" y="2" yaw="270" />
+  <xacro:tile name="tile_4_2" material="DT/curve_right" size="0.6" x="4" y="2" yaw="180" />
+  <xacro:tile name="tile_5_2" material="DT/asphalt" size="0.6" x="5" y="2" yaw="0" />
+  <xacro:tile name="tile_6_2" material="DT/curve_right" size="0.6" x="6" y="2" yaw="0" />
+  <xacro:tile name="tile_7_2" material="DT/curve_left" size="0.6" x="7" y="2" yaw="90" />
+  <xacro:tile name="tile_8_2" material="DT/asphalt" size="0.6" x="8" y="2" yaw="0" />
+  <xacro:tile name="tile_0_3" material="DT/asphalt" size="0.6" x="0" y="3" yaw="0" />
+  <xacro:tile name="tile_1_3" material="DT/straight" size="0.6" x="1" y="3" yaw="180" />
+  <xacro:tile name="tile_2_3" material="DT/asphalt" size="0.6" x="2" y="3" yaw="0" />
+  <xacro:tile name="tile_3_3" material="DT/asphalt" size="0.6" x="3" y="3" yaw="0" />
+  <xacro:tile name="tile_4_3" material="DT/asphalt" size="0.6" x="4" y="3" yaw="0" />
+  <xacro:tile name="tile_5_3" material="DT/asphalt" size="0.6" x="5" y="3" yaw="0" />
+  <xacro:tile name="tile_6_3" material="DT/straight" size="0.6" x="6" y="3" yaw="0" />
+  <xacro:tile name="tile_7_3" material="DT/asphalt" size="0.6" x="7" y="3" yaw="0" />
+  <xacro:tile name="tile_8_3" material="DT/asphalt" size="0.6" x="8" y="3" yaw="0" />
+  <xacro:tile name="tile_0_4" material="DT/asphalt" size="0.6" x="0" y="4" yaw="0" />
+  <xacro:tile name="tile_1_4" material="DT/straight" size="0.6" x="1" y="4" yaw="180" />
+  <xacro:tile name="tile_2_4" material="DT/asphalt" size="0.6" x="2" y="4" yaw="0" />
+  <xacro:tile name="tile_3_4" material="DT/asphalt" size="0.6" x="3" y="4" yaw="0" />
+  <xacro:tile name="tile_4_4" material="DT/curve_right" size="0.6" x="4" y="4" yaw="0" />
+  <xacro:tile name="tile_5_4" material="DT/straight" size="0.6" x="5" y="4" yaw="90" />
+  <xacro:tile name="tile_6_4" material="DT/curve_left" size="0.6" x="6" y="4" yaw="90" />
+  <xacro:tile name="tile_7_4" material="DT/asphalt" size="0.6" x="7" y="4" yaw="0" />
+  <xacro:tile name="tile_8_4" material="DT/asphalt" size="0.6" x="8" y="4" yaw="0" />
+  <xacro:tile name="tile_0_5" material="DT/asphalt" size="0.6" x="0" y="5" yaw="0" />
+  <xacro:tile name="tile_1_5" material="DT/straight" size="0.6" x="1" y="5" yaw="180" />
+  <xacro:tile name="tile_2_5" material="DT/asphalt" size="0.6" x="2" y="5" yaw="0" />
+  <xacro:tile name="tile_3_5" material="DT/curve_right" size="0.6" x="3" y="5" yaw="0" />
+  <xacro:tile name="tile_4_5" material="DT/curve_left" size="0.6" x="4" y="5" yaw="90" />
+  <xacro:tile name="tile_5_5" material="DT/asphalt" size="0.6" x="5" y="5" yaw="0" />
+  <xacro:tile name="tile_6_5" material="DT/asphalt" size="0.6" x="6" y="5" yaw="0" />
+  <xacro:tile name="tile_7_5" material="DT/asphalt" size="0.6" x="7" y="5" yaw="0" />
+  <xacro:tile name="tile_8_5" material="DT/asphalt" size="0.6" x="8" y="5" yaw="0" />
+  <xacro:tile name="tile_0_6" material="DT/asphalt" size="0.6" x="0" y="6" yaw="0" />
+  <xacro:tile name="tile_1_6" material="DT/straight" size="0.6" x="1" y="6" yaw="180" />
+  <xacro:tile name="tile_2_6" material="DT/asphalt" size="0.6" x="2" y="6" yaw="0" />
+  <xacro:tile name="tile_3_6" material="DT/straight" size="0.6" x="3" y="6" yaw="0" />
+  <xacro:tile name="tile_4_6" material="DT/asphalt" size="0.6" x="4" y="6" yaw="0" />
+  <xacro:tile name="tile_5_6" material="DT/asphalt" size="0.6" x="5" y="6" yaw="0" />
+  <xacro:tile name="tile_6_6" material="DT/asphalt" size="0.6" x="6" y="6" yaw="0" />
+  <xacro:tile name="tile_7_6" material="DT/asphalt" size="0.6" x="7" y="6" yaw="0" />
+  <xacro:tile name="tile_8_6" material="DT/asphalt" size="0.6" x="8" y="6" yaw="0" />
+  <xacro:tile name="tile_0_7" material="DT/asphalt" size="0.6" x="0" y="7" yaw="0" />
+  <xacro:tile name="tile_1_7" material="DT/curve_left" size="0.6" x="1" y="7" yaw="180" />
+  <xacro:tile name="tile_2_7" material="DT/straight" size="0.6" x="2" y="7" yaw="90" />
+  <xacro:tile name="tile_3_7" material="DT/curve_left" size="0.6" x="3" y="7" yaw="90" />
+  <xacro:tile name="tile_4_7" material="DT/asphalt" size="0.6" x="4" y="7" yaw="0" />
+  <xacro:tile name="tile_5_7" material="DT/asphalt" size="0.6" x="5" y="7" yaw="0" />
+  <xacro:tile name="tile_6_7" material="DT/asphalt" size="0.6" x="6" y="7" yaw="0" />
+  <xacro:tile name="tile_7_7" material="DT/asphalt" size="0.6" x="7" y="7" yaw="0" />
+  <xacro:tile name="tile_8_7" material="DT/asphalt" size="0.6" x="8" y="7" yaw="0" />
+  <xacro:tile name="tile_0_8" material="DT/asphalt" size="0.6" x="0" y="8" yaw="0" />
+  <xacro:tile name="tile_1_8" material="DT/asphalt" size="0.6" x="1" y="8" yaw="0" />
+  <xacro:tile name="tile_2_8" material="DT/asphalt" size="0.6" x="2" y="8" yaw="0" />
+  <xacro:tile name="tile_3_8" material="DT/asphalt" size="0.6" x="3" y="8" yaw="0" />
+  <xacro:tile name="tile_4_8" material="DT/asphalt" size="0.6" x="4" y="8" yaw="0" />
+  <xacro:tile name="tile_5_8" material="DT/asphalt" size="0.6" x="5" y="8" yaw="0" />
+  <xacro:tile name="tile_6_8" material="DT/asphalt" size="0.6" x="6" y="8" yaw="0" />
+  <xacro:tile name="tile_7_8" material="DT/asphalt" size="0.6" x="7" y="8" yaw="0" />
+  <xacro:tile name="tile_8_8" material="DT/asphalt" size="0.6" x="8" y="8" yaw="0" />
 </robot>

File: urdf/lidar.xacro (robot description, xacro)
@@ -1,40 +1,39 @@
 <robot xmlns:xacro="http://www.ros.org/wiki/xacro">
-    <joint name="lidar" type="fixed">
-        <origin rpy="0 0 0" xyz="0 0 0.6" />
-        <parent link="link_chassis" />
-        <child link="lidar_link" />
-    </joint>
-    <link name="lidar_link">
-    </link>
-    <gazebo reference="lidar_link">
-        <sensor name="lidar" type="ray">
-            <pose> 0 0 0 0 0 0 </pose>
-            <visualize>false</visualize>
-            <update_rate>15</update_rate>
-            <ray>
-                <scan>
-                    <horizontal>
-                        <samples>720</samples>
-                        <resolution>1</resolution>
-                        <min_angle>-3.14</min_angle>
-                        <max_angle>3.14</max_angle>
-                    </horizontal>
-                </scan>
-                <range>
-                    <min>2</min>
-                    <max>12</max>
-                    <resolution>0.1</resolution>
-                </range>
-                <noise>
-                  <type>gaussian</type>
-                  <mean>0.0</mean>
-                  <stddev>0.01</stddev>
-                </noise>
-            </ray>
-            <plugin name="laser_controller" filename="libgazebo_ros_laser.so">
-                <topicName>/mirte/scan</topicName>
-                <frameName>lidar_link</frameName>
-            </plugin>
-        </sensor>
-    </gazebo>
+  <joint name="lidar" type="fixed">
+    <origin rpy="0 0 0" xyz="0 0 0.6" />
+    <parent link="link_chassis" />
+    <child link="lidar_link" />
+  </joint>
+  <link name="lidar_link"></link>
+  <gazebo reference="lidar_link">
+    <sensor name="lidar" type="ray">
+      <pose>0 0 0 0 0 0</pose>
+      <visualize>false</visualize>
+      <update_rate>15</update_rate>
+      <ray>
+        <scan>
+          <horizontal>
+            <samples>720</samples>
+            <resolution>1</resolution>
+            <min_angle>-3.14</min_angle>
+            <max_angle>3.14</max_angle>
+          </horizontal>
+        </scan>
+        <range>
+          <min>2</min>
+          <max>12</max>
+          <resolution>0.1</resolution>
+        </range>
+        <noise>
+          <type>gaussian</type>
+          <mean>0.0</mean>
+          <stddev>0.01</stddev>
+        </noise>
+      </ray>
+      <plugin name="laser_controller" filename="libgazebo_ros_laser.so">
+        <topicName>/mirte/scan</topicName>
+        <frameName>lidar_link</frameName>
+      </plugin>
+    </sensor>
+  </gazebo>
 </robot>

File: urdf/macros.xacro (robot description, xacro)
@@ -3,21 +3,21 @@
   <xacro:macro name="inertia_box" params="x y z mass *origin">
     <inertial>
-      <mass value="${mass}"/>
+      <mass value="${mass}" />
       <xacro:insert_block name="origin" />
-      <inertia ixx="${mass / 12.0 * (y*y + z*z)}" ixy="0.0" ixz="0.0" iyy="${mass / 12.0 * (z*z + x*x)}" iyz="0.0" izz="${mass / 12.0 * (y*y + x*x)}"/>
+      <inertia ixx="${mass / 12.0 * (y*y + z*z)}" ixy="0.0" ixz="0.0" iyy="${mass / 12.0 * (z*z + x*x)}" iyz="0.0" izz="${mass / 12.0 * (y*y + x*x)}" />
     </inertial>
   </xacro:macro>
   <xacro:macro name="inertia_cylinder" params="r h mass *origin">
     <inertial>
-      <mass value="${mass}"/>
+      <mass value="${mass}" />
       <xacro:insert_block name="origin" />
-      <inertia ixx="${mass / 12 * (3*r*r + h*h)}" ixy="0" ixz="0" iyy="${mass / 12 * (3*r*r + h*h)}" iyz="0" izz="${mass / 2 * r * r}"/>
+      <inertia ixx="${mass / 12 * (3*r*r + h*h)}" ixy="0" ixz="0" iyy="${mass / 12 * (3*r*r + h*h)}" iyz="0" izz="${mass / 2 * r * r}" />
     </inertial>
   </xacro:macro>
   <xacro:macro name="inertia_sphere" params="r mass *origin">
     <inertial>
-      <mass value="${mass}"/>
-      <xacro:insert_block name="origin"/>
-      <inertia ixx="${2/5 * mass * r*r}" ixy = "0" ixz = "0" iyy="${2/5 * mass * r*r}" iyz = "0" izz="${2/5 * mass * r*r}"/>
+      <mass value="${mass}" />
+      <xacro:insert_block name="origin" />
+      <inertia ixx="${2/5 * mass * r*r}" ixy="0" ixz="0" iyy="${2/5 * mass * r*r}" iyz="0" izz="${2/5 * mass * r*r}" />
     </inertial>
   </xacro:macro>
@@ -25,66 +25,66 @@
     <link name="link_${name}">
       <xacro:inertia_cylinder r="${radius}" h="0.015" mass="${mass}">
-        <origin rpy="0 1.5707 1.5707" xyz="0 0 0"/>
+        <origin rpy="0 1.5707 1.5707" xyz="0 0 0" />
       </xacro:inertia_cylinder>
       <collision name="link_${name}_collision">
-        <origin rpy="0 1.5707 1.5707" xyz="0 0 0"/>
+        <origin rpy="0 1.5707 1.5707" xyz="0 0 0" />
         <geometry>
-          <cylinder length="0.015" radius="${radius}"/>
+          <mesh filename="file://$(find mirte_gazebo)/meshes/mirte_wheel.stl" scale="0.001 0.001 0.001" rpy="0 0 1.57079633" />
         </geometry>
       </collision>
       <visual name="link_${name}_visual">
-        <origin rpy="0 1.5707 1.5707" xyz="0 0 0"/>
+        <origin rpy="0 1.5707 1.5707" xyz="0 0 0" />
         <geometry>
-          <cylinder length="0.015" radius="${radius}"/>
+          <mesh filename="file://$(find mirte_gazebo)/meshes/mirte_wheel.stl" scale="0.001 0.001 0.001" rpy="0 0 1.57079633" />
         </geometry>
       </visual>
     </link>
     <gazebo reference="link_${name}">
-       <gravity>0</gravity>
+      <gravity>0</gravity>
     </gazebo>
     <joint name="joint_${name}" type="continuous">
       <xacro:insert_block name="origin" />
-      <child link="link_${name}"/>
-      <parent link="${parent}"/>
-      <axis rpy="0 0 0" xyz="0 1 0"/>
+      <child link="link_${name}" />
+      <parent link="${parent}" />
+      <axis rpy="0 0 0" xyz="0 1 0" />
       <xacro:insert_block name="content" />
     </joint>
     <transmission name="trans_${name}">
-     <type>transmission_interface/SimpleTransmission</type>
-     <joint name="joint_${name}">
-       <hardwareInterface>hardware_interface/VelocityJointInterface</hardwareInterface>
-     </joint>
-     <actuator name="motor_${name}">
-       <hardwareInterface>hardware_interface/VelocityJointInterface</hardwareInterface>
-       <mechanicalReduction>120</mechanicalReduction>
-     </actuator>
-   </transmission>
- </xacro:macro>
- <xacro:macro name="caster" params="name parent radius mass *origin" >
-   <link name="link_${name}">
-     <collision>
-       <xacro:insert_block name="origin" />
-       <geometry>
-         <sphere radius="${radius}"/>
-       </geometry>
-     </collision>
-     <visual>
-       <xacro:insert_block name="origin" />
-       <geometry>
-         <sphere radius="${radius}"/>
-       </geometry>
-       <material name="red"/>
-     </visual>
-     <xacro:inertia_sphere r="${radius}" mass="${mass}">
-       <xacro:insert_block name="origin" />
-     </xacro:inertia_sphere>
-   </link>
-   <gazebo reference="link_${name}">
-    <gravity>1</gravity>
-  </gazebo>
-   <joint name="fixed" type="fixed">
-     <parent link="${parent}"/>
-     <child link="link_${name}"/>
-   </joint>
- </xacro:macro>
+      <type>transmission_interface/SimpleTransmission</type>
+      <joint name="joint_${name}">
+        <hardwareInterface>hardware_interface/VelocityJointInterface</hardwareInterface>
+      </joint>
+      <actuator name="motor_${name}">
+        <hardwareInterface>hardware_interface/VelocityJointInterface</hardwareInterface>
+        <mechanicalReduction>120</mechanicalReduction>
+      </actuator>
+    </transmission>
+  </xacro:macro>
+  <xacro:macro name="caster" params="name parent radius mass *origin">
+    <link name="link_${name}">
+      <collision>
+        <xacro:insert_block name="origin" />
+        <geometry>
+          <sphere radius="${radius}" />
+        </geometry>
+      </collision>
+      <visual>
+        <xacro:insert_block name="origin" />
+        <geometry>
+          <sphere radius="${radius}" />
+        </geometry>
+        <material name="red" />
+      </visual>
+      <xacro:inertia_sphere r="${radius}" mass="${mass}">
+        <xacro:insert_block name="origin" />
+      </xacro:inertia_sphere>
+    </link>
+    <gazebo reference="link_${name}">
+      <gravity>1</gravity>
+    </gazebo>
+    <joint name="fixed" type="fixed">
+      <parent link="${parent}" />
+      <child link="link_${name}" />
+    </joint>
+  </xacro:macro>
 </robot>

File: urdf/materials.xacro (robot description, xacro)
@@ -2,29 +2,29 @@
 <robot name="mirte" xmlns:xacro="http://www.ros.org/wiki/xacro">
   <material name="black">
-    <color rgba="0.0 0.0 0.0 1.0"/>
+    <color rgba="0.0 0.0 0.0 1.0" />
   </material>
   <material name="blue">
-    <color rgba="0.203125 0.23828125 0.28515625 1.0"/>
+    <color rgba="0.203125 0.23828125 0.28515625 1.0" />
   </material>
   <material name="green">
-    <color rgba="0.0 0.8 0.0 1.0"/>
+    <color rgba="0.0 0.8 0.0 1.0" />
   </material>
   <material name="grey">
-    <color rgba="0.2 0.2 0.2 1.0"/>
+    <color rgba="0.2 0.2 0.2 1.0" />
   </material>
   <material name="orange">
-    <color rgba="1.0 0.423529411765 0.0392156862745 1.0"/>
+    <color rgba="1.0 0.423529411765 0.0392156862745 1.0" />
   </material>
   <material name="brown">
-    <color rgba="0.870588235294 0.811764705882 0.764705882353 1.0"/>
+    <color rgba="0.870588235294 0.811764705882 0.764705882353 1.0" />
   </material>
   <material name="red">
-    <color rgba="0.80078125 0.12890625 0.1328125 1.0"/>
+    <color rgba="0.80078125 0.12890625 0.1328125 1.0" />
   </material>
   <material name="white">
-    <color rgba="1.0 1.0 1.0 1.0"/>
+    <color rgba="1.0 1.0 1.0 1.0" />
   </material>
   <material name="wood">
-    <color rgba="1.0 0.0 1.0 1.0"/>
+    <color rgba="1.0 0.0 1.0 1.0" />
   </material>
   <gazebo reference="link_chassis">
@@ -37,8 +37,8 @@
   </gazebo>
   <gazebo reference="link_left_wheel">
-    <mu1 value="1.0"/>
-    <mu2 value="1.0"/>
-    <kp value="1000000.0"/>
-    <kd value= "100.0"/>
+    <mu1 value="1.0" />
+    <mu2 value="1.0" />
+    <kp value="1000000.0" />
+    <kd value="100.0" />
     <minDepth>0.001</minDepth>
     <maxVel>0.55</maxVel>
@@ -46,8 +46,8 @@
   </gazebo>
   <gazebo reference="link_right_wheel">
-    <mu1 value="1.0"/>
-    <mu2 value="1.0"/>
-    <kp value="1000000.0"/>
-    <kd value= "100.0"/>
+    <mu1 value="1.0" />
+    <mu2 value="1.0" />
+    <kp value="1000000.0" />
+    <kd value="100.0" />
     <minDepth>0.001</minDepth>
     <maxVel>0.55</maxVel>
