Commit message: Add duckytown generation + start sim

File: urdf/mirte.xacro (robot description, xacro)
@@ -1,30 +1,30 @@
-<?xml version="1.0" ?>
+<?xml version="1.0"?>
 <robot name="mirte" xmlns:xacro="http://www.ros.org/wiki/xacro">
-  <xacro:include filename="$(find mirte_gazebo)/urdf/materials.xacro"/>
-  <xacro:include filename="$(find mirte_gazebo)/urdf/macros.xacro"/>
-  <xacro:include filename="$(find mirte_gazebo)/urdf/ros_control.xacro"/>
-  <xacro:include filename="$(find mirte_gazebo)/urdf/lidar.xacro"/>
-  <xacro:include filename="$(find mirte_gazebo)/urdf/camera.xacro"/>
-<!--  <xacro:include filename="$(find mirte_gazebo)/urdf/ultrasonic.xacro"/> -->
+  <xacro:include filename="$(find mirte_gazebo)/urdf/materials.xacro" />
+  <xacro:include filename="$(find mirte_gazebo)/urdf/macros.xacro" />
+  <xacro:include filename="$(find mirte_gazebo)/urdf/ros_control.xacro" />
+  <xacro:include filename="$(find mirte_gazebo)/urdf/lidar.xacro" />
+  <xacro:include filename="$(find mirte_gazebo)/urdf/camera.xacro" />
+  <!--  <xacro:include filename="$(find mirte_gazebo)/urdf/ultrasonic.xacro"/> -->
   <xacro:property name="yaml_param_file" value="$(find mirte_gazebo)/config/mirte_dimensions.yaml" />
-  <xacro:property name="params" value="${load_yaml(yaml_param_file)}"/>
+  <xacro:property name="params" value="${load_yaml(yaml_param_file)}" />
   <link name="link_chassis">
     <!-- pose and inertial -->
     <pose>0 0 0.015 0 0 0</pose>
     <xacro:inertia_box x="${params['base_len']}" y="${params['base_width']}" z="${params['base_height']}" mass="${params['base_mass']}">
-      <origin rpy="0 0 0" xyz="0 0 0.015"/>
+      <origin rpy="0 0 0" xyz="0 0 0.015" />
     </xacro:inertia_box>
     <!-- body -->
     <collision name="collision_chassis">
       <geometry>
-        <mesh filename="file://$(find mirte_gazebo)/meshes/mirte_base.stl" scale="0.001 0.001 0.001"/>
+        <mesh filename="file://$(find mirte_gazebo)/meshes/mirte_base.stl" scale="0.001 0.001 0.001" rpy="0 0 1.57079633" />
       </geometry>
     </collision>
     <visual>
-      <origin rpy="0 0 0" xyz="0 0 0"/>
+      <origin rpy="0 0 0" xyz="0 0 0" />
       <geometry>
-        <mesh filename="file://$(find mirte_gazebo)/meshes/mirte_base.stl" scale="0.001 0.001 0.001"/>
+        <mesh filename="file://$(find mirte_gazebo)/meshes/mirte_base.stl" scale="0.001 0.001 0.001" rpy="0 0 1.57079633" />
       </geometry>
-      <material name="blue"/>
+      <material name="blue" />
     </visual>
   </link>
@@ -37,27 +37,27 @@
   </gazebo>
   <joint name="base_joint" type="fixed">
-    <parent link="base_link"/>
-    <child link="link_chassis"/>
+    <parent link="base_link" />
+    <child link="link_chassis" />
   </joint>
   <xacro:caster name="caster_wheel_back" parent="link_chassis" radius="${params['caster_wheel_radius']}" mass="${params['caster_wheel_mass']}">
-    <origin rpy=" 0 0 0" xyz="${params['caster_wheel_center_x_offset']} ${params['caster_wheel_center_y_offset']} ${params['caster_wheel_center_z_offset']}"/>
+    <origin rpy="0 0 0" xyz="${params['caster_wheel_center_x_offset']} ${params['caster_wheel_center_y_offset']} ${params['caster_wheel_center_z_offset']}" />
   </xacro:caster>
   <!-- NOTE: xacro parser adds joint_ -->
   <xacro:wheel name="left_wheel" parent="link_chassis" radius="${params['wheel_radius']}" mass="${params['wheel_mass']}">
-    <origin rpy="0 0 0" xyz="${params['wheel_center_x_offset']} ${params['wheel_center_y_offset']} ${params['wheel_center_z_offset']}"/>
+    <origin rpy="0 0 0" xyz="${params['wheel_center_x_offset']} ${params['wheel_center_y_offset']} ${params['wheel_center_z_offset']}" />
     <joint_options>
-      <limit effort="10" velocity="8"/>
-      <dynamics damping="0.0" friction="0.0"/>
+      <limit effort="10" velocity="8" />
+      <dynamics damping="0.0" friction="0.0" />
     </joint_options>
   </xacro:wheel>
   <!-- NOTE: xacro parser adds joint_ -->
   <xacro:wheel name="right_wheel" parent="link_chassis" radius="${params['wheel_radius']}" mass="${params['wheel_mass']}">
-    <origin rpy="0 0 0" xyz="${params['wheel_center_x_offset']} ${-1*params['wheel_center_y_offset']} ${params['wheel_center_z_offset']}"/>
+    <origin rpy="3.14 0 0" xyz="${params['wheel_center_x_offset']} ${-1*params['wheel_center_y_offset']} ${params['wheel_center_z_offset']}" />
     <joint_options>
-      <limit effort="10" velocity="8"/>
-      <dynamics damping="0.0" friction="0.0"/>
+      <limit effort="10" velocity="8" />
+      <dynamics damping="0.0" friction="0.0" />
     </joint_options>
   </xacro:wheel>
-<!--
+  <!--
   <xacro:ultrasonic_sensor name="left">
     <origin rpy="0 0 .45" xyz="0.085 0.04 0.022" />
@@ -67,11 +67,10 @@
   </xacro:ultrasonic_sensor>
 -->
-<gazebo>
-  <!-- <plugin name="gazebo_ros_control" filename="libgazebo_ros_control.so">
+  <gazebo>
+    <!-- <plugin name="gazebo_ros_control" filename="libgazebo_ros_control.so">
     <robotNamespace>/mirte-control</robotNamespace>
   </plugin> -->
- <plugin name="gazebo_ros_controller_manager" filename="libgazebo_ros_controller_manager.so">
-    </plugin>
-</gazebo>
-  <xacro:include filename="$(find mirte_gazebo)/urdf/diffdrive.xacro"/>
+    <plugin name="gazebo_ros_controller_manager" filename="libgazebo_ros_controller_manager.so"></plugin>
+  </gazebo>
+  <xacro:include filename="$(find mirte_gazebo)/urdf/diffdrive.xacro" />
 </robot>

File: urdf/ros_control.xacro (robot description, xacro)
@@ -1,7 +1,7 @@
 <?xml version="1.0"?>
 <robot xmlns:xacro="http://www.ros.org/wiki/xacro">
-<!-- TODO: currewntly this is also defined in the macros.xacro
+  <!-- TODO: currewntly this is also defined in the macros.xacro
  I think it should be over here -->
-<!--
+  <!--
 <transmission name="left_wheel_transmission">
   <type>transmission_interface/SimpleTransmission</type>
@@ -25,8 +25,8 @@
 </transmission>
 -->
-<gazebo>
+  <gazebo>
     <plugin filename="libgazebo_ros_control.so" name="gazebo_ros_control">
-        <robotNamespace>/mirte-control</robotNamespace>
+      <robotNamespace>/mirte-control</robotNamespace>
     </plugin>
-</gazebo>
+  </gazebo>
 </robot>

File: urdf/tile.xacro (robot description, xacro)
@@ -1,29 +1,29 @@
 <robot xmlns:xacro="http://www.ros.org/wiki/xacro">
- <xacro:macro name="tile" params="name material size x y yaw=0" >
-  <link name="${name}">
-    <inertial>
-      <mass value="10.0" />
-      <inertia  ixx="1.0" ixy="0.0"  ixz="0.0"  iyy="1.0"  iyz="0.0"  izz="1.0" />
-    </inertial>
-    <visual>
-      <origin xyz="${x * size} ${y * size} 0" rpy="0 0 ${pi / 180 * yaw}"/>
-      <geometry>
-        <box size="${size} ${size} .02" />
-      </geometry>
-    </visual>
-    <collision>
-      <origin xyz="${x * size} ${y * size} 0"/>
-      <geometry>
-        <box size="${size} ${size} .02" />
-      </geometry>
-    </collision>
-  </link>
-  <joint name="${name}_joint" type="fixed">
-    <parent link="dummy_link"/>
-    <child link="${name}"/>
-  </joint>
-  <gazebo reference="${name}">
-     <material>${material}</material>
-  </gazebo>
- </xacro:macro>
+  <xacro:macro name="tile" params="name material size x y yaw=0">
+    <link name="${name}">
+      <inertial>
+        <mass value="10.0" />
+        <inertia ixx="1.0" ixy="0.0" ixz="0.0" iyy="1.0" iyz="0.0" izz="1.0" />
+      </inertial>
+      <visual>
+        <origin xyz="${x * size} ${y * size} 0" rpy="0 0 ${pi / 180 * yaw}" />
+        <geometry>
+          <box size="${size} ${size} .02" />
+        </geometry>
+      </visual>
+      <collision>
+        <origin xyz="${x * size} ${y * size} 0" />
+        <geometry>
+          <box size="${size} ${size} .02" />
+        </geometry>
+      </collision>
+    </link>
+    <joint name="${name}_joint" type="fixed">
+      <parent link="dummy_link" />
+      <child link="${name}" />
+    </joint>
+    <gazebo reference="${name}">
+      <material>${material}</material>
+    </gazebo>
+  </xacro:macro>
 </robot>

File: urdf/ultrasonic.xacro (robot description, xacro)
@@ -1,77 +1,77 @@
 <?xml version="1.0"?>
 <robot xmlns:xacro="http://www.ros.org/wiki/xacro">
-<xacro:macro name="ultrasonic_sensor" params="name *origin">
-<joint name="sonar_${name}" type="fixed">
-    <axis xyz="0 1 0" />
-    <xacro:insert_block name="origin" />
-    <parent link="link_chassis"/>
-    <child link="base_sonar_${name}"/>
-</joint>
-<link name="base_sonar_${name}">
-    <collision>
-      <origin xyz="0 0 0" rpy="0 0 0"/>
-      <geometry>
-        <box size="0.01 0.05 0.037"/>
-      </geometry>
-    </collision>
-    <visual>
-      <origin xyz="0 0 0" rpy="0 0 0"/>
-      <geometry>
-        <box size="0.01 0.05 0.037"/>
-      </geometry>
-      <material name="blue"/>
-    </visual>
-    <inertial>
-      <mass value="0.0" />
-      <origin xyz="0 0 0" rpy="0 0 0"/>
-      <inertia ixx="0.0" ixy="0.0" ixz="0.0" iyy="0.0" iyz="0.0" izz="0.0" />
-    </inertial>
- </link>
-<gazebo reference="base_sonar_${name}">
-<sensor type="ray" name="range_sensor_${name}">
-   <visualize>false</visualize>
-    <ray>
-         <scan>
+  <xacro:macro name="ultrasonic_sensor" params="name *origin">
+    <joint name="sonar_${name}" type="fixed">
+      <axis xyz="0 1 0" />
+      <xacro:insert_block name="origin" />
+      <parent link="link_chassis" />
+      <child link="base_sonar_${name}" />
+    </joint>
+    <link name="base_sonar_${name}">
+      <collision>
+        <origin xyz="0 0 0" rpy="0 0 0" />
+        <geometry>
+          <box size="0.01 0.05 0.037" />
+        </geometry>
+      </collision>
+      <visual>
+        <origin xyz="0 0 0" rpy="0 0 0" />
+        <geometry>
+          <box size="0.01 0.05 0.037" />
+        </geometry>
+        <material name="blue" />
+      </visual>
+      <inertial>
+        <mass value="0.0" />
+        <origin xyz="0 0 0" rpy="0 0 0" />
+        <inertia ixx="0.0" ixy="0.0" ixz="0.0" iyy="0.0" iyz="0.0" izz="0.0" />
+      </inertial>
+    </link>
+    <gazebo reference="base_sonar_${name}">
+      <sensor type="ray" name="range_sensor_${name}">
+        <visualize>false</visualize>
+        <ray>
+          <scan>
             <horizontal>
-               <!-- for some reason 1 does not work, we neex 2x2 -->
-               <samples>2</samples>
-               <resolution>1</resolution>
-               <min_angle>-0.26</min_angle>
-               <max_angle>0.26</max_angle>
+              <!-- for some reason 1 does not work, we neex 2x2 -->
+              <samples>2</samples>
+              <resolution>1</resolution>
+              <min_angle>-0.26</min_angle>
+              <max_angle>0.26</max_angle>
             </horizontal>
             <vertical>
-               <samples>2</samples>
-               <resolution>1</resolution>
-               <min_angle>-0.014835</min_angle>
-               <max_angle>0.014835</max_angle>
+              <samples>2</samples>
+              <resolution>1</resolution>
+              <min_angle>-0.014835</min_angle>
+              <max_angle>0.014835</max_angle>
             </vertical>
-         </scan>
-         <range>
+          </scan>
+          <range>
             <min>0.01</min>
             <max>5</max>
             <resolution>0.01</resolution>
-         </range>
-      <!-- Using gazebo's noise instead of plugin's -->
-      <noise>
-        <type>gaussian</type>
-        <mean>0.0</mean>
-        <stddev>0.01</stddev>
-      </noise>
-    </ray>
-    <!-- Using gazebo's update rate instead of plugin's -->
-    <update_rate>30</update_rate>
-    <plugin name="gazebo_ros_range_controller_${name}" filename="libgazebo_ros_ray_sensor.so">
-      <!-- Change namespace and output topic so published topic is /rrbot/laser/scan -->
-      <ros>
-        <namespace>/mirte</namespace>
-        <remapping>~/out:=distance/${name}</remapping>
-      </ros>
-      <!-- Set output to sensor_msgs/Range to get same output type as gazebo_ros_range -->
-      <output_type>sensor_msgs/Range</output_type>
-      <!-- <frame_name> ommited, will default to range_link -->
-      <radiation_type>ultrasound</radiation_type>
-    </plugin>
-  </sensor>
+          </range>
+          <!-- Using gazebo's noise instead of plugin's -->
+          <noise>
+            <type>gaussian</type>
+            <mean>0.0</mean>
+            <stddev>0.01</stddev>
+          </noise>
+        </ray>
+        <!-- Using gazebo's update rate instead of plugin's -->
+        <update_rate>30</update_rate>
+        <plugin name="gazebo_ros_range_controller_${name}" filename="libgazebo_ros_ray_sensor.so">
+          <!-- Change namespace and output topic so published topic is /rrbot/laser/scan -->
+          <ros>
+            <namespace>/mirte</namespace>
+            <remapping>~/out:=distance/${name}</remapping>
+          </ros>
+          <!-- Set output to sensor_msgs/Range to get same output type as gazebo_ros_range -->
+          <output_type>sensor_msgs/Range</output_type>
+          <!-- <frame_name> ommited, will default to range_link -->
+          <radiation_type>ultrasound</radiation_type>
+        </plugin>
+      </sensor>
     </gazebo>
-</xacro:macro>
+  </xacro:macro>
 </robot>
