Commit message: change to tidy

File: urdf/camera.xacro (robot description, xacro)
@@ -1,2 +1,3 @@
+<?xml version="1.0"?>
 <robot xmlns:xacro="http://www.ros.org/wiki/xacro">
   <joint name="joint_camera" type="fixed">
@@ -5,5 +6,5 @@
     <child link="camera_link" />
   </joint>
-  <link name="camera_link"></link>
+  <link name="camera_link" />
   <gazebo reference="camera_link">
     <sensor type="camera" name="camera1">
@@ -28,5 +29,6 @@
         </distortion>
       </camera>
-      <plugin name="camera_controller" filename="libgazebo_ros_camera.so">
+      <plugin name="camera_controller"
+      filename="libgazebo_ros_camera.so">
         <ros>
           <namespace>custom_ns</namespace>

File: urdf/diffdrive.xacro (robot description, xacro)
@@ -2,5 +2,6 @@
 <robot>
   <gazebo>
-    <plugin name="differential_drive_controller" filename="libgazebo_ros_diff_drive.so">
+    <plugin name="differential_drive_controller"
+    filename="libgazebo_ros_diff_drive.so">
       <alwaysOn>false</alwaysOn>
       <legacyMode>false</legacyMode>
@@ -11,6 +12,8 @@
       <wheelDiameter>2</wheelDiameter>
       <torque>20</torque>
-      <commandTopic>/mirte_control/base_controller/cmd_vel</commandTopic>
-      <odometryTopic>/mirte_control/base_controller/odom</odometryTopic>
+      <commandTopic>
+      /mirte_control/base_controller/cmd_vel</commandTopic>
+      <odometryTopic>
+      /mirte_control/base_controller/odom</odometryTopic>
       <odometryFrame>odom</odometryFrame>
       <robotBaseFrame>base_footprint</robotBaseFrame>

File: urdf/duckietown.xacro (robot description, xacro)
@@ -1,4 +1,5 @@
 <?xml version="1.0"?>
-<robot name="duckietown" xmlns:xacro="http://www.ros.org/wiki/xacro">
+<robot xmlns:xacro="http://www.ros.org/wiki/xacro"
+name="duckietown">
   <xacro:include filename="$(find mirte_gazebo)/urdf/tile.xacro" />
   <!-- this dummy base is used to link all tiles to -->
@@ -6,5 +7,6 @@
     <inertial>
       <mass value="10.0" />
-      <inertia ixx="1.0" ixy="0.0" ixz="0.0" iyy="1.0" iyz="0.0" izz="1.0" />
+      <inertia ixx="1.0" ixy="0.0" ixz="0.0" iyy="1.0" iyz="0.0"
+      izz="1.0" />
     </inertial>
   </link>
@@ -13,84 +15,165 @@
   <xacro:tile name="curve_2" material="DT/Curve" size="0.6" x="1" y="-1"/>
   <xacro:tile name="straight_2" material="DT/Straight" size="0.6" x="0" y="-1"/> -->
-  <xacro:tile name="tile_0_0" material="DT/asphalt" size="0.6" x="0" y="0" yaw="0" />
-  <xacro:tile name="tile_1_0" material="DT/asphalt" size="0.6" x="1" y="0" yaw="0" />
-  <xacro:tile name="tile_2_0" material="DT/asphalt" size="0.6" x="2" y="0" yaw="0" />
-  <xacro:tile name="tile_3_0" material="DT/asphalt" size="0.6" x="3" y="0" yaw="0" />
-  <xacro:tile name="tile_4_0" material="DT/asphalt" size="0.6" x="4" y="0" yaw="0" />
-  <xacro:tile name="tile_5_0" material="DT/asphalt" size="0.6" x="5" y="0" yaw="0" />
-  <xacro:tile name="tile_6_0" material="DT/asphalt" size="0.6" x="6" y="0" yaw="0" />
-  <xacro:tile name="tile_7_0" material="DT/asphalt" size="0.6" x="7" y="0" yaw="0" />
-  <xacro:tile name="tile_8_0" material="DT/asphalt" size="0.6" x="8" y="0" yaw="0" />
-  <xacro:tile name="tile_0_1" material="DT/asphalt" size="0.6" x="0" y="1" yaw="0" />
-  <xacro:tile name="tile_1_1" material="DT/curve_left" size="0.6" x="1" y="1" yaw="270" />
-  <xacro:tile name="tile_2_1" material="DT/curve_left" size="0.6" x="2" y="1" yaw="0" />
-  <xacro:tile name="tile_3_1" material="DT/asphalt" size="0.6" x="3" y="1" yaw="0" />
-  <xacro:tile name="tile_4_1" material="DT/curve_left" size="0.6" x="4" y="1" yaw="270" />
-  <xacro:tile name="tile_5_1" material="DT/straight" size="0.6" x="5" y="1" yaw="270" />
-  <xacro:tile name="tile_6_1" material="DT/straight" size="0.6" x="6" y="1" yaw="270" />
-  <xacro:tile name="tile_7_1" material="DT/curve_left" size="0.6" x="7" y="1" yaw="0" />
-  <xacro:tile name="tile_8_1" material="DT/asphalt" size="0.6" x="8" y="1" yaw="0" />
-  <xacro:tile name="tile_0_2" material="DT/asphalt" size="0.6" x="0" y="2" yaw="0" />
-  <xacro:tile name="tile_1_2" material="DT/straight" size="0.6" x="1" y="2" yaw="180" />
-  <xacro:tile name="tile_2_2" material="DT/curve_right" size="0.6" x="2" y="2" yaw="270" />
-  <xacro:tile name="tile_3_2" material="DT/straight" size="0.6" x="3" y="2" yaw="270" />
-  <xacro:tile name="tile_4_2" material="DT/curve_right" size="0.6" x="4" y="2" yaw="180" />
-  <xacro:tile name="tile_5_2" material="DT/asphalt" size="0.6" x="5" y="2" yaw="0" />
-  <xacro:tile name="tile_6_2" material="DT/curve_right" size="0.6" x="6" y="2" yaw="0" />
-  <xacro:tile name="tile_7_2" material="DT/curve_left" size="0.6" x="7" y="2" yaw="90" />
-  <xacro:tile name="tile_8_2" material="DT/asphalt" size="0.6" x="8" y="2" yaw="0" />
-  <xacro:tile name="tile_0_3" material="DT/asphalt" size="0.6" x="0" y="3" yaw="0" />
-  <xacro:tile name="tile_1_3" material="DT/straight" size="0.6" x="1" y="3" yaw="180" />
-  <xacro:tile name="tile_2_3" material="DT/asphalt" size="0.6" x="2" y="3" yaw="0" />
-  <xacro:tile name="tile_3_3" material="DT/asphalt" size="0.6" x="3" y="3" yaw="0" />
-  <xacro:tile name="tile_4_3" material="DT/asphalt" size="0.6" x="4" y="3" yaw="0" />
-  <xacro:tile name="tile_5_3" material="DT/asphalt" size="0.6" x="5" y="3" yaw="0" />
-  <xacro:tile name="tile_6_3" material="DT/straight" size="0.6" x="6" y="3" yaw="0" />
-  <xacro:tile name="tile_7_3" material="DT/asphalt" size="0.6" x="7" y="3" yaw="0" />
-  <xacro:tile name="tile_8_3" material="DT/asphalt" size="0.6" x="8" y="3" yaw="0" />
-  <xacro:tile name="tile_0_4" material="DT/asphalt" size="0.6" x="0" y="4" yaw="0" />
-  <xacro:tile name="tile_1_4" material="DT/straight" size="0.6" x="1" y="4" yaw="180" />
-  <xacro:tile name="tile_2_4" material="DT/asphalt" size="0.6" x="2" y="4" yaw="0" />
-  <xacro:tile name="tile_3_4" material="DT/asphalt" size="0.6" x="3" y="4" yaw="0" />
-  <xacro:tile name="tile_4_4" material="DT/curve_right" size="0.6" x="4" y="4" yaw="0" />
-  <xacro:tile name="tile_5_4" material="DT/straight" size="0.6" x="5" y="4" yaw="90" />
-  <xacro:tile name="tile_6_4" material="DT/curve_left" size="0.6" x="6" y="4" yaw="90" />
-  <xacro:tile name="tile_7_4" material="DT/asphalt" size="0.6" x="7" y="4" yaw="0" />
-  <xacro:tile name="tile_8_4" material="DT/asphalt" size="0.6" x="8" y="4" yaw="0" />
-  <xacro:tile name="tile_0_5" material="DT/asphalt" size="0.6" x="0" y="5" yaw="0" />
-  <xacro:tile name="tile_1_5" material="DT/straight" size="0.6" x="1" y="5" yaw="180" />
-  <xacro:tile name="tile_2_5" material="DT/asphalt" size="0.6" x="2" y="5" yaw="0" />
-  <xacro:tile name="tile_3_5" material="DT/curve_right" size="0.6" x="3" y="5" yaw="0" />
-  <xacro:tile name="tile_4_5" material="DT/curve_left" size="0.6" x="4" y="5" yaw="90" />
-  <xacro:tile name="tile_5_5" material="DT/asphalt" size="0.6" x="5" y="5" yaw="0" />
-  <xacro:tile name="tile_6_5" material="DT/asphalt" size="0.6" x="6" y="5" yaw="0" />
-  <xacro:tile name="tile_7_5" material="DT/asphalt" size="0.6" x="7" y="5" yaw="0" />
-  <xacro:tile name="tile_8_5" material="DT/asphalt" size="0.6" x="8" y="5" yaw="0" />
-  <xacro:tile name="tile_0_6" material="DT/asphalt" size="0.6" x="0" y="6" yaw="0" />
-  <xacro:tile name="tile_1_6" material="DT/straight" size="0.6" x="1" y="6" yaw="180" />
-  <xacro:tile name="tile_2_6" material="DT/asphalt" size="0.6" x="2" y="6" yaw="0" />
-  <xacro:tile name="tile_3_6" material="DT/straight" size="0.6" x="3" y="6" yaw="0" />
-  <xacro:tile name="tile_4_6" material="DT/asphalt" size="0.6" x="4" y="6" yaw="0" />
-  <xacro:tile name="tile_5_6" material="DT/asphalt" size="0.6" x="5" y="6" yaw="0" />
-  <xacro:tile name="tile_6_6" material="DT/asphalt" size="0.6" x="6" y="6" yaw="0" />
-  <xacro:tile name="tile_7_6" material="DT/asphalt" size="0.6" x="7" y="6" yaw="0" />
-  <xacro:tile name="tile_8_6" material="DT/asphalt" size="0.6" x="8" y="6" yaw="0" />
-  <xacro:tile name="tile_0_7" material="DT/asphalt" size="0.6" x="0" y="7" yaw="0" />
-  <xacro:tile name="tile_1_7" material="DT/curve_left" size="0.6" x="1" y="7" yaw="180" />
-  <xacro:tile name="tile_2_7" material="DT/straight" size="0.6" x="2" y="7" yaw="90" />
-  <xacro:tile name="tile_3_7" material="DT/curve_left" size="0.6" x="3" y="7" yaw="90" />
-  <xacro:tile name="tile_4_7" material="DT/asphalt" size="0.6" x="4" y="7" yaw="0" />
-  <xacro:tile name="tile_5_7" material="DT/asphalt" size="0.6" x="5" y="7" yaw="0" />
-  <xacro:tile name="tile_6_7" material="DT/asphalt" size="0.6" x="6" y="7" yaw="0" />
-  <xacro:tile name="tile_7_7" material="DT/asphalt" size="0.6" x="7" y="7" yaw="0" />
-  <xacro:tile name="tile_8_7" material="DT/asphalt" size="0.6" x="8" y="7" yaw="0" />
-  <xacro:tile name="tile_0_8" material="DT/asphalt" size="0.6" x="0" y="8" yaw="0" />
-  <xacro:tile name="tile_1_8" material="DT/asphalt" size="0.6" x="1" y="8" yaw="0" />
-  <xacro:tile name="tile_2_8" material="DT/asphalt" size="0.6" x="2" y="8" yaw="0" />
-  <xacro:tile name="tile_3_8" material="DT/asphalt" size="0.6" x="3" y="8" yaw="0" />
-  <xacro:tile name="tile_4_8" material="DT/asphalt" size="0.6" x="4" y="8" yaw="0" />
-  <xacro:tile name="tile_5_8" material="DT/asphalt" size="0.6" x="5" y="8" yaw="0" />
-  <xacro:tile name="tile_6_8" material="DT/asphalt" size="0.6" x="6" y="8" yaw="0" />
-  <xacro:tile name="tile_7_8" material="DT/asphalt" size="0.6" x="7" y="8" yaw="0" />
-  <xacro:tile name="tile_8_8" material="DT/asphalt" size="0.6" x="8" y="8" yaw="0" />
+  <xacro:tile name="tile_0_0" material="DT/asphalt" size="0.6"
+  x="0" y="0" yaw="0" />
+  <xacro:tile name="tile_1_0" material="DT/asphalt" size="0.6"
+  x="1" y="0" yaw="0" />
+  <xacro:tile name="tile_2_0" material="DT/asphalt" size="0.6"
+  x="2" y="0" yaw="0" />
+  <xacro:tile name="tile_3_0" material="DT/asphalt" size="0.6"
+  x="3" y="0" yaw="0" />
+  <xacro:tile name="tile_4_0" material="DT/asphalt" size="0.6"
+  x="4" y="0" yaw="0" />
+  <xacro:tile name="tile_5_0" material="DT/asphalt" size="0.6"
+  x="5" y="0" yaw="0" />
+  <xacro:tile name="tile_6_0" material="DT/asphalt" size="0.6"
+  x="6" y="0" yaw="0" />
+  <xacro:tile name="tile_7_0" material="DT/asphalt" size="0.6"
+  x="7" y="0" yaw="0" />
+  <xacro:tile name="tile_8_0" material="DT/asphalt" size="0.6"
+  x="8" y="0" yaw="0" />
+  <xacro:tile name="tile_0_1" material="DT/asphalt" size="0.6"
+  x="0" y="1" yaw="0" />
+  <xacro:tile name="tile_1_1" material="DT/curve_left" size="0.6"
+  x="1" y="1" yaw="270" />
+  <xacro:tile name="tile_2_1" material="DT/curve_left" size="0.6"
+  x="2" y="1" yaw="0" />
+  <xacro:tile name="tile_3_1" material="DT/asphalt" size="0.6"
+  x="3" y="1" yaw="0" />
+  <xacro:tile name="tile_4_1" material="DT/curve_left" size="0.6"
+  x="4" y="1" yaw="270" />
+  <xacro:tile name="tile_5_1" material="DT/straight" size="0.6"
+  x="5" y="1" yaw="270" />
+  <xacro:tile name="tile_6_1" material="DT/straight" size="0.6"
+  x="6" y="1" yaw="270" />
+  <xacro:tile name="tile_7_1" material="DT/curve_left" size="0.6"
+  x="7" y="1" yaw="0" />
+  <xacro:tile name="tile_8_1" material="DT/asphalt" size="0.6"
+  x="8" y="1" yaw="0" />
+  <xacro:tile name="tile_0_2" material="DT/asphalt" size="0.6"
+  x="0" y="2" yaw="0" />
+  <xacro:tile name="tile_1_2" material="DT/straight" size="0.6"
+  x="1" y="2" yaw="180" />
+  <xacro:tile name="tile_2_2" material="DT/curve_right" size="0.6"
+  x="2" y="2" yaw="270" />
+  <xacro:tile name="tile_3_2" material="DT/straight" size="0.6"
+  x="3" y="2" yaw="270" />
+  <xacro:tile name="tile_4_2" material="DT/curve_right" size="0.6"
+  x="4" y="2" yaw="180" />
+  <xacro:tile name="tile_5_2" material="DT/asphalt" size="0.6"
+  x="5" y="2" yaw="0" />
+  <xacro:tile name="tile_6_2" material="DT/curve_right" size="0.6"
+  x="6" y="2" yaw="0" />
+  <xacro:tile name="tile_7_2" material="DT/curve_left" size="0.6"
+  x="7" y="2" yaw="90" />
+  <xacro:tile name="tile_8_2" material="DT/asphalt" size="0.6"
+  x="8" y="2" yaw="0" />
+  <xacro:tile name="tile_0_3" material="DT/asphalt" size="0.6"
+  x="0" y="3" yaw="0" />
+  <xacro:tile name="tile_1_3" material="DT/straight" size="0.6"
+  x="1" y="3" yaw="180" />
+  <xacro:tile name="tile_2_3" material="DT/asphalt" size="0.6"
+  x="2" y="3" yaw="0" />
+  <xacro:tile name="tile_3_3" material="DT/asphalt" size="0.6"
+  x="3" y="3" yaw="0" />
+  <xacro:tile name="tile_4_3" material="DT/asphalt" size="0.6"
+  x="4" y="3" yaw="0" />
+  <xacro:tile name="tile_5_3" material="DT/asphalt" size="0.6"
+  x="5" y="3" yaw="0" />
+  <xacro:tile name="tile_6_3" material="DT/straight" size="0.6"
+  x="6" y="3" yaw="0" />
+  <xacro:tile name="tile_7_3" material="DT/asphalt" size="0.6"
+  x="7" y="3" yaw="0" />
+  <xacro:tile name="tile_8_3" material="DT/asphalt" size="0.6"
+  x="8" y="3" yaw="0" />
+  <xacro:tile name="tile_0_4" material="DT/asphalt" size="0.6"
+  x="0" y="4" yaw="0" />
+  <xacro:tile name="tile_1_4" material="DT/straight" size="0.6"
+  x="1" y="4" yaw="180" />
+  <xacro:tile name="tile_2_4" material="DT/asphalt" size="0.6"
+  x="2" y="4" yaw="0" />
+  <xacro:tile name="tile_3_4" material="DT/asphalt" size="0.6"
+  x="3" y="4" yaw="0" />
+  <xacro:tile name="tile_4_4" material="DT/curve_right" size="0.6"
+  x="4" y="4" yaw="0" />
+  <xacro:tile name="tile_5_4" material="DT/straight" size="0.6"
+  x="5" y="4" yaw="90" />
+  <xacro:tile name="tile_6_4" material="DT/curve_left" size="0.6"
+  x="6" y="4" yaw="90" />
+  <xacro:tile name="tile_7_4" material="DT/asphalt" size="0.6"
+  x="7" y="4" yaw="0" />
+  <xacro:tile name="tile_8_4" material="DT/asphalt" size="0.6"
+  x="8" y="4" yaw="0" />
+  <xacro:tile name="tile_0_5" material="DT/asphalt" size="0.6"
+  x="0" y="5" yaw="0" />
+  <xacro:tile name="tile_1_5" material="DT/straight" size="0.6"
+  x="1" y="5" yaw="180" />
+  <xacro:tile name="tile_2_5" material="DT/asphalt" size="0.6"
+  x="2" y="5" yaw="0" />
+  <xacro:tile name="tile_3_5" material="DT/curve_right" size="0.6"
+  x="3" y="5" yaw="0" />
+  <xacro:tile name="tile_4_5" material="DT/curve_left" size="0.6"
+  x="4" y="5" yaw="90" />
+  <xacro:tile name="tile_5_5" material="DT/asphalt" size="0.6"
+  x="5" y="5" yaw="0" />
+  <xacro:tile name="tile_6_5" material="DT/asphalt" size="0.6"
+  x="6" y="5" yaw="0" />
+  <xacro:tile name="tile_7_5" material="DT/asphalt" size="0.6"
+  x="7" y="5" yaw="0" />
+  <xacro:tile name="tile_8_5" material="DT/asphalt" size="0.6"
+  x="8" y="5" yaw="0" />
+  <xacro:tile name="tile_0_6" material="DT/asphalt" size="0.6"
+  x="0" y="6" yaw="0" />
+  <xacro:tile name="tile_1_6" material="DT/straight" size="0.6"
+  x="1" y="6" yaw="180" />
+  <xacro:tile name="tile_2_6" material="DT/asphalt" size="0.6"
+  x="2" y="6" yaw="0" />
+  <xacro:tile name="tile_3_6" material="DT/straight" size="0.6"
+  x="3" y="6" yaw="0" />
+  <xacro:tile name="tile_4_6" material="DT/asphalt" size="0.6"
+  x="4" y="6" yaw="0" />
+  <xacro:tile name="tile_5_6" material="DT/asphalt" size="0.6"
+  x="5" y="6" yaw="0" />
+  <xacro:tile name="tile_6_6" material="DT/asphalt" size="0.6"
+  x="6" y="6" yaw="0" />
+  <xacro:tile name="tile_7_6" material="DT/asphalt" size="0.6"
+  x="7" y="6" yaw="0" />
+  <xacro:tile name="tile_8_6" material="DT/asphalt" size="0.6"
+  x="8" y="6" yaw="0" />
+  <xacro:tile name="tile_0_7" material="DT/asphalt" size="0.6"
+  x="0" y="7" yaw="0" />
+  <xacro:tile name="tile_1_7" material="DT/curve_left" size="0.6"
+  x="1" y="7" yaw="180" />
+  <xacro:tile name="tile_2_7" material="DT/straight" size="0.6"
+  x="2" y="7" yaw="90" />
+  <xacro:tile name="tile_3_7" material="DT/curve_left" size="0.6"
+  x="3" y="7" yaw="90" />
+  <xacro:tile name="tile_4_7" material="DT/asphalt" size="0.6"
+  x="4" y="7" yaw="0" />
+  <xacro:tile name="tile_5_7" material="DT/asphalt" size="0.6"
+  x="5" y="7" yaw="0" />
+  <xacro:tile name="tile_6_7" material="DT/asphalt" size="0.6"
+  x="6" y="7" yaw="0" />
+  <xacro:tile name="tile_7_7" material="DT/asphalt" size="0.6"
+  x="7" y="7" yaw="0" />
+  <xacro:tile name="tile_8_7" material="DT/asphalt" size="0.6"
+  x="8" y="7" yaw="0" />
+  <xacro:tile name="tile_0_8" material="DT/asphalt" size="0.6"
+  x="0" y="8" yaw="0" />
+  <xacro:tile name="tile_1_8" material="DT/asphalt" size="0.6"
+  x="1" y="8" yaw="0" />
+  <xacro:tile name="tile_2_8" material="DT/asphalt" size="0.6"
+  x="2" y="8" yaw="0" />
+  <xacro:tile name="tile_3_8" material="DT/asphalt" size="0.6"
+  x="3" y="8" yaw="0" />
+  <xacro:tile name="tile_4_8" material="DT/asphalt" size="0.6"
+  x="4" y="8" yaw="0" />
+  <xacro:tile name="tile_5_8" material="DT/asphalt" size="0.6"
+  x="5" y="8" yaw="0" />
+  <xacro:tile name="tile_6_8" material="DT/asphalt" size="0.6"
+  x="6" y="8" yaw="0" />
+  <xacro:tile name="tile_7_8" material="DT/asphalt" size="0.6"
+  x="7" y="8" yaw="0" />
+  <xacro:tile name="tile_8_8" material="DT/asphalt" size="0.6"
+  x="8" y="8" yaw="0" />
 </robot>

File: urdf/lidar.xacro (robot description, xacro)
@@ -1,2 +1,3 @@
+<?xml version="1.0"?>
 <robot xmlns:xacro="http://www.ros.org/wiki/xacro">
   <joint name="lidar" type="fixed">
@@ -5,5 +6,5 @@
     <child link="lidar_link" />
   </joint>
-  <link name="lidar_link"></link>
+  <link name="lidar_link" />
   <gazebo reference="lidar_link">
     <sensor name="lidar" type="ray">
@@ -31,5 +32,6 @@
         </noise>
       </ray>
-      <plugin name="laser_controller" filename="libgazebo_ros_laser.so">
+      <plugin name="laser_controller"
+      filename="libgazebo_ros_laser.so">
         <topicName>/mirte/scan</topicName>
         <frameName>lidar_link</frameName>

File: urdf/macros.xacro (robot description, xacro)
@@ -1,9 +1,11 @@
 <?xml version="1.0"?>
-<robot name="mirte" xmlns:xacro="http://www.ros.org/wiki/xacro">
+<robot xmlns:xacro="http://www.ros.org/wiki/xacro" name="mirte">
   <xacro:macro name="inertia_box" params="x y z mass *origin">
     <inertial>
       <mass value="${mass}" />
       <xacro:insert_block name="origin" />
-      <inertia ixx="${mass / 12.0 * (y*y + z*z)}" ixy="0.0" ixz="0.0" iyy="${mass / 12.0 * (z*z + x*x)}" iyz="0.0" izz="${mass / 12.0 * (y*y + x*x)}" />
+      <inertia ixx="${mass / 12.0 * (y*y + z*z)}" ixy="0.0"
+      ixz="0.0" iyy="${mass / 12.0 * (z*z + x*x)}" iyz="0.0"
+      izz="${mass / 12.0 * (y*y + x*x)}" />
     </inertial>
   </xacro:macro>
@@ -12,5 +14,7 @@
       <mass value="${mass}" />
       <xacro:insert_block name="origin" />
-      <inertia ixx="${mass / 12 * (3*r*r + h*h)}" ixy="0" ixz="0" iyy="${mass / 12 * (3*r*r + h*h)}" iyz="0" izz="${mass / 2 * r * r}" />
+      <inertia ixx="${mass / 12 * (3*r*r + h*h)}" ixy="0" ixz="0"
+      iyy="${mass / 12 * (3*r*r + h*h)}" iyz="0"
+      izz="${mass / 2 * r * r}" />
     </inertial>
   </xacro:macro>
@@ -19,10 +23,14 @@
       <mass value="${mass}" />
       <xacro:insert_block name="origin" />
-      <inertia ixx="${2/5 * mass * r*r}" ixy="0" ixz="0" iyy="${2/5 * mass * r*r}" iyz="0" izz="${2/5 * mass * r*r}" />
+      <inertia ixx="${2/5 * mass * r*r}" ixy="0" ixz="0"
+      iyy="${2/5 * mass * r*r}" iyz="0"
+      izz="${2/5 * mass * r*r}" />
     </inertial>
   </xacro:macro>
-  <xacro:macro name="wheel" params="name parent radius mass *origin **content">
+  <xacro:macro name="wheel"
+  params="name parent radius mass *origin **content">
     <link name="link_${name}">
-      <xacro:inertia_cylinder r="${radius}" h="0.015" mass="${mass}">
+      <xacro:inertia_cylinder r="${radius}" h="0.015"
+      mass="${mass}">
         <origin rpy="0 1.5707 1.5707" xyz="0 0 0" />
       </xacro:inertia_cylinder>
@@ -30,5 +38,6 @@
         <origin rpy="0 1.5707 1.5707" xyz="0 0 0" />
         <geometry>
-          <mesh filename="file://$(find mirte_gazebo)/meshes/mirte_wheel.stl" scale="0.001 0.001 0.001" rpy="0 0 1.57079633" />
+          <mesh filename="file://$(find mirte_gazebo)/meshes/mirte_wheel.stl"
+          scale="0.001 0.001 0.001" rpy="0 0 1.57079633" />
         </geometry>
       </collision>
@@ -36,5 +45,6 @@
         <origin rpy="0 1.5707 1.5707" xyz="0 0 0" />
         <geometry>
-          <mesh filename="file://$(find mirte_gazebo)/meshes/mirte_wheel.stl" scale="0.001 0.001 0.001" rpy="0 0 1.57079633" />
+          <mesh filename="file://$(find mirte_gazebo)/meshes/mirte_wheel.stl"
+          scale="0.001 0.001 0.001" rpy="0 0 1.57079633" />
         </geometry>
       </visual>
@@ -53,13 +63,16 @@
       <type>transmission_interface/SimpleTransmission</type>
       <joint name="joint_${name}">
-        <hardwareInterface>hardware_interface/VelocityJointInterface</hardwareInterface>
+        <hardwareInterface>
+        hardware_interface/VelocityJointInterface</hardwareInterface>
       </joint>
       <actuator name="motor_${name}">
-        <hardwareInterface>hardware_interface/VelocityJointInterface</hardwareInterface>
+        <hardwareInterface>
+        hardware_interface/VelocityJointInterface</hardwareInterface>
         <mechanicalReduction>120</mechanicalReduction>
       </actuator>
     </transmission>
   </xacro:macro>
-  <xacro:macro name="caster" params="name parent radius mass *origin">
+  <xacro:macro name="caster"
+  params="name parent radius mass *origin">
     <link name="link_${name}">
       <collision>

File: urdf/materials.xacro (robot description, xacro)
@@ -1,4 +1,4 @@
 <?xml version="1.0"?>
-<robot name="mirte" xmlns:xacro="http://www.ros.org/wiki/xacro">
+<robot xmlns:xacro="http://www.ros.org/wiki/xacro" name="mirte">
   <material name="black">
     <color rgba="0.0 0.0 0.0 1.0" />
