Commit message: change to tidy

File: urdf/mirte.xacro (robot description, xacro)
@@ -1,4 +1,4 @@
 <?xml version="1.0"?>
-<robot name="mirte" xmlns:xacro="http://www.ros.org/wiki/xacro">
+<robot xmlns:xacro="http://www.ros.org/wiki/xacro" name="mirte">
   <xacro:include filename="$(find mirte_gazebo)/urdf/materials.xacro" />
   <xacro:include filename="$(find mirte_gazebo)/urdf/macros.xacro" />
@@ -7,10 +7,14 @@
   <xacro:include filename="$(find mirte_gazebo)/urdf/camera.xacro" />
   <!--  <xacro:include filename="$(find mirte_gazebo)/urdf/ultrasonic.xacro"/> -->
-  <xacro:property name="yaml_param_file" value="$(find mirte_gazebo)/config/mirte_dimensions.yaml" />
-  <xacro:property name="params" value="${load_yaml(yaml_param_file)}" />
+  <xacro:property name="yaml_param_file"
+  value="$(find mirte_gazebo)/config/mirte_dimensions.yaml" />
+  <xacro:property name="params"
+  value="${load_yaml(yaml_param_file)}" />
   <link name="link_chassis">
     <!-- pose and inertial -->
     <pose>0 0 0.015 0 0 0</pose>
-    <xacro:inertia_box x="${params['base_len']}" y="${params['base_width']}" z="${params['base_height']}" mass="${params['base_mass']}">
+    <xacro:inertia_box x="${params['base_len']}"
+    y="${params['base_width']}" z="${params['base_height']}"
+    mass="${params['base_mass']}">
       <origin rpy="0 0 0" xyz="0 0 0.015" />
     </xacro:inertia_box>
@@ -18,5 +22,6 @@
     <collision name="collision_chassis">
       <geometry>
-        <mesh filename="file://$(find mirte_gazebo)/meshes/mirte_base.stl" scale="0.001 0.001 0.001" rpy="0 0 1.57079633" />
+        <mesh filename="file://$(find mirte_gazebo)/meshes/mirte_base.stl"
+        scale="0.001 0.001 0.001" rpy="0 0 1.57079633" />
       </geometry>
     </collision>
@@ -24,5 +29,6 @@
       <origin rpy="0 0 0" xyz="0 0 0" />
       <geometry>
-        <mesh filename="file://$(find mirte_gazebo)/meshes/mirte_base.stl" scale="0.001 0.001 0.001" rpy="0 0 1.57079633" />
+        <mesh filename="file://$(find mirte_gazebo)/meshes/mirte_base.stl"
+        scale="0.001 0.001 0.001" rpy="0 0 1.57079633" />
       </geometry>
       <material name="blue" />
@@ -40,10 +46,16 @@
     <child link="link_chassis" />
   </joint>
-  <xacro:caster name="caster_wheel_back" parent="link_chassis" radius="${params['caster_wheel_radius']}" mass="${params['caster_wheel_mass']}">
-    <origin rpy="0 0 0" xyz="${params['caster_wheel_center_x_offset']} ${params['caster_wheel_center_y_offset']} ${params['caster_wheel_center_z_offset']}" />
+  <xacro:caster name="caster_wheel_back" parent="link_chassis"
+  radius="${params['caster_wheel_radius']}"
+  mass="${params['caster_wheel_mass']}">
+    <origin rpy="0 0 0"
+    xyz="${params['caster_wheel_center_x_offset']} ${params['caster_wheel_center_y_offset']} ${params['caster_wheel_center_z_offset']}" />
   </xacro:caster>
   <!-- NOTE: xacro parser adds joint_ -->
-  <xacro:wheel name="left_wheel" parent="link_chassis" radius="${params['wheel_radius']}" mass="${params['wheel_mass']}">
-    <origin rpy="0 0 0" xyz="${params['wheel_center_x_offset']} ${params['wheel_center_y_offset']} ${params['wheel_center_z_offset']}" />
+  <xacro:wheel name="left_wheel" parent="link_chassis"
+  radius="${params['wheel_radius']}"
+  mass="${params['wheel_mass']}">
+    <origin rpy="0 0 0"
+    xyz="${params['wheel_center_x_offset']} ${params['wheel_center_y_offset']} ${params['wheel_center_z_offset']}" />
     <joint_options>
       <limit effort="10" velocity="8" />
@@ -52,6 +64,9 @@
   </xacro:wheel>
   <!-- NOTE: xacro parser adds joint_ -->
-  <xacro:wheel name="right_wheel" parent="link_chassis" radius="${params['wheel_radius']}" mass="${params['wheel_mass']}">
-    <origin rpy="3.14 0 0" xyz="${params['wheel_center_x_offset']} ${-1*params['wheel_center_y_offset']} ${params['wheel_center_z_offset']}" />
+  <xacro:wheel name="right_wheel" parent="link_chassis"
+  radius="${params['wheel_radius']}"
+  mass="${params['wheel_mass']}">
+    <origin rpy="3.14 0 0"
+    xyz="${params['wheel_center_x_offset']} ${-1*params['wheel_center_y_offset']} ${params['wheel_center_z_offset']}" />
     <joint_options>
       <limit effort="10" velocity="8" />
@@ -71,5 +86,6 @@
     <robotNamespace>/mirte-control</robotNamespace>
   </plugin> -->
-    <plugin name="gazebo_ros_controller_manager" filename="libgazebo_ros_controller_manager.so"></plugin>
+    <plugin name="gazebo_ros_controller_manager"
+    filename="libgazebo_ros_controller_manager.so" />
   </gazebo>
   <xacro:include filename="$(find mirte_gazebo)/urdf/diffdrive.xacro" />

File: urdf/ros_control.xacro (robot description, xacro)
@@ -26,5 +26,6 @@
 -->
   <gazebo>
-    <plugin filename="libgazebo_ros_control.so" name="gazebo_ros_control">
+    <plugin filename="libgazebo_ros_control.so"
+    name="gazebo_ros_control">
       <robotNamespace>/mirte-control</robotNamespace>
     </plugin>

File: urdf/tile.xacro (robot description, xacro)
@@ -1,2 +1,3 @@
+<?xml version="1.0"?>
 <robot xmlns:xacro="http://www.ros.org/wiki/xacro">
   <xacro:macro name="tile" params="name material size x y yaw=0">
@@ -4,8 +5,10 @@
       <inertial>
         <mass value="10.0" />
-        <inertia ixx="1.0" ixy="0.0" ixz="0.0" iyy="1.0" iyz="0.0" izz="1.0" />
+        <inertia ixx="1.0" ixy="0.0" ixz="0.0" iyy="1.0" iyz="0.0"
+        izz="1.0" />
       </inertial>
       <visual>
-        <origin xyz="${x * size} ${y * size} 0" rpy="0 0 ${pi / 180 * yaw}" />
+        <origin xyz="${x * size} ${y * size} 0"
+        rpy="0 0 ${pi / 180 * yaw}" />
         <geometry>
           <box size="${size} ${size} .02" />

File: urdf/ultrasonic.xacro (robot description, xacro)
@@ -25,5 +25,6 @@
         <mass value="0.0" />
         <origin xyz="0 0 0" rpy="0 0 0" />
-        <inertia ixx="0.0" ixy="0.0" ixz="0.0" iyy="0.0" iyz="0.0" izz="0.0" />
+        <inertia ixx="0.0" ixy="0.0" ixz="0.0" iyy="0.0" iyz="0.0"
+        izz="0.0" />
       </inertial>
     </link>
@@ -61,5 +62,6 @@
         <!-- Using gazebo's update rate instead of plugin's -->
         <update_rate>30</update_rate>
-        <plugin name="gazebo_ros_range_controller_${name}" filename="libgazebo_ros_ray_sensor.so">
+        <plugin name="gazebo_ros_range_controller_${name}"
+        filename="libgazebo_ros_ray_sensor.so">
           <!-- Change namespace and output topic so published topic is /rrbot/laser/scan -->
           <ros>
