Commit message: add sonar + fix formatting

File: urdf/materials.xacro (robot description, xacro)
@@ -2,29 +2,29 @@
 <robot xmlns:xacro="http://www.ros.org/wiki/xacro" name="mirte">
   <material name="black">
-    <color rgba="0.0 0.0 0.0 1.0" />
+    <color rgba="0.0 0.0 0.0 1.0"/>
   </material>
   <material name="blue">
-    <color rgba="0.203125 0.23828125 0.28515625 1.0" />
+    <color rgba="0.203125 0.23828125 0.28515625 1.0"/>
   </material>
   <material name="green">
-    <color rgba="0.0 0.8 0.0 1.0" />
+    <color rgba="0.0 0.8 0.0 1.0"/>
   </material>
   <material name="grey">
-    <color rgba="0.2 0.2 0.2 1.0" />
+    <color rgba="0.2 0.2 0.2 1.0"/>
   </material>
   <material name="orange">
-    <color rgba="1.0 0.423529411765 0.0392156862745 1.0" />
+    <color rgba="1.0 0.423529411765 0.0392156862745 1.0"/>
   </material>
   <material name="brown">
-    <color rgba="0.870588235294 0.811764705882 0.764705882353 1.0" />
+    <color rgba="0.870588235294 0.811764705882 0.764705882353 1.0"/>
   </material>
   <material name="red">
-    <color rgba="0.80078125 0.12890625 0.1328125 1.0" />
+    <color rgba="0.80078125 0.12890625 0.1328125 1.0"/>
   </material>
   <material name="white">
-    <color rgba="1.0 1.0 1.0 1.0" />
+    <color rgba="1.0 1.0 1.0 1.0"/>
   </material>
   <material name="wood">
-    <color rgba="1.0 0.0 1.0 1.0" />
+    <color rgba="1.0 0.0 1.0 1.0"/>
   </material>
   <gazebo reference="link_chassis">
@@ -37,8 +37,8 @@
   </gazebo>
   <gazebo reference="link_left_wheel">
-    <mu1 value="1.0" />
-    <mu2 value="1.0" />
-    <kp value="1000000.0" />
-    <kd value="100.0" />
+    <mu1 value="1.0"/>
+    <mu2 value="1.0"/>
+    <kp value="1000000.0"/>
+    <kd value="100.0"/>
     <minDepth>0.001</minDepth>
     <maxVel>0.55</maxVel>
@@ -46,8 +46,8 @@
   </gazebo>
   <gazebo reference="link_right_wheel">
-    <mu1 value="1.0" />
-    <mu2 value="1.0" />
-    <kp value="1000000.0" />
-    <kd value="100.0" />
+    <mu1 value="1.0"/>
+    <mu2 value="1.0"/>
+    <kp value="1000000.0"/>
+    <kd value="100.0"/>
     <minDepth>0.001</minDepth>
     <maxVel>0.55</maxVel>

File: urdf/mirte.xacro (robot description, xacro)
@@ -1,36 +1,30 @@
 <?xml version="1.0"?>
 <robot xmlns:xacro="http://www.ros.org/wiki/xacro" name="mirte">
-  <xacro:include filename="$(find mirte_gazebo)/urdf/materials.xacro" />
-  <xacro:include filename="$(find mirte_gazebo)/urdf/macros.xacro" />
-  <xacro:include filename="$(find mirte_gazebo)/urdf/ros_control.xacro" />
+  <xacro:include filename="$(find mirte_gazebo)/urdf/materials.xacro"/>
+  <xacro:include filename="$(find mirte_gazebo)/urdf/macros.xacro"/>
+  <xacro:include filename="$(find mirte_gazebo)/urdf/ros_control.xacro"/>
   <!-- <xacro:include filename="$(find mirte_gazebo)/urdf/lidar.xacro" /> -->
   <!-- <xacro:include filename="$(find mirte_gazebo)/urdf/camera.xacro" /> -->
-   <xacro:include filename="$(find mirte_gazebo)/urdf/ultrasonic.xacro"/>
-  <xacro:property name="yaml_param_file"
-  value="$(find mirte_gazebo)/config/mirte_dimensions.yaml" />
-  <xacro:property name="params"
-  value="${xacro.load_yaml(yaml_param_file)}" />
+  <xacro:include filename="$(find mirte_gazebo)/urdf/ultrasonic.xacro"/>
+  <xacro:property name="yaml_param_file" value="$(find mirte_gazebo)/config/mirte_dimensions.yaml"/>
+  <xacro:property name="params" value="${xacro.load_yaml(yaml_param_file)}"/>
   <link name="link_chassis">
     <!-- pose and inertial -->
     <pose>0 0 0.015 0 0 0</pose>
-    <xacro:inertia_box x="${params['base_len']}"
-    y="${params['base_width']}" z="${params['base_height']}"
-    mass="${params['base_mass']}">
-      <origin rpy="0 0 0" xyz="0 0 0.015" />
+    <xacro:inertia_box x="${params['base_len']}" y="${params['base_width']}" z="${params['base_height']}" mass="${params['base_mass']}">
+      <origin rpy="0 0 0" xyz="0 0 0.015"/>
     </xacro:inertia_box>
     <!-- body -->
     <collision name="collision_chassis">
       <geometry>
-        <mesh filename="file://$(find mirte_gazebo)/meshes/mirte_base.stl"
-        scale="0.001 0.001 0.001" rpy="0 0 1.57079633" />
+        <mesh filename="file://$(find mirte_gazebo)/meshes/mirte_base.stl" scale="0.001 0.001 0.001" rpy="0 0 1.57079633"/>
       </geometry>
     </collision>
     <visual>
-      <origin rpy="0 0 0" xyz="0 0 0" />
+      <origin rpy="0 0 0" xyz="0 0 0"/>
       <geometry>
-        <mesh filename="file://$(find mirte_gazebo)/meshes/mirte_base.stl"
-        scale="0.001 0.001 0.001" rpy="0 0 1.57079633" />
+        <mesh filename="file://$(find mirte_gazebo)/meshes/mirte_base.stl" scale="0.001 0.001 0.001" rpy="0 0 1.57079633"/>
       </geometry>
-      <material name="blue" />
+      <material name="blue"/>
     </visual>
   </link>
@@ -38,56 +32,44 @@
     <gravity>0</gravity>
   </gazebo>
-  <link name="base_link" />
+  <link name="base_link"/>
   <gazebo reference="base_link">
     <gravity>0</gravity>
   </gazebo>
   <joint name="base_joint" type="fixed">
-    <parent link="base_link" />
-    <child link="link_chassis" />
+    <parent link="base_link"/>
+    <child link="link_chassis"/>
   </joint>
-  <xacro:caster name="caster_wheel_back" parent="link_chassis"
-  radius="${params['caster_wheel_radius']}"
-  mass="${params['caster_wheel_mass']}">
-    <origin rpy="0 0 0"
-    xyz="${params['caster_wheel_center_x_offset']} ${params['caster_wheel_center_y_offset']} ${params['caster_wheel_center_z_offset']}" />
+  <xacro:caster name="caster_wheel_back" parent="link_chassis" radius="${params['caster_wheel_radius']}" mass="${params['caster_wheel_mass']}">
+    <origin rpy="0 0 0" xyz="${params['caster_wheel_center_x_offset']} ${params['caster_wheel_center_y_offset']} ${params['caster_wheel_center_z_offset']}"/>
   </xacro:caster>
   <!-- NOTE: xacro parser adds joint_ -->
-  <xacro:wheel name="left_wheel" parent="link_chassis"
-  radius="${params['wheel_radius']}" visualRot="1"
-  mass="${params['wheel_mass']}">
-    <origin rpy="0 0 0"
-    xyz="${params['wheel_center_x_offset']} ${params['wheel_center_y_offset']} ${params['wheel_center_z_offset']}" />
+  <xacro:wheel name="left_wheel" parent="link_chassis" radius="${params['wheel_radius']}" visualRot="1" mass="${params['wheel_mass']}">
+    <origin rpy="0 0 0" xyz="${params['wheel_center_x_offset']} ${params['wheel_center_y_offset']} ${params['wheel_center_z_offset']}"/>
     <joint_options>
-      <limit effort="10" velocity="8" />
-      <dynamics damping="0.0" friction="0.0" />
+      <limit effort="10" velocity="8"/>
+      <dynamics damping="0.0" friction="0.0"/>
     </joint_options>
   </xacro:wheel>
   <!-- NOTE: xacro parser adds joint_ -->
-  <xacro:wheel name="right_wheel" parent="link_chassis"
-  radius="${params['wheel_radius']}" mass="${params['wheel_mass']}"
-  visualRot="0">
-    <origin rpy="0 0 0"
-    xyz="${params['wheel_center_x_offset']} ${-1*params['wheel_center_y_offset']} ${params['wheel_center_z_offset']}" />
+  <xacro:wheel name="right_wheel" parent="link_chassis" radius="${params['wheel_radius']}" mass="${params['wheel_mass']}" visualRot="0">
+    <origin rpy="0 0 0" xyz="${params['wheel_center_x_offset']} ${-1*params['wheel_center_y_offset']} ${params['wheel_center_z_offset']}"/>
     <joint_options>
-      <limit effort="10" velocity="8" />
-      <dynamics damping="0.0" friction="0.0" />
+      <limit effort="10" velocity="8"/>
+      <dynamics damping="0.0" friction="0.0"/>
     </joint_options>
   </xacro:wheel>
   <xacro:ultrasonic_sensor name="left">
-    <origin rpy="0 0 .45" xyz="0.085 0.04 0.022" />
+    <origin rpy="0 0 .45" xyz="0.085 0.04 0.022"/>
   </xacro:ultrasonic_sensor>
-<!--
   <xacro:ultrasonic_sensor name="right">
-    <origin rpy="0 0 -0.45" xyz="0.085 -0.04 0.022" />
-  </xacro:ultrasonic_sensor> -->
+    <origin rpy="0 0 -0.45" xyz="0.085 -0.04 0.022"/>
+  </xacro:ultrasonic_sensor>
   <gazebo>
-    <plugin name="gazebo_ros_control"
-    filename="libgazebo_ros_control.so">
+    <plugin name="gazebo_ros_control" filename="libgazebo_ros_control.so">
       <robotNamespace>/mirte-control</robotNamespace>
       <parameters>$(find mirte_gazebo)/config/mirte_diff_drive.yaml</parameters>
     </plugin>
-    <plugin name="gazebo_ros_controller_manager"
-    filename="libgazebo_ros_controller_manager.so" />
+    <plugin name="gazebo_ros_controller_manager" filename="libgazebo_ros_controller_manager.so"/>
   </gazebo>
-  <xacro:include filename="$(find mirte_gazebo)/urdf/diffdrive.xacro" />
+  <xacro:include filename="$(find mirte_gazebo)/urdf/diffdrive.xacro"/>
 </robot>

File: urdf/ros_control.xacro (robot description, xacro)
@@ -26,6 +26,5 @@
 -->
   <gazebo>
-    <plugin filename="libgazebo_ros_control.so"
-    name="gazebo_ros_control">
+    <plugin filename="libgazebo_ros_control.so" name="gazebo_ros_control">
       <robotNamespace>/mirte-control</robotNamespace>
     </plugin>

File: urdf/tile.xacro (robot description, xacro)
@@ -4,25 +4,23 @@
     <link name="${name}">
       <inertial>
-        <mass value="10.0" />
-        <inertia ixx="1.0" ixy="0.0" ixz="0.0" iyy="1.0" iyz="0.0"
-        izz="1.0" />
+        <mass value="10.0"/>
+        <inertia ixx="1.0" ixy="0.0" ixz="0.0" iyy="1.0" iyz="0.0" izz="1.0"/>
       </inertial>
       <visual>
-        <origin xyz="${x * size} ${y * size} 0"
-        rpy="0 0 ${pi / 180 * yaw}" />
+        <origin xyz="${x * size} ${y * size} 0" rpy="0 0 ${pi / 180 * yaw}"/>
         <geometry>
-          <box size="${size} ${size} .02" />
+          <box size="${size} ${size} .02"/>
         </geometry>
       </visual>
       <collision>
-        <origin xyz="${x * size} ${y * size} 0" />
+        <origin xyz="${x * size} ${y * size} 0"/>
         <geometry>
-          <box size="${size} ${size} .02" />
+          <box size="${size} ${size} .02"/>
         </geometry>
       </collision>
     </link>
     <joint name="${name}_joint" type="fixed">
-      <parent link="dummy_link" />
-      <child link="${name}" />
+      <parent link="dummy_link"/>
+      <child link="${name}"/>
     </joint>
     <gazebo reference="${name}">

File: urdf/ultrasonic.xacro (robot description, xacro)
@@ -2,30 +2,29 @@
 <robot xmlns:xacro="http://www.ros.org/wiki/xacro">
   <xacro:macro name="ultrasonic_sensor" params="name *origin">
-<xacro:property name="sonar_angle_max" value="${radians(15)}" />
+    <xacro:property name="sonar_angle_max" value="${radians(15)}"/>
     <joint name="sonar_${name}" type="fixed">
-      <axis xyz="0 1 0" />
-      <xacro:insert_block name="origin" />
-      <parent link="link_chassis" />
-      <child link="base_sonar_${name}" />
+      <axis xyz="0 1 0"/>
+      <xacro:insert_block name="origin"/>
+      <parent link="link_chassis"/>
+      <child link="base_sonar_${name}"/>
     </joint>
     <link name="base_sonar_${name}">
       <collision>
-        <origin xyz="0 0 0" rpy="0 0 0" />
+        <origin xyz="0 0 0" rpy="0 0 0"/>
         <geometry>
-          <box size="0.01 0.05 0.037" />
+          <box size="0.01 0.05 0.037"/>
         </geometry>
       </collision>
       <visual>
-        <origin xyz="0 0 0" rpy="0 0 0" />
+        <origin xyz="0 0 0" rpy="0 0 0"/>
         <geometry>
-          <box size="0.01 0.05 0.037" />
+          <box size="0.01 0.05 0.037"/>
         </geometry>
-        <material name="blue" />
+        <material name="blue"/>
       </visual>
       <inertial>
-        <mass value="0.0" />
-        <origin xyz="0 0 0" rpy="0 0 0" />
-        <inertia ixx="0.0" ixy="0.0" ixz="0.0" iyy="0.0" iyz="0.0"
-        izz="0.0" />
+        <mass value="0.0"/>
+        <origin xyz="0 0 0" rpy="0 0 0"/>
+        <inertia ixx="0.0" ixy="0.0" ixz="0.0" iyy="0.0" iyz="0.0" izz="0.0"/>
       </inertial>
     </link>
@@ -45,5 +44,6 @@
               <samples>4</samples>
               <resolution>1</resolution>
-              <min_angle>0</min_angle> <!-- Don't look to much at the floor-->
+              <min_angle>0</min_angle>
+              <!-- Don't look at the floor-->
               <max_angle>${sonar_angle_max/4}</max_angle>
             </vertical>
@@ -63,12 +63,11 @@
         <!-- Using gazebo's update rate instead of plugin's -->
         <update_rate>30</update_rate>
-          <plugin name="laser_controller"
-      filename="libgazebo_ros_laser.so">
-        <topicName>/mirte/scan2</topicName>
-              <output_type>sensor_msgs/Range</output_type>
-      <radiation_type>ultrasound</radiation_type>
-        <frameName>base_sonar_${name}</frameName>
-      </plugin>
-<!--         <plugin name="gazebo_ros_head_hokuyo_controlle" filename="libgazebo_ros_range_sensor.so" >
+        <plugin name="laser_controller_sonar${name}" filename="libgazebo_ros_laser.so">
+          <topicName>/mirte/scanSonar${name}</topicName>
+          <output_type>sensor_msgs/Range</output_type>
+          <radiation_type>ultrasound</radiation_type>
+          <frameName>base_sonar_${name}</frameName>
+        </plugin>
+        <!--         <plugin name="gazebo_ros_head_hokuyo_controlle" filename="libgazebo_ros_range_sensor.so" >
   <ros>
     <remapping>~/out:=/jemoeder</remapping>
