Commit message: cones, mirte cam done

File: urdf/camera.xacro (robot description, xacro)
@@ -3,13 +3,18 @@
   <joint name="joint_camera" type="fixed">
     <origin xyz="0.1 0 0.035" rpy="0 0 0"/>
-    <parent link="link_chassis"/>
-    <child link="camera_link"/>
+    <parent>link_chassis</parent>
+    <child>camera_link</child>
   </joint>
-  <link name="camera_link"/>
-  <gazebo reference="camera_link">
-    <sensor type="camera" name="camera1">
-      <update_rate>10</update_rate>
-      <camera name="head">
-        <horizontal_fov>1.2</horizontal_fov>
+  <link name="camera_link">
+  <!-- <gazebo reference="camera_link"> -->
+  <sensor name="camera_sensor" type="camera">
+  <always_on>true</always_on>
+  <visualize>true</visualize>
+  <update_rate>30</update_rate>
+  <topic>camera/image_raw</topic>
+  <gz_frame_id>camera_rgb_frame</gz_frame_id>
+  <camera name="intel_realsense_r200">
+    <camera_info_topic>camera/camera_info</camera_info_topic>
+<horizontal_fov>1.2</horizontal_fov>
         <image>
           <width>640</width>
@@ -27,5 +32,9 @@
           <p1>0.0</p1>
           <p2>0.0</p2>
-        </distortion>
+        </distortion>  </camera>
+</sensor>
+    <!-- <sensor type="camera" name="camera1">
+      <update_rate>10</update_rate>
+      <camera name="head">
       </camera>
       <plugin name="camera_controller" filename="libgazebo_ros_camera.so">
@@ -39,5 +48,6 @@
         <hack_baseline>0.07</hack_baseline>
       </plugin>
-    </sensor>
-  </gazebo>
+    </sensor> -->
+  <!-- </gazebo> -->
+  </link>
 </robot>

File: urdf/duckieModels.xacro (robot description, xacro)
@@ -144,5 +144,5 @@
             <script>
               <name>${type}/${type}</name>
-              <uri>file://$(find mirte_gazebo)/models/${type}/materials/scripts/${type}.material</uri>
+              <uri>file://$(find mirte_gazebo)/models/${type}/meshes/${type}.mtl</uri>
             </script>
           </material>
@@ -271,3 +271,144 @@
     </model>
   </xacro:macro>
+  <xacro:macro name="model" params="name type size x y yaw=0 static=1 scale=1">
+        <!-- START GENERATED SCALES AND OFFSETS-->
+<!--
+    <xacro:property name="model_scale" value="${1}"/>
+      <xacro:property name="z_offset" value="${0}"/> -->
+<xacro:if value="${type == 'sign_blank'}">
+        <xacro:property name="model_scale" value="${0.19415283233733935}"/>
+        <xacro:property name="z_offset" value="${0}"/>
+      </xacro:if>
+      <xacro:if value="${type == 'building'}">
+        <xacro:property name="model_scale" value="${0.2898550724637681}"/>
+        <xacro:property name="z_offset" value="${0}"/>
+      </xacro:if>
+      <xacro:if value="${type == 'house'}">
+        <xacro:property name="model_scale" value="${0.20755956855837843}"/>
+        <xacro:property name="z_offset" value="${0.024247}"/>
+      </xacro:if>
+      <xacro:if value="${type == 'cone'}">
+        <xacro:property name="model_scale" value="${0.03172296965063494}"/>
+        <xacro:property name="z_offset" value="${0}"/>
+      </xacro:if>
+      <xacro:if value="${type == 'truck'}">
+        <xacro:property name="model_scale" value="${0.1927574101731193}"/>
+        <xacro:property name="z_offset" value="${1.072166}"/>
+      </xacro:if>
+      <xacro:if value="${type == 'tree'}">
+        <xacro:property name="model_scale" value="${0.28054126509522415}"/>
+        <xacro:property name="z_offset" value="${0.003644}"/>
+      </xacro:if>
+      <xacro:if value="${type == 'duckiebot'}">
+        <xacro:property name="model_scale" value="${8.126777732629012}"/>
+        <xacro:property name="z_offset" value="${0.03311}"/>
+      </xacro:if>
+      <xacro:if value="${type == 'sign_left_T_intersect'}">
+        <xacro:property name="model_scale" value="${4.34593654932638}"/>
+        <xacro:property name="z_offset" value="${0}"/>
+      </xacro:if>
+      <xacro:if value="${type == 'sign_4_way_intersect'}">
+        <xacro:property name="model_scale" value="${4.34593654932638}"/>
+        <xacro:property name="z_offset" value="${0}"/>
+      </xacro:if>
+      <xacro:if value="${type == 'sign_yield'}">
+        <xacro:property name="model_scale" value="${4.34593654932638}"/>
+        <xacro:property name="z_offset" value="${0}"/>
+      </xacro:if>
+      <xacro:if value="${type == 'sign_no_right_turn'}">
+        <xacro:property name="model_scale" value="${4.34593654932638}"/>
+        <xacro:property name="z_offset" value="${0}"/>
+      </xacro:if>
+      <xacro:if value="${type == 'sign_duck_crossing'}">
+        <xacro:property name="model_scale" value="${4.34593654932638}"/>
+        <xacro:property name="z_offset" value="${0}"/>
+      </xacro:if>
+      <xacro:if value="${type == 'sign_no_left_turn'}">
+        <xacro:property name="model_scale" value="${4.34593654932638}"/>
+        <xacro:property name="z_offset" value="${0}"/>
+      </xacro:if>
+      <xacro:if value="${type == 'sign_stop'}">
+        <xacro:property name="model_scale" value="${4.34593654932638}"/>
+        <xacro:property name="z_offset" value="${0}"/>
+      </xacro:if>
+      <xacro:if value="${type == 'sign_do_not_enter'}">
+        <xacro:property name="model_scale" value="${4.34593654932638}"/>
+        <xacro:property name="z_offset" value="${0}"/>
+      </xacro:if>
+      <xacro:if value="${type == 'bus'}">
+        <xacro:property name="model_scale" value="${0.22667415295835838}"/>
+        <xacro:property name="z_offset" value="${-4.396879}"/>
+      </xacro:if>
+      <xacro:if value="${type == 'sign_t_light_ahead'}">
+        <xacro:property name="model_scale" value="${4.34593654932638}"/>
+        <xacro:property name="z_offset" value="${0}"/>
+      </xacro:if>
+      <xacro:if value="${type == 'sign_right_T_intersect'}">
+        <xacro:property name="model_scale" value="${4.34593654932638}"/>
+        <xacro:property name="z_offset" value="${0}"/>
+      </xacro:if>
+      <xacro:if value="${type == 'sign_pedestrian'}">
+        <xacro:property name="model_scale" value="${4.34593654932638}"/>
+        <xacro:property name="z_offset" value="${0}"/>
+      </xacro:if>
+      <xacro:if value="${type == 'sign_oneway_left'}">
+        <xacro:property name="model_scale" value="${4.34593654932638}"/>
+        <xacro:property name="z_offset" value="${0}"/>
+      </xacro:if>
+      <xacro:if value="${type == 'trafficlight'}">
+        <xacro:property name="model_scale" value="${2.7362925425083047}"/>
+        <xacro:property name="z_offset" value="${0.014439}"/>
+      </xacro:if>
+      <xacro:if value="${type == 'sign_oneway_right'}">
+        <xacro:property name="model_scale" value="${4.34593654932638}"/>
+        <xacro:property name="z_offset" value="${0}"/>
+      </xacro:if>
+      <xacro:if value="${type == 'sign_T_intersect'}">
+        <xacro:property name="model_scale" value="${4.34593654932638}"/>
+        <xacro:property name="z_offset" value="${0}"/>
+      </xacro:if>
+      <xacro:if value="${type == 'duckie'}">
+        <xacro:property name="model_scale" value="${0.6585788789802037}"/>
+        <xacro:property name="z_offset" value="${-0.113989}"/>
+      </xacro:if>
+      <xacro:if value="${type == 'barrier'}">
+        <xacro:property name="model_scale" value="${0.8748906386701663}"/>
+        <xacro:property name="z_offset" value="${0}"/>
+      </xacro:if>
+      <!-- END GENERATED -->
+       <model name="model_${name}">
+      <static>${static}</static>
+                <pose>${x * size} ${y * size} ${z_offset*size * model_scale * scale + 0.01} ${radians(90)} -0  ${radians(yaw)}</pose>
+    <link name="link_${name}">
+      <collision name="collision_${name}">
+        <geometry>
+          <mesh>
+      <scale>${size * model_scale * scale} ${size * model_scale * scale} ${size * model_scale * scale}</scale>
+            <!-- <scale>0.0254 0.0254 0.0254</scale> -->
+            <uri>model://${type}/meshes/${type}.obj</uri>
+          </mesh>
+        </geometry>
+      </collision>
+      <visual name="visual_${name}">
+        <geometry>
+          <mesh>
+      <pose>${x * size} ${y * size} ${z_offset*size * model_scale * scale + 0.01} ${radians(90)} -0  ${radians(yaw)}</pose>
+      <scale>${size * model_scale * scale} ${size * model_scale * scale} ${size * model_scale * scale}</scale>
+            <!-- <scale>0.0254 0.0254 0.0254</scale> -->
+            <uri>model://${type}/meshes/${type}.obj</uri>
+          </mesh>
+        </geometry>
+      </visual>
+    </link>
+  </model>
+  <!-- <model name="model_${name}">
+      <pose>${x * size} ${y * size} ${z_offset*size * model_scale * scale + 0.01} ${radians(90)} -0  ${radians(yaw)}</pose>
+      <static>${static}</static>
+      <scale>${size * model_scale * scale} ${size * model_scale * scale} ${size * model_scale * scale}</scale>
+      <include>
+      <scale>0.5 0.5 0.5</scale>
+        <uri>model://${type}</uri>
+      </include>
+    </model> -->
+    </xacro:macro>
 </robot>

File: urdf/macros.xacro (robot description, xacro)
@@ -49,5 +49,5 @@
     </inertial>
   </xacro:macro>
-  <xacro:macro name="wheel" params="name parent radius mass visualRot  *pose **content">
+  <xacro:macro name="wheel" params="name parent radius mass visualRot mult=1  *pose **content">
     <link name="link_${name}">
       <xacro:insert_block name="pose"/>
@@ -95,5 +95,5 @@
       <axis>
         <rpy>0 0 0</rpy>
-        <xyz>0 1 0</xyz>
+        <xyz>0 0 ${mult}</xyz>
       </axis>
       <xacro:insert_block name="content"/>

File: urdf/mirte.xacro (robot description, xacro)
@@ -4,5 +4,5 @@
     <xacro:arg name="sonar_enable" default="false"/>
     <xacro:arg name="intensity_enable" default="false"/>
-    <xacro:arg name="camera_enable" default="false"/>
+    <xacro:arg name="camera_enable" default="true"/>
     <xacro:arg name="lidar_enable" default="false"/>
     <xacro:arg name="realsense_enable" default="false"/>
@@ -88,5 +88,5 @@
     </xacro:caster>
     <!-- NOTE: xacro parser adds joint_ -->
-    <xacro:wheel name="left_wheel" parent="link_chassis" radius="${params['wheel_radius']}" visualRot="1" mass="${params['wheel_mass']}">
+    <xacro:wheel name="left_wheel" parent="link_chassis" radius="${params['wheel_radius']}" visualRot="1" mass="${params['wheel_mass']}" mult="-1">
       <pose>${params['wheel_center_x_offset']} ${params['wheel_center_y_offset']} ${params['wheel_center_z_offset']} ${pi/2} ${pi/2} 0</pose>
       <!-- <origin><rpy>0 0 0</rpy><xyz>${params['wheel_center_x_offset']} ${params['wheel_center_y_offset']} ${params['wheel_center_z_offset']}</xyz></origin> -->
@@ -97,5 +97,5 @@
     </xacro:wheel>
     <!-- NOTE: xacro parser adds joint_ -->
-    <xacro:wheel name="right_wheel" parent="link_chassis" radius="${params['wheel_radius']}" mass="${params['wheel_mass']}" visualRot="0">
+    <xacro:wheel name="right_wheel" parent="link_chassis" radius="${params['wheel_radius']}" mass="${params['wheel_mass']}" visualRot="0" mult="1">
       <pose>${params['wheel_center_x_offset']} ${-1*params['wheel_center_y_offset']} ${params['wheel_center_z_offset']} ${pi/2} ${pi/2} ${pi}</pose>
       <!-- <origin><rpy>0 0 0</rpy><xyz></xyz></origin> -->
@@ -122,4 +122,21 @@
       </xacro:ir_sensor>
     </xacro:if>
+    <plugin filename="gz-sim-diff-drive-system" name="gz::sim::systems::DiffDrive">
+  <!-- Remove <ros> tag. -->
+  <!-- wheels -->
+  <left_joint>joint_left_wheel</left_joint>
+  <right_joint>joint_right_wheel</right_joint>
+  <!-- kinematics -->
+  <wheel_separation>0.14</wheel_separation>
+  <wheel_radius>0.0325</wheel_radius> <!-- computed from <wheel_diameter> in the original plugin-->
+  <!-- limits -->
+  <max_linear_acceleration>1</max_linear_acceleration> <!-- computed from <max_linear_acceleration> in the original plugin-->
+  <topic>cmd_vel</topic> <!-- from <commant_topic> -->
+  <odom_topic>odom</odom_topic> <!-- from <odometry_topic> -->
+  <frame_id>odom</frame_id> <!-- from <odometry_frame> -->
+  <child_frame_id>base_footprint</child_frame_id> <!-- from <robot_base_frame> -->
+  <odom_publisher_frequency>30</odom_publisher_frequency> <!-- from <update_rate>-->
+  <tf_topic>/tf</tf_topic> <!-- Short topic name for tf output -->
+</plugin>
     <!-- <gazebo>
     <plugin name="gazebo_ros_control" filename="libgazebo_ros_control.so">

File: urdf/realsense-depth.xacro (robot description, xacro)
@@ -16,13 +16,14 @@
     <!-- Camera link -->
     <link name="${prefix}rs200_camera">
-      <visual>
+      <visual name="vis_${prefix}_rs200_cam">
         <origin rpy="0 0 0" xyz="0 0 0"/>
         <geometry>
-          <mesh filename="package://mirte_gazebo/models/realsense_camera/meshes/realsense.dae"/>
+          <mesh>
+           <filename>package://mirte_gazebo/models/realsense_camera/meshes/realsense.dae</filename></mesh>
         </geometry>
       </visual>
-      <collision name="realsense_collision">
+      <collision name="coll_${prefix}_rs200_cam">
         <geometry>
-          <box size="0.0078 0.130 0.0192"/>
+          <box><size>0.0078 0.130 0.0192</size></box>
         </geometry>
       </collision>
@@ -30,11 +31,13 @@
         <mass value="0.0615752"/>
         <origin rpy="0 0 0" xyz="0 0 0"/>
-        <inertia ixx="9.108e-05" ixy="0" ixz="0" iyy="2.51e-06" iyz="0" izz="8.931e-05"/>
+        <inertia>
+         <ixx>9.108e-05</ixx> <ixy>0</ixy><ixz>0</ixz><iyy>2.51e-06</iyy><iyz>0</iyz><izz>8.931e-05</izz>
+         </inertia>
       </inertial>
     </link>
     <!-- Connect camera to parent frame-->
     <joint name="${prefix}realsense_joint" type="fixed">
-      <parent link="${parent}"/>
-      <child link="${prefix}rs200_camera"/>
+      <parent>${parent}</parent>
+      <child>${prefix}rs200_camera</child>
       <xacro:insert_block name="origin"/>
     </joint>
@@ -43,10 +46,11 @@
     <!-- Joints positioning the virtual links with respect to the camera main link-->
     <joint name="${prefix}depth_joint" type="fixed">
-      <parent link="${prefix}rs200_camera"/>
-      <child link="${prefix}depth"/>
+      <parent>${prefix}rs200_camera</parent>
+      <child>${prefix}depth</child>
       <origin xyz="0 -0 0.004" rpy="0 0 0"/>
     </joint>
-    <gazebo reference="${prefix}rs200_camera">
-      <sensor name="realsense_contact" type="contact">
+    <!-- <gazebo reference="${prefix}rs200_camera"> -->
+    <!-- TODO: later weer terugzetten! -->
+      <!-- <sensor name="realsense_contact" type="contact">
         <always_on>true</always_on>
         <update_rate>30.0</update_rate>
@@ -57,6 +61,6 @@
           <test2 name="ir" value="$(arg intensity_enable)"/>
           <arg val="2 + 2xir + lidar"/>
-          <!-- See https://github.com/gazebosim/sdformat/issues/333 for why the strange naming. Get the correct name by running xacro mirte.xacro > test.xml && gz sdf -p test.xml > robot.xml and look for the name-->
-          <!-- This strange calculation should make sure that when adding/removing lidar and ir sensors, the collision name still is correct -->
+          <!- - See https://github.com/gazebosim/sdformat/issues/333 for why the strange naming. Get the correct name by running xacro mirte.xacro > test.xml && gz sdf -p test.xml > robot.xml and look for the name- ->
+          <!- - This strange calculation should make sure that when adding/removing lidar and ir sensors, the collision name still is correct - ->
           <collision>base_link_fixed_joint_lump__realsense_collision_collision_${lidar + 2*ir + 2}</collision>
         </contact>
@@ -66,12 +70,15 @@
         </plugin>
       </sensor>
-    </gazebo>
-    <gazebo reference="${prefix}depth">
-      <sensor name="depth_camera" type="depth">
-        <always_on>true</always_on>
-        <visualize>False</visualize>
-        <update_rate>10</update_rate>
-        <camera name="camera">
-          <horizontal_fov>2.5</horizontal_fov>
+    </gazebo> -->
+    <!-- <gazebo reference="${prefix}depth"> -->
+    <sensor name="camera_sensor_depth" type="camera">
+  <always_on>true</always_on>
+  <visualize>true</visualize>
+  <update_rate>30</update_rate>
+  <topic>camera/image_raw</topic>
+  <gz_frame_id>camera_rgb_frame</gz_frame_id>
+  <camera name="intel_realsense_r200">
+    <camera_info_topic>camera/camera_info</camera_info_topic>
+<horizontal_fov>2.5</horizontal_fov>
           <image>
             <width>640</width>
@@ -82,7 +89,23 @@
             <near>0.02</near>
             <far>2</far>
-          </clip>
-        </camera>
-        <plugin name="depth_camera_controller" filename="libgazebo_ros_depth_camera.so">
+          </clip>  </camera>
+</sensor>
+      <sensor name="depth_camera1" type="depth_camera">
+          <update_rate>10</update_rate>
+          <topic>depth_camera</topic>
+          <camera>
+            <horizontal_fov>1.05</horizontal_fov>
+            <image>
+              <width>256</width>
+              <height>256</height>
+              <format>R_FLOAT32</format>
+            </image>
+            <clip>
+              <near>0.1</near>
+              <far>10.0</far>
+            </clip>
+          </camera>
+          </sensor>
+        <!-- <plugin name="depth_camera_controller" filename="libgazebo_ros_depth_camera.so">
           <alwaysOn>1</alwaysOn>
           <updateRate>10.0</updateRate>
@@ -95,5 +118,5 @@
         </plugin>
       </sensor>
-    </gazebo>
+    </gazebo> -->
   </xacro:macro>
 </robot>
