Commit message: cleanups and style fixes

File: urdf/camera.xacro (robot description, xacro)
@@ -7,14 +7,14 @@
   </joint>
   <link name="camera_link">
-  <!-- <gazebo reference="camera_link"> -->
-  <sensor name="camera_sensor" type="camera">
-  <always_on>true</always_on>
-  <visualize>true</visualize>
-  <update_rate>30</update_rate>
-  <topic>camera/image_raw</topic>
-  <gz_frame_id>camera_rgb_frame</gz_frame_id>
-  <camera name="intel_realsense_r200">
-    <camera_info_topic>camera/camera_info</camera_info_topic>
-<horizontal_fov>1.2</horizontal_fov>
+    <!-- <gazebo reference="camera_link"> -->
+    <sensor name="camera_sensor" type="camera">
+      <always_on>true</always_on>
+      <visualize>true</visualize>
+      <update_rate>30</update_rate>
+      <topic>camera/image_raw</topic>
+      <gz_frame_id>camera_rgb_frame</gz_frame_id>
+      <camera name="intel_realsense_r200">
+        <camera_info_topic>camera/camera_info</camera_info_topic>
+        <horizontal_fov>1.2</horizontal_fov>
         <image>
           <width>640</width>
@@ -32,6 +32,7 @@
           <p1>0.0</p1>
           <p2>0.0</p2>
-        </distortion>  </camera>
-</sensor>
+        </distortion>
+      </camera>
+    </sensor>
     <!-- <sensor type="camera" name="camera1">
       <update_rate>10</update_rate>
@@ -49,5 +50,5 @@
       </plugin>
     </sensor> -->
-  <!-- </gazebo> -->
+    <!-- </gazebo> -->
   </link>
 </robot>

File: urdf/duckieModels.xacro (robot description, xacro)
@@ -272,135 +272,135 @@
   </xacro:macro>
   <xacro:macro name="model" params="name type size x y yaw=0 static=1 scale=1">
-        <!-- START GENERATED SCALES AND OFFSETS-->
-<!--
+    <!-- START GENERATED SCALES AND OFFSETS-->
+    <!--
     <xacro:property name="model_scale" value="${1}"/>
       <xacro:property name="z_offset" value="${0}"/> -->
-<xacro:if value="${type == 'sign_blank'}">
-        <xacro:property name="model_scale" value="${0.19415283233733935}"/>
-        <xacro:property name="z_offset" value="${0}"/>
-      </xacro:if>
-      <xacro:if value="${type == 'building'}">
-        <xacro:property name="model_scale" value="${0.2898550724637681}"/>
-        <xacro:property name="z_offset" value="${0}"/>
-      </xacro:if>
-      <xacro:if value="${type == 'house'}">
-        <xacro:property name="model_scale" value="${0.20755956855837843}"/>
-        <xacro:property name="z_offset" value="${0.024247}"/>
-      </xacro:if>
-      <xacro:if value="${type == 'cone'}">
-        <xacro:property name="model_scale" value="${0.03172296965063494}"/>
-        <xacro:property name="z_offset" value="${3.5}"/>
-      </xacro:if>
-      <xacro:if value="${type == 'truck'}">
-        <xacro:property name="model_scale" value="${0.1927574101731193}"/>
-        <xacro:property name="z_offset" value="${1.072166}"/>
-      </xacro:if>
-      <xacro:if value="${type == 'tree'}">
-        <xacro:property name="model_scale" value="${0.28054126509522415}"/>
-        <xacro:property name="z_offset" value="${0.003644}"/>
-      </xacro:if>
-      <xacro:if value="${type == 'duckiebot'}">
-        <xacro:property name="model_scale" value="${8.126777732629012}"/>
-        <xacro:property name="z_offset" value="${0.03311}"/>
-      </xacro:if>
-      <xacro:if value="${type == 'sign_left_T_intersect'}">
-        <xacro:property name="model_scale" value="${4.34593654932638}"/>
-        <xacro:property name="z_offset" value="${0}"/>
-      </xacro:if>
-      <xacro:if value="${type == 'sign_4_way_intersect'}">
-        <xacro:property name="model_scale" value="${4.34593654932638}"/>
-        <xacro:property name="z_offset" value="${0}"/>
-      </xacro:if>
-      <xacro:if value="${type == 'sign_yield'}">
-        <xacro:property name="model_scale" value="${4.34593654932638}"/>
-        <xacro:property name="z_offset" value="${0}"/>
-      </xacro:if>
-      <xacro:if value="${type == 'sign_no_right_turn'}">
-        <xacro:property name="model_scale" value="${4.34593654932638}"/>
-        <xacro:property name="z_offset" value="${0}"/>
-      </xacro:if>
-      <xacro:if value="${type == 'sign_duck_crossing'}">
-        <xacro:property name="model_scale" value="${4.34593654932638}"/>
-        <xacro:property name="z_offset" value="${0}"/>
-      </xacro:if>
-      <xacro:if value="${type == 'sign_no_left_turn'}">
-        <xacro:property name="model_scale" value="${4.34593654932638}"/>
-        <xacro:property name="z_offset" value="${0}"/>
-      </xacro:if>
-      <xacro:if value="${type == 'sign_stop'}">
-        <xacro:property name="model_scale" value="${4.34593654932638}"/>
-        <xacro:property name="z_offset" value="${0}"/>
-      </xacro:if>
-      <xacro:if value="${type == 'sign_do_not_enter'}">
-        <xacro:property name="model_scale" value="${4.34593654932638}"/>
-        <xacro:property name="z_offset" value="${0}"/>
-      </xacro:if>
-      <xacro:if value="${type == 'bus'}">
-        <xacro:property name="model_scale" value="${0.22667415295835838}"/>
-        <xacro:property name="z_offset" value="${-4.396879}"/>
-      </xacro:if>
-      <xacro:if value="${type == 'sign_t_light_ahead'}">
-        <xacro:property name="model_scale" value="${4.34593654932638}"/>
-        <xacro:property name="z_offset" value="${0}"/>
-      </xacro:if>
-      <xacro:if value="${type == 'sign_right_T_intersect'}">
-        <xacro:property name="model_scale" value="${4.34593654932638}"/>
-        <xacro:property name="z_offset" value="${0}"/>
-      </xacro:if>
-      <xacro:if value="${type == 'sign_pedestrian'}">
-        <xacro:property name="model_scale" value="${4.34593654932638}"/>
-        <xacro:property name="z_offset" value="${0}"/>
-      </xacro:if>
-      <xacro:if value="${type == 'sign_oneway_left'}">
-        <xacro:property name="model_scale" value="${4.34593654932638}"/>
-        <xacro:property name="z_offset" value="${0}"/>
-      </xacro:if>
-      <xacro:if value="${type == 'trafficlight'}">
-        <xacro:property name="model_scale" value="${2.7362925425083047}"/>
-        <xacro:property name="z_offset" value="${0.014439}"/>
-      </xacro:if>
-      <xacro:if value="${type == 'sign_oneway_right'}">
-        <xacro:property name="model_scale" value="${4.34593654932638}"/>
-        <xacro:property name="z_offset" value="${0}"/>
-      </xacro:if>
-      <xacro:if value="${type == 'sign_T_intersect'}">
-        <xacro:property name="model_scale" value="${4.34593654932638}"/>
-        <xacro:property name="z_offset" value="${0}"/>
-      </xacro:if>
-      <xacro:if value="${type == 'duckie'}">
-        <xacro:property name="model_scale" value="${0.6585788789802037}"/>
-        <xacro:property name="z_offset" value="${-0.113989}"/>
-      </xacro:if>
-      <xacro:if value="${type == 'barrier'}">
-        <xacro:property name="model_scale" value="${0.8748906386701663}"/>
-        <xacro:property name="z_offset" value="${0}"/>
-      </xacro:if>
-      <!-- END GENERATED -->
-       <model name="model_${name}">
+    <xacro:if value="${type == 'sign_blank'}">
+      <xacro:property name="model_scale" value="${0.19415283233733935}"/>
+      <xacro:property name="z_offset" value="${0}"/>
+    </xacro:if>
+    <xacro:if value="${type == 'building'}">
+      <xacro:property name="model_scale" value="${0.2898550724637681}"/>
+      <xacro:property name="z_offset" value="${0}"/>
+    </xacro:if>
+    <xacro:if value="${type == 'house'}">
+      <xacro:property name="model_scale" value="${0.20755956855837843}"/>
+      <xacro:property name="z_offset" value="${0.024247}"/>
+    </xacro:if>
+    <xacro:if value="${type == 'cone'}">
+      <xacro:property name="model_scale" value="${0.03172296965063494}"/>
+      <xacro:property name="z_offset" value="${3.5}"/>
+    </xacro:if>
+    <xacro:if value="${type == 'truck'}">
+      <xacro:property name="model_scale" value="${0.1927574101731193}"/>
+      <xacro:property name="z_offset" value="${1.072166}"/>
+    </xacro:if>
+    <xacro:if value="${type == 'tree'}">
+      <xacro:property name="model_scale" value="${0.28054126509522415}"/>
+      <xacro:property name="z_offset" value="${0.003644}"/>
+    </xacro:if>
+    <xacro:if value="${type == 'duckiebot'}">
+      <xacro:property name="model_scale" value="${8.126777732629012}"/>
+      <xacro:property name="z_offset" value="${0.03311}"/>
+    </xacro:if>
+    <xacro:if value="${type == 'sign_left_T_intersect'}">
+      <xacro:property name="model_scale" value="${4.34593654932638}"/>
+      <xacro:property name="z_offset" value="${0}"/>
+    </xacro:if>
+    <xacro:if value="${type == 'sign_4_way_intersect'}">
+      <xacro:property name="model_scale" value="${4.34593654932638}"/>
+      <xacro:property name="z_offset" value="${0}"/>
+    </xacro:if>
+    <xacro:if value="${type == 'sign_yield'}">
+      <xacro:property name="model_scale" value="${4.34593654932638}"/>
+      <xacro:property name="z_offset" value="${0}"/>
+    </xacro:if>
+    <xacro:if value="${type == 'sign_no_right_turn'}">
+      <xacro:property name="model_scale" value="${4.34593654932638}"/>
+      <xacro:property name="z_offset" value="${0}"/>
+    </xacro:if>
+    <xacro:if value="${type == 'sign_duck_crossing'}">
+      <xacro:property name="model_scale" value="${4.34593654932638}"/>
+      <xacro:property name="z_offset" value="${0}"/>
+    </xacro:if>
+    <xacro:if value="${type == 'sign_no_left_turn'}">
+      <xacro:property name="model_scale" value="${4.34593654932638}"/>
+      <xacro:property name="z_offset" value="${0}"/>
+    </xacro:if>
+    <xacro:if value="${type == 'sign_stop'}">
+      <xacro:property name="model_scale" value="${4.34593654932638}"/>
+      <xacro:property name="z_offset" value="${0}"/>
+    </xacro:if>
+    <xacro:if value="${type == 'sign_do_not_enter'}">
+      <xacro:property name="model_scale" value="${4.34593654932638}"/>
+      <xacro:property name="z_offset" value="${0}"/>
+    </xacro:if>
+    <xacro:if value="${type == 'bus'}">
+      <xacro:property name="model_scale" value="${0.22667415295835838}"/>
+      <xacro:property name="z_offset" value="${-4.396879}"/>
+    </xacro:if>
+    <xacro:if value="${type == 'sign_t_light_ahead'}">
+      <xacro:property name="model_scale" value="${4.34593654932638}"/>
+      <xacro:property name="z_offset" value="${0}"/>
+    </xacro:if>
+    <xacro:if value="${type == 'sign_right_T_intersect'}">
+      <xacro:property name="model_scale" value="${4.34593654932638}"/>
+      <xacro:property name="z_offset" value="${0}"/>
+    </xacro:if>
+    <xacro:if value="${type == 'sign_pedestrian'}">
+      <xacro:property name="model_scale" value="${4.34593654932638}"/>
+      <xacro:property name="z_offset" value="${0}"/>
+    </xacro:if>
+    <xacro:if value="${type == 'sign_oneway_left'}">
+      <xacro:property name="model_scale" value="${4.34593654932638}"/>
+      <xacro:property name="z_offset" value="${0}"/>
+    </xacro:if>
+    <xacro:if value="${type == 'trafficlight'}">
+      <xacro:property name="model_scale" value="${2.7362925425083047}"/>
+      <xacro:property name="z_offset" value="${0.014439}"/>
+    </xacro:if>
+    <xacro:if value="${type == 'sign_oneway_right'}">
+      <xacro:property name="model_scale" value="${4.34593654932638}"/>
+      <xacro:property name="z_offset" value="${0}"/>
+    </xacro:if>
+    <xacro:if value="${type == 'sign_T_intersect'}">
+      <xacro:property name="model_scale" value="${4.34593654932638}"/>
+      <xacro:property name="z_offset" value="${0}"/>
+    </xacro:if>
+    <xacro:if value="${type == 'duckie'}">
+      <xacro:property name="model_scale" value="${0.6585788789802037}"/>
+      <xacro:property name="z_offset" value="${-0.113989}"/>
+    </xacro:if>
+    <xacro:if value="${type == 'barrier'}">
+      <xacro:property name="model_scale" value="${0.8748906386701663}"/>
+      <xacro:property name="z_offset" value="${0}"/>
+    </xacro:if>
+    <!-- END GENERATED -->
+    <model name="model_${name}">
       <static>${static}</static>
-                <pose>${x * size} ${y * size} ${z_offset*size * model_scale * scale + 0.01} ${radians(90)} -0  ${radians(yaw)}</pose>
-    <link name="link_${name}">
-      <collision name="collision_${name}">
-        <geometry>
-          <mesh>
-      <scale>${size * model_scale * scale} ${size * model_scale * scale} ${size * model_scale * scale}</scale>
-            <!-- <scale>0.0254 0.0254 0.0254</scale> -->
-            <uri>model://${type}/meshes/${type}.obj</uri>
-          </mesh>
-        </geometry>
-      </collision>
-      <visual name="visual_${name}">
-        <geometry>
-          <mesh>
       <pose>${x * size} ${y * size} ${z_offset*size * model_scale * scale + 0.01} ${radians(90)} -0  ${radians(yaw)}</pose>
-      <scale>${size * model_scale * scale} ${size * model_scale * scale} ${size * model_scale * scale}</scale>
-            <!-- <scale>0.0254 0.0254 0.0254</scale> -->
-            <uri>model://${type}/meshes/${type}.obj</uri>
-          </mesh>
-        </geometry>
-      </visual>
-    </link>
-  </model>
-  <!-- <model name="model_${name}">
+      <link name="link_${name}">
+        <collision name="collision_${name}">
+          <geometry>
+            <mesh>
+              <scale>${size * model_scale * scale} ${size * model_scale * scale} ${size * model_scale * scale}</scale>
+              <!-- <scale>0.0254 0.0254 0.0254</scale> -->
+              <uri>model://${type}/meshes/${type}.obj</uri>
+            </mesh>
+          </geometry>
+        </collision>
+        <visual name="visual_${name}">
+          <geometry>
+            <mesh>
+              <pose>${x * size} ${y * size} ${z_offset*size * model_scale * scale + 0.01} ${radians(90)} -0  ${radians(yaw)}</pose>
+              <scale>${size * model_scale * scale} ${size * model_scale * scale} ${size * model_scale * scale}</scale>
+              <!-- <scale>0.0254 0.0254 0.0254</scale> -->
+              <uri>model://${type}/meshes/${type}.obj</uri>
+            </mesh>
+          </geometry>
+        </visual>
+      </link>
+    </model>
+    <!-- <model name="model_${name}">
       <pose>${x * size} ${y * size} ${z_offset*size * model_scale * scale + 0.01} ${radians(90)} -0  ${radians(yaw)}</pose>
       <static>${static}</static>
@@ -411,4 +411,4 @@
       </include>
     </model> -->
-    </xacro:macro>
+  </xacro:macro>
 </robot>

File: urdf/includedMacro.xacro (robot description, xacro)
@@ -2,11 +2,10 @@
 <robot xmlns:xacro="http://www.ros.org/wiki/xacro">
   <xacro:macro name="person" params="name size x y yaw=0 static=1 scale=1">
-        <xacro:property name="model_scale" value="${1}"/>
-      <xacro:property name="z_offset" value="${0}"/>
-   <model name='person_standing'>
-      <link name='link'>
+    <xacro:property name="model_scale" value="${1}"/>
+    <xacro:property name="z_offset" value="${0}"/>
+    <model name="person_standing">
+      <link name="link">
         <inertial>
-      <!-- <origin xyz="${size} ${y * size} 0"/> -->
-      <pose>${x * size} ${y * size} ${z_offset*size * model_scale * scale + 0.01} 0 -0  ${radians(yaw)}</pose>
+          <pose>${x * size} ${y * size} ${z_offset*size * model_scale * scale + 0.01} 0 -0  ${radians(yaw)}</pose>
           <mass>80</mass>
           <inertia>
@@ -19,5 +18,5 @@
           </inertia>
         </inertial>
-        <collision name='bottom'>
+        <collision name="bottom">
           <pose>0 -0.1 0.01 0 0 0</pose>
           <geometry>
@@ -34,16 +33,18 @@
           </surface>
         </collision>
-        <collision name='person'>
+        <collision name="person">
           <pose>0 0 0.02 0.04 0 0</pose>
           <geometry>
-            <mesh>              <scale>${scale} ${ scale} ${ scale}</scale>
+            <mesh>
+              <scale>${scale} ${ scale} ${ scale}</scale>
               <uri>model://person_standing/meshes/standing.dae</uri>
             </mesh>
           </geometry>
         </collision>
-        <visual name='visual'>
+        <visual name="visual">
           <pose>0 0 0.02 0.04 0 0</pose>
           <geometry>
-            <mesh>              <scale>${scale} ${ scale} ${ scale}</scale>
+            <mesh>
+              <scale>${scale} ${ scale} ${ scale}</scale>
               <uri>model://person_standing/meshes/standing.dae</uri>
             </mesh>
@@ -53,5 +54,4 @@
         <enable_wind>false</enable_wind>
       </link>
-      <!-- <origin xyz="${size} ${y * size} 0"/> -->
       <pose>${x * size} ${y * size} ${z_offset*size * model_scale * scale + 0.01} 0 -0  ${radians(yaw)}</pose>
       <static>${static}</static>
@@ -94,13 +94,6 @@
               <scale>${size * model_scale * scale} ${size * model_scale * scale} ${size * model_scale * scale}</scale>
               <uri>model://person_standing/meshes/person_standing.obj</uri>
-              <!-- <pose>${x * size} ${y * size}  ${z_offset*size * model_scale * scale + 0.01} ${radians(90)} -0 0</pose> -->
             </mesh>
           </geometry>
-          <!-- <material>
-            <script>
-              <name>${type}/${type}</name>
-              <uri>file://$(find mirte_gazebo)/models/${type}/materials/scripts/${type}.material</uri>
-            </script>
-          </material> -->
         </visual>
         <self_collide>0</self_collide>
@@ -108,5 +101,4 @@
         <kinematic>0</kinematic>
       </link>
-      <!-- <pose>${x * size} ${y * size}  ${z_offset*size * model_scale * scale + 0.01} ${radians(90)} -0 0</pose> -->
     </model>
   </xacro:macro>

File: urdf/macros.xacro (robot description, xacro)
@@ -114,10 +114,10 @@
   <xacro:macro name="caster" params="name parent radius mass *pose">
     <link name="link_${name}">
-    <inertial>
+      <inertial>
         <mass>10.0</mass>
         <!-- <origin rpy="0 0 0" xyz="0 0 0"/> -->
         <inertia>
-         <!-- <ixx>9.108e-05</ixx> <ixy>0</ixy><ixz>0</ixz><iyy>2.51e-06</iyy><iyz>0</iyz><izz>8.931e-05</izz> -->
-         </inertia>
+          <!-- <ixx>9.108e-05</ixx> <ixy>0</ixy><ixz>0</ixz><iyy>2.51e-06</iyy><iyz>0</iyz><izz>8.931e-05</izz> -->
+        </inertia>
       </inertial>
       <xacro:insert_block name="pose"/>

File: urdf/mirte.xacro (robot description, xacro)
@@ -7,7 +7,5 @@
     <xacro:arg name="lidar_enable" default="false"/>
     <xacro:arg name="realsense_enable" default="false"/>
-    <!-- <xacro:include filename="$(find mirte_gazebo)/urdf/materials.xacro"/> -->
     <xacro:include filename="$(find mirte_gazebo)/urdf/macros.xacro"/>
-    <!-- <xacro:include filename="$(find mirte_gazebo)/urdf/ros_control.xacro"/> -->
     <test value="$(arg sonar_enable)" name="sonar_enable"/>
     <test value="$(arg intensity_enable)" name="intensity_enable"/>
@@ -20,7 +18,4 @@
       <xacro:include filename="$(find mirte_gazebo)/urdf/ir.xacro"/>
     </xacro:if>
-    <!-- <xacro:if value="$(arg camera_enable)">
-      <xacro:include filename="$(find mirte_gazebo)/urdf/camera.xacro"/>
-    </xacro:if> -->
     <xacro:if value="$(arg sonar_enable)">
       <xacro:include filename="$(find mirte_gazebo)/urdf/ultrasonic.xacro"/>
@@ -88,5 +83,4 @@
     <xacro:wheel name="left_wheel" parent="link_chassis" radius="${params['wheel_radius']}" visualRot="1" mass="${params['wheel_mass']}" mult="-1">
       <pose>${params['wheel_center_x_offset']} ${params['wheel_center_y_offset']} ${params['wheel_center_z_offset']} ${pi/2} ${pi/2} 0</pose>
-      <!-- <origin><rpy>0 0 0</rpy><xyz>${params['wheel_center_x_offset']} ${params['wheel_center_y_offset']} ${params['wheel_center_z_offset']}</xyz></origin> -->
       <joint_options>
         <limit effort="10" velocity="8"/>
@@ -97,6 +91,4 @@
     <xacro:wheel name="right_wheel" parent="link_chassis" radius="${params['wheel_radius']}" mass="${params['wheel_mass']}" visualRot="0" mult="1">
       <pose>${params['wheel_center_x_offset']} ${-1*params['wheel_center_y_offset']} ${params['wheel_center_z_offset']} ${pi/2} ${pi/2} ${pi}</pose>
-      <!-- <origin><rpy>0 0 0</rpy><xyz></xyz></origin> -->
-      <!-- <origin rpy="0 0 0" xyz="${params['wheel_center_x_offset']} ${-1*params['wheel_center_y_offset']} ${params['wheel_center_z_offset']}"/> -->
       <joint_options>
         <limit effort="10" velocity="8"/>
@@ -121,37 +113,28 @@
     </xacro:if>
     <plugin filename="gz-sim-diff-drive-system" name="gz::sim::systems::DiffDrive">
-  <!-- Remove <ros> tag. -->
-  <!-- wheels -->
-  <left_joint>joint_left_wheel</left_joint>
-  <right_joint>joint_right_wheel</right_joint>
-  <!-- kinematics -->
-  <wheel_separation>0.14</wheel_separation>
-  <wheel_radius>0.0325</wheel_radius> <!-- computed from <wheel_diameter> in the original plugin-->
-  <!-- limits -->
-  <max_linear_acceleration>1</max_linear_acceleration> <!-- computed from <max_linear_acceleration> in the original plugin-->
-  <topic>cmd_vel</topic> <!-- from <commant_topic> -->
-  <odom_topic>odom</odom_topic> <!-- from <odometry_topic> -->
-  <frame_id>odom</frame_id> <!-- from <odometry_frame> -->
-  <child_frame_id>base_footprint</child_frame_id> <!-- from <robot_base_frame> -->
-  <odom_publisher_frequency>30</odom_publisher_frequency> <!-- from <update_rate>-->
-  <tf_topic>/tf</tf_topic> <!-- Short topic name for tf output -->
-</plugin>
-    <!-- <gazebo>
-    <plugin name="gazebo_ros_control" filename="libgazebo_ros_control.so">
-      <robotNamespace>/mirte</robotNamespace>
-      <!- - <parameters>$(find mirte_gazebo)/config/mirte_diff_drive.yaml</parameters> -->
-    <!-- </plugin> -->
-    <!-- <plugin name="gazebo_ros_controller_manager" filename="libgazebo_ros_controller_manager.so"/> - ->
-  </gazebo> -->
-    <!-- <xacro:include filename="$(find mirte_gazebo)/urdf/diffdrive.xacro"/>
-  <gazebo>
-    <plugin name="p3d" filename="libgazebo_ros_p3d.so">
-      <!- -  <robotNamespace>/prius</robotNamespace> - ->
-      <bodyName>base_link</bodyName>
-      <topicName>base_pose_ground_truth</topicName>
-      <frameName>map</frameName>
-      <updateRate>10.0</updateRate>
+      <!-- Remove <ros> tag. -->
+      <!-- wheels -->
+      <left_joint>joint_left_wheel</left_joint>
+      <right_joint>joint_right_wheel</right_joint>
+      <!-- kinematics -->
+      <wheel_separation>0.14</wheel_separation>
+      <wheel_radius>0.0325</wheel_radius>
+      <!-- computed from <wheel_diameter> in the original plugin-->
+      <!-- limits -->
+      <max_linear_acceleration>1</max_linear_acceleration>
+      <!-- computed from <max_linear_acceleration> in the original plugin-->
+      <topic>cmd_vel</topic>
+      <!-- from <commant_topic> -->
+      <odom_topic>odom</odom_topic>
+      <!-- from <odometry_topic> -->
+      <frame_id>odom</frame_id>
+      <!-- from <odometry_frame> -->
+      <child_frame_id>base_footprint</child_frame_id>
+      <!-- from <robot_base_frame> -->
+      <odom_publisher_frequency>30</odom_publisher_frequency>
+      <!-- from <update_rate>-->
+      <tf_topic>/tf</tf_topic>
+      <!-- Short topic name for tf output -->
     </plugin>
-  </gazebo> -->
   </model>
 </sdf>
