Commit message: cleanups and style fixes

File: urdf/realsense-RS200.macro.xacro (robot description, xacro)
@@ -1,4 +1,4 @@
 <?xml version="1.0"?>
-THIS FILE IS NOT IN USE
+<!-- THIS FILE IS NOT IN USE -->
 <!--Develped by Daniel Ordonez 22.05.2018 - daniels.ordonez@gmail.com
     INFORMATION:
@@ -17,12 +17,12 @@
     <link name="${prefix}rs200_camera">
       <visual>
-    <geometry>
-        <!-- <geometry> -->
-              <mesh>
-                <!-- <scale>0.0254 0.0254 0.0254</scale> -->
-                <uri>model://curve_left_1/meshes/curve_left_1.obj</uri>
-                <!-- <uri>model://realsense_camera/meshes/realsense.obj</uri> -->
-              </mesh>
-            <!-- </geometry> -->
+        <geometry>
+          <!-- <geometry> -->
+          <mesh>
+            <!-- <scale>0.0254 0.0254 0.0254</scale> -->
+            <uri>model://curve_left_1/meshes/curve_left_1.obj</uri>
+            <!-- <uri>model://realsense_camera/meshes/realsense.obj</uri> -->
+          </mesh>
+          <!-- </geometry> -->
           <!-- <mesh filename="model://realsense_camera/meshes/realsense.dae"/> -->
         </geometry>

File: urdf/realsense-depth.xacro (robot description, xacro)
@@ -16,36 +16,29 @@
     <!-- Camera link -->
     <link name="${prefix}rs200_camera">
-            <!-- <origin rpy="${pi/2} ${pi/2} ${pi/2}" xyz="0 0 0"/> -->
-          <pose>0.1 0 0.035 0 0 0</pose>
+      <pose>0.1 0 0.035 0 0 0</pose>
       <visual name="vis_${prefix}_rs200_cam">
-      <pose>0 0 0 ${pi/2} 0 0</pose>
-       <!-- <origin>
-          <rpy>${pi/2} 0 0</rpy>
-          <xyz>0 0 0</xyz>
-        </origin>     -->
+        <pose>0 0 0 ${pi/2} 0 0</pose>
         <geometry>
-                <!-- <origin rpy="${pi/2} ${pi/2} ${pi/2}" xyz="0 0 0"/> -->
-        <!-- <geometry> -->
-              <mesh>
-                              <!-- <origin rpy="${pi/2} ${pi/2} ${pi/2}" xyz="0 0 0"/> -->
-                <!-- <scale>0.0254 0.0254 0.0254</scale> -->
-                <!-- <uri>model://curve_left_1/meshes/curve_left_1.obj</uri> -->
-                <uri>model://realsense_camera/meshes/realsense.obj</uri>
-              </mesh>
-            <!-- </geometry> -->
-          <!-- <mesh filename="model://realsense_camera/meshes/realsense.dae"/> -->
+          <mesh>
+            <uri>model://realsense_camera/meshes/realsense.obj</uri>
+          </mesh>
         </geometry>
       </visual>
       <collision name="coll_${prefix}_rs200_cam">
         <geometry>
-          <box><size>0.0078 0.130 0.0192</size></box>
+          <box>
+            <size>0.0078 0.130 0.0192</size>
+          </box>
         </geometry>
       </collision>
       <inertial>
-        <!-- <mass value="0.0"/> -->
-        <!-- <origin rpy="0 0 0" xyz="0 0 0"/> -->
         <inertia>
-         <ixx>9.108e-05</ixx> <ixy>0</ixy><ixz>0</ixz><iyy>2.51e-06</iyy><iyz>0</iyz><izz>8.931e-05</izz>
-         </inertia>
+          <ixx>9.108e-05</ixx>
+          <ixy>0</ixy>
+          <ixz>0</ixz>
+          <iyy>2.51e-06</iyy>
+          <iyz>0</iyz>
+          <izz>8.931e-05</izz>
+        </inertia>
       </inertial>
     </link>
@@ -54,6 +47,4 @@
       <parent>${parent}</parent>
       <child>${prefix}rs200_camera</child>
-          <!-- <pose>0.1 0 0.035 0 0 0</pose> -->
-      <!-- <xacro:insert_block name="origin"/> -->
     </joint>
     <!-- Virtual links representing the cameras positons and orientations-->
@@ -62,39 +53,16 @@
       <parent>${prefix}rs200_camera</parent>
       <child>${prefix}depth</child>
-      <!-- <origin xyz="0 -0 0.004" rpy="0 0 0"/> -->
     </joint>
-    <!-- <gazebo reference="${prefix}rs200_camera"> -->
-    <!-- TODO: later weer terugzetten! -->
-      <!-- <sensor name="realsense_contact" type="contact">
+    <link name="${prefix}depth">
+      <pose>0.13 0 0.045 0 0 0</pose>
+      <sensor name="camera_sensor_depth" type="camera">
         <always_on>true</always_on>
-        <update_rate>30.0</update_rate>
-        <contact>
-          <xacro:property name="lidar" value="$(arg lidar_enable)"/>
-          <xacro:property name="ir" value="$(arg intensity_enable)"/>
-          <test2 name="lidar" value="$(arg lidar_enable)"/>
-          <test2 name="ir" value="$(arg intensity_enable)"/>
-          <arg val="2 + 2xir + lidar"/>
-          <!- - See https://github.com/gazebosim/sdformat/issues/333 for why the strange naming. Get the correct name by running xacro mirte.xacro > test.xml && gz sdf -p test.xml > robot.xml and look for the name- ->
-          <!- - This strange calculation should make sure that when adding/removing lidar and ir sensors, the collision name still is correct - ->
-          <collision>base_link_fixed_joint_lump__realsense_collision_collision_${lidar + 2*ir + 2}</collision>
-        </contact>
-        <plugin name="gripper_bumper" filename="libgazebo_ros_bumper.so">
-          <bumperTopicName>realsense_contact</bumperTopicName>
-          <frameName>${prefix}rs200_camera</frameName>
-        </plugin>
-      </sensor>
-    </gazebo> -->
-    <!-- <gazebo reference="${prefix}depth"> -->
-    <link name="${prefix}depth">
-              <pose>0.13 0 0.045 0 0 0</pose>
-    <sensor name="camera_sensor_depth" type="camera">
-  <always_on>true</always_on>
-  <visualize>true</visualize>
-  <update_rate>10</update_rate>
-  <topic>camera/image_raw</topic>
-  <gz_frame_id>camera_rgb_frame</gz_frame_id>
-  <camera name="intel_realsense_r200">
-    <camera_info_topic>camera/camera_info</camera_info_topic>
-<horizontal_fov>2.5</horizontal_fov>
+        <visualize>true</visualize>
+        <update_rate>10</update_rate>
+        <topic>camera/image_raw</topic>
+        <gz_frame_id>camera_rgb_frame</gz_frame_id>
+        <camera name="intel_realsense_r200">
+          <camera_info_topic>camera/camera_info</camera_info_topic>
+          <horizontal_fov>2.5</horizontal_fov>
           <image>
             <width>640</width>
@@ -105,15 +73,15 @@
             <near>0.02</near>
             <far>2</far>
-          </clip>  </camera>
-</sensor>
-   <sensor name="depth_camera1" type="depth_camera">
-  <always_on>true</always_on>
-  <visualize>true</visualize>
-  <update_rate>10</update_rate>
-  <topic>depth_camera</topic>
-  <gz_frame_id>camera_rgb_frame</gz_frame_id>
-  <camera name="intel_realsense_r200_depth">
-    <!-- <camera_info_topic>camera/camera_info</camera_info_topic> -->
-<horizontal_fov>2.5</horizontal_fov>
+          </clip>
+        </camera>
+      </sensor>
+      <sensor name="depth_camera1" type="depth_camera">
+        <always_on>true</always_on>
+        <visualize>true</visualize>
+        <update_rate>10</update_rate>
+        <topic>depth_camera</topic>
+        <gz_frame_id>camera_rgb_frame</gz_frame_id>
+        <camera name="intel_realsense_r200_depth">
+          <horizontal_fov>2.5</horizontal_fov>
           <image>
             <width>640</width>
@@ -124,36 +92,8 @@
             <near>0.02</near>
             <far>2</far>
-          </clip>  </camera>
-</sensor>
-      <!-- <sensor name="depth_camera1" type="camera">
-          <update_rate>10</update_rate>
-          <!- - <topic>depth_camera</topic> - ->
-          <topic>camera/image_raw</topic>
-          <camera>
-            <horizontal_fov>2.5</horizontal_fov>
-            <image>
-              <width>512</width>
-              <height>512</height>
-              <!- - <format>R_FLOAT32</format> - ->
-            </image>
-            <clip>
-              <near>0.001</near>
-              <far>2</far>
-            </clip>
-          </camera>
-          </sensor> -->
-          </link>
-        <!-- <plugin name="depth_camera_controller" filename="libgazebo_ros_depth_camera.so">
-          <alwaysOn>1</alwaysOn>
-          <updateRate>10.0</updateRate>
-          <imageTopicName>image_raw</imageTopicName>
-          <pointCloudTopicName>points</pointCloudTopicName>
-          <cameraInfoTopicName>camera_info</cameraInfoTopicName>
-          <cameraName>depth_cam</cameraName>
-          <frameName>${prefix}depth</frameName>
-          <pointCloudCutoff>0.001</pointCloudCutoff>
-        </plugin>
+          </clip>
+        </camera>
       </sensor>
-    </gazebo> -->
+    </link>
   </xacro:macro>
 </robot>

File: urdf/static_cam.xacro (robot description, xacro)
@@ -1,54 +1,55 @@
+<?xml version="1.0"?>
 <robot xmlns:xacro="http://www.ros.org/wiki/xacro" name="mirte">
-    <xacro:macro name="static_cam" params="">
-        <model name="top_down_cam">
-        <static>true</static>
-            <link name="top_down_link">
-            <static>1</static>
-                <sensor name="top_down_camera_sensor" type="camera">
-                    <always_on>true</always_on>
-                    <visualize>true</visualize>
-                    <update_rate>10</update_rate>
-                    <topic>top_down_camera/image_raw</topic>
-                    <gz_frame_id>top_down_camera_rgb_frame</gz_frame_id>
-                    <camera name="top_down_camera">
-                        <camera_info_topic>camera/camera_info</camera_info_topic>
-                        <!-- <horizontal_fov>2.5</horizontal_fov> -->
-                        <image>
-                            <width>640</width>
-                            <height>640</height>
-                            <format>R8G8B8</format>
-                        </image>
-                        <clip>
-                            <near>0.02</near>
-                            <far>6</far>
-                        </clip>
-                    </camera>
-                </sensor>
-                <static>1</static>
+  <xacro:macro name="static_cam" params="">
+    <model name="top_down_cam">
+      <static>true</static>
+      <link name="top_down_link">
+        <static>1</static>
+        <sensor name="top_down_camera_sensor" type="camera">
+          <always_on>true</always_on>
+          <visualize>true</visualize>
+          <update_rate>10</update_rate>
+          <topic>top_down_camera/image_raw</topic>
+          <gz_frame_id>top_down_camera_rgb_frame</gz_frame_id>
+          <camera name="top_down_camera">
+            <camera_info_topic>camera/camera_info</camera_info_topic>
+            <!-- <horizontal_fov>2.5</horizontal_fov> -->
+            <image>
+              <width>640</width>
+              <height>640</height>
+              <format>R8G8B8</format>
+            </image>
+            <clip>
+              <near>0.02</near>
+              <far>6</far>
+            </clip>
+          </camera>
+        </sensor>
+        <static>1</static>
+        <pose>1.688 1.36 4 0 1.57 0</pose>
+        <link name="top_down_link">
+          <static>1</static>
+          <collision name="collision_tile_7_4">
+            <geometry>
+              <mesh>
+                <scale>0.5 0.5 0.5</scale>
+                <!-- <scale>0.0254 0.0254 0.0254</scale> -->
+                <uri>model://floor/meshes/floor.obj</uri>
+              </mesh>
+            </geometry>
+          </collision>
+          <visual name="visual_tile_7_4">
+            <geometry>
+              <mesh>
                 <pose>1.688 1.36 4 0 1.57 0</pose>
-                <link name="top_down_link">
-                <static>1</static>
-                    <collision name="collision_tile_7_4">
-                        <geometry>
-                            <mesh>
-                                <scale>0.5 0.5 0.5</scale>
-                                <!-- <scale>0.0254 0.0254 0.0254</scale> -->
-                                <uri>model://floor/meshes/floor.obj</uri>
-                            </mesh>
-                        </geometry>
-                    </collision>
-                    <visual name="visual_tile_7_4">
-                        <geometry>
-                            <mesh>
-                                <pose>1.688 1.36 4 0 1.57 0</pose>
-                                <scale>0.5 0.5 0.5</scale>
-                                <!-- <scale>0.0254 0.0254 0.0254</scale> -->
-                                <uri>model://floor/meshes/floor.obj</uri>
-                            </mesh>
-                        </geometry>
-                    </visual>
-                </link>
-            </link>
-        </model>
-    </xacro:macro>
+                <scale>0.5 0.5 0.5</scale>
+                <!-- <scale>0.0254 0.0254 0.0254</scale> -->
+                <uri>model://floor/meshes/floor.obj</uri>
+              </mesh>
+            </geometry>
+          </visual>
+        </link>
+      </link>
+    </model>
+  </xacro:macro>
 </robot>

File: urdf/tileWorld.xacro (robot description, xacro)
@@ -3,29 +3,29 @@
   <xacro:macro name="tileWorld" params="name material size x y yaw=0 z_offset=0 model_scale=1 scale=1">
     <model name="unit_box_${name}">
-         <model name="model_${name}">
-      <static>1</static>
+      <model name="model_${name}">
+        <static>1</static>
+        <pose>${x * size} ${y * size} ${z_offset*size * model_scale * scale + 0.01} ${radians(90)} -0  ${radians(yaw)}</pose>
+        <link name="link_${name}">
+          <collision name="collision_${name}">
+            <geometry>
+              <mesh>
+                <scale>${size * model_scale * scale} ${size * model_scale * scale} ${size * model_scale * scale}</scale>
+                <!-- <scale>0.0254 0.0254 0.0254</scale> -->
+                <uri>model://${material}/meshes/${material}.obj</uri>
+              </mesh>
+            </geometry>
+          </collision>
+          <visual name="visual_${name}">
+            <geometry>
+              <mesh>
                 <pose>${x * size} ${y * size} ${z_offset*size * model_scale * scale + 0.01} ${radians(90)} -0  ${radians(yaw)}</pose>
-    <link name="link_${name}">
-      <collision name="collision_${name}">
-        <geometry>
-          <mesh>
-      <scale>${size * model_scale * scale} ${size * model_scale * scale} ${size * model_scale * scale}</scale>
-            <!-- <scale>0.0254 0.0254 0.0254</scale> -->
-            <uri>model://${material}/meshes/${material}.obj</uri>
-          </mesh>
-        </geometry>
-      </collision>
-      <visual name="visual_${name}">
-        <geometry>
-          <mesh>
-      <pose>${x * size} ${y * size} ${z_offset*size * model_scale * scale + 0.01} ${radians(90)} -0  ${radians(yaw)}</pose>
-      <scale>${size * model_scale * scale} ${size * model_scale * scale} ${size * model_scale * scale}</scale>
-            <!-- <scale>0.0254 0.0254 0.0254</scale> -->
-            <uri>model://${material}/meshes/${material}.obj</uri>
-          </mesh>
-        </geometry>
-      </visual>
-    </link>
-  </model>
+                <scale>${size * model_scale * scale} ${size * model_scale * scale} ${size * model_scale * scale}</scale>
+                <!-- <scale>0.0254 0.0254 0.0254</scale> -->
+                <uri>model://${material}/meshes/${material}.obj</uri>
+              </mesh>
+            </geometry>
+          </visual>
+        </link>
+      </model>
     </model>
   </xacro:macro>
