Commit message: lab 3 world + ir

File: urdf/ir.xacro (robot description, xacro)
@@ -1,34 +1,61 @@
 <?xml version="1.0"?>
 <robot xmlns:xacro="http://www.ros.org/wiki/xacro">
-  <xacro:macro name="ir_sensor" params="name *origin">
+  <xacro:macro name="ir_sensor" params="name *pose">
     <!-- <xacro:property name="ir_angle_max" value="${radians(15)}"/> -->
     <joint name="ir_${name}" type="fixed">
-      <axis xyz="0 1 0"/>
-      <xacro:insert_block name="origin"/>
-      <parent link="link_chassis"/>
-      <child link="base_ir_${name}"/>
+      <!-- <axis xyz="0 1 0"/> -->
+      <!-- <xacro:insert_block name="origin"/> -->
+      <parent>link_chassis</parent>
+      <child>base_ir_${name}</child>
     </joint>
     <link name="base_ir_${name}">
-      <collision>
+          <xacro:insert_block name="pose"/>
+      <collision name="collision_ir_${name}">
+      <!-- <name>collision_ir_${name}</name> -->
         <origin xyz="0 0 0" rpy="0 0 0"/>
         <geometry>
-          <box size="0.01 0.05 0.037"/>
-        </geometry>
+ <box>
+          <size>
+          0.01 0.01 0.01
+          </size></box>        </geometry>
       </collision>
-      <visual>
+      <visual name="visual_ir_${name}">
         <origin xyz="0 0 0" rpy="0 0 0"/>
         <geometry>
-          <box size="0.01 0.01 0.01"/>
+          <box>
+          <size>
+          0.01 0.01 0.01
+          </size></box>
         </geometry>
-        <material name="yellow"/>
+        <material >
+        <ambient>0.0 0.5 0.5</ambient>
+        </material>
       </visual>
-      <inertial>
+      <!-- <inertial>
         <mass value="0.0"/>
         <origin xyz="0 0 0" rpy="0 0 0"/>
-        <inertia ixx="0.0" ixy="0.0" ixz="0.0" iyy="0.0" iyz="0.0" izz="0.0"/>
-      </inertial>
-    </link>
-    <gazebo reference="base_ir_${name}">
-      <sensor type="camera" name="camera_ir_${name}">
+        <inertia> <ixx>0.0 ixy="0.0" ixz="0.0" iyy="0.0" iyz="0.0" izz="0.0"/>
+      </inertial>  -->
+      <sensor name="ir_cam_${name}" type="camera">
+        <always_on>true</always_on>
+        <visualize>true</visualize>
+        <update_rate>10</update_rate>
+        <topic>camera_${name}/image_raw</topic>
+        <gz_frame_id>camera_rgb_frame</gz_frame_id>
+        <camera name="head">
+          <!-- <camera_info_topic>camera/camera_info</camera_info_topic> -->
+          <horizontal_fov>1.2</horizontal_fov>
+          <image>
+            <width>1</width>
+            <height>1</height>
+            <format>L8</format>
+          </image>
+          <clip>
+            <near>0.0001</near>
+            <far>1</far>
+          </clip>
+        </camera>
+      </sensor>
+      <!-- <sensor type="camera" name="camera_ir_${name}">
         <update_rate>5</update_rate>
         <camera name="head">
@@ -50,6 +77,6 @@
           <cameraName>camera_ir_${name}</cameraName>
         </plugin>
-      </sensor>
-    </gazebo>
+      </sensor> -->
+    </link>
   </xacro:macro>
 </robot>

File: urdf/mirte.xacro (robot description, xacro)
@@ -106,8 +106,8 @@
     <xacro:if value="$(arg intensity_enable)">
       <xacro:ir_sensor name="left">
-        <origin rpy="0 ${radians(90)} 0" xyz="0.0785 0.022 0.002"/>
+        <pose>0.0785 0.022 0.002 0 ${radians(90)} 0</pose>
       </xacro:ir_sensor>
       <xacro:ir_sensor name="right">
-        <origin rpy="0 ${radians(90)} 0" xyz="0.0785 -0.022 0.002"/>
+              <pose>0.0785 -0.022 0.002 0 ${radians(90)} 0</pose>
       </xacro:ir_sensor>
     </xacro:if>
