Commit message: Cleanup and mesh replacement

File: mirte_master_description/urdf/mirte_master.xacro (robot description, xacro)
@@ -81,10 +81,7 @@
     </visual>
     <collision>
-      <origin
-        xyz="0 0 0"
-        rpy="0 0 0" />
-      <geometry>
-        <mesh
-          filename="package://mirte_master_description/meshes/wheel_fl.STL" />
+      <origin xyz="0 0 0.025" />
+      <geometry>
+        <cylinder radius="0.053" length="0.055" />
       </geometry>
     </collision>
@@ -134,10 +131,7 @@
     </visual>
     <collision>
-      <origin
-        xyz="0 0 0"
-        rpy="0 0 0" />
-      <geometry>
-        <mesh
-          filename="package://mirte_master_description/meshes/wheel_br.STL" />
+      <origin xyz="0 0 -0.025" />
+      <geometry>
+        <cylinder radius="0.053" length="0.055" />
       </geometry>
     </collision>
@@ -187,10 +181,7 @@
     </visual>
     <collision>
-      <origin
-        xyz="0 0 0"
-        rpy="0 0 0" />
-      <geometry>
-        <mesh
-          filename="package://mirte_master_description/meshes/wheel_fr.STL" />
+      <origin xyz="0 0 -0.025" />
+      <geometry>
+        <cylinder radius="0.053" length="0.055" />
       </geometry>
     </collision>
@@ -240,10 +231,7 @@
     </visual>
     <collision>
-      <origin
-        xyz="0 0 0"
-        rpy="0 0 0" />
-      <geometry>
-        <mesh
-          filename="package://mirte_master_description/meshes/wheel_bl.STL" />
+      <origin xyz="0 0 0.025" />
+      <geometry>
+        <cylinder radius="0.053" length="0.055" />
       </geometry>
     </collision>
@@ -687,634 +675,6 @@
   </joint>
   <xacro:if value="$(arg flag_enable)">
-    <link
-      name="flag">
-      <inertial>
-        <origin
-          xyz="0.0249185518105129 -0.170067519347241 -0.000222734216111346"
-          rpy="0 0 0" />
-        <mass
-          value="0.0374187697708756" />
-        <inertia
-          ixx="0.00108799032272128"
-          ixy="-6.06514391971722E-05"
-          ixz="-2.07236681084901E-07"
-          iyy="7.05873812366136E-05"
-          iyz="-1.13163625013946E-06"
-          izz="0.00115807893485493" />
-      </inertial>
-      <visual>
-        <geometry>
-          <mesh
-            filename="package://mirte_master_description/meshes/flag.STL" />
-        </geometry>
-        <material
-          name="">
-          <color
-            rgba="0.796078431372549 0.823529411764706 0.937254901960784 1" />
-        </material>
-      </visual>
-      <collision>
-        <geometry>
-          <mesh
-            filename="package://mirte_master_description/meshes/flag.STL" />
-        </geometry>
-      </collision>
-    </link>
-    <joint
-      name="flag_joint"
-      type="fixed">
-      <origin
-        xyz="-0.0496954854378495 0.124843221166346 0.625600000000005"
-        rpy="1.5707963267949 0 1.61494047314374" />
-      <parent
-        link="base_link" />
-      <child
-        link="flag" />
-    </joint>
+    <xacro:include filename="$(mirte_master_description/urdf/flag.xacro)" />
   </xacro:if>
-  <link
-    name="arm_Rot">
-    <inertial>
-      <origin
-        xyz="-1.27894101951934E-05 0.0208058767653727 0.00585680210359747"
-        rpy="0 0 0" />
-      <mass
-        value="0.0689676051678483" />
-      <inertia
-        ixx="1.10736817655159E-05"
-        ixy="-9.06572517495388E-09"
-        ixz="-2.13237951815141E-10"
-        iyy="2.24480121987499E-05"
-        iyz="-4.10984989642458E-07"
-        izz="1.70252517510809E-05" />
-    </inertial>
-    <visual>
-      <origin
-        xyz="0 0 0"
-        rpy="0 0 0" />
-      <geometry>
-        <mesh
-          filename="package://mirte_master_description/meshes/arm_Rot.STL" />
-      </geometry>
-      <material
-        name="">
-        <color
-          rgba="0.792156862745098 0.819607843137255 0.933333333333333 1" />
-      </material>
-    </visual>
-    <collision>
-      <origin
-        xyz="0 0 0"
-        rpy="0 0 0" />
-      <geometry>
-        <mesh
-          filename="package://mirte_master_description/meshes/arm_Rot.STL" />
-      </geometry>
-    </collision>
-  </link>
-  <joint
-    name="arm_Rot_joint"
-    type="revolute">
-    <origin
-      xyz="0 -0.079274 0.06"
-      rpy="1.5708 0 3.1416" />
-    <parent
-      link="base_link" />
-    <child
-      link="arm_Rot" />
-    <axis
-      xyz="0 1 0" />
-    <limit
-      lower="${pi/-2}"
-      upper="${pi/2}"
-      effort="2"
-      velocity="2"
-      />
-  </joint>
-  <link
-    name="arm_Shoulder">
-    <inertial>
-      <origin
-        xyz="0.0764974362945755 0.000442680770353329 -4.93690401059954E-09"
-        rpy="0 0 0" />
-      <mass
-        value="0.104616018825837" />
-      <inertia
-        ixx="3.85677839717214E-05"
-        ixy="1.84827309047044E-08"
-        ixz="1.42612941509626E-12"
-        iyy="2.54245117502168E-05"
-        iyz="-2.05142765424474E-12"
-        izz="5.51611966703411E-05" />
-    </inertial>
-    <visual>
-      <origin
-        xyz="0 0 0"
-        rpy="0 0 0" />
-      <geometry>
-        <mesh
-          filename="package://mirte_master_description/meshes/arm_Shoulder.STL" />
-      </geometry>
-      <material
-        name="">
-        <color
-          rgba="0.501960784313725 0.501960784313725 0.501960784313725 1" />
-      </material>
-    </visual>
-    <collision>
-      <origin
-        xyz="0 0 0"
-        rpy="0 0 0" />
-      <geometry>
-        <mesh
-          filename="package://mirte_master_description/meshes/arm_Shoulder.STL" />
-      </geometry>
-    </collision>
-  </link>
-  <joint
-    name="arm_Shoulder_joint"
-    type="revolute">
-    <origin
-      xyz="0 0.0281 -0.00625"
-      rpy="3.1416 0 1.5708" />
-    <parent
-      link="arm_Rot" />
-    <child
-      link="arm_Shoulder" />
-    <axis
-      xyz="1 0 0" />
-      <limit
-      lower="${pi/-2}"
-      upper="${pi/2}"
-      effort="2"
-      velocity="2"
-      />
-  </joint>
-  <link
-    name="arm_Elbow">
-    <inertial>
-      <origin
-        xyz="0.000768647609078278 0.0642294520091309 -2.34835863116567E-08"
-        rpy="0 0 0" />
-      <mass
-        value="0.0709795960901316" />
-      <inertia
-        ixx="2.06491501981418E-05"
-        ixy="1.76077623308388E-08"
-        ixz="-6.06300089698489E-13"
-        iyy="2.45686930201746E-05"
-        iyz="3.04033870141042E-12"
-        izz="3.79131240892547E-05" />
-    </inertial>
-    <visual>
-      <origin
-        xyz="0 0 0"
-        rpy="0 0 0" />
-      <geometry>
-        <mesh
-          filename="package://mirte_master_description/meshes/arm_Elbow.STL" />
-      </geometry>
-      <material
-        name="">
-        <color
-          rgba="0.501960784313725 0.501960784313725 0.501960784313725 1" />
-      </material>
-    </visual>
-    <collision>
-      <origin
-        xyz="0 0 0"
-        rpy="0 0 0" />
-      <geometry>
-        <mesh
-          filename="package://mirte_master_description/meshes/arm_Elbow.STL" />
-      </geometry>
-    </collision>
-  </link>
-  <joint
-    name="arm_Elbow_joint"
-    type="revolute">
-    <origin
-      xyz="0.1378 0 0"
-      rpy="-3.1416 0 1.5708" />
-    <parent
-      link="arm_Shoulder" />
-    <child
-      link="arm_Elbow" />
-    <axis
-      xyz="1 0 0" />
-      <limit
-      lower="${pi/-2}"
-      upper="${pi/2}"
-      effort="2"
-      velocity="2"
-      />
-  </joint>
-  <link
-    name="arm_Wrist">
-    <inertial>
-      <origin
-        xyz="0.0225315136140379 0.000488092971965825 -2.74405760168628E-06"
-        rpy="0 0 0" />
-      <mass
-        value="0.0464803878756425" />
-      <inertia
-        ixx="1.36228105923869E-05"
-        ixy="-2.7486243117372E-08"
-        ixz="-2.82180089490711E-08"
-        iyy="7.22412070962973E-06"
-        iyz="3.4652740053439E-09"
-        izz="1.75204377049058E-05" />
-    </inertial>
-    <visual>
-      <origin
-        xyz="0 0 0"
-        rpy="0 0 0" />
-      <geometry>
-        <mesh
-          filename="package://mirte_master_description/meshes/arm_Wrist.STL" />
-      </geometry>
-      <material
-        name="">
-        <color
-          rgba="0.501960784313725 0.501960784313725 0.501960784313725 1" />
-      </material>
-    </visual>
-    <collision>
-      <origin
-        xyz="0 0 0"
-        rpy="0 0 0" />
-      <geometry>
-        <mesh
-          filename="package://mirte_master_description/meshes/arm_Wrist.STL" />
-      </geometry>
-    </collision>
-  </link>
-  <joint
-    name="arm_Wrist_joint"
-    type="revolute">
-    <origin
-      xyz="-0.00014 0.14265 0"
-      rpy="3.1416 0 1.5708" />
-    <parent
-      link="arm_Elbow" />
-    <child
-      link="arm_Wrist" />
-    <axis
-      xyz="1 0 0" />
-      <limit
-      lower="${pi/-2}"
-      upper="${pi/2}"
-      effort="2"
-      velocity="2"
-      />
-  </joint>
-  <link
-    name="Gripper">
-    <inertial>
-      <origin
-        xyz="0.0128439388984141 0.00467107677719844 -0.023531822516204"
-        rpy="0 0 0" />
-      <mass
-        value="0.0109603788959771" />
-      <inertia
-        ixx="1.64287457972505E-06"
-        ixy="-2.54915969005551E-10"
-        ixz="-3.17766452649769E-07"
-        iyy="2.96639543247368E-06"
-        iyz="-7.8877045337556E-08"
-        izz="1.49193844890504E-06" />
-    </inertial>
-    <visual>
-      <origin
-        xyz="0 0 0"
-        rpy="0 0 0" />
-      <geometry>
-        <mesh
-          filename="package://mirte_master_description/meshes/Gripper.STL" />
-      </geometry>
-      <material
-        name="">
-        <color
-          rgba="0.792156862745098 0.819607843137255 0.933333333333333 1" />
-      </material>
-    </visual>
-    <collision>
-      <origin
-        xyz="0 0 0"
-        rpy="0 0 0" />
-      <geometry>
-        <mesh
-          filename="package://mirte_master_description/meshes/Gripper.STL" />
-      </geometry>
-    </collision>
-  </link>
-  <joint
-    name="Gripper_joint"
-    type="revolute">
-    <origin
-      xyz="0.0435 -0.012 0.0045"
-      rpy="-1.5708 0 0" />
-    <parent
-      link="arm_Wrist" />
-    <child
-      link="Gripper" />
-    <axis
-      xyz="0 0 1" />
-      <limit
-      lower="0"
-      upper="${pi/2}"
-      effort="2"
-      velocity="2"
-      />
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
Commit message: Update V2

File: mirte_master_description/urdf/mirte_master.xacro (robot description, xacro)
@@ -11,4 +11,9 @@
   <!-- TODO FIX -->
   <!-- <xacro:include filename="$(find mirte_master_gazebo)/urdf/mirte_master_description.gazebo" /> -->
+  <xacro:include filename="$(find gazebo_sensor_collection)/urdf/cameras/rgbd/orbbec_astra_pro_plus.urdf.xacro"/>
+  <!-- TODO: CHANGE TO CAMERA -->
+  <xacro:sensor_orbbec_astra_pro_plus name="camera" parent="base_link" color="black">
+    <origin xyz="0.01 -0.146658788505756 0.0427000000000005" rpy="0 0 ${radians(-90)}" />
+  </xacro:sensor_orbbec_astra_pro_plus>
   <link
     name="base_link">
@@ -515,5 +520,5 @@
       xyz="0 0 0" />
   </joint>
-  <link
+  <!-- <link
     name="depth_cam">
     <inertial>
@@ -567,5 +572,5 @@
     <axis
       xyz="0 0 0" />
-  </joint>
+  </joint> -->
   <link
     name="lidar">

Commit message: Wheels are nearly controllable

File: mirte_master_description/urdf/mirte_master.xacro (robot description, xacro)
@@ -6,10 +6,10 @@
 <robot
   name="mirte_master" xmlns:xacro="http://ros.org/wiki/xacro">
-  <xacro:arg name="flag_enable" default="false" />
-  <!-- <xacro:property name="pi" value="3.1415" /> -->
+  <xacro:arg name="flag_enable" default="False" />
+  <xacro:arg name="arm_enable" default="False" />
   <!-- Bring in simulation data for Gazebo. -->
-  <!-- TODO FIX -->
-  <!-- <xacro:include filename="$(find mirte_master_gazebo)/urdf/mirte_master_description.gazebo" /> -->
-  <xacro:include filename="$(find gazebo_sensor_collection)/urdf/cameras/rgbd/orbbec_astra_pro_plus.urdf.xacro"/>
+  <xacro:include filename="$(find mirte_master_description)/urdf/mirte_master_base.gazebo.xacro" />
+  <xacro:include
+    filename="$(find gazebo_sensor_collection)/urdf/cameras/rgbd/orbbec_astra_pro_plus.urdf.xacro" />
   <!-- TODO: CHANGE TO CAMERA -->
   <xacro:sensor_orbbec_astra_pro_plus name="camera" parent="base_link" color="black">
@@ -98,19 +98,23 @@
       xyz="0.153 -0.085 -0.0455"
       rpy="1.5708 0 -1.5708" />
-    <parent
-      link="base_link" />
-    <child
-      link="wheel_fl" />
-    <axis
-      xyz="0 0 -1" />
-  </joint>
+    <parent link="base_link" />
+    <child link="wheel_fl" />
+    <axis xyz="0 0 -1" />
+    <dynamics damping="3.0" friction="5.0" />
+  </joint>
+  <transmission name="wheel_trans_fl">
+    <type>transmission_interface/SimpleTransmission</type>
+    <joint name="wheel_joint_fl">
+        <hardwareInterface>hardware_interface/VelocityJointInterface</hardwareInterface>
+    </joint>
+    <actuator name="wheel_act_fl">
+        <mechanicalReduction>1</mechanicalReduction>
+    </actuator>
+</transmission>
   <link
     name="wheel_br">
     <inertial>
-      <origin
-        xyz="-1.0009E-10 2.9473E-10 -0.025064"
-        rpy="0 0 0" />
-      <mass
-        value="0.26661" />
+      <origin xyz="-1.0009E-10 2.9473E-10 -0.025064" />
+      <mass value="0.26661" />
       <inertia
         ixx="8.0546E-05"
@@ -148,19 +152,23 @@
       xyz="-0.153 0.085 -0.0455"
       rpy="1.5708 0 -1.5708" />
-    <parent
-      link="base_link" />
-    <child
-      link="wheel_br" />
-    <axis
-      xyz="0 0 1" />
-  </joint>
+    <parent link="base_link" />
+    <child link="wheel_br" />
+    <axis xyz="0 0 1" />
+    <dynamics damping="3.0" friction="5.0" />
+  </joint>
+  <transmission name="wheel_trans_br">
+    <type>transmission_interface/SimpleTransmission</type>
+    <joint name="wheel_joint_br">
+        <hardwareInterface>hardware_interface/VelocityJointInterface</hardwareInterface>
+    </joint>
+    <actuator name="wheel_act_br">
+        <mechanicalReduction>1</mechanicalReduction>
+    </actuator>
+  </transmission>
   <link
     name="wheel_fr">
     <inertial>
-      <origin
-        xyz="-1.9E-10 2.1252E-10 -0.025064"
-        rpy="0 0 0" />
-      <mass
-        value="0.26661" />
+      <origin xyz="-1.9E-10 2.1252E-10 -0.025064" />
+      <mass value="0.26661" />
       <inertia
         ixx="8.0546E-05"
@@ -172,7 +180,7 @@
     </inertial>
     <visual>
-      <origin
-        xyz="0 0 0"
-        rpy="0 0 0" />
+      <!-- <origin
+        xyz="0 0 0"
+        rpy="0 0 0" /> -->
       <geometry>
         <mesh
@@ -198,17 +206,22 @@
       xyz="-0.153 -0.085 -0.0455"
       rpy="1.5708 0 -1.5708" />
-    <parent
-      link="base_link" />
-    <child
-      link="wheel_fr" />
-    <axis
-      xyz="0 0 1" />
-  </joint>
+    <parent link="base_link" />
+    <child link="wheel_fr" />
+    <axis xyz="0 0 1" />
+    <dynamics damping="3.0" friction="5.0" />
+  </joint>
+  <transmission name="wheel_trans_fr">
+    <type>transmission_interface/SimpleTransmission</type>
+    <joint name="wheel_joint_fr">
+        <hardwareInterface>hardware_interface/VelocityJointInterface</hardwareInterface>
+    </joint>
+    <actuator name="wheel_act_fr">
+        <mechanicalReduction>1</mechanicalReduction>
+    </actuator>
+</transmission>
   <link
     name="wheel_bl">
     <inertial>
-      <origin
-        xyz="-1.9E-10 2.1252E-10 0.024936"
-        rpy="0 0 0" />
+      <origin xyz="-1.9E-10 2.1252E-10 0.024936" />
       <mass
         value="0.26661" />
@@ -248,11 +261,18 @@
       xyz="0.153 0.085 -0.0455"
       rpy="1.5708 0 -1.5708" />
-    <parent
-      link="base_link" />
-    <child
-      link="wheel_bl" />
-    <axis
-      xyz="0 0 -1" />
-  </joint>
+    <parent link="base_link" />
+    <child link="wheel_bl" />
+    <axis xyz="0 0 -1" />
+    <dynamics damping="3.0" friction="5.0" />
+  </joint>
+  <transmission name="wheel_trans_bl">
+    <type>transmission_interface/SimpleTransmission</type>
+    <joint name="wheel_joint_bl">
+        <hardwareInterface>hardware_interface/VelocityJointInterface</hardwareInterface>
+    </joint>
+    <actuator name="wheel_act_bl">
+        <mechanicalReduction>1</mechanicalReduction>
+    </actuator>
+</transmission>
   <link
     name="cam_front">
@@ -528,5 +548,6 @@
       <mass
         value="0.188133920196831" />
-      <inertia
+      <inerti  <xacro:arg name="flag_enable" default="False" />
+a
         ixx="6.91459455879894E-05"
         ixy="2.54332859259088E-06"
@@ -682,4 +703,6 @@
     <xacro:include filename="$(mirte_master_description/urdf/flag.xacro)" />
   </xacro:if>
-  <xacro:include filename="$(find mirte_master_description)/urdf/arm.xacro" />
+  <xacro:if value="$(arg arm_enable)">
+    <xacro:include filename="$(find mirte_master_description)/urdf/arm.xacro" />
+  </xacro:if>
 </robot>
