Commit message: Tried mecanum drive plugin

File: mirte_master_description/urdf/mirte_master.xacro (robot description, xacro)
@@ -8,4 +8,6 @@
   <xacro:arg name="flag_enable" default="False" />
   <xacro:arg name="arm_enable" default="False" />
+  <xacro:arg name="screen_enable" default="False" />
+  <xacro:arg name="front_camera_enable" default="False" />
   <!-- Bring in simulation data for Gazebo. -->
   <xacro:include filename="$(find mirte_master_description)/urdf/mirte_master_base.gazebo.xacro" />
@@ -16,4 +18,10 @@
     <origin xyz="0.01 -0.146658788505756 0.0427000000000005" rpy="0 0 ${radians(-90)}" />
   </xacro:sensor_orbbec_astra_pro_plus>
+  <link name="base_footprint"></link>
+  <joint name="base_link_joint" type="fixed">
+    <origin xyz="0 0 0.10" rpy="0 0 0" />
+    <parent link="base_footprint" />
+    <child link="base_link" />
+  </joint>
   <link
     name="base_link">
@@ -106,10 +114,10 @@
     <type>transmission_interface/SimpleTransmission</type>
     <joint name="wheel_joint_fl">
-        <hardwareInterface>hardware_interface/VelocityJointInterface</hardwareInterface>
+      <hardwareInterface>hardware_interface/VelocityJointInterface</hardwareInterface>
     </joint>
     <actuator name="wheel_act_fl">
-        <mechanicalReduction>1</mechanicalReduction>
+      <mechanicalReduction>1</mechanicalReduction>
     </actuator>
-</transmission>
+  </transmission>
   <link
     name="wheel_br">
@@ -160,8 +168,8 @@
     <type>transmission_interface/SimpleTransmission</type>
     <joint name="wheel_joint_br">
-        <hardwareInterface>hardware_interface/VelocityJointInterface</hardwareInterface>
+      <hardwareInterface>hardware_interface/VelocityJointInterface</hardwareInterface>
     </joint>
     <actuator name="wheel_act_br">
-        <mechanicalReduction>1</mechanicalReduction>
+      <mechanicalReduction>1</mechanicalReduction>
     </actuator>
   </transmission>
@@ -214,10 +222,10 @@
     <type>transmission_interface/SimpleTransmission</type>
     <joint name="wheel_joint_fr">
-        <hardwareInterface>hardware_interface/VelocityJointInterface</hardwareInterface>
+      <hardwareInterface>hardware_interface/VelocityJointInterface</hardwareInterface>
     </joint>
     <actuator name="wheel_act_fr">
-        <mechanicalReduction>1</mechanicalReduction>
+      <mechanicalReduction>1</mechanicalReduction>
     </actuator>
-</transmission>
+  </transmission>
   <link
     name="wheel_bl">
@@ -269,63 +277,62 @@
     <type>transmission_interface/SimpleTransmission</type>
     <joint name="wheel_joint_bl">
-        <hardwareInterface>hardware_interface/VelocityJointInterface</hardwareInterface>
+      <hardwareInterface>hardware_interface/VelocityJointInterface</hardwareInterface>
     </joint>
     <actuator name="wheel_act_bl">
-        <mechanicalReduction>1</mechanicalReduction>
+      <mechanicalReduction>1</mechanicalReduction>
     </actuator>
-</transmission>
-  <link
-    name="cam_front">
-    <inertial>
-      <origin
-        xyz="-0.00010069 -0.00018452 0.0033961"
-        rpy="0 0 0" />
-      <mass
-        value="0.0022023" />
-      <inertia
-        ixx="7.901E-08"
-        ixy="-1.4438E-25"
-        ixz="5.502E-24"
-        iyy="1.049E-07"
-        iyz="-1.0016E-23"
-        izz="1.3983E-07" />
-    </inertial>
-    <visual>
-      <origin
-        xyz="0 0 0"
-        rpy="0 0 0" />
-      <geometry>
-        <mesh
-          filename="package://mirte_master_description/meshes/cam_front.STL" />
-      </geometry>
-      <material
-        name="">
-        <color
-          rgba="0.79608 0.82353 0.93725 1" />
-      </material>
-    </visual>
-    <collision>
-      <origin
-        xyz="0 0 0"
-        rpy="0 0 0" />
-      <geometry>
-        <mesh
-          filename="package://mirte_master_description/meshes/cam_front.STL" />
-      </geometry>
-    </collision>
-  </link>
-  <joint
-    name="cam_joint_front"
-    type="fixed">
-    <origin
-      xyz="0 -0.1325 -0.0285"
-      rpy="1.5708 0 0" />
-    <parent
-      link="base_link" />
-    <child
-      link="cam_front" />
-    <axis
-      xyz="0 0 0" />
-  </joint>
+  </transmission>
+  <xacro:if value="$(arg front_camera_enable)">
+    <link
+      name="cam_front">
+      <inertial>
+        <origin
+          xyz="-0.00010069 -0.00018452 0.0033961"
+          rpy="0 0 0" />
+        <mass
+          value="0.0022023" />
+        <inertia
+          ixx="7.901E-08"
+          ixy="-1.4438E-25"
+          ixz="5.502E-24"
+          iyy="1.049E-07"
+          iyz="-1.0016E-23"
+          izz="1.3983E-07" />
+      </inertial>
+      <visual>
+        <origin
+          xyz="0 0 0"
+          rpy="0 0 0" />
+        <geometry>
+          <mesh
+            filename="package://mirte_master_description/meshes/cam_front.STL" />
+        </geometry>
+        <material
+          name="">
+          <color
+            rgba="0.79608 0.82353 0.93725 1" />
+        </material>
+      </visual>
+      <!-- <collision>
+  <origin
+  xyz="0 0 0"
+  rpy="0 0 0" />
+  <geometry>
+    <mesh
+    filename="package://mirte_master_description/meshes/cam_front.STL" />
+  </geometry>
+</collision> -->
+    </link>
+    <joint
+      name="cam_joint_front"
+      type="fixed">
+      <origin
+        xyz="0 -0.1325 -0.0285"
+        rpy="1.5708 0 0" />
+      <parent link="base_link" />
+      <child link="cam_front" />
+      <!-- <axis xyz="0 0 0" /> -->
+    </joint>
+  </xacro:if>
   <link
     name="ultrasonic_fl">
@@ -647,57 +654,59 @@
       xyz="0 0 0" />
   </joint>
-  <link
-    name="screen">
-    <inertial>
-      <origin
-        xyz="-1.24638847975239E-07 0.0013371323974908 0.00160606068028191"
-        rpy="0 0 0" />
-      <mass
-        value="0.00357270774970056" />
-      <inertia
-        ixx="1.29976980207027E-07"
-        ixy="-1.78182996362165E-11"
-        ixz="-4.24689246841474E-13"
-        iyy="2.09902246549457E-07"
-        iyz="1.92672613573332E-09"
-        izz="3.37075734369407E-07" />
-    </inertial>
-    <visual>
-      <origin
-        xyz="0 0 0"
-        rpy="0 0 0" />
-      <geometry>
-        <mesh
-          filename="package://mirte_master_description/meshes/screen.STL" />
-      </geometry>
-      <material
-        name="">
-        <color
-          rgba="0.768627450980392 0.768627450980392 0.768627450980392 1" />
-      </material>
-    </visual>
-    <collision>
-      <origin
-        xyz="0 0 0"
-        rpy="0 0 0" />
-      <geometry>
-        <mesh
-          filename="package://mirte_master_description/meshes/screen.STL" />
-      </geometry>
-    </collision>
-  </link>
-  <joint
-    name="screen_joint"
-    type="fixed">
-    <origin
-      xyz="0 0.121521156261136 0.0540000000000046"
-      rpy="1.5707963267949 0 -3.14159265358979" />
-    <parent
-      link="base_link" />
-    <child
-      link="screen" />
-    <axis
-      xyz="0 0 0" />
-  </joint>
+  <xacro:if value="$(arg screen_enable)">
+    <link
+      name="screen">
+      <inertial>
+        <origin
+          xyz="-1.24638847975239E-07 0.0013371323974908 0.00160606068028191"
+          rpy="0 0 0" />
+        <mass
+          value="0.00357270774970056" />
+        <inertia
+          ixx="1.29976980207027E-07"
+          ixy="-1.78182996362165E-11"
+          ixz="-4.24689246841474E-13"
+          iyy="2.09902246549457E-07"
+          iyz="1.92672613573332E-09"
+          izz="3.37075734369407E-07" />
+      </inertial>
+      <visual>
+        <origin
+          xyz="0 0 0"
+          rpy="0 0 0" />
+        <geometry>
+          <mesh
+            filename="package://mirte_master_description/meshes/screen.STL" />
+        </geometry>
+        <material
+          name="">
+          <color
+            rgba="0.768627450980392 0.768627450980392 0.768627450980392 1" />
+        </material>
+      </visual>
+      <collision>
+        <origin
+          xyz="0 0 0"
+          rpy="0 0 0" />
+        <geometry>
+          <mesh
+            filename="package://mirte_master_description/meshes/screen.STL" />
+        </geometry>
+      </collision>
+    </link>
+    <joint
+      name="screen_joint"
+      type="fixed">
+      <origin
+        xyz="0 0.121521156261136 0.0540000000000046"
+        rpy="1.5707963267949 0 -3.14159265358979" />
+      <parent
+        link="base_link" />
+      <child
+        link="screen" />
+      <axis
+        xyz="0 0 0" />
+    </joint>
+  </xacro:if>
   <xacro:if value="$(arg flag_enable)">
     <xacro:include filename="$(mirte_master_description/urdf/flag.xacro)" />

File: mirte_master_description/urdf/mirte_master_base.gazebo.xacro (robot description, xacro)
@@ -5,8 +5,8 @@
     <gazebo>
       <plugin name="mirte_master_mechanum_drive" filename="libgazebo_ros_mecanum_drive.so">
-        <commandTopic>cmd_vel</commandTopic>
+        <commandTopic>mobile_base_controller/cmd_vel</commandTopic>
         <odometryTopic>odom</odometryTopic>
         <odometryFrame>odom</odometryFrame>
-        <robotBaseFrame>base_link</robotBaseFrame>
+        <robotBaseFrame>base_footprint</robotBaseFrame>
         <LeftRear>wheel_joint_bl</LeftRear>
         <LeftFront>wheel_joint_fl</LeftFront>
@@ -22,5 +22,8 @@
         <wheelDiameter>0.106</wheelDiameter> <!--Was 0.13-->
         <publishOdom>true</publishOdom>
-        <isRollerModel>true</isRollerModel>
+        <isRollerModel>false</isRollerModel>
+        <plugin name="gazebo_ros_control" filename="libgazebo_ros_control.so">
+          <robotNamespace>/mirte</robotNamespace>
+        </plugin>
       </plugin>
     </gazebo>
@@ -69,4 +72,5 @@
     <material>Gazebo/White</material>
     <gravity>true</gravity>
+    <selfCollide>false</selfCollide>
   </gazebo>
   <!-- Individual link colouring still needed in Gazebo 2.x -->

Commit message: Attempt at making wheels better, but the physics don't work out

File: mirte_master_description/urdf/mirte_master.xacro (robot description, xacro)
@@ -20,5 +20,5 @@
   <link name="base_footprint"></link>
   <joint name="base_link_joint" type="fixed">
-    <origin xyz="0 0 0.10" rpy="0 0 0" />
+    <origin xyz="0 0 0.10" rpy="0 0 ${radians(90)}" />
     <parent link="base_footprint" />
     <child link="base_link" />
@@ -54,10 +54,13 @@
     </visual>
     <collision>
-      <origin
-        xyz="0 0 0"
-        rpy="0 0 0" />
-      <geometry>
-        <mesh
-          filename="package://mirte_master_description/meshes/base_link.STL" />
+      <origin xyz="0 0 -0.03" />
+      <geometry>
+        <box size="0.19 0.28 0.06" />
+      </geometry>
+    </collision>
+    <collision>
+      <origin xyz="0 0.05 0.045" />
+      <geometry>
+        <box size="0.18 0.16 0.05" />
       </geometry>
     </collision>

File: mirte_master_description/urdf/mirte_master_base.gazebo.xacro (robot description, xacro)
@@ -14,17 +14,17 @@
         <RightRear>wheel_joint_br</RightRear>
         <odometryRate>20</odometryRate>
-        <publishWheelTF>false</publishWheelTF>
+        <publishWheelTF>true</publishWheelTF>
         <publishWheelJointState>true</publishWheelJointState>
-        <WheelTorque>30</WheelTorque>
+        <WheelTorque>0.100</WheelTorque>
         <WheelSeparationW>0.170</WheelSeparationW>
         <WheelSeparationL>0.306</WheelSeparationL>
-        <wheelAccel>5</wheelAccel>
+        <wheelAccel>2.5</wheelAccel>
         <wheelDiameter>0.106</wheelDiameter> <!--Was 0.13-->
         <publishOdom>true</publishOdom>
         <isRollerModel>false</isRollerModel>
+      </plugin>
         <plugin name="gazebo_ros_control" filename="libgazebo_ros_control.so">
-          <robotNamespace>/mirte</robotNamespace>
+          <robotNamespace>/</robotNamespace>
         </plugin>
-      </plugin>
     </gazebo>
     <!--

File: mirte_master_description/urdf/wheel.gazebo.xacro (robot description, xacro)
@@ -3,9 +3,9 @@
     <xacro:macro name="wheel_gazebo" params="name">
         <gazebo reference="${name}">
-            <selfCollide>false</selfCollide>
+            <!-- <selfCollide>false</selfCollide> -->
             <gravity>true</gravity>
-            <mu1>30</mu1>
-            <mu2>30</mu2>
-            <!-- <kp>1e50</kp> -->
+            <mu1>5.0</mu1>
+            <mu2>5.0</mu2>
+            <!-- <kp>1e2</kp> -->
             <!-- <kd>1e50</kd> -->
             <material>Gazebo/DarkGrey</material>
