Commit message: A somewhat stable simulation

File: mirte_master_description/urdf/mirte_master.xacro (robot description, xacro)
@@ -10,4 +10,13 @@
   <xacro:arg name="screen_enable" default="False" />
   <xacro:arg name="front_camera_enable" default="False" />
+  <xacro:arg name="sonar_enable" default="False" />
+  <xacro:arg name="lidar_enable" default="False" />
+  <xacro:arg name="depth_camera_enable" default="False" />
+  <xacro:property name="wheel_radius" value="0.053" />
+  <xacro:property name="wheel_length" value="0.055" />
+  <xacro:property name="wheel_mass" value="0.26661" />
+  <xacro:property name="wheel_velocity" value="10" />
+  <xacro:property name="wheel_effort" value="10" /> <!-- 5 -->
+  <xacro:property name="base_mass" value="4.0815" /> <!-- 3.0815 -->
   <!-- Bring in simulation data for Gazebo. -->
   <xacro:include filename="$(find mirte_master_description)/urdf/mirte_master_base.gazebo.xacro" />
@@ -15,10 +24,12 @@
     filename="$(find gazebo_sensor_collection)/urdf/cameras/rgbd/orbbec_astra_pro_plus.urdf.xacro" />
   <!-- TODO: CHANGE TO CAMERA -->
-  <xacro:sensor_orbbec_astra_pro_plus name="camera" parent="base_link" color="black">
-    <origin xyz="0.01 -0.146658788505756 0.0427000000000005" rpy="0 0 ${radians(-90)}" />
-  </xacro:sensor_orbbec_astra_pro_plus>
+  <xacro:if value="$(arg depth_camera_enable)">
+    <xacro:sensor_orbbec_astra_pro_plus name="camera" parent="base_link" color="black">
+      <origin xyz="0.01 -0.146658788505756 0.0427" rpy="0 0 ${radians(-90)}" />
+    </xacro:sensor_orbbec_astra_pro_plus>
+  </xacro:if>
   <link name="base_footprint"></link>
   <joint name="base_link_joint" type="fixed">
-    <origin xyz="0 0 0.10" rpy="0 0 ${radians(90)}" />
+    <origin xyz="0 0 0.10" rpy="0 0 0" />
     <parent link="base_footprint" />
     <child link="base_link" />
@@ -27,9 +38,7 @@
     name="base_link">
     <inertial>
-      <origin
-        xyz="-0.00024285 0.0082178 -0.0037661"
-        rpy="0 0 0" /> F <mass
-        value="3.0815" />
-      <inertia
+      <!-- <origin xyz="-0.00024285 0.0082178 -0.0037661" /> -->
+      <mass value="${base_mass}" />
+      <!-- <inertia
         ixx="0.01245"
         ixy="-6.0298E-07"
@@ -37,18 +46,18 @@
         iyy="0.0091262"
         iyz="-0.00017974"
-        izz="0.020706" />
+        izz="0.020706" /> -->
+      <inertia
+        ixx="${base_mass * (0.06**2 + 0.28**2) / 12}"
+        iyy="${base_mass * (0.19**2 + 0.06**2) / 12}"
+        izz="${base_mass * (0.19**2 + 0.28**2) / 12}"
+        ixy="0" ixz="0" iyz="0" />
     </inertial>
     <visual>
-      <origin
-        xyz="0 0 0"
-        rpy="0 0 0" />
       <geometry>
         <mesh
           filename="package://mirte_master_description/meshes/base_link.STL" />
       </geometry>
-      <material
-        name="">
-        <color
-          rgba="0.52941 0.54902 0.54902 1" />
+      <material name="">
+        <color rgba="0.52941 0.54902 0.54902 1" />
       </material>
     </visual>
@@ -69,29 +78,19 @@
     name="wheel_fl">
     <inertial>
-      <origin
-        xyz="-1.1211E-10 2.9249E-10 0.024936"
-        rpy="0 0 0" />
-      <mass
-        value="0.26661" />
+      <origin xyz="0 0 0.025" />
+      <mass value="${wheel_mass}" />
       <inertia
-        ixx="8.0546E-05"
-        ixy="1.9673E-15"
-        ixz="1.226E-14"
-        iyy="8.0546E-05"
-        iyz="9.6889E-15"
-        izz="9.3196E-05" />
+        ixx="${wheel_mass * (3 * (wheel_radius**2) + (wheel_length**2)) / 12}"
+        iyy="${wheel_mass * (3 * (wheel_radius**2) + (wheel_length**2)) / 12}"
+        izz="${wheel_mass * (wheel_radius **2) / 2}"
+        ixy="0" ixz="0" iyz="0" />
     </inertial>
     <visual>
-      <origin
-        xyz="0 0 0"
-        rpy="0 0 0" />
       <geometry>
         <mesh
           filename="package://mirte_master_description/meshes/wheel_fl.STL" />
       </geometry>
-      <material
-        name="">
-        <color
-          rgba="0.79216 0.81961 0.93333 1" />
+      <material name="">
+        <color rgba="0.79216 0.81961 0.93333 1" />
       </material>
     </visual>
@@ -99,5 +98,5 @@
       <origin xyz="0 0 0.025" />
       <geometry>
-        <cylinder radius="0.053" length="0.055" />
+        <cylinder radius="${wheel_radius}" length="${wheel_length}" />
       </geometry>
     </collision>
@@ -113,4 +112,5 @@
     <axis xyz="0 0 -1" />
     <dynamics damping="3.0" friction="5.0" />
+    <limit velocity="${wheel_velocity}" effort="${wheel_effort}"/>
   </joint>
   <transmission name="wheel_trans_fl">
@@ -126,26 +126,19 @@
     name="wheel_br">
     <inertial>
-      <origin xyz="-1.0009E-10 2.9473E-10 -0.025064" />
-      <mass value="0.26661" />
+      <origin xyz="0 0 0.025" />
+      <mass value="${wheel_mass}" />
       <inertia
-        ixx="8.0546E-05"
-        ixy="4.8209E-17"
-        ixz="1.2652E-14"
-        iyy="8.0546E-05"
-        iyz="1.7571E-14"
-        izz="9.3196E-05" />
+        ixx="${wheel_mass * (3 * (wheel_radius**2) + (wheel_length**2)) / 12}"
+        iyy="${wheel_mass * (3 * (wheel_radius**2) + (wheel_length**2)) / 12}"
+        izz="${wheel_mass * (wheel_radius **2) / 2}"
+        ixy="0" ixz="0" iyz="0" />
     </inertial>
     <visual>
-      <origin
-        xyz="0 0 0"
-        rpy="0 0 0" />
       <geometry>
         <mesh
           filename="package://mirte_master_description/meshes/wheel_br.STL" />
       </geometry>
-      <material
-        name="">
-        <color
-          rgba="0.79216 0.81961 0.93333 1" />
+      <material name="">
+        <color rgba="0.79216 0.81961 0.93333 1" />
       </material>
     </visual>
@@ -153,5 +146,5 @@
       <origin xyz="0 0 -0.025" />
       <geometry>
-        <cylinder radius="0.053" length="0.055" />
+        <cylinder radius="${wheel_radius}" length="${wheel_length}" />
       </geometry>
     </collision>
@@ -165,6 +158,7 @@
     <parent link="base_link" />
     <child link="wheel_br" />
-    <axis xyz="0 0 1" />
+    <axis xyz="0 0 -1" />
     <dynamics damping="3.0" friction="5.0" />
+    <limit velocity="${wheel_velocity}" effort="${wheel_effort}"/>
   </joint>
   <transmission name="wheel_trans_br">
@@ -180,26 +174,19 @@
     name="wheel_fr">
     <inertial>
-      <origin xyz="-1.9E-10 2.1252E-10 -0.025064" />
-      <mass value="0.26661" />
+      <origin xyz="0 0 0.025" />
+      <mass value="${wheel_mass}" />
       <inertia
-        ixx="8.0546E-05"
-        ixy="-4.5866E-15"
-        ixz="7.6917E-14"
-        iyy="8.0546E-05"
-        iyz="9.6011E-15"
-        izz="9.3196E-05" />
+        ixx="${wheel_mass * (3 * (wheel_radius**2) + (wheel_length**2)) / 12}"
+        iyy="${wheel_mass * (3 * (wheel_radius**2) + (wheel_length**2)) / 12}"
+        izz="${wheel_mass * (wheel_radius **2) / 2}"
+        ixy="0" ixz="0" iyz="0" />
     </inertial>
     <visual>
-      <!-- <origin
-        xyz="0 0 0"
-        rpy="0 0 0" /> -->
       <geometry>
         <mesh
           filename="package://mirte_master_description/meshes/wheel_fr.STL" />
       </geometry>
-      <material
-        name="">
-        <color
-          rgba="0.79216 0.81961 0.93333 1" />
+      <material name="">
+        <color rgba="0.79216 0.81961 0.93333 1" />
       </material>
     </visual>
@@ -207,5 +194,5 @@
       <origin xyz="0 0 -0.025" />
       <geometry>
-        <cylinder radius="0.053" length="0.055" />
+        <cylinder radius="${wheel_radius}" length="${wheel_length}" />
       </geometry>
     </collision>
@@ -219,6 +206,7 @@
     <parent link="base_link" />
     <child link="wheel_fr" />
-    <axis xyz="0 0 1" />
+    <axis xyz="0 0 -1" />
     <dynamics damping="3.0" friction="5.0" />
+    <limit velocity="${wheel_velocity}" effort="${wheel_effort}"/>
   </joint>
   <transmission name="wheel_trans_fr">
@@ -234,27 +222,19 @@
     name="wheel_bl">
     <inertial>
-      <origin xyz="-1.9E-10 2.1252E-10 0.024936" />
-      <mass
-        value="0.26661" />
+      <origin xyz="0 0 0.025" />
+      <mass value="${wheel_mass}" />
       <inertia
-        ixx="8.0546E-05"
-        ixy="-4.5761E-15"
-        ixz="7.6918E-14"
-        iyy="8.0546E-05"
-        iyz="9.5856E-15"
-        izz="9.3196E-05" />
+        ixx="${wheel_mass * (3 * (wheel_radius**2) + (wheel_length**2)) / 12}"
+        iyy="${wheel_mass * (3 * (wheel_radius**2) + (wheel_length**2)) / 12}"
+        izz="${wheel_mass * (wheel_radius **2) / 2}"
+        ixy="0" ixz="0" iyz="0" />
     </inertial>
     <visual>
-      <origin
-        xyz="0 0 0"
-        rpy="0 0 0" />
       <geometry>
         <mesh
           filename="package://mirte_master_description/meshes/wheel_bl.STL" />
       </geometry>
-      <material
-        name="">
-        <color
-          rgba="0.79216 0.81961 0.93333 1" />
+      <material name="">
+        <color rgba="0.79216 0.81961 0.93333 1" />
       </material>
     </visual>
@@ -262,5 +242,5 @@
       <origin xyz="0 0 0.025" />
       <geometry>
-        <cylinder radius="0.053" length="0.055" />
+        <cylinder radius="${wheel_radius}" length="${wheel_length}" />
       </geometry>
     </collision>
@@ -276,4 +256,5 @@
     <axis xyz="0 0 -1" />
     <dynamics damping="3.0" friction="5.0" />
+    <limit velocity="${wheel_velocity}" effort="${wheel_effort}"/>
   </joint>
   <transmission name="wheel_trans_bl">
@@ -338,216 +319,218 @@
     </joint>
   </xacro:if>
-  <link
-    name="ultrasonic_fl">
-    <inertial>
-      <origin
-        xyz="-4.30733527062924E-05 0.00367564883489804 -6.99136578631437E-05"
-        rpy="0 0 0" />
-      <mass
-        value="0.00383513951999247" />
-      <inertia
-        ixx="1.59365628586768E-07"
-        ixy="-8.54250314742639E-10"
-        ixz="-3.40905422018191E-09"
-        iyy="7.68751523460336E-07"
-        iyz="2.65062440645508E-09"
-        izz="7.26221149125628E-07" />
-    </inertial>
-    <visual>
-      <origin
-        xyz="0 0 0"
-        rpy="0 0 0" />
-      <geometry>
-        <mesh
-          filename="package://mirte_master_description/meshes/ultrasonic_fl.STL" />
-      </geometry>
-      <material
-        name="">
-        <color
-          rgba="0.792156862745098 0.819607843137255 0.933333333333333 1" />
-      </material>
-    </visual>
-    <collision>
-      <origin
-        xyz="0 0 0"
-        rpy="0 0 0" />
-      <geometry>
-        <mesh
-          filename="package://mirte_master_description/meshes/ultrasonic_fl.STL" />
-      </geometry>
-    </collision>
-  </link>
-  <joint
-    name="ultrasonic_joint_fl"
-    type="fixed">
-    <origin
-      xyz="0.05297775289576 -0.120282421780502 -0.031"
-      rpy="3.14159265358979 0 0.296705972839036" />
-    <parent
-      link="base_link" />
-    <child
-      link="ultrasonic_fl" />
-    <axis
-      xyz="0 0 0" />
-  </joint>
-  <link
-    name="ultrasonic_fr">
-    <inertial>
-      <origin
-        xyz="-4.30733527063201E-05 0.00367564883489799 -6.99136578631784E-05"
-        rpy="0 0 0" />
-      <mass
-        value="0.00383513951999245" />
-      <inertia
-        ixx="1.59365628586767E-07"
-        ixy="-8.54250314742507E-10"
-        ixz="-3.40905422018182E-09"
-        iyy="7.6875152346034E-07"
-        iyz="2.65062440645522E-09"
-        izz="7.26221149125632E-07" />
-    </inertial>
-    <visual>
-      <origin
-        xyz="0 0 0"
-        rpy="0 0 0" />
-      <geometry>
-        <mesh
-          filename="package://mirte_master_description/meshes/ultrasonic_fr.STL" />
-      </geometry>
-      <material
-        name="">
-        <color
-          rgba="0.792156862745098 0.819607843137255 0.933333333333333 1" />
-      </material>
-    </visual>
-    <collision>
-      <origin
-        xyz="0 0 0"
-        rpy="0 0 0" />
-      <geometry>
-        <mesh
-          filename="package://mirte_master_description/meshes/ultrasonic_fr.STL" />
-      </geometry>
-    </collision>
-  </link>
-  <joint
-    name="ultrasonic_joint_fr"
-    type="fixed">
-    <origin
-      xyz="-0.05297775289576 -0.120282421780502 -0.031"
-      rpy="3.14159265358979 0 -0.296705972839036" />
-    <parent
-      link="base_link" />
-    <child
-      link="ultrasonic_fr" />
-    <axis
-      xyz="0 0 0" />
-  </joint>
-  <link
-    name="ultrasonic_bl">
-    <inertial>
-      <origin
-        xyz="-4.30733527062716E-05 0.00367564883489804 -6.9913657863175E-05"
-        rpy="0 0 0" />
-      <mass
-        value="0.00383513951999244" />
-      <inertia
-        ixx="1.59365628586767E-07"
-        ixy="-8.54250314742494E-10"
-        ixz="-3.40905422018206E-09"
-        iyy="7.68751523460339E-07"
-        iyz="2.6506244064553E-09"
-        izz="7.26221149125632E-07" />
-    </inertial>
-    <visual>
-      <origin
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
File: mirte_master_description/urdf/mirte_master_base.gazebo.xacro (robot description, xacro)
@@ -8,5 +8,5 @@
         <odometryTopic>odom</odometryTopic>
         <odometryFrame>odom</odometryFrame>
-        <robotBaseFrame>base_footprint</robotBaseFrame>
+        <robotBaseFrame>base_link</robotBaseFrame>
         <LeftRear>wheel_joint_bl</LeftRear>
         <LeftFront>wheel_joint_fl</LeftFront>
@@ -14,13 +14,13 @@
         <RightRear>wheel_joint_br</RightRear>
         <odometryRate>20</odometryRate>
-        <publishWheelTF>true</publishWheelTF>
+        <publishWheelTF>false</publishWheelTF>
         <publishWheelJointState>true</publishWheelJointState>
-        <WheelTorque>0.100</WheelTorque>
+        <WheelTorque>50</WheelTorque>
         <WheelSeparationW>0.170</WheelSeparationW>
-        <WheelSeparationL>0.306</WheelSeparationL>
-        <wheelAccel>2.5</wheelAccel>
-        <wheelDiameter>0.106</wheelDiameter> <!--Was 0.13-->
+        <WheelSeparationL>0.3</WheelSeparationL> <!-- 3.06 -->
+        <wheelAccel>1</wheelAccel>
+        <wheelDiameter>0.1</wheelDiameter> <!-- 1.06 Was 0.13-->
         <publishOdom>true</publishOdom>
-        <isRollerModel>false</isRollerModel>
+        <isRollerModel>true</isRollerModel>
       </plugin>
         <plugin name="gazebo_ros_control" filename="libgazebo_ros_control.so">

File: mirte_master_description/urdf/wheel.gazebo.xacro (robot description, xacro)
@@ -5,8 +5,8 @@
             <!-- <selfCollide>false</selfCollide> -->
             <gravity>true</gravity>
-            <mu1>5.0</mu1>
-            <mu2>5.0</mu2>
-            <!-- <kp>1e2</kp> -->
-            <!-- <kd>1e50</kd> -->
+            <mu1>2.5</mu1>
+            <mu2>2.5</mu2>
+            <!-- <kp>1e15</kp> --> <!-- <kp>1e2</kp> -->
+            <!-- <kd>1e13</kd> --> <!-- <kd>1e50</kd> -->
             <material>Gazebo/DarkGrey</material>
         </gazebo>

Commit message: Fix the driving of mirte

File: mirte_master_description/urdf/mirte_master.xacro (robot description, xacro)
@@ -13,9 +13,12 @@
   <xacro:arg name="lidar_enable" default="False" />
   <xacro:arg name="depth_camera_enable" default="False" />
+  <!-- Disable momentum on the main body, makes the simulation behave slightly nicer, at the cost of
+  inaccuracies (It is better toggle this when the robot hits the ground)-->
+  <xacro:arg name="kinematic_only" default="False" />
   <xacro:property name="wheel_radius" value="0.053" />
   <xacro:property name="wheel_length" value="0.055" />
   <xacro:property name="wheel_mass" value="0.26661" />
-  <xacro:property name="wheel_velocity" value="10" />
-  <xacro:property name="wheel_effort" value="10" /> <!-- 5 -->
+  <xacro:property name="wheel_velocity" value="8" /> <!-- Was 10 based on calc-->
+  <xacro:property name="wheel_effort" value="5" /> <!-- 5 -->
   <xacro:property name="base_mass" value="4.0815" /> <!-- 3.0815 -->
   <!-- Bring in simulation data for Gazebo. -->
@@ -23,5 +26,4 @@
   <xacro:include
     filename="$(find gazebo_sensor_collection)/urdf/cameras/rgbd/orbbec_astra_pro_plus.urdf.xacro" />
-  <!-- TODO: CHANGE TO CAMERA -->
   <xacro:if value="$(arg depth_camera_enable)">
     <xacro:sensor_orbbec_astra_pro_plus name="camera" parent="base_link" color="black">
@@ -31,5 +33,5 @@
   <link name="base_footprint"></link>
   <joint name="base_link_joint" type="fixed">
-    <origin xyz="0 0 0.10" rpy="0 0 0" />
+    <origin xyz="0 0 0.10" rpy="0 0 ${radians(90)}" />
     <parent link="base_footprint" />
     <child link="base_link" />
@@ -38,5 +40,5 @@
     name="base_link">
     <inertial>
-      <!-- <origin xyz="-0.00024285 0.0082178 -0.0037661" /> -->
+      <origin xyz="-0.00024285 0.0082178 -0.0037661" />
       <mass value="${base_mass}" />
       <!-- <inertia
@@ -112,5 +114,5 @@
     <axis xyz="0 0 -1" />
     <dynamics damping="3.0" friction="5.0" />
-    <limit velocity="${wheel_velocity}" effort="${wheel_effort}"/>
+    <limit velocity="${wheel_velocity}" effort="${wheel_effort}" />
   </joint>
   <transmission name="wheel_trans_fl">
@@ -160,5 +162,5 @@
     <axis xyz="0 0 -1" />
     <dynamics damping="3.0" friction="5.0" />
-    <limit velocity="${wheel_velocity}" effort="${wheel_effort}"/>
+    <limit velocity="${wheel_velocity}" effort="${wheel_effort}" />
   </joint>
   <transmission name="wheel_trans_br">
@@ -208,5 +210,5 @@
     <axis xyz="0 0 -1" />
     <dynamics damping="3.0" friction="5.0" />
-    <limit velocity="${wheel_velocity}" effort="${wheel_effort}"/>
+    <limit velocity="${wheel_velocity}" effort="${wheel_effort}" />
   </joint>
   <transmission name="wheel_trans_fr">
@@ -256,5 +258,5 @@
     <axis xyz="0 0 -1" />
     <dynamics damping="3.0" friction="5.0" />
-    <limit velocity="${wheel_velocity}" effort="${wheel_effort}"/>
+    <limit velocity="${wheel_velocity}" effort="${wheel_effort}" />
   </joint>
   <transmission name="wheel_trans_bl">
@@ -698,5 +700,5 @@
   </xacro:if>
   <xacro:if value="$(arg flag_enable)">
-    <xacro:include filename="$(mirte_master_description/urdf/flag.xacro)" />
+    <xacro:include filename="$(find mirte_master_description)/urdf/flag.xacro" />
   </xacro:if>
   <xacro:if value="$(arg arm_enable)">

File: mirte_master_description/urdf/mirte_master_base.gazebo.xacro (robot description, xacro)
@@ -5,8 +5,8 @@
     <gazebo>
       <plugin name="mirte_master_mechanum_drive" filename="libgazebo_ros_mecanum_drive.so">
-        <commandTopic>mobile_base_controller/cmd_vel</commandTopic>
+        <commandTopic>mobile_base_controller/cmd_vel_corrected</commandTopic>
         <odometryTopic>odom</odometryTopic>
         <odometryFrame>odom</odometryFrame>
-        <robotBaseFrame>base_link</robotBaseFrame>
+        <robotBaseFrame>base_footprint</robotBaseFrame>
         <LeftRear>wheel_joint_bl</LeftRear>
         <LeftFront>wheel_joint_fl</LeftFront>
@@ -17,10 +17,10 @@
         <publishWheelJointState>true</publishWheelJointState>
         <WheelTorque>50</WheelTorque>
-        <WheelSeparationW>0.170</WheelSeparationW>
-        <WheelSeparationL>0.3</WheelSeparationL> <!-- 3.06 -->
-        <wheelAccel>1</wheelAccel>
+        <WheelSeparationW>0.28</WheelSeparationW>
+        <WheelSeparationL>0.175</WheelSeparationL> <!-- 3.06 -->
+        <wheelAccel>5</wheelAccel>
         <wheelDiameter>0.1</wheelDiameter> <!-- 1.06 Was 0.13-->
         <publishOdom>true</publishOdom>
-        <isRollerModel>true</isRollerModel>
+        <isRollerModel>false</isRollerModel>
       </plugin>
         <plugin name="gazebo_ros_control" filename="libgazebo_ros_control.so">
@@ -72,5 +72,6 @@
     <material>Gazebo/White</material>
     <gravity>true</gravity>
-    <selfCollide>false</selfCollide>
+    <kinematic>$(arg kinematic_only)</kinematic>
+    <!-- <selfCollide>false</selfCollide> -->
   </gazebo>
   <!-- Individual link colouring still needed in Gazebo 2.x -->
@@ -111,7 +112,7 @@
        the body level. -->
   <xacro:include filename="$(find mirte_master_description)/urdf/wheel.gazebo.xacro" />
-  <xacro:wheel_gazebo name="wheel_bl" />
-  <xacro:wheel_gazebo name="wheel_br" />
-  <xacro:wheel_gazebo name="wheel_fl"/>
-  <xacro:wheel_gazebo name="wheel_fr"/>
+  <xacro:wheel_gazebo id="bl" />
+  <xacro:wheel_gazebo id="br" />
+  <xacro:wheel_gazebo id="fl"/>
+  <xacro:wheel_gazebo id="fr"/>
 </robot>

File: mirte_master_description/urdf/wheel.gazebo.xacro (robot description, xacro)
@@ -1,14 +1,20 @@
 <?xml version="1.0"?>
 <robot xmlns:xacro="http://ros.org/wiki/xacro">
-    <xacro:macro name="wheel_gazebo" params="name">
-        <gazebo reference="${name}">
-            <!-- <selfCollide>false</selfCollide> -->
+    <xacro:macro name="wheel_gazebo" params="id">
+        <gazebo reference="wheel_${id}">
+            <selfCollide>false</selfCollide>
             <gravity>true</gravity>
-            <mu1>2.5</mu1>
-            <mu2>2.5</mu2>
+            <mu1>0.0</mu1> <!--2.5-->
+            <mu2>0.0</mu2> <!--2.5-->
             <!-- <kp>1e15</kp> --> <!-- <kp>1e2</kp> -->
             <!-- <kd>1e13</kd> --> <!-- <kd>1e50</kd> -->
             <material>Gazebo/DarkGrey</material>
         </gazebo>
+        <gazebo reference="wheel_joint_${id}">
+            <ode>
+                <implicit_spring_damper>true</implicit_spring_damper>
+            </ode>
+            <!-- < -->
+        </gazebo>
     </xacro:macro>
 </robot>
