Commit message: Version 1.1.0

File: mirte_master_description/urdf/arm.xacro (robot description, xacro)
@@ -48,5 +48,5 @@
             rpy="1.5708 0 3.1416" />
         <parent
-            link="base_link" />
+            link="frame_link" />
         <child
             link="arm_Rot" />

File: mirte_master_description/urdf/flag.xacro (robot description, xacro)
@@ -42,5 +42,5 @@
         rpy="1.5707963267949 0 1.61494047314374" />
       <parent
-        link="base_link" />
+        link="frame_link" />
       <child
         link="flag" />

File: mirte_master_description/urdf/lidar.xacro (robot description, xacro)
@@ -48,5 +48,5 @@
       rpy="-1.5707963267949 0 -1.5707963267949" />
     <parent
-      link="base_link" />
+      link="frame_link" />
     <child
       link="lidar_base" />

File: mirte_master_description/urdf/mirte_master.xacro (robot description, xacro)
@@ -13,15 +13,12 @@
   <xacro:arg name="lidar_enable" default="True" />
   <xacro:arg name="depth_camera_enable" default="False" />
-  <!-- Disable momentum on the main body, makes the simulation behave slightly nicer, at the cost of
-  inaccuracies (It is better toggle this when the robot hits the ground)-->
-  <!-- BETTER IDEA: use http://wiki.ros.org/timed_roslaunch to launch a custom nodes which sets the
-  link to kinematic  -->
-  <xacro:arg name="kinematic_only" default="False" />
+  <xacro:arg name="imu_enable" default="True" />
   <xacro:property name="wheel_radius" value="0.050" />
   <xacro:property name="wheel_length" value="0.055" />
-  <xacro:property name="wheel_mass" value="0.26661" />
+  <xacro:property name="wheel_mass" value="2.15" /> <!-- 0.26661 -->
+  <!-- Currently unused -->
   <xacro:property name="wheel_velocity" value="8" /> <!-- Was 10 based on calc-->
-  <xacro:property name="wheel_effort" value="5" /> <!-- 5 -->
-  <xacro:property name="base_mass" value="4.0815" /> <!-- 3.0815 -->
+  <xacro:property name="wheel_effort" value="5" />
+  <xacro:property name="base_mass" value="5.0" /> <!-- 4.0815 --> <!-- 3.0815 -->
   <!-- Used for sonar by mirte-gazebo -->
   <material name="blue">
@@ -33,26 +30,28 @@
     filename="$(find gazebo_sensor_collection)/urdf/cameras/rgbd/orbbec_astra_pro_plus.urdf.xacro" />
   <xacro:if value="$(arg depth_camera_enable)">
-    <xacro:sensor_orbbec_astra_pro_plus name="camera" parent="base_link" color="black">
+    <xacro:sensor_orbbec_astra_pro_plus name="camera" parent="frame_link" color="black">
       <origin xyz="0.01 -0.146658788505756 0.0427" rpy="0 0 ${radians(-90)}" />
     </xacro:sensor_orbbec_astra_pro_plus>
   </xacro:if>
-  <link name="base_footprint"></link>
-  <joint name="base_link_joint" type="fixed">
+  <xacro:if value="$(arg imu_enable)">
+    <link name="imu_link" />
+    <joint name="imu_joint" type="fixed">
+      <origin xyz="0 0 0.10" />
+      <parent link="base_link" />
+      <child link="imu_link" />
+    </joint>
+  </xacro:if>
+  <link name="base_link" />
+  <joint name="frame_base_joint" type="fixed">
     <origin xyz="0 0 0.10" rpy="0 0 ${radians(90)}" />
-    <parent link="base_footprint" />
-    <child link="base_link" />
+    <parent link="base_link" />
+    <child link="frame_link" />
   </joint>
   <link
-    name="base_link">
+    name="frame_link">
     <inertial>
-      <origin xyz="-0.00024285 0.0082178 -0.0037661" />
+      <!-- Lower the center of mass for less woble as a result of accelaration -->
+      <origin xyz="-0.00024285 0.0082178 ${-0.0037661 - 0.04}" />
       <mass value="${base_mass}" />
-      <!-- <inertia
-        ixx="0.01245"
-        ixy="-6.0298E-07"
-        ixz="-7.3071E-07"
-        iyy="0.0091262"
-        iyz="-0.00017974"
-        izz="0.020706" /> -->
       <inertia
         ixx="${base_mass * (0.06**2 + 0.28**2) / 12}"
@@ -64,5 +63,5 @@
       <geometry>
         <mesh
-          filename="package://mirte_master_description/meshes/base_link.STL" />
+          filename="package://mirte_master_description/meshes/frame_link.STL" />
       </geometry>
       <material name="">
@@ -133,5 +132,5 @@
   </link>
   <link
-    name="wheel_fl">
+    name="wheel_left_front">
     <inertial>
       <origin xyz="0 0 0.025" />
@@ -146,5 +145,5 @@
       <geometry>
         <mesh
-          filename="package://mirte_master_description/meshes/wheel_fl.STL" />
+          filename="package://mirte_master_description/meshes/wheel_left_front.STL" />
       </geometry>
       <material name="">
@@ -160,26 +159,27 @@
   </link>
   <joint
-    name="wheel_joint_fl"
+    name="wheel_left_front_joint"
     type="continuous">
     <origin
       xyz="0.153 -0.085 -0.0455"
       rpy="1.5708 0 -1.5708" />
-    <parent link="base_link" />
-    <child link="wheel_fl" />
+    <parent link="frame_link" />
+    <child link="wheel_left_front" />
     <axis xyz="0 0 -1" />
-    <dynamics damping="3.0" friction="5.0" />
-    <limit velocity="${wheel_velocity}" effort="${wheel_effort}" />
+    <!--<dynamics
+    damping="3.0" friction="5.0" />
+    <limit velocity="${wheel_velocity}" effort="${wheel_effort}" /> -->
   </joint>
-  <transmission name="wheel_trans_fl">
+  <transmission name="wheel_left_front_transmission">
     <type>transmission_interface/SimpleTransmission</type>
-    <joint name="wheel_joint_fl">
+    <joint name="wheel_left_front_joint">
       <hardwareInterface>hardware_interface/VelocityJointInterface</hardwareInterface>
     </joint>
-    <actuator name="wheel_act_fl">
+    <actuator name="wheel_left_front_actuator">
       <mechanicalReduction>1</mechanicalReduction>
     </actuator>
   </transmission>
   <link
-    name="wheel_br">
+    name="wheel_left_rear">
     <inertial>
       <origin xyz="0 0 0.025" />
@@ -194,5 +194,5 @@
       <geometry>
         <mesh
-          filename="package://mirte_master_description/meshes/wheel_br.STL" />
+          filename="package://mirte_master_description/meshes/wheel_left_rear.STL" />
       </geometry>
       <material name="">
@@ -201,5 +201,5 @@
     </visual>
     <collision>
-      <origin xyz="0 0 -0.025" />
+      <origin xyz="0 0 0.025" />
       <geometry>
         <cylinder radius="${wheel_radius}" length="${wheel_length}" />
@@ -208,28 +208,28 @@
   </link>
   <joint
-    name="wheel_joint_br"
+    name="wheel_left_rear_joint"
     type="continuous">
     <origin
-      xyz="-0.153 0.085 -0.0455"
+      xyz="0.153 0.085 -0.0455"
       rpy="1.5708 0 -1.5708" />
-    <parent link="base_link" />
-    <child link="wheel_br" />
+    <parent link="frame_link" />
+    <child link="wheel_left_rear" />
     <axis xyz="0 0 -1" />
-    <dynamics damping="3.0" friction="5.0" />
-    <limit velocity="${wheel_velocity}" effort="${wheel_effort}" />
+    <!-- <dynamics damping="3.0" friction="5.0" />
+  <limit velocity="${wheel_velocity}" effort="${wheel_effort}" />-->
   </joint>
-  <transmission name="wheel_trans_br">
+  <transmission name="wheel_left_rear_transmission">
     <type>transmission_interface/SimpleTransmission</type>
-    <joint name="wheel_joint_br">
+    <joint name="wheel_left_rear_joint">
       <hardwareInterface>hardware_interface/VelocityJointInterface</hardwareInterface>
     </joint>
-    <actuator name="wheel_act_br">
+    <actuator name="wheel_left_rear_actuator">
       <mechanicalReduction>1</mechanicalReduction>
     </actuator>
   </transmission>
   <link
-    name="wheel_fr">
+    name="wheel_right_front">
     <inertial>
-      <origin xyz="0 0 0.025" />
+      <origin xyz="0 0 -0.025" />
       <mass value="${wheel_mass}" />
       <inertia
@@ -242,5 +242,5 @@
       <geometry>
         <mesh
-          filename="package://mirte_master_description/meshes/wheel_fr.STL" />
+          filename="package://mirte_master_description/meshes/wheel_right_front.STL" />
       </geometry>
       <material name="">
@@ -256,28 +256,28 @@
   </link>
   <joint
-    name="wheel_joint_fr"
+    name="wheel_right_front_joint"
     type="continuous">
     <origin
       xyz="-0.153 -0.085 -0.0455"
       rpy="1.5708 0 -1.5708" />
-    <parent link="base_link" />
-    <child link="wheel_fr" />
+    <parent link="frame_link" />
+    <child link="wheel_right_front" />
     <axis xyz="0 0 -1" />
-    <dynamics damping="3.0" friction="5.0" />
-    <limit velocity="${wheel_velocity}" effort="${wheel_effort}" />
+    <!-- <dynamics damping="3.0" friction="5.0" />
+    <limit velocity="${wheel_velocity}" effort="${wheel_effort}" /> -->
   </joint>
-  <transmission name="wheel_trans_fr">
+  <transmission name="wheel_right_front_transmission">
     <type>transmission_interface/SimpleTransmission</type>
-    <joint name="wheel_joint_fr">
+    <joint name="wheel_right_front_joint">
       <hardwareInterface>hardware_interface/VelocityJointInterface</hardwareInterface>
     </joint>
-    <actuator name="wheel_act_fr">
+    <actuator name="wheel_right_front_actuator">
       <mechanicalReduction>1</mechanicalReduction>
     </actuator>
   </transmission>
   <link
-    name="wheel_bl">
+    name="wheel_right_rear">
     <inertial>
-      <origin xyz="0 0 0.025" />
+      <origin xyz="0 0 -0.025" />
       <mass value="${wheel_mass}" />
       <inertia
@@ -290,5 +290,5 @@
       <geometry>
         <mesh
-          filename="package://mirte_master_description/meshes/wheel_bl.STL" />
+          filename="package://mirte_master_description/meshes/wheel_right_rear.STL" />
       </geometry>
       <material name="">
@@ -297,5 +297,5 @@
     </visual>
     <collision>
-      <origin xyz="0 0 0.025" />
+      <origin xyz="0 0 -0.025" />
       <geometry>
         <cylinder radius="${wheel_radius}" length="${wheel_length}" />
@@ -304,21 +304,22 @@
   </link>
   <joint
-    name="wheel_joint_bl"
+    name="wheel_right_rear_joint"
     type="continuous">
     <origin
-      xyz="0.153 0.085 -0.0455"
+      xyz="-0.153 0.085 -0.0455"
       rpy="1.5708 0 -1.5708" />
-    <parent link="base_link" />
-    <child link="wheel_bl" />
+    <parent link="frame_link" />
+    <child link="wheel_right_rear" />
     <axis xyz="0 0 -1" />
-    <dynamics damping="3.0" friction="5.0" />
-    <limit velocity="${wheel_velocity}" effort="${wheel_effort}" />
+    <!--<dynamics
+    damping="3.0" friction="5.0" />
+    <limit velocity="${wheel_velocity}" effort="${wheel_effort}" />-->
   </joint>
-  <transmission name="wheel_trans_bl">
+  <transmission name="wheel_right_rear_transmission">
     <type>transmission_interface/SimpleTransmission</type>
-    <joint name="wheel_joint_bl">
+    <joint name="wheel_right_rear_joint">
       <hardwareInterface>hardware_interface/VelocityJointInterface</hardwareInterface>
     </joint>
-    <actuator name="wheel_act_bl">
+    <actuator name="wheel_right_rear_actuator">
       <mechanicalReduction>1</mechanicalReduction>
     </actuator>
@@ -355,13 +356,15 @@
         </material>
       </visual>
-      <!-- <collision>
-  <origin
-  xyz="0 0 0"
-  rpy="0 0 0" />
-  <geometry>
-    <mesh
-    filename="package://mirte_master_description/meshes/cam_front.STL" />
-  </geometry>
-</collision> -->
+<!--
+      <collision>
+        <origin
+          xyz="0 0 0"
+          rpy="0 0 0" />
+        <geometry>
+          <mesh
+            filename="package://mirte_master_description/meshes/cam_front.STL" />
+        </geometry>
+      </collision>
+ -->
     </link>
     <joint
@@ -371,7 +374,7 @@
         xyz="0 -0.1325 -0.0285"
         rpy="1.5708 0 0" />
-      <parent link="base_link" />
+      <parent link="frame_link" />
       <child link="cam_front" />
-      <!-- <axis xyz="0 0 0" /> -->
+      <axis xyz="0 0 0" />
     </joint>
   </xacro:if>
@@ -381,5 +384,5 @@
       <!-- Move the link so the rest will line up easier -->
       <!-- <origin xyz="0 0 -0.031" /> -->
-      <parent link="base_link" />
+      <parent link="frame_link" />
       <child link="link_chassis" />
     </joint>
@@ -457,5 +460,5 @@
         rpy="1.5707963267949 0 -3.14159265358979" />
       <parent
-        link="base_link" />
+        link="frame_link" />
       <child
         link="screen" />

File: mirte_master_description/urdf/mirte_master_base.gazebo.xacro (robot description, xacro)
@@ -1,38 +1,11 @@
 <?xml version="1.0"?>
 <robot xmlns:xacro="http://ros.org/wiki/xacro">
-  <!-- <gazebo> -->
   <!-- ros_control plugin -->
   <gazebo>
-    <plugin name="mirte_master_mechanum_drive" filename="libgazebo_ros_mecanum_drive.so">
-      <commandTopic>mobile_base_controller/cmd_vel_corrected</commandTopic>
-      <odometryTopic>mobile_base_controller/odom</odometryTopic>
-      <odometryFrame>odom</odometryFrame>
-      <robotBaseFrame>base_footprint</robotBaseFrame>
-      <LeftRear>wheel_joint_bl</LeftRear>
-      <LeftFront>wheel_joint_fl</LeftFront>
-      <RightFront>wheel_joint_fr</RightFront>
-      <RightRear>wheel_joint_br</RightRear>
-      <odometryRate>20</odometryRate>
-      <publishWheelTF>false</publishWheelTF>
-      <publishWheelJointState>true</publishWheelJointState>
-      <WheelTorque>50</WheelTorque>
-      <WheelSeparationW>0.28</WheelSeparationW>
-      <WheelSeparationL>0.175</WheelSeparationL> <!-- 3.06 -->
-      <wheelAccel>5</wheelAccel>
-      <wheelDiameter>0.1</wheelDiameter> <!-- 1.06 Was 0.13-->
-      <publishOdom>true</publishOdom>
-      <isRollerModel>false</isRollerModel>
-    </plugin>
     <plugin name="gazebo_ros_control" filename="libgazebo_ros_control.so">
       <robotNamespace>/</robotNamespace>
     </plugin>
-  </gazebo>
-  <!--
-    <plugin name="gazebo_ros_control" filename="libgazebo_ros_control.so">
-      <robotNamespace>/</robotNamespace>
-    </plugin> -->
-  <!-- <plugin name="ridgeback_ros_force_based_move"
-    filename="libridgeback_ros_force_based_move.so">
-      <robotNamespace>/</robotNamespace>
+    <plugin name="ridgeback_ros_force_based_move" filename="libridgeback_ros_force_based_move.so">
+      <robotNamespace>/mobile_base_controller</robotNamespace>
       <commandTopic>cmd_vel</commandTopic>
       <odometryTopic>odom</odometryTopic>
@@ -40,31 +13,27 @@
       <odometryRate>25.0</odometryRate>
       <robotBaseFrame>base_link</robotBaseFrame>
-      <cmdVelTimeOut>0.25</cmdVelTimeOut> -->
-  <!-- Don't publish a transform: the controller does it. -->
-  <!-- <publishOdometryTf>0</publishOdometryTf>
+      <cmdVelTimeOut>0.25</cmdVelTimeOut>
+      <!-- Don't publish a transform: the controller does it. -->
+      <publishOdometryTf>0</publishOdometryTf>
       <yaw_velocity_p_gain>500.0</yaw_velocity_p_gain>
       <x_velocity_p_gain>10000.0</x_velocity_p_gain>
       <y_velocity_p_gain>10000.0</y_velocity_p_gain>
-    </plugin> -->
-  <!-- <plugin name="imu_controller" filename="libhector_gazebo_ros_imu.so">
-      <robotNamespace>/</robotNamespace>
-      <updateRate>50.0</updateRate>
-      <bodyName>imu_link</bodyName>
-      <topicName>imu/data</topicName>
-      <frameId>base_link</frameId>
-      <accelDrift>0.005 0.005 0.005</accelDrift>
-      <accelGaussianNoise>0.005 0.005 0.005</accelGaussianNoise>
-      <rateDrift>0.00005 0.00005 0.00005</rateDrift>
-      <rateGaussianNoise>0.00005 0.00005 0.00005</rateGaussianNoise>
-      <headingDrift>0.005</headingDrift>
-      <headingGaussianNoise>0.005</headingGaussianNoise>
-    </plugin> -->
-  <!-- <plugin name="gazebo_ros_joint_state_publisher"
-    filename="libgazebo_ros_joint_state_publisher.so">
-      <jointName>front_rocker</jointName>
-      <robotNamespace>/</robotNamespace>
-      <updateRate>50.0</updateRate>
-    </plugin> -->
-  <!-- </gazebo> -->
+    </plugin>
+    <xacro:if value="$(arg imu_enable)">
+      <plugin name="imu_controller" filename="libhector_gazebo_ros_imu.so">
+        <robotNamespace>/mirte</robotNamespace>
+        <updateRate>50.0</updateRate>
+        <bodyName>imu_link</bodyName>
+        <topicName>imu/data</topicName>
+        <frameId>base_link</frameId>
+        <accelDrift>0.005 0.005 0.005</accelDrift>
+        <accelGaussianNoise>0.005 0.005 0.005</accelGaussianNoise>
+        <rateDrift>0.00005 0.00005 0.00005</rateDrift>
+        <rateGaussianNoise>0.00005 0.00005 0.00005</rateGaussianNoise>
+        <headingDrift>0.005</headingDrift>
+        <headingGaussianNoise>0.005</headingGaussianNoise>
+      </plugin>
+    </xacro:if>
+  </gazebo>
   <!-- All static links get collapsed down to base_link in Gazebo, so that's
        the one to apply the colour to (in Gazebo 5+). -->
@@ -72,6 +41,4 @@
     <material>Gazebo/White</material>
     <gravity>true</gravity>
-    <kinematic>$(arg kinematic_only)</kinematic>
-    <!-- <selfCollide>false</selfCollide> -->
   </gazebo>
   <!-- Individual link colouring still needed in Gazebo 2.x -->
@@ -112,7 +79,7 @@
        the body level. -->
   <xacro:include filename="$(find mirte_master_description)/urdf/wheel.gazebo.xacro" />
-  <xacro:wheel_gazebo id="bl" />
-  <xacro:wheel_gazebo id="br" />
-  <xacro:wheel_gazebo id="fl" />
-  <xacro:wheel_gazebo id="fr" />
+  <xacro:wheel_gazebo id="left_front" />
+  <xacro:wheel_gazebo id="left_rear" />
+  <xacro:wheel_gazebo id="right_front" />
+  <xacro:wheel_gazebo id="right_rear" />
 </robot>

File: mirte_master_description/urdf/wheel.gazebo.xacro (robot description, xacro)
@@ -5,15 +5,7 @@
             <selfCollide>false</selfCollide>
             <gravity>true</gravity>
-            <mu1>0.0</mu1> <!--2.5-->
-            <mu2>0.0</mu2> <!--2.5-->
-            <!-- <kp>1e15</kp> --> <!-- <kp>1e2</kp> -->
-            <!-- <kd>1e13</kd> --> <!-- <kd>1e50</kd> -->
+            <mu1>0.0</mu1>
+            <mu2>0.0</mu2>
             <material>Gazebo/DarkGrey</material>
-        </gazebo>
-        <gazebo reference="wheel_joint_${id}">
-            <ode>
-                <implicit_spring_damper>true</implicit_spring_damper>
-            </ode>
-            <!-- < -->
         </gazebo>
     </xacro:macro>
