Commit message: Allow multi sim

File: mirte_master_description/urdf/lidar.xacro (robot description, xacro)
@@ -90,6 +90,6 @@
             </ray>
             <plugin name="lidar" filename="libgazebo_ros_laser.so">
-                <topicName>/scan</topicName>
-                <frameName>lidar_link</frameName>
+                <topicName>scan</topicName>
+                <frameName>${tf_namespace}lidar_link</frameName>
             </plugin>
         </sensor>

File: mirte_master_description/urdf/mirte_master.xacro (robot description, xacro)
@@ -14,4 +14,16 @@
   <xacro:arg name="depth_camera_enable" default="False" />
   <xacro:arg name="imu_enable" default="True" />
+  <xacro:arg name="use_namespace" default="False"/>
+  <xacro:arg name="namespace_name" default="" />
+  <xacro:if value="$(arg use_namespace)" >
+    <xacro:property name="camera_name" value="$(arg namespace_name)/camera" lazy_eval="False"/>
+    <xacro:property name="namespace" value="$(arg namespace_name)" scope="global" lazy_eval="False"/>
+    <xacro:property name="tf_namespace" value="$(arg namespace_name)/" scope="global" lazy_eval="False"/>
+  </xacro:if>
+  <xacro:unless value="$(arg use_namespace)">
+    <xacro:property name="camera_name" value="camera" lazy_eval="False"/>
+    <xacro:property name="namespace" value="" scope="global" lazy_eval="False"/>
+    <xacro:property name="tf_namespace" value="" scope="global" lazy_eval="False"/>
+  </xacro:unless>
   <xacro:property name="wheel_radius" value="0.050" />
   <xacro:property name="wheel_length" value="0.055" />
@@ -30,5 +42,5 @@
     filename="$(find gazebo_sensor_collection_description)/urdf/cameras/rgbd/orbbec_astra_pro_plus.urdf.xacro" />
   <xacro:if value="$(arg depth_camera_enable)">
-    <xacro:sensor_orbbec_astra_pro_plus name="camera" parent="frame_link" color="black">
+    <xacro:sensor_orbbec_astra_pro_plus name="${camera_name}" parent="frame_link" color="black">
       <origin xyz="0.01 -0.146658788505756 0.0427" rpy="0 0 ${radians(-90)}" />
     </xacro:sensor_orbbec_astra_pro_plus>

File: mirte_master_description/urdf/mirte_master_base.gazebo.xacro (robot description, xacro)
@@ -4,8 +4,8 @@
   <gazebo>
     <plugin name="gazebo_ros_control" filename="libgazebo_ros_control.so">
-      <robotNamespace>/</robotNamespace>
+      <robotNamespace>/${namespace}</robotNamespace>
     </plugin>
     <plugin name="ridgeback_ros_force_based_move" filename="libridgeback_ros_force_based_move.so">
-      <robotNamespace>/mobile_base_controller</robotNamespace>
+      <robotNamespace>/${tf_namespace}mobile_base_controller</robotNamespace>
       <commandTopic>cmd_vel</commandTopic>
       <odometryTopic>odom</odometryTopic>
@@ -22,5 +22,5 @@
     <xacro:if value="$(arg imu_enable)">
       <plugin name="imu_controller" filename="libhector_gazebo_ros_imu.so">
-        <robotNamespace>/mirte</robotNamespace>
+        <robotNamespace>/${tf_namespace}mirte</robotNamespace>
         <updateRate>50.0</updateRate>
         <bodyName>imu_link</bodyName>

File: mirte_master_description/urdf/wheel.gazebo.xacro (robot description, xacro)
@@ -2,5 +2,5 @@
 <robot xmlns:xacro="http://ros.org/wiki/xacro">
     <xacro:macro name="wheel_gazebo" params="id">
-        <gazebo reference="wheel_${id}">
+        <gazebo reference="wheel_${id}"> <!-- ${tf_namespace}-->
             <selfCollide>false</selfCollide>
             <gravity>true</gravity>

Commit message: Optionally fix lidar frame

File: mirte_master_description/urdf/lidar.xacro (robot description, xacro)
@@ -1,6 +1,5 @@
 <?xml version="1.0" encoding="UTF-8"?>
 <robot xmlns:xacro="http://www.ros.org/wiki/xacro">
-    <link
-    name="lidar_base">
+  <link name="lidar_base">
     <inertial>
       <origin
@@ -55,43 +54,62 @@
   <link name="lidar_link"></link>
   <joint name="lidar_joint" type="fixed">
-    <origin rpy="${radians(90)} ${radians(0)} 0"/>
-    <parent link="lidar_base"/>
-    <child link="lidar_link"/>
+    <origin rpy="${radians(90)} ${radians(0)} 0" />
+    <parent link="lidar_base" />
+    <child link="lidar_link" />
     <axis xyz="0 0 0" />
   </joint>
-    <gazebo reference="lidar_link">
-        <sensor type="ray" name="lidar">
-            <pose>0 0 0 0 0 0</pose>
-            <visualize>false</visualize>
-            <update_rate>10</update_rate>
-            <ray>
-                <scan>
-                    <horizontal>
-                        <samples>500</samples>
-                        <resolution>1</resolution>
-                        <min_angle>${-pi}</min_angle>
-                        <max_angle>${pi}</max_angle>
-                    </horizontal>
-                </scan>
-                <range>
-                    <min>0.05</min>
-                    <max>10.0</max> <!-- Could be anything between 10-12 depeding on conditions according to the spec sheet-->
-                    <resolution>0.015</resolution>
-                </range>
-                <noise>
-                    <type>gaussian</type>
-                    <!-- Noise parameters based on published spec for Hokuyo laser
+  <xacro:if value="$(arg use_correct_laser_frame)">
+    <link name="laser"></link>
+    <joint name="laser_joint" type="fixed">
+      <origin rpy="0 0 ${radians(90)}" />
+      <parent link="lidar_link" />
+      <child link="laser" />
+      <axis xyz="0 0 0" />
+    </joint>
+    <xacro:property name="lidar_sensor_link" value="laser" />
+  </xacro:if>
+  <xacro:unless value="$(arg use_correct_laser_frame)">
+    <xacro:property name="lidar_sensor_link" value="lidar_link" />
+  </xacro:unless>
+  <gazebo reference="${lidar_sensor_link}">
+    <sensor type="ray" name="lidar">
+      <xacro:if value="$(arg use_correct_laser_frame)">
+        <pose>0 0 0 0 0 0</pose>
+      </xacro:if>
+      <xacro:unless value="$(arg use_correct_laser_frame)">
+        <pose>0 0 0 0 0 0</pose>
+      </xacro:unless>
+      <visualize>false</visualize>
+      <update_rate>10</update_rate>
+      <ray>
+        <scan>
+          <horizontal>
+            <samples>500</samples>
+            <resolution>1</resolution>
+            <min_angle>${-pi}</min_angle>
+            <max_angle>${pi}</max_angle>
+          </horizontal>
+        </scan>
+        <range>
+          <min>0.05</min>
+          <max>10.0</max> <!-- Could be anything between 10-12 depeding on conditions according to
+          the spec sheet-->
+          <resolution>0.015</resolution>
+        </range>
+        <noise>
+          <type>gaussian</type>
+          <!-- Noise parameters based on published spec for Hokuyo laser
                 achieving "+-30mm" accuracy at range < 10m.  A mean of 0.0m and
                 stddev of 0.01m will put 99.7% of samples within 0.03m of the true
                 reading. -->
-                    <mean>0.0</mean>
-                    <stddev>0.01</stddev>
-                </noise>
-            </ray>
-            <plugin name="lidar" filename="libgazebo_ros_laser.so">
-                <topicName>scan</topicName>
-                <frameName>lidar_link</frameName>
-            </plugin>
-        </sensor>
-    </gazebo>
+          <mean>0.0</mean>
+          <stddev>0.01</stddev>
+        </noise>
+      </ray>
+      <plugin name="lidar" filename="libgazebo_ros_laser.so">
+        <topicName>scan</topicName>
+        <frameName>${lidar_sensor_link}</frameName>
+      </plugin>
+    </sensor>
+  </gazebo>
 </robot>

File: mirte_master_description/urdf/mirte_master.xacro (robot description, xacro)
@@ -26,4 +26,5 @@
     <xacro:property name="tf_namespace" value="" scope="global" lazy_eval="False"/>
   </xacro:unless>
+  <xacro:arg name="use_correct_laser_frame" default="False" />
   <xacro:property name="wheel_radius" value="0.050" />
   <xacro:property name="wheel_length" value="0.055" />
