Commit message: Ported descroption to ROS2 humble and gazebo classic

File: mirte_master_description/urdf/lidar.xacro (robot description, xacro)
@@ -22,5 +22,5 @@
       <geometry>
         <mesh
-          filename="package://mirte_master_description/meshes/lidar.STL" />
+          filename="file://$(find mirte_master_description)/meshes/lidar.STL" />
       </geometry>
       <material
@@ -36,5 +36,5 @@
       <geometry>
         <mesh
-          filename="package://mirte_master_description/meshes/lidar.STL" />
+          filename="file://$(find mirte_master_description)/meshes/lidar.STL" />
       </geometry>
     </collision>
@@ -72,5 +72,6 @@
     <xacro:property name="lidar_sensor_link" value="lidar_link" />
   </xacro:unless>
-  <gazebo reference="${lidar_sensor_link}">
+<!--
+  <gazebo reference="lidar_link">
     <sensor type="ray" name="lidar">
       <xacro:if value="$(arg use_correct_laser_frame)">
@@ -93,23 +94,51 @@
         <range>
           <min>0.05</min>
-          <max>10.0</max> <!-- Could be anything between 10-12 depeding on conditions according to
-          the spec sheet-->
+          <max>10.0</max>
           <resolution>0.015</resolution>
         </range>
         <noise>
           <type>gaussian</type>
-          <!-- Noise parameters based on published spec for Hokuyo laser
-                achieving "+-30mm" accuracy at range < 10m.  A mean of 0.0m and
-                stddev of 0.01m will put 99.7% of samples within 0.03m of the true
-                reading. -->
           <mean>0.0</mean>
           <stddev>0.01</stddev>
         </noise>
       </ray>
-      <plugin name="lidar" filename="libgazebo_ros_laser.so">
-        <topicName>scan</topicName>
-        <frameName>${lidar_sensor_link}</frameName>
+      <plugin name="gazebo_lidar" filename="libgazebo_ros_laser.so">
+        <ros>
+          <remapping>~/out:=scan</remapping>
+        </ros>
+        <output_type>sensor_msgs/LaserScan</output_type>
+        <frame_name>${lidar_sensor_link}</frame_name>
       </plugin>
     </sensor>
   </gazebo>
+-->
+  <gazebo reference="lidar_link">
+        <sensor name="lidar" type="ray">
+            <pose> 0 0 0 0 0 0 </pose>
+            <visualize>false</visualize>
+            <update_rate>10</update_rate>
+            <ray>
+                <scan>
+                    <horizontal>
+                        <samples>360</samples>
+                        <resolution>1</resolution>
+                        <min_angle>-3.14</min_angle>
+                        <max_angle>3.14</max_angle>
+                    </horizontal>
+                </scan>
+                <range>
+                    <min>0.02</min>
+                    <max>12</max>
+                    <resolution>0.01</resolution>
+                </range>
+            </ray>
+            <plugin name="laser_controller" filename="libgazebo_ros_ray_sensor.so">
+                <ros>
+                    <remapping>~/out:=scan</remapping>
+                </ros>
+                <output_type>sensor_msgs/LaserScan</output_type>
+                <frame_name>lidar_link</frame_name>
+            </plugin>
+        </sensor>
+    </gazebo>
 </robot>

File: mirte_master_description/urdf/mirte_master.xacro (robot description, xacro)
@@ -1,7 +1,3 @@
 <?xml version="1.0" encoding="utf-8"?>
-<!-- This URDF was automatically created by SolidWorks to URDF Exporter! Originally created by
-Stephen Brawner (brawner@gmail.com)
-     Commit Version: 1.6.0-4-g7f85cfe  Build Version: 1.6.7995.38578
-     For more information, please see http://wiki.ros.org/sw_urdf_exporter -->
 <robot
   name="mirte_master" xmlns:xacro="http://ros.org/wiki/xacro">
@@ -10,8 +6,8 @@
   <xacro:arg name="screen_enable" default="False" />
   <xacro:arg name="front_camera_enable" default="False" />
-  <xacro:arg name="sonar_enable" default="True" />
+  <xacro:arg name="sonar_enable" default="False" />
   <xacro:arg name="lidar_enable" default="True" />
   <xacro:arg name="depth_camera_enable" default="False" />
-  <xacro:arg name="imu_enable" default="True" />
+  <xacro:arg name="imu_enable" default="False" />
   <xacro:arg name="use_namespace" default="False"/>
   <xacro:arg name="namespace_name" default="" />
@@ -26,20 +22,15 @@
     <xacro:property name="tf_namespace" value="" scope="global" lazy_eval="False"/>
   </xacro:unless>
-  <xacro:arg name="use_correct_laser_frame" default="False" />
+  <xacro:arg name="use_correct_laser_frame" default="True" />
   <xacro:property name="wheel_radius" value="0.050" />
   <xacro:property name="wheel_length" value="0.055" />
-  <xacro:property name="wheel_mass" value="2.15" /> <!-- 0.26661 -->
-  <!-- Currently unused -->
-  <xacro:property name="wheel_velocity" value="8" /> <!-- Was 10 based on calc-->
+  <xacro:property name="wheel_mass" value="2.15" />
+  <xacro:property name="wheel_velocity" value="8" />
   <xacro:property name="wheel_effort" value="5" />
-  <xacro:property name="base_mass" value="5.0" /> <!-- 4.0815 --> <!-- 3.0815 -->
-  <!-- Used for sonar by mirte-gazebo -->
+  <xacro:property name="base_mass" value="5.0" />
   <material name="blue">
     <color rgba="0.203125 0.23828125 0.28515625 1.0" />
   </material>
-  <!-- Bring in simulation data for Gazebo. -->
   <xacro:include filename="$(find mirte_master_description)/urdf/mirte_master_base.gazebo.xacro" />
-  <xacro:include
-    filename="$(find gazebo_sensor_collection_description)/urdf/cameras/rgbd/orbbec_astra_pro_plus.urdf.xacro" />
   <xacro:if value="$(arg depth_camera_enable)">
     <xacro:sensor_orbbec_astra_pro_plus name="${camera_name}" parent="frame_link" color="black">
@@ -64,5 +55,4 @@
     name="frame_link">
     <inertial>
-      <!-- Lower the center of mass for less woble as a result of accelaration -->
       <origin xyz="-0.00024285 0.0082178 ${-0.0037661 - 0.04}" />
       <mass value="${base_mass}" />
@@ -76,5 +66,5 @@
       <geometry>
         <mesh
-          filename="package://mirte_master_description/meshes/frame_link.STL" />
+          filename="file://$(find mirte_master_description)/meshes/frame_link.STL" />
       </geometry>
       <material name="">
@@ -82,5 +72,4 @@
       </material>
     </visual>
-    <!-- Add visuals for ultra sonic sensors-->
     <visual>
       <origin
@@ -88,5 +77,5 @@
         rpy="3.14159265358979 0 0.296705972839036" />
       <geometry>
-        <mesh filename="package://mirte_master_description/meshes/ultrasonic_fl.STL" />
+        <mesh filename="file://$(find mirte_master_description)/meshes/ultrasonic_fl.STL" />
       </geometry>
       <material name="blue" />
@@ -97,5 +86,5 @@
         rpy="3.14159265358979 0 -0.296705972839036" />
       <geometry>
-        <mesh filename="package://mirte_master_description/meshes/ultrasonic_fr.STL" />
+        <mesh filename="file://$(find mirte_master_description)/meshes/ultrasonic_fr.STL" />
       </geometry>
       <material name="blue" />
@@ -106,5 +95,5 @@
         rpy="3.14159265358979 0 2.84488668075076" />
       <geometry>
-        <mesh filename="package://mirte_master_description/meshes/ultrasonic_bl.STL" />
+        <mesh filename="file://$(find mirte_master_description)/meshes/ultrasonic_bl.STL" />
       </geometry>
       <material name="blue" />
@@ -115,5 +104,5 @@
         rpy="3.14159265358979 0 -2.84488668075076" />
       <geometry>
-        <mesh filename="package://mirte_master_description/meshes/ultrasonic_br.STL" />
+        <mesh filename="file://$(find mirte_master_description)/meshes/ultrasonic_br.STL" />
       </geometry>
       <material name="blue" />
@@ -158,5 +147,5 @@
       <geometry>
         <mesh
-          filename="package://mirte_master_description/meshes/wheel_left_front.STL" />
+          filename="file://$(find mirte_master_description)/meshes/wheel_left_front.STL" />
       </geometry>
       <material name="">
@@ -180,7 +169,4 @@
     <child link="wheel_left_front" />
     <axis xyz="0 0 -1" />
-    <!--<dynamics
-    damping="3.0" friction="5.0" />
-    <limit velocity="${wheel_velocity}" effort="${wheel_effort}" /> -->
   </joint>
   <transmission name="wheel_left_front_transmission">
@@ -207,5 +193,5 @@
       <geometry>
         <mesh
-          filename="package://mirte_master_description/meshes/wheel_left_rear.STL" />
+          filename="file://$(find mirte_master_description)/meshes/wheel_left_rear.STL" />
       </geometry>
       <material name="">
@@ -229,6 +215,4 @@
     <child link="wheel_left_rear" />
     <axis xyz="0 0 -1" />
-    <!-- <dynamics damping="3.0" friction="5.0" />
-  <limit velocity="${wheel_velocity}" effort="${wheel_effort}" />-->
   </joint>
   <transmission name="wheel_left_rear_transmission">
@@ -255,5 +239,5 @@
       <geometry>
         <mesh
-          filename="package://mirte_master_description/meshes/wheel_right_front.STL" />
+          filename="file://$(find mirte_master_description)/meshes/wheel_right_front.STL" />
       </geometry>
       <material name="">
@@ -277,6 +261,4 @@
     <child link="wheel_right_front" />
     <axis xyz="0 0 -1" />
-    <!-- <dynamics damping="3.0" friction="5.0" />
-    <limit velocity="${wheel_velocity}" effort="${wheel_effort}" /> -->
   </joint>
   <transmission name="wheel_right_front_transmission">
@@ -303,5 +285,5 @@
       <geometry>
         <mesh
-          filename="package://mirte_master_description/meshes/wheel_right_rear.STL" />
+          filename="file://$(find mirte_master_description)/meshes/wheel_right_rear.STL" />
       </geometry>
       <material name="">
@@ -325,7 +307,4 @@
     <child link="wheel_right_rear" />
     <axis xyz="0 0 -1" />
-    <!--<dynamics
-    damping="3.0" friction="5.0" />
-    <limit velocity="${wheel_velocity}" effort="${wheel_effort}" />-->
   </joint>
   <transmission name="wheel_right_rear_transmission">
@@ -361,5 +340,5 @@
         <geometry>
           <mesh
-            filename="package://mirte_master_description/meshes/cam_front.STL" />
+            filename="file://$(find mirte_master_description)/meshes/cam_front.STL" />
         </geometry>
         <material
@@ -369,15 +348,4 @@
         </material>
       </visual>
-<!--
-      <collision>
-        <origin
-          xyz="0 0 0"
-          rpy="0 0 0" />
-        <geometry>
-          <mesh
-            filename="package://mirte_master_description/meshes/cam_front.STL" />
-        </geometry>
-      </collision>
- -->
     </link>
     <joint
@@ -395,6 +363,4 @@
     <xacro:include filename="$(find mirte_master_description)/urdf/ultrasonic.xacro" />
     <joint name="chassis_base_joint" type="fixed">
-      <!-- Move the link so the rest will line up easier -->
-      <!-- <origin xyz="0 0 -0.031" /> -->
       <parent link="frame_link" />
       <child link="link_chassis" />
@@ -448,5 +414,5 @@
         <geometry>
           <mesh
-            filename="package://mirte_master_description/meshes/screen.STL" />
+            filename="file://$(find mirte_master_description)/meshes/screen.STL" />
         </geometry>
         <material
@@ -462,5 +428,5 @@
         <geometry>
           <mesh
-            filename="package://mirte_master_description/meshes/screen.STL" />
+            filename="file://$(find mirte_master_description)/meshes/screen.STL" />
         </geometry>
       </collision>

File: mirte_master_description/urdf/mirte_master_base.gazebo.xacro (robot description, xacro)
@@ -1,23 +1,5 @@
 <?xml version="1.0"?>
 <robot xmlns:xacro="http://ros.org/wiki/xacro">
-  <!-- ros_control plugin -->
   <gazebo>
-    <plugin name="gazebo_ros_control" filename="libgazebo_ros_control.so">
-      <robotNamespace>/${namespace}</robotNamespace>
-    </plugin>
-    <plugin name="ridgeback_ros_force_based_move" filename="libridgeback_ros_force_based_move.so">
-      <robotNamespace>/${tf_namespace}mobile_base_controller</robotNamespace>
-      <commandTopic>cmd_vel</commandTopic>
-      <odometryTopic>odom</odometryTopic>
-      <odometryFrame>odom</odometryFrame>
-      <odometryRate>25.0</odometryRate>
-      <robotBaseFrame>base_link</robotBaseFrame>
-      <cmdVelTimeOut>0.25</cmdVelTimeOut>
-      <!-- Don't publish a transform: the controller does it. -->
-      <publishOdometryTf>0</publishOdometryTf>
-      <yaw_velocity_p_gain>500.0</yaw_velocity_p_gain>
-      <x_velocity_p_gain>10000.0</x_velocity_p_gain>
-      <y_velocity_p_gain>10000.0</y_velocity_p_gain>
-    </plugin>
     <xacro:if value="$(arg imu_enable)">
       <plugin name="imu_controller" filename="libhector_gazebo_ros_imu.so">
@@ -36,46 +18,8 @@
     </xacro:if>
   </gazebo>
-  <!-- All static links get collapsed down to base_link in Gazebo, so that's
-       the one to apply the colour to (in Gazebo 5+). -->
   <gazebo reference="base_link">
     <material>Gazebo/White</material>
     <gravity>true</gravity>
   </gazebo>
-  <!-- Individual link colouring still needed in Gazebo 2.x -->
-  <!-- <gazebo reference="chassis_link">
-    <material>Gazebo/DarkGrey</material>
-  </gazebo>
-  <gazebo reference="top_link">
-    <material>Gazebo/DarkGrey</material>
-  </gazebo>
-  <gazebo reference="left_side_cover_link">
-    <material>Gazebo/Yellow</material>
-  </gazebo>
-  <gazebo reference="right_side_cover_link">
-    <material>Gazebo/Yellow</material>
-  </gazebo>
-  <gazebo reference="front_cover_link">
-    <material>Gazebo/DarkGrey</material>
-  </gazebo>
-  <gazebo reference="rear_cover_link">
-    <material>Gazebo/DarkGrey</material>
-  </gazebo>
-  <gazebo reference="front_lights_link">
-    <material>Gazebo/White</material>
-  </gazebo>
-  <gazebo reference="rear_lights_link">
-    <material>Gazebo/Red</material>
-  </gazebo>
-  <gazebo reference="front_rocker_link">
-    <material>Gazebo/DarkGrey</material>
-  </gazebo>
-  <gazebo reference="rear_rocker_link">
-    <material>Gazebo/DarkGrey</material>
-  </gazebo>
-  <gazebo reference="axle_link">
-    <material>Gazebo/DarkGrey</material>
-  </gazebo> -->
-  <!-- Wheel friction to zero, as movement is handled by applying forces at
-       the body level. -->
   <xacro:include filename="$(find mirte_master_description)/urdf/wheel.gazebo.xacro" />
   <xacro:wheel_gazebo id="left_front" />
@@ -83,3 +27,4 @@
   <xacro:wheel_gazebo id="right_front" />
   <xacro:wheel_gazebo id="right_rear" />
+  <xacro:include filename="$(find mirte_master_description)/urdf/ros2_control.xacro"/>
 </robot>

File: mirte_master_description/urdf/ultrasonic.xacro (robot description, xacro)
@@ -31,4 +31,5 @@
       </inertial> -->
     </link>
+<!--
     <gazebo reference="base_sonar_${name}">
       <sensor type="ray" name="range_sensor_${name}">
@@ -37,5 +38,4 @@
           <scan>
             <horizontal>
-              <!-- for some reason 1 does not work, we neex 2x2 -->
               <samples>4</samples>
               <resolution>1</resolution>
@@ -47,5 +47,4 @@
               <resolution>1</resolution>
               <min_angle>0</min_angle>
-              <!-- Don't look at the floor-->
               <max_angle>${sonar_angle_max/4}</max_angle>
             </vertical>
@@ -56,5 +55,4 @@
             <resolution>0.01</resolution>
           </range>
-          <!-- Using gazebo's noise instead of plugin's -->
           <noise>
             <type>gaussian</type>
@@ -63,5 +61,4 @@
           </noise>
         </ray>
-        <!-- Using gazebo's update rate instead of plugin's -->
         <update_rate>30</update_rate>
         <plugin name="laser_controller_sonar${name}" filename="libgazebo_ros_laser.so">
@@ -73,4 +70,5 @@
       </sensor>
     </gazebo>
+ -->
   </xacro:macro>
 </robot>

File: mirte_master_description/urdf/wheel.gazebo.xacro (robot description, xacro)
@@ -2,5 +2,5 @@
 <robot xmlns:xacro="http://ros.org/wiki/xacro">
     <xacro:macro name="wheel_gazebo" params="id">
-        <gazebo reference="wheel_${id}"> <!-- ${tf_namespace}-->
+        <gazebo reference="wheel_${id}">
             <selfCollide>false</selfCollide>
             <gravity>true</gravity>
