Commit message: Fix stylings

File: urdf/mirte/ir.xacro (robot description, xacro)
@@ -35,10 +35,10 @@
         <visualize>false</visualize>
         <topic>camera_${name}/image_raw</topic>
-<ros>
-        <imageTopicName>camera_${name}/image_raw</imageTopicName>
-        <cameraInfoTopicName>camera_${name}/cam_info</cameraInfoTopicName>
-        <!-- <depthImageTopicName>[your depth image topic]</depthImageTopicName>
+        <ros>
+          <imageTopicName>camera_${name}/image_raw</imageTopicName>
+          <cameraInfoTopicName>camera_${name}/cam_info</cameraInfoTopicName>
+          <!-- <depthImageTopicName>[your depth image topic]</depthImageTopicName>
         <pointCloudTopicName>[your point cloud topic]</pointCloudTopicName> -->
-     </ros>
+        </ros>
         <camera name="head">
           <horizontal_fov>1.2</horizontal_fov>

File: urdf/mirte/macros.xacro (robot description, xacro)
@@ -20,5 +20,5 @@
       <xacro:insert_block name="origin"/>
       <inertia ixx="${2/5 * mass * r*r}" ixy="0" ixz="0" iyy="${2/5 * mass * r*r}" iyz="0" izz="${2/5 * mass * r*r}"/>
-            <!-- <inertia ixx="0" ixy="0" ixz="0" iyy="0" iyz="0" izz="0"/> -->
+      <!-- <inertia ixx="0" ixy="0" ixz="0" iyy="0" iyz="0" izz="0"/> -->
     </inertial>
   </xacro:macro>
@@ -31,7 +31,7 @@
         <origin rpy="0 1.5707 1.5707" xyz="0 0 0"/>
         <geometry>
-          <sphere  radius="${radius}"/>
+          <sphere radius="${radius}"/>
         </geometry>
-                <surface>
+        <surface>
           <friction>
             <ode>
@@ -62,5 +62,5 @@
           <mesh filename="file://$(find mirte_gazebo)/meshes/wheel.stl" scale="1 1 1" rpy="0 0 ${pi*0 + visualRot*pi}"/>
         </geometry>
-                <!-- <origin rpy="0 1.5707 1.5707" xyz="0 0 0"/>
+        <!-- <origin rpy="0 1.5707 1.5707" xyz="0 0 0"/>
         <geometry>
           <cylinder length="0.015" radius="${radius}"/>

File: urdf/mirte/mirte.xacro (robot description, xacro)
@@ -69,5 +69,5 @@
     <parent link="base_footprint"/>
     <child link="base_link"/>
-     <origin rpy="0 0 0" xyz="0 0 0.018"/>
+    <origin rpy="0 0 0" xyz="0 0 0.018"/>
   </joint>
   <link name="base_link"/>
@@ -124,5 +124,5 @@
       <rpy_offset>0.0 0.0 0.0</rpy_offset>
       <gaussian_noise>0.01</gaussian_noise>
-     </plugin>
+    </plugin>
   </gazebo>
   <gazebo>

File: urdf/mirte/realsense-depth.xacro (robot description, xacro)
@@ -92,11 +92,11 @@
         </camera>
         <plugin name="camera_controller_depth" filename="libgazebo_ros_camera.so">
-            <ros>
-              <namespace>/mirte</namespace>
-              <remapping>camera_depth/image_raw:=camera_rgb/image_raw</remapping>
-              <remapping>camera_depth/camera_info:=camera_rgb/camera_info</remapping>
-              <remapping>camera_depth/depth/image_raw:=camera_depth/depth_image_raw</remapping>
-              <remapping>camera_depth/depth/camera_info:=camera_depth/camera_depth_info</remapping>
-            </ros>
+          <ros>
+            <namespace>/mirte</namespace>
+            <remapping>camera_depth/image_raw:=camera_rgb/image_raw</remapping>
+            <remapping>camera_depth/camera_info:=camera_rgb/camera_info</remapping>
+            <remapping>camera_depth/depth/image_raw:=camera_depth/depth_image_raw</remapping>
+            <remapping>camera_depth/depth/camera_info:=camera_depth/camera_depth_info</remapping>
+          </ros>
           <camera_name>camera_depth</camera_name>
           <frame_name>${prefix}depth_cloud</frame_name>

File: urdf/static_cam.xacro (robot description, xacro)
@@ -12,9 +12,9 @@
           <topic>top_down_camera/image_raw</topic>
           <ros>
-        <imageTopicName>top_down_camera/image_raw</imageTopicName>
-        <cameraInfoTopicName>top_down_camera/cam_info</cameraInfoTopicName>
-        <!-- <depthImageTopicName>[your depth image topic]</depthImageTopicName>
+            <imageTopicName>top_down_camera/image_raw</imageTopicName>
+            <cameraInfoTopicName>top_down_camera/cam_info</cameraInfoTopicName>
+            <!-- <depthImageTopicName>[your depth image topic]</depthImageTopicName>
         <pointCloudTopicName>[your point cloud topic]</pointCloudTopicName> -->
-     </ros>
+          </ros>
           <gz_frame_id>top_down_camera_rgb_frame</gz_frame_id>
           <camera name="top_down_camera">
@@ -31,10 +31,10 @@
             </clip>
           </camera>
-           <plugin name="camera_controller_top_down" filename="libgazebo_ros_camera.so">
-          <camera_name>camera_top_down</camera_name>
-          <frame_name>base_top_down</frame_name>
-          <frameName>base_top_down</frameName>
-          <cameraName>camera_top_down</cameraName>
-        </plugin>
+          <plugin name="camera_controller_top_down" filename="libgazebo_ros_camera.so">
+            <camera_name>camera_top_down</camera_name>
+            <frame_name>base_top_down</frame_name>
+            <frameName>base_top_down</frameName>
+            <cameraName>camera_top_down</cameraName>
+          </plugin>
         </sensor>
         <static>1</static>
