Commit message: Fixed package naming issues after move

File: mirte_description/mirte_pioneer_description/urdf/mirte/lidar.xacro (robot description, xacro)
@@ -10,5 +10,5 @@
       <origin rpy="0 0 0" xyz="0 0 -0.03"/>
       <geometry>
-        <mesh filename="file://$(find mirte_gazebo)/meshes/lidar.stl" scale="0.001 0.001 0.001" rpy="0 0 1.57079633"/>
+        <mesh filename="file://$(find mirte_pioneer_description)/meshes/lidar.stl" scale="0.001 0.001 0.001" rpy="0 0 1.57079633"/>
       </geometry>
     </visual>
@@ -16,5 +16,5 @@
       <origin rpy="0 0 0" xyz="0 0 -0.03"/>
       <geometry>
-        <mesh filename="file://$(find mirte_gazebo)/meshes/lidar.stl" scale="0.001 0.001 0.001" rpy="0 0 1.57079633"/>
+        <mesh filename="file://$(find mirte_pioneer_description)/meshes/lidar.stl" scale="0.001 0.001 0.001" rpy="0 0 1.57079633"/>
       </geometry>
     </collision>

File: mirte_description/mirte_pioneer_description/urdf/mirte/macros.xacro (robot description, xacro)
@@ -60,5 +60,5 @@
         <origin rpy="0 1.5707 ${1.5707 + visualRot*pi}" xyz="-0 0.0 0"/>
         <geometry>
-          <mesh filename="file://$(find mirte_gazebo)/meshes/wheel.stl" scale="1 1 1" rpy="0 0 ${pi*0 + visualRot*pi}"/>
+          <mesh filename="file://$(find mirte_pioneer_description)/meshes/wheel.stl" scale="1 1 1" rpy="0 0 ${pi*0 + visualRot*pi}"/>
         </geometry>
         <!-- <origin rpy="0 1.5707 1.5707" xyz="0 0 0"/>

File: mirte_description/mirte_pioneer_description/urdf/mirte/mirte.xacro (robot description, xacro)
@@ -6,6 +6,6 @@
   <xacro:arg name="lidar_enable" default="true"/>
   <xacro:arg name="realsense_enable" default="true"/>
-  <xacro:include filename="$(find mirte_gazebo)/urdf/mirte/materials.xacro"/>
-  <xacro:include filename="$(find mirte_gazebo)/urdf/mirte/macros.xacro"/>
+  <xacro:include filename="$(find mirte_pioneer_description)/urdf/mirte/materials.xacro"/>
+  <xacro:include filename="$(find mirte_pioneer_description)/urdf/mirte/macros.xacro"/>
   <test value="$(arg sonar_enable)" name="sonar_enable"/>
   <test value="$(arg intensity_enable)" name="intensity_enable"/>
@@ -13,19 +13,19 @@
   <test value="$(arg lidar_enable)" name="lidar_enable"/>
   <xacro:if value="$(arg lidar_enable)">
-    <xacro:include filename="$(find mirte_gazebo)/urdf/mirte/lidar.xacro"/>
+    <xacro:include filename="$(find mirte_pioneer_description)/urdf/mirte/lidar.xacro"/>
   </xacro:if>
   <xacro:if value="$(arg intensity_enable)">
-    <xacro:include filename="$(find mirte_gazebo)/urdf/mirte/ir.xacro"/>
+    <xacro:include filename="$(find mirte_pioneer_description)/urdf/mirte/ir.xacro"/>
   </xacro:if>
   <xacro:if value="$(arg camera_enable)">
-    <xacro:include filename="$(find mirte_gazebo)/urdf/mirte/camera.xacro"/>
+    <xacro:include filename="$(find mirte_pioneer_description)/urdf/mirte/camera.xacro"/>
   </xacro:if>
   <xacro:if value="$(arg sonar_enable)">
-    <xacro:include filename="$(find mirte_gazebo)/urdf/mirte/ultrasonic.xacro"/>
+    <xacro:include filename="$(find mirte_pioneer_description)/urdf/mirte/ultrasonic.xacro"/>
   </xacro:if>
   <xacro:if value="$(arg realsense_enable)">
-    <xacro:include filename="$(find mirte_gazebo)/urdf/mirte/realsense.xacro"/>
+    <xacro:include filename="$(find mirte_pioneer_description)/urdf/mirte/realsense.xacro"/>
   </xacro:if>
-  <xacro:property name="yaml_param_file" value="$(find mirte_gazebo)/config/mirte_dimensions.yaml"/>
+  <xacro:property name="yaml_param_file" value="$(find mirte_pioneer_description)/config/mirte_dimensions.yaml"/>
   <xacro:property name="params" value="${xacro.load_yaml(yaml_param_file)}"/>
   <link name="link_chassis">
@@ -38,5 +38,5 @@
     <collision name="collision_chassis">
       <geometry>
-        <mesh filename="file://$(find mirte_gazebo)/meshes/mirte_base.stl" scale="0.001 0.001 0.001" rpy="0 0 1.57079633"/>
+        <mesh filename="file://$(find mirte_pioneer_description)/meshes/mirte_base.stl" scale="0.001 0.001 0.001" rpy="0 0 1.57079633"/>
       </geometry>
     </collision>
@@ -44,5 +44,5 @@
       <origin rpy="0 0 0" xyz="0 0 0"/>
       <geometry>
-        <mesh filename="file://$(find mirte_gazebo)/meshes/mirte_base.stl" scale="0.001 0.001 0.001" rpy="0 0 1.57079633"/>
+        <mesh filename="file://$(find mirte_pioneer_description)/meshes/mirte_base.stl" scale="0.001 0.001 0.001" rpy="0 0 1.57079633"/>
       </geometry>
       <material name="blue"/>
@@ -109,5 +109,5 @@
     </xacro:ir_sensor>
   </xacro:if>
-  <xacro:include filename="$(find mirte_gazebo)/urdf/mirte/diffdrive.xacro"/>
+  <xacro:include filename="$(find mirte_pioneer_description)/urdf/mirte/diffdrive.xacro"/>
   <gazebo>
     <plugin name="gazebo_ros_p3d" filename="libgazebo_ros_p3d.so">

File: mirte_description/mirte_pioneer_description/urdf/mirte/realsense-depth.xacro (robot description, xacro)
@@ -19,5 +19,5 @@
         <origin rpy="0 0 0" xyz="0 0 0"/>
         <geometry>
-          <mesh filename="file://$(find mirte_gazebo)/models/realsense_camera/meshes/realsense.dae"/>
+          <mesh filename="file://$(find mirte_pioneer_description)/models/realsense_camera/meshes/realsense.dae"/>
         </geometry>
       </visual>

File: mirte_description/mirte_pioneer_description/urdf/mirte/realsense.xacro (robot description, xacro)
@@ -1,5 +1,5 @@
 <?xml version="1.0"?>
 <robot xmlns:xacro="http://www.ros.org/wiki/xacro">
-  <xacro:include filename="$(find mirte_gazebo)/urdf/mirte/realsense-depth.xacro"/>
+  <xacro:include filename="$(find mirte_pioneer_description)/urdf/mirte/realsense-depth.xacro"/>
   <xacro:realsense-depth prefix="mirte_" parent="link_chassis">
     <origin xyz="0.1 0 0.035" rpy="0 0 0"/>
