Commit message: One joint of the arm for testing

File: mirte_description/mirte_master_description/urdf/arm.xacro (robot description, xacro)
@@ -23,19 +23,19 @@
             <geometry>
                 <mesh
-                    filename="package://mirte_master_description/meshes/arm_Rot.STL" />
-            </geometry>
-            <material
-                name="">
-                <color
-                    rgba="0.792156862745098 0.819607843137255 0.933333333333333 1" />
-            </material>
-        </visual>
-        <collision>
-            <origin
-                xyz="0 0 0"
-                rpy="0 0 0" />
-            <geometry>
-                <mesh
-                    filename="package://mirte_master_description/meshes/arm_Rot.STL" />
+                    filename="file://$(find mirte_master_description)/meshes/arm_Rot.STL" />
+            </geometry>
+            <material
+                name="">
+                <color
+                    rgba="0.792156862745098 0.819607843137255 0.933333333333333 1" />
+            </material>
+        </visual>
+        <collision>
+            <origin
+                xyz="0 0 0"
+                rpy="0 0 0" />
+            <geometry>
+                <mesh
+                    filename="file://$(find mirte_master_description)/meshes/arm_Rot.STL" />
             </geometry>
         </collision>
@@ -60,4 +60,5 @@
         />
     </joint>
+<!--
     <link
         name="arm_Shoulder">
@@ -82,5 +83,5 @@
             <geometry>
                 <mesh
-                    filename="package://mirte_master_description/meshes/arm_Shoulder.STL" />
+                    filename="file://$(find mirte_master_description)/meshes/arm_Shoulder.STL" />
             </geometry>
             <material
@@ -96,5 +97,5 @@
             <geometry>
                 <mesh
-                    filename="package://mirte_master_description/meshes/arm_Shoulder.STL" />
+                    filename="file://$(find mirte_master_description)/meshes/arm_Shoulder.STL" />
             </geometry>
         </collision>
@@ -141,5 +142,5 @@
             <geometry>
                 <mesh
-                    filename="package://mirte_master_description/meshes/arm_Elbow.STL" />
+                    filename="file://$(find mirte_master_description)/meshes/arm_Elbow.STL" />
             </geometry>
             <material
@@ -155,5 +156,5 @@
             <geometry>
                 <mesh
-                    filename="package://mirte_master_description/meshes/arm_Elbow.STL" />
+                    filename="file://$(find mirte_master_description)/meshes/arm_Elbow.STL" />
             </geometry>
         </collision>
@@ -200,5 +201,5 @@
             <geometry>
                 <mesh
-                    filename="package://mirte_master_description/meshes/arm_Wrist.STL" />
+                    filename="file://$(find mirte_master_description)/meshes/arm_Wrist.STL" />
             </geometry>
             <material
@@ -214,5 +215,5 @@
             <geometry>
                 <mesh
-                    filename="package://mirte_master_description/meshes/arm_Wrist.STL" />
+                    filename="file://$(find mirte_master_description)/meshes/arm_Wrist.STL" />
             </geometry>
         </collision>
@@ -259,19 +260,19 @@
             <geometry>
                 <mesh
-                    filename="package://mirte_master_description/meshes/Gripper.STL" />
-            </geometry>
-            <material
-                name="">
-                <color
-                    rgba="0.792156862745098 0.819607843137255 0.933333333333333 1" />
-            </material>
-        </visual>
-        <collision>
-            <origin
-                xyz="0 0 0"
-                rpy="0 0 0" />
-            <geometry>
-                <mesh
-                    filename="package://mirte_master_description/meshes/Gripper.STL" />
+                    filename="file://$(find mirte_master_description)/meshes/Gripper.STL" />
+            </geometry>
+            <material
+                name="">
+                <color
+                    rgba="0.792156862745098 0.819607843137255 0.933333333333333 1" />
+            </material>
+        </visual>
+        <collision>
+            <origin
+                xyz="0 0 0"
+                rpy="0 0 0" />
+            <geometry>
+                <mesh
+                    filename="file://$(find mirte_master_description)/meshes/Gripper.STL" />
             </geometry>
         </collision>
@@ -318,19 +319,19 @@
             <geometry>
                 <mesh
-                    filename="package://mirte_master_description/meshes/_gripper_link_r.STL" />
-            </geometry>
-            <material
-                name="">
-                <color
-                    rgba="0.792156862745098 0.819607843137255 0.933333333333333 1" />
-            </material>
-        </visual>
-        <collision>
-            <origin
-                xyz="0 0 0"
-                rpy="0 0 0" />
-            <geometry>
-                <mesh
-                    filename="package://mirte_master_description/meshes/_gripper_link_r.STL" />
+                    filename="file://$(find mirte_master_description)/meshes/_gripper_link_r.STL" />
+            </geometry>
+            <material
+                name="">
+                <color
+                    rgba="0.792156862745098 0.819607843137255 0.933333333333333 1" />
+            </material>
+        </visual>
+        <collision>
+            <origin
+                xyz="0 0 0"
+                rpy="0 0 0" />
+            <geometry>
+                <mesh
+                    filename="file://$(find mirte_master_description)/meshes/_gripper_link_r.STL" />
             </geometry>
         </collision>
@@ -376,19 +377,19 @@
             <geometry>
                 <mesh
-                    filename="package://mirte_master_description/meshes/gripper_finger_r.STL" />
-            </geometry>
-            <material
-                name="">
-                <color
-                    rgba="0.792156862745098 0.819607843137255 0.933333333333333 1" />
-            </material>
-        </visual>
-        <collision>
-            <origin
-                xyz="0 0 0"
-                rpy="0 0 0" />
-            <geometry>
-                <mesh
-                    filename="package://mirte_master_description/meshes/gripper_finger_r.STL" />
+                    filename="file://$(find mirte_master_description)/meshes/gripper_finger_r.STL" />
+            </geometry>
+            <material
+                name="">
+                <color
+                    rgba="0.792156862745098 0.819607843137255 0.933333333333333 1" />
+            </material>
+        </visual>
+        <collision>
+            <origin
+                xyz="0 0 0"
+                rpy="0 0 0" />
+            <geometry>
+                <mesh
+                    filename="file://$(find mirte_master_description)/meshes/gripper_finger_r.STL" />
             </geometry>
         </collision>
@@ -434,19 +435,19 @@
             <geometry>
                 <mesh
-                    filename="package://mirte_master_description/meshes/_gripper_link_l.STL" />
-            </geometry>
-            <material
-                name="">
-                <color
-                    rgba="0.792156862745098 0.819607843137255 0.933333333333333 1" />
-            </material>
-        </visual>
-        <collision>
-            <origin
-                xyz="0 0 0"
-                rpy="0 0 0" />
-            <geometry>
-                <mesh
-                    filename="package://mirte_master_description/meshes/_gripper_link_l.STL" />
+                    filename="file://$(find mirte_master_description)/meshes/_gripper_link_l.STL" />
+            </geometry>
+            <material
+                name="">
+                <color
+                    rgba="0.792156862745098 0.819607843137255 0.933333333333333 1" />
+            </material>
+        </visual>
+        <collision>
+            <origin
+                xyz="0 0 0"
+                rpy="0 0 0" />
+            <geometry>
+                <mesh
+                    filename="file://$(find mirte_master_description)/meshes/_gripper_link_l.STL" />
             </geometry>
         </collision>
@@ -492,19 +493,19 @@
             <geometry>
                 <mesh
-                    filename="package://mirte_master_description/meshes/gripper_finger_l.STL" />
-            </geometry>
-            <material
-                name="">
-                <color
-                    rgba="0.792156862745098 0.819607843137255 0.933333333333333 1" />
-            </material>
-        </visual>
-        <collision>
-            <origin
-                xyz="0 0 0"
-                rpy="0 0 0" />
-            <geometry>
-                <mesh
-                    filename="package://mirte_master_description/meshes/gripper_finger_l.STL" />
+                    filename="file://$(find mirte_master_description)/meshes/gripper_finger_l.STL" />
+            </geometry>
+            <material
+                name="">
+                <color
+                    rgba="0.792156862745098 0.819607843137255 0.933333333333333 1" />
+            </material>
+        </visual>
+        <collision>
+            <origin
+                xyz="0 0 0"
+                rpy="0 0 0" />
+            <geometry>
+                <mesh
+                    filename="file://$(find mirte_master_description)/meshes/gripper_finger_l.STL" />
             </geometry>
         </collision>
@@ -550,19 +551,19 @@
             <geometry>
                 <mesh
-                    filename="package://mirte_master_description/meshes/_Gripper_r.STL" />
-            </geometry>
-            <material
-                name="">
-                <color
-                    rgba="0.792156862745098 0.819607843137255 0.933333333333333 1" />
-            </material>
-        </visual>
-        <collision>
-            <origin
-                xyz="0 0 0"
-                rpy="0 0 0" />
-            <geometry>
-                <mesh
-                    filename="package://mirte_master_description/meshes/_Gripper_r.STL" />
+                    filename="file://$(find mirte_master_description)/meshes/_Gripper_r.STL" />
+            </geometry>
+            <material
+                name="">
+                <color
+                    rgba="0.792156862745098 0.819607843137255 0.933333333333333 1" />
+            </material>
+        </visual>
+        <collision>
+            <origin
+                xyz="0 0 0"
+                rpy="0 0 0" />
+            <geometry>
+                <mesh
+                    filename="file://$(find mirte_master_description)/meshes/_Gripper_r.STL" />
             </geometry>
         </collision>
@@ -586,3 +587,4 @@
             velocity="0" />
     </joint>
+-->
 </robot>

File: mirte_description/mirte_master_description/urdf/mirte_master.xacro (robot description, xacro)
@@ -3,9 +3,9 @@
   name="mirte_master" xmlns:xacro="http://ros.org/wiki/xacro">
   <xacro:arg name="flag_enable" default="False" />
-  <xacro:arg name="arm_enable" default="False" />
+  <xacro:arg name="arm_enable" default="True" />
   <xacro:arg name="screen_enable" default="False" />
   <xacro:arg name="front_camera_enable" default="False" />
   <xacro:arg name="sonar_enable" default="False" />
-  <xacro:arg name="lidar_enable" default="True" />
+  <xacro:arg name="lidar_enable" default="False" />
   <xacro:arg name="depth_camera_enable" default="False" />
   <xacro:arg name="imu_enable" default="False" />

Commit message: Added ros2 control for the arm and gripper

File: mirte_description/mirte_master_description/urdf/arm.xacro (robot description, xacro)
@@ -60,5 +60,4 @@
         />
     </joint>
-<!--
     <link
         name="arm_Shoulder">
@@ -587,4 +586,3 @@
             velocity="0" />
     </joint>
--->
 </robot>

File: mirte_description/mirte_master_description/urdf/ros2_control.xacro (robot description, xacro)
@@ -41,4 +41,24 @@
         <state_interface name="effort" />
     </joint>
+    <joint name="arm_Rot_joint">
+        <command_interface name="position"/>
+        <state_interface name="position" />
+    </joint>
+    <joint name="arm_Shoulder_joint">
+        <command_interface name="position"/>
+        <state_interface name="position" />
+    </joint>
+    <joint name="arm_Elbow_joint">
+        <command_interface name="position"/>
+        <state_interface name="position" />
+    </joint>
+    <joint name="arm_Wrist_joint">
+        <command_interface name="position"/>
+        <state_interface name="position" />
+    </joint>
+    <joint name="Gripper_joint">
+        <command_interface name="position"/>
+        <state_interface name="position" />
+    </joint>
   </ros2_control>
 <gazebo>

Commit message: Added temporary simple gripper with mimicing

File: mirte_description/mirte_master_description/urdf/arm.xacro (robot description, xacro)
@@ -296,5 +296,6 @@
         />
     </joint>
-    <link
+<!--
+   <link
         name="_gripper_link_r">
         <inertial>
@@ -528,4 +529,5 @@
             velocity="0" />
     </joint>
+-->
     <link
         name="_Gripper_r">
@@ -579,10 +581,12 @@
             link="_Gripper_r" />
         <axis
-            xyz="0 0 1" />
-        <limit
-            lower="0"
+            xyz="0 -1 0" />
+        <limit
+            lower="-${pi/2}"
             upper="0"
-            effort="0"
-            velocity="0" />
+            effort="2"
+            velocity="2"
+        />
+        <mimic joint="Gripper_joint" multiplier="-1"/>
     </joint>
 </robot>

File: mirte_description/mirte_master_description/urdf/ros2_control.xacro (robot description, xacro)
@@ -43,19 +43,31 @@
     <joint name="arm_Rot_joint">
         <command_interface name="position"/>
-        <state_interface name="position" />
+        <state_interface name="position"/>
+   </joint>
+    <joint name="arm_Shoulder_joint">
+        <command_interface name="position"/>
+        <state_interface name="position">
+          <param name="initial_value">-1.56</param>
+        </state_interface>
     </joint>
-    <joint name="arm_Shoulder_joint">
+    <joint name="arm_Elbow_joint">
+        <command_interface name="position"/>
+        <state_interface name="position">
+          <param name="initial_value">-1.56</param>
+        </state_interface>
+    </joint>
+    <joint name="arm_Wrist_joint">
+        <command_interface name="position"/>
+        <state_interface name="position">
+          <param name="initial_value">1.56</param>
+        </state_interface>
+    </joint>
+    <joint name="Gripper_joint">
         <command_interface name="position"/>
         <state_interface name="position" />
     </joint>
-    <joint name="arm_Elbow_joint">
-        <command_interface name="position"/>
-        <state_interface name="position" />
-    </joint>
-    <joint name="arm_Wrist_joint">
-        <command_interface name="position"/>
-        <state_interface name="position" />
-    </joint>
-    <joint name="Gripper_joint">
+    <joint name="_Gripper_joint_r">
+        <param name="mimic">Gripper_joint</param>
+        <param name="multiplier">-1</param>
         <command_interface name="position"/>
         <state_interface name="position" />

Commit message: Added rest of the gripper, still simple control

File: mirte_description/mirte_master_description/urdf/arm.xacro (robot description, xacro)
@@ -290,11 +290,10 @@
             xyz="0 -1 0" />
         <limit
-            lower="0"
-            upper="${pi/2}"
+            lower="-.20"
+            upper="0.25"
             effort="2"
             velocity="2"
         />
     </joint>
-<!--
    <link
         name="_gripper_link_r">
@@ -348,5 +347,5 @@
             link="_gripper_link_r" />
         <axis
-            xyz="0 0 1" />
+            xyz="0 -1 0" />
         <limit
             lower="0"
@@ -354,4 +353,5 @@
             effort="0"
             velocity="0" />
+        <mimic joint="Gripper_joint" multiplier="1.4"/>
     </joint>
     <link
@@ -464,5 +464,5 @@
             link="_gripper_link_l" />
         <axis
-            xyz="0 0 1" />
+            xyz="0 -1 0" />
         <limit
             lower="0"
@@ -470,4 +470,5 @@
             effort="0"
             velocity="0" />
+        <mimic joint="Gripper_joint" multiplier="-1.4"/>
     </joint>
     <link
@@ -529,5 +530,4 @@
             velocity="0" />
     </joint>
--->
     <link
         name="_Gripper_r">
@@ -583,6 +583,6 @@
             xyz="0 -1 0" />
         <limit
-            lower="-${pi/2}"
-            upper="0"
+            lower="-.25"
+            upper="0.20"
             effort="2"
             velocity="2"

File: mirte_description/mirte_master_description/urdf/ros2_control.xacro (robot description, xacro)
@@ -73,4 +73,24 @@
         <state_interface name="position" />
     </joint>
+    <joint name="_gripper_link_joint_l">
+        <param name="mimic">Gripper_joint</param>
+        <param name="multiplier">-1.4</param>
+        <command_interface name="position"/>
+        <state_interface name="position" />
+    </joint>
+    <joint name="_gripper_link_joint_r">
+        <param name="mimic">Gripper_joint</param>
+        <param name="multiplier">-1.4</param>
+        <command_interface name="position"/>
+        <state_interface name="position" />
+    </joint>
+    <joint name="gripper_finger_joint_l">
+        <command_interface name="position"/>
+        <state_interface name="position" />
+    </joint>
+    <joint name="gripper_finger_joint_r">
+        <command_interface name="position"/>
+        <state_interface name="position" />
+    </joint>
   </ros2_control>
 <gazebo>
