Commit message: Initial attempt on ultrasonic, still failing on NaN values

File: mirte_description/mirte_master_description/urdf/mirte_master.xacro (robot description, xacro)
@@ -6,5 +6,5 @@
   <xacro:arg name="screen_enable" default="False" />
   <xacro:arg name="front_camera_enable" default="False" />
-  <xacro:arg name="sonar_enable" default="False" />
+  <xacro:arg name="sonar_enable" default="True" />
   <xacro:arg name="lidar_enable" default="True" />
   <xacro:arg name="depth_camera_enable" default="False" />
@@ -71,40 +71,4 @@
         <color rgba="0.52941 0.54902 0.54902 1" />
       </material>
-    </visual>
-    <visual>
-      <origin
-        xyz="0.05297775289576 -0.120282421780502 -0.031"
-        rpy="3.14159265358979 0 0.296705972839036" />
-      <geometry>
-        <mesh filename="file://$(find mirte_master_description)/meshes/ultrasonic_fl.STL" />
-      </geometry>
-      <material name="blue" />
-    </visual>
-    <visual>
-      <origin
-        xyz="-0.05297775289576 -0.120282421780502 -0.031"
-        rpy="3.14159265358979 0 -0.296705972839036" />
-      <geometry>
-        <mesh filename="file://$(find mirte_master_description)/meshes/ultrasonic_fr.STL" />
-      </geometry>
-      <material name="blue" />
-    </visual>
-    <visual>
-      <origin
-        xyz="0.0565606470918482 0.119187021096338 -0.031"
-        rpy="3.14159265358979 0 2.84488668075076" />
-      <geometry>
-        <mesh filename="file://$(find mirte_master_description)/meshes/ultrasonic_bl.STL" />
-      </geometry>
-      <material name="blue" />
-    </visual>
-    <visual>
-      <origin
-        xyz="-0.0565606470918482 0.119187021096338 -0.031"
-        rpy="3.14159265358979 0 -2.84488668075076" />
-      <geometry>
-        <mesh filename="file://$(find mirte_master_description)/meshes/ultrasonic_br.STL" />
-      </geometry>
-      <material name="blue" />
     </visual>
     <collision>

File: mirte_description/mirte_master_description/urdf/ultrasonic.xacro (robot description, xacro)
@@ -12,63 +12,55 @@
     </joint>
     <link name="base_sonar_${name}">
-      <!-- <collision>
-        <origin xyz="0 0 0" rpy="0 0 0"/>
+      <visual>
+        <origin rpy="0 0 ${radians(-90)}" />
         <geometry>
-          <box size="0.01 0.05 0.037"/>
+          <mesh filename="file://$(find mirte_master_description)/meshes/ultrasonic_fl.STL" />
         </geometry>
-      </collision> -->
-      <visual>
-        <origin xyz="0 0 0" rpy="0 0 0"/>
-        <geometry>
-          <box size="0.01 0.05 0.037"/>
-        </geometry>
-        <material name="blue"/>
+        <material name="blue" />
       </visual>
-      <!-- <inertial>
-        <mass value="0.0"/>
-        <origin xyz="0 0 0" rpy="0 0 0"/>
-        <inertia ixx="0.0" ixy="0.0" ixz="0.0" iyy="0.0" iyz="0.0" izz="0.0"/>
-      </inertial> -->
     </link>
-<!--
     <gazebo reference="base_sonar_${name}">
       <sensor type="ray" name="range_sensor_${name}">
         <visualize>false</visualize>
-        <ray>
-          <scan>
-            <horizontal>
-              <samples>4</samples>
+          <ray>
+            <scan>
+              <horizontal>
+                <!-- for some reason 1 does not work, we neex 2x2 -->
+                <samples>2</samples>
+                <resolution>1</resolution>
+                <min_angle>-0.26</min_angle>
+                <max_angle>0.26</max_angle>
+              </horizontal>
+            <vertical>
+              <samples>2</samples>
               <resolution>1</resolution>
-              <min_angle>${-sonar_angle_max/2}</min_angle>
-              <max_angle>${sonar_angle_max/2}</max_angle>
-            </horizontal>
-            <vertical>
-              <samples>4</samples>
-              <resolution>1</resolution>
-              <min_angle>0</min_angle>
-              <max_angle>${sonar_angle_max/4}</max_angle>
+              <min_angle>-0.014835</min_angle>
+              <max_angle>0.014835</max_angle>
             </vertical>
-          </scan>
-          <range>
-            <min>0.025</min>
-            <max>5</max>
-            <resolution>0.01</resolution>
-          </range>
-          <noise>
-            <type>gaussian</type>
-            <mean>0.0</mean>
-            <stddev>0.01</stddev>
-          </noise>
-        </ray>
-        <update_rate>30</update_rate>
-        <plugin name="laser_controller_sonar${name}" filename="libgazebo_ros_laser.so">
-          <topicName>mirte/scanSonar${name}</topicName>
-          <output_type>sensor_msgs/Range</output_type>
-          <radiation_type>ultrasound</radiation_type>
-          <frameName>base_sonar_${name}</frameName>
-        </plugin>
-      </sensor>
-    </gazebo>
- -->
+         </scan>
+         <range>
+           <min>0.03</min>
+           <max>4</max>
+           <resolution>0.01</resolution>
+         </range>
+         <!-- Using gazebo's noise instead of plugin's -->
+         <noise>
+           <type>gaussian</type>
+           <mean>0.0</mean>
+           <stddev>0.01</stddev>
+         </noise>
+       </ray>
+       <!-- Using gazebo's update rate instead of plugin's -->
+       <update_rate>30</update_rate>
+       <plugin name="gazebo_ros_range_controller_${name}" filename="libgazebo_ros_ray_sensor.so">
+         <ros>
+           <namespace>/mirte</namespace>
+           <remapping>~/out:=distance/${name}</remapping>
+         </ros>
+         <output_type>sensor_msgs/Range</output_type>
+         <radiation_type>ultrasound</radiation_type>
+       </plugin>
+     </sensor>
+   </gazebo>
   </xacro:macro>
 </robot>
